File: Krake_V1/LCD.kicad_sch (KiCad schematic)
At the start: 0 parts

Commit message: The arduino IDE file replaced the older IDE file. This Arduino IDE contains LCD print and a mute button.
Parts:
- added C301: 100nF, Capacitor_SMD:C_0603_1608Metric_Pad1.08x0.95mm_HandSolder, symbol Device:C
- added C302: 47uF 16V, Capacitor_SMD:CP_Elec_5x5.4, symbol Device:C_Polarized
- added Q301: BSS138, Package_TO_SOT_SMD:SOT-23, symbol Transistor_FET:BSS138
- added R301, R302, R303, R311, R312: 4K7, Resistor_SMD:R_0603_1608Metric_Pad0.98x0.95mm_HandSolder, symbol Device:R
- added R304: 1K, Resistor_SMD:R_0603_1608Metric_Pad0.98x0.95mm_HandSolder, symbol Device:R
- added R305, R307, R309, R310: 1R0, Resistor_SMD:R_0603_1608Metric_Pad0.98x0.95mm_HandSolder, symbol Device:R
- added R306, R308: DNI, Resistor_SMD:R_0603_1608Metric_Pad0.98x0.95mm_HandSolder, symbol Device:R
- added RV301: POT 0.375 10K, GeneralPurposeAlarmDevicePCB:Potentiometer_Bourns_3386P_Vertical, symbol GPAD_SCH_LIB:POT 0.375 10K
- added TP401: Vcc_LCD, TestPoint:TestPoint_Loop_D2.54mm_Drill1.5mm_Beaded, symbol Connector:TestPoint
- added TP402: nINT, TestPoint:TestPoint_Loop_D2.54mm_Drill1.5mm_Beaded, symbol Connector:TestPoint
- added U301: PCF8574AT_3_518, Package_SO:SOIC-16W_7.5x10.3mm_P1.27mm, symbol GPAD_SCH_LIB:PCF8574AT_3_518
- added U302: LCD_20x4_Character-GPAD_SCH_LIB, GPAD:LCD_2004A, symbol GPAD_SCH_LIB:LCD_20x4_Character-GPAD_SCH_LIB
Connections:
- new net: R311.1, R312.2, U301.7 (P3)
- new net: R302.1, R307.1, U301.2 (A1)
- new net: Q301.1 (G), R312.1
- new net: R303.1, R309.1, U301.1 (A0)
- new net: U301.10 (P5), U302.12 (DB5)
- new net: U301.11 (P6), U302.13 (DB6)
- new net: U301.12 (P7), U302.14 (DB7)
- new net: R304.1, TP402.1, U301.13 (~{INT})
- new net: R301.1, R305.1, U301.3 (A2)
- new net: U301.4 (P0), U302.4 (RS)
- new net: U301.5 (P1), U302.5 (R/W)
- new net: U301.6 (P2), U302.6 (E)
- new net: U301.9 (P4), U302.11 (DB4)
- new net: R306.1, R308.2, RV301.2, U302.3 (VO)
- new net: Q301.3 (D), U302.16 (K)
- new net +5V: R310.2
- new net GND: C301.2, C302.2, Q301.2 (S), R305.2, R307.2, R308.1, R309.2, RV301.1, U301.8 (VSS), U302.1 (VSS), U302.10 (DB3), U302.17 (MH1), U302.18 (MH2), U302.19 (MH3), U302.20 (MH4), U302.7 (DB0), U302.8 (DB1), U302.9 (DB2)
- new net SCL: U301.14 (SCL)
- new net SDA: U301.15 (SDA)
- new net Vcc_LCD: C301.1, C302.1, R301.2, R302.2, R303.2, R304.2, R306.2, R310.1, R311.2, RV301.3, TP401.1, U301.16 (VDD), U302.15 (A), U302.2 (VDD)
Other:
- note added: "LCD compnents including I2C interface."
- note added: "Wiring of I2C to LCD from: https://alselectro.wordpress.com/2016/05/12/serial-lcd-i2c-module-pcf8574/"
