File: Krake_V1/Krake_V1.kicad_sch (KiCad schematic)
At the start: 61 parts, among them J1 Barrel_Jack_Switch_SMT, Q301 BSS138, U1 LM7805_TO220, U301 PCF8574AT_3_518, U302 LCD_20x4_Character-GPAD_SCH_L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

Commit message: The arduino IDE file replaced the older IDE file. This Arduino IDE contains LCD print and a mute button.
Parts:
- added H4: MountingHole_Pad_3.5mm, GeneralPurposeAlarmDevicePCB:MountingHole_3.5mm_Pad_Via, symbol GPAD_SCH_LIB:MountingHole_Pad_3.5mm
- added R1: LDR03, OptoDevice:R_LDR_10x8.5mm_P7.6mm_Vertical, symbol Sensor_Optical:LDR03
- D1: DK_Detail_Page /product-detail/en/lite-on-inc/LTL2R3KEK/160-1682-ND/573572 -> /product-detail/en/lite-on-inc/LTW-2R3D7/160-1772-ND/1277121; Digi-Key_PN 160-1682-ND -> 160-1772-ND; MPN (none) -> LTW-2R3D7
- D3, D4, D5, D6, D7, D8: footprint PubInv_KiCad_PCB:LED_5mm_Radial -> GeneralPurposeAlarmDevicePCB:LED_5mm_Radial; DK_Detail_Page /product-detail/en/lite-on-inc/LTL2R3KEK/160-1682-ND/573572 -> /product-detail/en/lite-on-inc/LTW-2R3D7/160-1772-ND/1277121; Digi-Key_PN 160-1682-ND -> 160-1772-ND; MPN (none) -> LTW-2R3D7
- H2, H3, H4: footprint PubInv_KiCad_PCB:MountingHole_3.5mm_Pad_Via -> GeneralPurposeAlarmDevicePCB:MountingHole_3.5mm_Pad_Via
- J1: footprint PubInv_KiCad_PCB:BarrelJack_CLIFF_FC681465S_SMT_Horizontal -> GeneralPurposeAlarmDevicePCB:BarrelJack_CLIFF_FC681465S_SMT_Horizontal
- MF1: Distributor 1 Nagham -> PublicInvention; Distributor 1 PN ENCLOSURE_KiCad-Krake_VER1 -> ENCLOSURE_GPAD_VER1
- U302: footprint GeneralPurposeAlarmDevicePCB:LCD_2004A -> GPAD:LCD_2004A; Distributor 1 eBay Aliexpress -> Aliexpress; Distributor 1 PN 403534100457 -> https://www.aliexpress.com/item/3256803213374992.html; Distributor 2 Amazon / Aliexpress -> Amazon; Distributor 2 PN https://www.amazon.com/GeeekPi-Interface-Adapter-Backlight-Raspberry/dp/B07QLRD3TM/ref=sr_1_2 / https://www.aliexpress.com/item/3256803213374992.html -> https://www.amazon.com/GeeekPi-Interface-Adapter-Backlight-Raspberry/dp/B07QLRD3TM/ref=sr_1_2
- gave numbers to parts that had none: 2
Connections:
- net GND: now also H4.1, R1.1
- net SCL: now also ESP1.17 (O22); no longer ESP1.24 (TX2)
- net SDA: now also ESP1.20 (O21); no longer ESP1.25 (RX2)
- net at ESP1.12 (O34): now also R1.2
- net at ESP1.18 (TX0): no longer DF_Player1.2 (RX)
- net at ESP1.19 (RX0): no longer DF_Player1.3 (TX)
- new net: DF_Player1.2 (RX), ESP1.24 (TX2)
- new net: DF_Player1.3 (TX), ESP1.25 (RX2)
- no-connect marks 12 -> 22
Other:
- removed sheet LCD
- note added: "Mute Button"
- moved on the sheet: C301, C302, Q301, R301, R302, R303, R304, R305, R306, R307, R308, R309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

Commit message: schematic and PCB update.
Parts:
- DF_Player1: footprint (none) -> DF_PLAYER1:DF PLAYER
- LS1: footprint (none) -> speaker:Speaker
- U302: footprint GPAD:LCD_2004A -> LCD 20x4Library:LCD_2004A
Connections:
- net GND: now also DF_Player1.8 (SPK_2), LS1.1
- net Vcc_LCD: no longer C301.1, C302.1, R301.2, R302.2, R303.2, R304.2, R306.2, R310.1, R311.2, RV301.3, TP401.1, U301.16 (VDD), U302.15 (A), U302.2 (VDD)
- net SCL: no longer names the net of ESP1.17 (O22), U301.14 (SCL)
- net SDA: no longer names the net of ESP1.20 (O21), U301.15 (SDA)
- new net: C301.1, C302.1, R301.2, R302.2, R303.2, R304.2, R306.2, R310.1, R311.2, RV301.3, TP401.1, U301.16 (VDD), U302.15 (A), U302.2 (VDD)
Other:
- moved on the sheet: C1, C2, C3, C301, C302, C4, C5, C6, C7, D1, D2, D3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

Commit message: Update the PCBA And Edit the ESP32 Footprint
Other:
- note added: "ON /OFF Button"
Changed lines of the file:
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@@
+    (effects (font (size 1.27 1.27)) (justify left bottom))
+  )
+  (text "ON /OFF Button" (at 12.446 59.69 0)
     (effects (font (size 1.27 1.27)) (justify left bottom))
   )
