File: Krake_V1/Krake_V1.kicad_pcb (KiCad board)
At the start: 2 copper layers, 60 parts, among them J1 Barrel_Jack_Switch_SMT, Q1 BSS138, U1 LM7805_TO220, U2 PCF8574AT_3_518, U3 LCD_20x4_Character-GPAD_SCH_L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

Commit message: schematic and PCB update.
Parts:
- removed S1, S2: SWITCH_TACTILE_SPST-NO_0.05A_24V, PubInv_KiCad_PCB:Switch_Tactile_THT_6x6mm
- added DF_Player1: ~, DF_PLAYER1:DF PLAYER, F.Cu at (139.8, 88.5)
- added LS1: Speaker, speaker:Speaker, F.Cu at (145.4, 115.1)
- D2, D3, D4, D5, D6, D7: footprint PubInv_KiCad_PCB:LED_5mm_Radial -> GeneralPurposeAlarmDevicePCB:LED_5mm_Radial; moved to B.Cu
- D8: moved to B.Cu
- H1, H2, H3, H4: footprint PubInv_KiCad_PCB:MountingHole_3.5mm_Pad_Via -> GeneralPurposeAlarmDevicePCB:MountingHole_3.5mm_Pad_Via
- J1: footprint PubInv_KiCad_PCB:BarrelJack_CLIFF_FC681465S_SMT_Horizontal -> GeneralPurposeAlarmDevicePCB:BarrelJack_CLIFF_FC681465S_SMT_Horizontal
- U3: footprint GeneralPurposeAlarmDevicePCB:LCD_2004A -> LCD 20x4Library:LCD_2004A
- moved D2 453.3 mm to (213.4, 80.4)
- moved D6 451.6 mm to (213.3, 95.2)
- moved D3 449.4 mm to (213.4, 72.8)
- moved D7 447.9 mm to (213.3, 87.5)
- moved D5 444.5 mm to (213.4, 57.5)
- moved D4 441.4 mm to (213.4, 65.1)
- moved R16 438.1 mm to (214.4, 38.9), turned to 90 degrees
- moved R14 434.3 mm to (209.9, 38.8), turned to 90 degrees
- moved R13 432.4 mm to (207.4, 38.8), turned to 90 degrees
- moved R15 431.6 mm to (212.4, 38.9), turned to 90 degrees
- moved R18 427.8 mm to (205.0, 38.9), turned to 90 degrees
- moved R17 425.8 mm to (202.3, 38.9), turned to 90 degrees
- moved U3 329.3 mm to (168.0, -29.8), turned to 180 degrees
- moved H1 185.3 mm to (220.0, 28.1)
- moved H2 179.2 mm to (219.9, 121.1)
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Connections:
- net /Vcc_LCD renamed Net-(U2-VDD)
- ESP1 pad 17: unconnected-(ESP1-O22-Pad17) -> Net-(ESP1-O22)
- ESP1 pad 18: Net-(DF_Player1-RX) -> unconnected-(ESP1-TX0-Pad18)
- ESP1 pad 19: Net-(DF_Player1-TX) -> unconnected-(ESP1-RX0-Pad19)
- ESP1 pad 20: unconnected-(ESP1-O21-Pad20) -> Net-(ESP1-O21)
- ESP1 pad 24: /SCL -> Net-(DF_Player1-RX)
- ESP1 pad 25: /SDA -> Net-(DF_Player1-TX)
- U2 pad 14: /SCL -> Net-(ESP1-O22)
- U2 pad 15: /SDA -> Net-(ESP1-O21)
Routing:
- net Net-(ESP1-O15): track 0.00 -> 76.5 mm, vias 0 -> 2
- net Net-(ESP1-O2): track 0.00 -> 73.4 mm, vias 0 -> 2
- net Net-(ESP1-O4): track 0.00 -> 71.1 mm, vias 0 -> 2
- net Net-(D6-Pad1): track 0.00 -> 62.8 mm, vias 0 -> 2
- net Net-(U2-A1): track 2.26 -> 61.1 mm, vias 0 -> 2
- net Net-(ESP1-O5): track 0.00 -> 57.1 mm, vias 0 -> 2
- net Net-(D8-Pad1): track 13.7 -> 70.8 mm, vias 0 -> 2
- net Net-(D7-Pad1): track 0.00 -> 55.4 mm, vias 0 -> 2
- net Net-(ESP1-O34): track 0.00 -> 55.3 mm
- net Net-(DF_Player1-SPK_1): track 0.00 -> 54.1 mm, vias 0 -> 2
- net Net-(ESP1-O18): track 0.00 -> 52.4 mm, vias 0 -> 2
- net Net-(D2-Pad1): track 0.00 -> 46.7 mm, vias 0 -> 2
- net Net-(ESP1-3V3): track 60.0 -> 105.6 mm, vias 0 -> 2
- net Net-(ESP1-O19): track 0.00 -> 42.7 mm, vias 0 -> 2
- net Net-(Q1-G): track 47.0 -> 7.93 mm
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- added copper zone on F.Cu, net GND
Other:
- board outline added: 107.5 x 102 mm
- copper layers 2 -> 4

Commit message: Placed the files for LCD debugging in a factory test file.
Routing:
- net Net-(ESP1-O4): track 71.1 -> 66.5 mm
- net Net-(ESP1-O5): track 57.1 -> 52.5 mm
- net Net-(ESP1-O2): track 73.4 -> 71.6 mm
Changed lines of the file:
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@@
   (via (at 202.325 34.175) (size 0.5) (drill 0.3) (layers "F.Cu" "B.Cu") (net 31))
   (via (at 191 63.9) (size 0.5) (drill 0.3) (layers "F.Cu" "B.Cu") (net 31))
-  (segment (start 202.325 34.175) (end 194.975 34.175) (width 0.5) (layer "B.Cu") (net 31))
-  (segment (start 190.975 63.875) (end 191 63.9) (width 0.5) (layer "B.Cu") (net 31))
-  (segment (start 187.25 40.875) (end 188.55 42.175) (width 0.5) (layer "B.Cu") (net 31))
-  (segment (start 194.975 34.175) (end 193.828079 34.175) (width 0.5) (layer "B.Cu") (net 31))
-  (segment (start 190.975 42.5) (end 190.975 63.875) (width 0.5) (layer "B.Cu") (net 31))
-  (segment (start 188.875 42.5) (end 190.975 42.5) (width 0.5) (layer "B.Cu") (net 31))
-  (segment (start 188.55 42.175) (end 188.875 42.5) (width 0.5) (layer "B.Cu") (net 31))
-  (segment (start 193.828079 34.175) (end 187.25 40.753079) (width 0.5) (layer "B.Cu") (net 31))
-  (segment (start 187.25 40.753079) (end 187.25 40.875) (width 0.5) (layer "B.Cu") (net 31))
+  (segment (start 197.612 32.512) (end 196.85 31.75) (width 0.5) (layer "B.Cu") (net 31))
+  (segment (start 193.802 31.75) (end 191.625 33.927) (width 0.5) (layer "B.Cu") (net 31))
+  (segment (start 197.612 34.036) (end 197.612 32.512) (width 0.5) (layer "B.Cu") (net 31))
+  (segment (start 196.85 31.75) (end 193.802 31.75) (width 0.5) (layer "B.Cu") (net 31))
+  (segment (start 197.751 34.175) (end 197.612 34.036) (width 0.5) (layer "B.Cu") (net 31))
+  (segment (start 191.625 63.275) (end 191 63.9) (width 0.5) (layer "B.Cu") (net 31))
+  (segment (start 202.325 34.175) (end 197.751 34.175) (width 0.5) (layer "B.Cu") (net 31))
+  (segment (start 191.625 33.927) (end 191.625 63.275) (width 0.5) (layer "B.Cu") (net 31))
   (segment (start 195.835 69.2916) (end 192.4334 69.2916) (width 0.5) (layer "F.Cu") (net 32))
   (segment (start 192.4334 69.2916) (end 192.325 69.4) (width 0.5) (layer "F.Cu") (net 32))
@@
   (via (at 192.325 69.4) (size 0.5) (drill 0.3) (layers "F.Cu" "B.Cu") (net 32))
   (via (at 204.975 35.05) (size 0.5) (drill 0.3) (layers "F.Cu" "B.Cu") (net 32))
-  (segment (start 189.731971 41.075) (end 192.25 41.075) (width 0.5) (layer "B.Cu") (net 32))
-  (segment (start 192.25 69.325) (end 192.325 69.4) (width 0.5) (layer "B.Cu") (net 32))
-  (segment (start 196.125 35.075) (end 196.15 35.05) (width 0.5) (layer "B.Cu") (net 32))
-  (segment (start 196.810051 35.05) (end 196.785051 35.075) (width 0.5) (layer "B.Cu") (net 32))
-  (segment (start 193.943029 35.05) (end 188.825 40.168029) (width 0.5) (layer "B.Cu") (net 32))
-  (segment (start 196.785051 35.075) (end 196.05 35.075) (width 0.5) (layer "B.Cu") (net 32))
-  (segment (start 188.825 40.168029) (end 189.731971 41.075) (width 0.5) (layer "B.Cu") (net 32))
-  (segment (start 196.15 35.05) (end 193.943029 35.05) (width 0.5) (layer "B.Cu") (net 32))
+  (segment (start 196.810051 35.05) (end 196.046051 35.814) (width 0.5) (layer "B.Cu") (net 32))
+  (segment (start 196.046051 35.814) (end 193.179029 35.814) (width 0.5) (layer "B.Cu") (net 32))
+  (segment (start 192.325 36.668029) (end 192.325 69.4) (width 0.5) (layer "B.Cu") (net 32))
   (segment (start 204.975 35.05) (end 196.810051 35.05) (width 0.5) (layer "B.Cu") (net 32))
-  (segment (start 196.05 35.075) (end 196.125 35.075) (width 0.5) (layer "B.Cu") (net 32))
-  (segment (start 192.25 41.075) (end 192.25 69.325) (width 0.5) (layer "B.Cu") (net 32))
+  (segment (start 193.179029 35.814) (end 192.325 36.668029) (width 0.5) (layer "B.Cu") (net 32))
   (segment (start 150.8 62.225) (end 148.45 62.225) (width 0.5) (layer "F.Cu") (net 34))
   (via (at 148.45 62.225) (size 0.5) (drill 0.3) (layers "F.Cu" "B.Cu") (net 34))
@@
   (via (at 207.425 35.825) (size 0.5) (drill 0.3) (layers "F.Cu" "B.Cu") (net 35))
   (via (at 193.15 84.425) (size 0.5) (drill 0.3) (layers "F.Cu" "B.Cu") (net 35))
-  (segment (start 190.15 39.832979) (end 192.807979 39.832979) (width 0.5) (layer "B.Cu") (net 35))
-  (segment (start 194.207979 35.775) (end 190.15 39.832979) (width 0.5) (layer "B.Cu") (net 35))
-  (segment (start 196.975 35.775) (end 194.207979 35.775) (width 0.5) (layer "B.Cu") (net 35))
+  (segment (start 193.15 37.736) (end 193.15 84.4) (width 0.5) (layer "B.Cu") (net 35))
+  (segment (start 194.31 36.576) (end 193.15 37.736) (width 0.5) (layer "B.Cu") (net 35))
+  (segment (start 207.425 35.825) (end 197.025 35.825) (width 0.5) (layer "B.Cu") (net 35))
   (segment (start 193.15 84.4) (end 193.15 84.425) (width 0.5) (layer "B.Cu") (net 35))
+  (segment (start 196.274 36.576) (end 194.31 36.576) (width 0.5) (layer "B.Cu") (net 35))
   (segment (start 193.15 84.425) (end 193.125 84.425) (width 0.5) (layer "B.Cu") (net 35))
-  (segment (start 193.2 40.225) (end 193.2 84.35) (width 0.5) (layer "B.Cu") (net 35))
-  (segment (start 193.2 84.35) (end 193.15 84.4) (width 0.5) (layer "B.Cu") (net 35))
-  (segment (start 207.425 35.825) (end 197.025 35.825) (width 0.5) (layer "B.Cu") (net 35))
-  (segment (start 192.807979 39.832979) (end 193.2 40.225) (width 0.5) (layer "B.Cu") (net 35))
+  (segment (start 197.025 35.825) (end 196.274 36.576) (width 0.5) (layer "B.Cu") (net 35))
   (segment (start 193.125 84.425) (end 193.15 84.4) (width 0.5) (layer "B.Cu") (net 35))
-  (segment (start 197.025 35.825) (end 196.975 35.775) (width 0.5) (layer "B.Cu") (net 35))
   (segment (start 209.9 37.925) (end 209.875 37.9) (width 0.5) (layer "F.Cu") (net 36))
   (segment (start 193.6634 89.6116) (end 193.65 89.625) (width 0.5) (layer "F.Cu") (net 36))
@@
   (via (at 209.875 36.625) (size 0.5) (drill 0.3) (layers "F.Cu" "B.Cu") (net 36))
   (via (at 193.65 89.625) (size 0.5) (drill 0.3) (layers "F.Cu" "B.Cu") (net 36))
-  (segment (start 193.536777 37.711777) (end 194.25 38.425) (width 0.5) (layer "B.Cu") (net 36))
-  (segment (start 209.875 36.625) (end 197.6 36.625) (width 0.5) (layer "B.Cu") (net 36))
-  (segment (start 194.470477 36.502451) (end 193.261151 37.711777) (width 0.5) (layer "B.Cu") (net 36))
-  (segment (start 193.261151 37.711777) (end 193.536777 37.711777) (width 0.5) (layer "B.Cu") (net 36))
-  (segment (start 196.353272 36.675) (end 196.180723 36.502451) (width 0.5) (layer "B.Cu") (net 36))
-  (segment (start 197.55 36.675) (end 196.353272 36.675) (width 0.5) (layer "B.Cu") (net 36))
-  (segment (start 196.180723 36.502451) (end 194.470477 36.502451) (width 0.5) (layer "B.Cu") (net 36))
-  (segment (start 194.25 38.425) (end 194.25 89.025) (width 0.5) (layer "B.Cu") (net 36))
-  (segment (start 194.25 89.025) (end 193.65 89.625) (width 0.5) (layer "B.Cu") (net 36))
-  (segment (start 197.6 36.625) (end 197.55 36.675) (width 0.5) (layer "B.Cu") (net 36))
+  (segment (start 194.056 89.219) (end 193.65 89.625) (width 0.5) (layer "B.Cu") (net 36))
+  (segment (start 194.056 38.1) (end 194.056 89.219) (width 0.5) (layer "B.Cu") (net 36))
+  (segment (start 196.596 37.338) (end 194.818 37.338) (width 0.5) (layer "B.Cu") (net 36))
+  (segment (start 197.309 36.625) (end 196.596 37.338) (width 0.5) (layer "B.Cu") (net 36))
+  (segment (start 194.818 37.338) (end 194.056 38.1) (width 0.5) (layer "B.Cu") (net 36))
+  (segment (start 209.875 36.625) (end 197.309 36.625) (width 0.5) (layer "B.Cu") (net 36))
   (segment (start 212.425 37.9625) (end 212.425 36.675) (width 0.5) (layer "F.Cu") (net 37))
   (segment (start 195.835 94.6916) (end 198.0666 94.6916) (width 0.5) (layer "F.Cu") (net 37))

Commit message: Update the PCBA And Edit the ESP32 Footprint
Parts:
- removed H3, H4: MountingHole_Pad_3.5mm, GeneralPurposeAlarmDevicePCB:MountingHole_3.5mm_Pad_Via
- U3: moved to B.Cu
- moved U3 133.2 mm to (122.8, 95.5), turned to 90 degrees
- moved J1 118.5 mm to (95.8, 73.8), turned to 0 degrees
- moved F1 115.9 mm to (98.0, 60.2), turned to -90 degrees
- moved LS1 64.8 mm to (101.8, 67.1), turned to 90 degrees
- moved TP4 51.0 mm to (184.4, 82.0)
- moved C4 46.2 mm to (113.6, 140.3)
- moved C1 45.6 mm to (124.6, 134.5)
- moved C7 45.6 mm to (123.0, 143.2)
- moved C8 45.6 mm to (110.0, 82.7)
- moved ESP1 45.6 mm to (148.4, 53.9)
- moved R10 45.6 mm to (114.4, 85.2)
- moved R11 45.6 mm to (114.4, 87.7)
- moved R12 45.6 mm to (114.4, 90.2)
- moved R14 45.6 mm to (180.6, 73.8)
- moved R15 45.6 mm to (183.1, 73.8)
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Routing:
- net Net-(U2-VDD): track 54.4 -> 286.7 mm
- net GND: track 48.3 -> 235.3 mm, vias 2 -> 8
- net +5V: track 67.5 -> 228.6 mm, vias 1 -> 3
- net Net-(DF_Player1-RX): track 0.00 -> 133.5 mm
- net Net-(DF_Player1-TX): track 0.00 -> 111.0 mm
- net Net-(Q1-D): track 0.00 -> 88.2 mm, vias 0 -> 2
- net Net-(D1-A): track 0.00 -> 85.8 mm, vias 0 -> 2
- net Net-(ESP1-O21): track 2.35 -> 87.2 mm, vias 1 -> 2
- net Net-(U2-P0): track 2.43 -> 58.9 mm
- net Net-(U2-P1): track 2.41 -> 56.0 mm, vias 1 -> 2
- net Net-(ESP1-O22): track 2.36 -> 55.7 mm, vias 1 -> 0
- net Net-(U2-P3): track 9.14 -> 56.0 mm, vias 1 -> 2
- net Net-(U2-P2): track 2.40 -> 46.2 mm
- net +3.3V: track 10.7 -> 54.1 mm, vias 0 -> 2
- net Net-(U2-~{INT}): track 36.9 -> 79.1 mm
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- added copper zone on B.Cu, net GND
- added copper zone on In1.Cu, net GND
- added copper zone on In2.Cu, net GND
Other:
- board size 107.5 x 102 mm -> 98.4 x 102.4 mm

Commit message: Adding Rotary Encoder to Krake
Parts:
- removed DF_Player1: ~, DF_PLAYER1:DF PLAYER
- removed ESP1: ~, esp32 15 pin Library:esp32
- removed LS1: Speaker, speaker:Speaker
- removed U3: LCD_20x4_Character-GPAD_SCH_LIB, LCD 20x4Library:LCD_2004A
- added ESP32_DEVKITV1: ~, esp32 15 pin Library:esp32, F.Cu at (135.0, 60.2)
- added H3: MountingHole_Pad_3.5mm, GeneralPurposeAlarmDevicePCB:MountingHole_3.5mm_Pad_Via, F.Cu at (183.9, 128.3)
- added H4: MountingHole_Pad_3.5mm, GeneralPurposeAlarmDevicePCB:MountingHole_3.5mm_Pad_Via, F.Cu at (128.2, 126.2)
- added J2: SPK, Connector_PinHeader_1.27mm:PinHeader_1x02_P1.27mm_Vertical, F.Cu at (132.1, 73.7)
- added J3: 5_DFPLAYER1, Connector_PinHeader_1.00mm:PinHeader_1x09_P1.00mm_Vertical, F.Cu at (129.2, 68.7)
- added J4_LCD1: Conn_01x04, Connector_PinSocket_2.54mm:PinSocket_1x04_P2.54mm_Vertical, F.Cu at (129.5, 54.4)
- added TP6: TestPoint, TestPoint:TestPoint_Loop_D2.54mm_Drill1.5mm_Beaded, F.Cu at (183.1, 76.3)
- D2, D3, D4, D5, D6, D7, D8: moved to F.Cu
- moved Q1 109.9 mm to (37.5, 140.1)
- moved H2 102.5 mm to (182.8, 39.4), turned to 90 degrees
- moved D6 95.7 mm to (146.8, 37.9), turned to 90 degrees
- moved J1 91.4 mm to (180.1, 109.3), turned to 180 degrees
- moved D7 86.5 mm to (153.7, 37.9), turned to 90 degrees
- moved C5 86.0 mm to (178.3, 88.6), turned to 90 degrees
- moved C7 84.6 mm to (182.4, 82.9), turned to 90 degrees
- moved TP1 84.6 mm to (170.2, 116.7)
- moved C4 84.3 mm to (182.4, 91.5), turned to 90 degrees
- moved C8 83.5 mm to (37.2, 123.5)
- moved R10 83.5 mm to (41.6, 126.0)
- moved R12 83.5 mm to (41.6, 131.1)
- moved R5 83.5 mm to (41.6, 113.5)
- moved R6 83.5 mm to (41.6, 116.0)
- moved R7 83.5 mm to (41.6, 118.5)
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Connections:
- U2 pad 14: Net-(ESP1-O22) -> unconnected-(U2-SCL-Pad14)
- U2 pad 15: Net-(ESP1-O21) -> unconnected-(U2-SDA-Pad15)
Routing:
- net Net-(U2-VDD): track 286.7 -> 0.00 mm, vias 1 -> 0
- net GND: track 235.3 -> 0.00 mm, vias 8 -> 0
- net +5V: track 228.6 -> 0.00 mm, vias 3 -> 0
- net Net-(DF_Player1-RX): track 133.5 -> 0.00 mm
- net Net-(DF_Player1-TX): track 111.0 -> 0.00 mm
- net Net-(ESP32_DEVKITV1-3V3): track 105.4 -> 0.00 mm, vias 2 -> 0
- net Net-(Q1-D): track 88.2 -> 0.00 mm, vias 2 -> 0
- net Net-(ESP1-O21): track 87.2 -> 0.00 mm, vias 2 -> 0
- net Net-(D1-A): track 85.8 -> 0.00 mm, vias 2 -> 0
- net Net-(U3-VO): track 80.5 -> 0.00 mm
- net Net-(U2-~{INT}): track 79.1 -> 0.00 mm, vias 2 -> 0
- net Net-(ESP32_DEVKITV1-GPIO15): track 76.5 -> 0.00 mm, vias 2 -> 0
- net Net-(ESP32_DEVKITV1-GPIO2): track 70.7 -> 0.00 mm, vias 2 -> 0
- net Net-(D8-Pad1): track 67.8 -> 0.00 mm, vias 1 -> 0
- net Net-(ESP32_DEVKITV1-GPIO4): track 66.5 -> 0.00 mm, vias 2 -> 0
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- removed copper zone on B.Cu, net GND
- removed copper zone on F.Cu, net GND
- removed copper zone on In1.Cu, net GND
- removed copper zone on In2.Cu, net GND
Other:
- board outline removed
