File: PCBa_KRAKE/PCBa_KRAKE.kicad_sch (KiCad schematic)
At the start: 55 parts, among them J101 Barrel_Jack_Switch_SMT, J102 0.100_2Pin, J103 0.100_2Pin, J105 S04B-XASK-1(LF)(SN)Rev2, U101 LM7805_TO220, U102 PI_ATMEGA328P-AU-InOrder

Commit message: Adding ESP32_WROOM_32D symbol library and schematic in the GPAD_SCH_LIB.kicad_sym and editted the visibility of PINS 15 38 39 and 32 and canged their electical type.
Parts:
- added U999: ESP32-WROOM-32D, RF_Module:ESP32-WROOM-32D, symbol GPAD_SCH_LIB:ESP32-WROOM-32D-PINORDER
Connections:
- net GND: now also U999.1 (GND), U999.15 (GND), U999.38 (GND), U999.39 (GND)

Commit message: Deleted the 16mhz quarts crystal, deleted the sheild footprint.
Parts:
- removed A101: Arduino_UNO_R3_Shield, GeneralPurposeAlarmDevicePCB:Arduino_UNO_R3_NoMountingHoles3D, symbol GPAD_SCH_LIB:Arduino_UNO_R3_Shield
- removed C104, C107: 39pF, Capacitor_SMD:C_0603_1608Metric_Pad1.08x0.95mm_HandSolder, symbol Device:C
- removed R111: 330R, Resistor_SMD:R_0603_1608Metric_Pad0.98x0.95mm_HandSolder, symbol Device:R
- removed XTAL101: 16MHZ 20PF HC-49S/SMD, Crystal:Crystal_SMD_HC49-SD, symbol Device:Crystal
Connections:
- net GND: no longer U999.1 (GND), U999.15 (GND), U999.38 (GND), U999.39 (GND)

Commit message: Connected the SPI bus to the ESP32.
Connections:
- net CIPO: now also U999.8 (IO32)
- net COPI: now also U999.11 (IO26)
- net SPI_SCK: now also U999.10 (IO25)
- net nCS: now also U999.9 (IO33)
Changed lines of the file:
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@@
+    (stroke (width 0) (type default))
+  )
+  (wire (pts (xy -53.34 109.22) (xy -35.56 109.22))
     (stroke (width 0) (type default))
   )
@@
     (stroke (width 0) (type default))
   )
+  (wire (pts (xy -53.34 114.3) (xy -35.56 114.3))
+    (stroke (width 0) (type default))
+  )
   (wire (pts (xy 60.96 66.04) (xy 60.96 86.36))
     (stroke (width 0) (type default))
   )
+  (wire (pts (xy -54.61 116.84) (xy -35.56 116.84))
+    (stroke (width 0) (type default))
+  )
   (wire (pts (xy 52.07 97.79) (xy 57.15 97.79))
     (stroke (width 0) (type default))
@@
   )
   (wire (pts (xy 74.93 87.63) (xy 72.39 87.63))
+    (stroke (width 0) (type default))
+  )
+  (wire (pts (xy -54.61 111.76) (xy -35.56 111.76))
     (stroke (width 0) (type default))
   )
@@
     )
   )
+  (global_label "SPI_SCK" (shape input) (at -53.34 114.3 180) (fields_autoplaced)
+    (effects (font (size 1.27 1.27)) (justify right))
+    (property "Intersheetrefs" "${INTERSHEET_REFS}" (at -63.393 114.3 0)
+      (effects (font (size 1.27 1.27)) (justify right) hide)
+    )
+  )
   (global_label "ControllerTX" (shape input) (at 50.8 184.15 0) (fields_autoplaced)
     (effects (font (size 1.27 1.27)) (justify left))
@@
     )
   )
+  (global_label "nCS" (shape input) (at -54.61 111.76 180) (fields_autoplaced)
+    (effects (font (size 1.27 1.27)) (justify right))
+    (property "Intersheetrefs" "${INTERSHEET_REFS}" (at -60.4901 111.76 0)
+      (effects (font (size 1.27 1.27)) (justify right) hide)
+    )
+  )
   (global_label "Attenuate" (shape output) (at 72.39 93.98 180) (fields_autoplaced)
     (effects (font (size 1.27 1.27)) (justify right))
@@
     )
   )
+  (global_label "CIPO" (shape output) (at -53.34 109.22 180) (fields_autoplaced)
+    (effects (font (size 1.27 1.27)) (justify right))
+    (property "Intersheetrefs" "${INTERSHEET_REFS}" (at -60.0669 109.22 0)
+      (effects (font (size 1.27 1.27)) (justify right) hide)
+    )
+  )
   (global_label "nCS" (shape output) (at 96.52 157.48 180) (fields_autoplaced)
     (effects (font (size 1.27 1.27)) (justify right))
@@
       (effects (font (size 1.27 1.27)) (justify right) hide)
     )
+  )
+  (global_label "COPI" (shape input) (at -54.61 116.84 180) (fields_autoplaced)
+    (effects (font (size 1.27 1.27)) (justify right))
+    (property "Intersheetrefs" "${INTERSHEET_REFS}" (at -61.3369 116.84 0)
+      (effects (font (size 1.27 1.27)) (justify right) hide)
+    )

Commit message: replaced the ATMEGA328P with esp32_wroom_32D
Parts:
- added C? (x2): 100nF, Capacitor_SMD:C_0603_1608Metric_Pad1.08x0.95mm_HandSolder, symbol Device:C
- added C?: 47uF 16V, Capacitor_SMD:CP_Elec_5x5.4, symbol Device:C_Polarized
- added D?: Schottky 2A, Diode_SMD:D_SMB, symbol Device:D_Schottky
- added R?: 10K, Resistor_SMD:R_0603_1608Metric_Pad0.98x0.95mm_HandSolder, symbol Device:R
- added R?: 1R0, Resistor_SMD:R_0603_1608Metric_Pad0.98x0.95mm_HandSolder, symbol Device:R
- added S?: SWITCH_TACTILE_SPST-NO_0.05A_24V, GeneralPurposeAlarmDevicePCB:Switch_Tactile_THT_6x6mm, symbol GPAD_SCH_LIB:SWITCH_TACTILE_SPST-NO_0.05A_24V
- added TP?: VccController, TestPoint:TestPoint_Loop_D2.54mm_Drill1.5mm_Beaded, symbol Connector:TestPoint
Connections:
- net +5V: now also R?.2
- net Attenuate: now also U999.12 (IO27)
- net ControllerRX: now also U999.35 (TXD0/IO1)
- net ControllerTX: now also U999.34 (RXD0/IO3)
- net GND: now also U999.1 (GND), U999.15 (GND), U999.38 (GND), U999.39 (GND), C?.2, C?.2, S?.3, S?.4
- net Light0: now also U999.26 (IO4)
- net Light1: now also U999.29 (IO5)
- net Light2: now also U999.14 (IO12)
- net Light3: now also U999.16 (IO13)
- net Light4: now also U999.13 (IO14)
- net PC0: now also U999.30 (IO18)
- net PC1: now also U999.28 (IO17)
- net PC2: now also U999.27 (IO16)
- net PC3: now also U999.24 (IO2)
- net SCL: now also U999.36 (IO22)
- net SDA: now also U999.33 (IO21)
- net Switch_Mute: now also U999.37 (IO23)
- net Tone: now also U999.23 (IO15)
- net VccController: now also U999.2 (VDD), C?.1, C?.1, D?.1 (K), R?.1, R?.2, TP?.1
- net nRESET: now also U999.31 (IO19), C?.1, D?.2 (A), R?.1, S?.1, S?.2
- net nRTS: now also C?.2
- no-connect marks 2 -> 4
Other:
- note added: "controls boot"
- moved on the sheet: C103, C106, C110, C111, C112, D102, D103, MF103, R101, R102, R103, R108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

Commit message: PCBa_KRAKE schematic fix input output pin connections to ESP32.
Connections:
- net ControllerRX: now also U999.34 (RXD0/IO3); no longer U999.35 (TXD0/IO1)
- net ControllerTX: now also U999.35 (TXD0/IO1); no longer U999.34 (RXD0/IO3)

Commit message: PCBa_KRAKE.kicad_sch all input and output signals migrated to ESP32 except the DFplayer.
Parts:
- removed C? (x2): 100nF, Capacitor_SMD:C_0603_1608Metric_Pad1.08x0.95mm_HandSolder, symbol Device:C
- removed C?: 47uF 16V, Capacitor_SMD:CP_Elec_5x5.4, symbol Device:C_Polarized
- removed D?: Schottky 2A, Diode_SMD:D_SMB, symbol Device:D_Schottky
- removed R?: 10K, Resistor_SMD:R_0603_1608Metric_Pad0.98x0.95mm_HandSolder, symbol Device:R
- removed R?: 1R0, Resistor_SMD:R_0603_1608Metric_Pad0.98x0.95mm_HandSolder, symbol Device:R
- removed S?: SWITCH_TACTILE_SPST-NO_0.05A_24V, GeneralPurposeAlarmDevicePCB:Switch_Tactile_THT_6x6mm, symbol GPAD_SCH_LIB:SWITCH_TACTILE_SPST-NO_0.05A_24V
- removed TP?: VccController, TestPoint:TestPoint_Loop_D2.54mm_Drill1.5mm_Beaded, symbol Connector:TestPoint
Connections:
- net Attenuate: no longer U999.12 (IO27)
- net Light0: now also U999.23 (IO15); no longer U999.26 (IO4)
- net Light1: now also U999.26 (IO4); no longer U999.29 (IO5)
- net Light2: now also U999.29 (IO5); no longer U999.14 (IO12)
- net Light3: now also U999.30 (IO18); no longer U999.16 (IO13)
- net Light4: now also U999.31 (IO19); no longer U999.13 (IO14)
- net PC0: no longer U999.30 (IO18)
- net PC1: no longer U999.28 (IO17)
- net PC2: no longer U999.27 (IO16)
- net PC3: no longer U999.24 (IO2)
- net Switch_Mute: now also U999.6 (IO34); no longer U999.37 (IO23)
- net Tone: no longer U999.23 (IO15)
- net VccController: no longer U999.2 (VDD)
- net nRESET: now also U999.3 (EN); no longer U999.31 (IO19)
Other:
- moved on the sheet: C103, C106, C110, C111, C112, D102, D103, R101, R102, R103, R108, R109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

Commit message: PCBa_KRAKE.kicad_sch adding 3v3 voltage regulator.
Parts:
- added C? (x3): 47uF 16V, Capacitor_SMD:CP_Elec_5x5.4, symbol Device:C_Polarized
- added C? (x3): 100nF, Capacitor_SMD:C_0603_1608Metric_Pad1.08x0.95mm_HandSolder, symbol Device:C
- added R?: 1R0, Resistor_SMD:R_0603_1608Metric_Pad0.98x0.95mm_HandSolder, symbol Device:R
- added U?: AMS1117-3.3, Package_TO_SOT_SMD:SOT-223-3_TabPin2, symbol Regulator_Linear:AMS1117-3.3
Connections:
- net +5V: now also C?.1, C?.1, U?.3 (VI)
- net GND: now also C?.2, C?.2, C?.2, C?.2, C?.2, C?.2, U?.1 (GND)
- net at U999.2 (VDD): now also C?.1, C?.1, R?.1
- new net +3.3V: C?.1, C?.1, R?.2, U?.2 (VO)

Commit message: Adding the DFplayer schematic symbol to the GPAD_SCH_LIB.
Parts:
- added J?: Conn_01x08, symbol GPAD_SCH_LIB:DFPlayermini_241116
Changed lines of the file:
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@@
+    )
+  )
+  (symbol (lib_id "GPAD_SCH_LIB:DFPlayermini_241116") (at -173.99 138.43 0) (unit 1)
+    (in_bom yes) (on_board yes) (dnp no) (fields_autoplaced)
+    (property "Reference" "J?" (at -163.83 124.46 0)
+      (effects (font (size 1.27 1.27)))
+    )
+    (property "Value" "Conn_01x08" (at -163.83 127 0)
+      (effects (font (size 1.27 1.27)))
+    )
+    (property "Footprint" "" (at -173.99 138.43 0)
+      (effects (font (size 1.27 1.27)) hide)
+    )
+    (property "Datasheet" "~" (at -173.99 138.43 0)
+      (effects (font (size 1.27 1.27)) hide)
+    )
+    (pin "9")
+    (pin "1")
+    (pin "10")
+    (pin "11")
+    (pin "12")
+    (pin "13")
+    (pin "14")
+    (pin "15")
+    (pin "16")
+    (pin "2")
+    (pin "3")
+    (pin "4")
+    (pin "5")
+    (pin "6")
+    (pin "7")
+    (pin "8")
+    (instances
+      (project "PCBa_KRAKE"
+        (path "/412a327d-1ee3-473e-bc00-1545004b7edf"
+          (reference "J?") (unit 1)
+        )
+      )
     )
   )
