File: PCBa_KRAKE/PCBa_KRAKE.kicad_sch (KiCad schematic)
At the start: 60 parts, among them J101 Barrel_Jack_Switch_SMT, J102 0.100_2Pin, J103 0.100_2Pin, J105 S04B-XASK-1(LF)(SN)Rev2, U101 LM7805_TO220, U102 PI_ATMEGA328P-AU-InOrder, U999 ESP32-WROOM-32D

Commit message: Added the datasheet for the DFPlayer.
Parts:
- J1: renamed from J?; footprint (none) -> GeneralPurposeAlarmDevicePCB:DFPlayer_mini_20241116
- gave numbers to parts that had none: 8
Changed lines of the file:
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@@
   (symbol (lib_id "Regulator_Linear:AMS1117-3.3") (at -162.56 43.18 0) (unit 1)
     (in_bom yes) (on_board yes) (dnp no) (fields_autoplaced)
-    (property "Reference" "U?" (at -162.56 36.83 0)
+    (property "Reference" "U1" (at -162.56 36.83 0)
       (effects (font (size 1.27 1.27)))
     )
@@
       (project "PCBa_KRAKE"
         (path "/412a327d-1ee3-473e-bc00-1545004b7edf"
-          (reference "U?") (unit 1)
+          (reference "U1") (unit 1)
         )
       )
@@
   (symbol (lib_id "Device:C_Polarized") (at -137.16 48.26 0) (unit 1)
     (in_bom yes) (on_board yes) (dnp no)
-    (property "Reference" "C?" (at -134.1628 47.0916 0)
+    (property "Reference" "C6" (at -134.1628 47.0916 0)
       (effects (font (size 1.27 1.27)) (justify left))
     )
@@
       (project "PCBa_KRAKE"
         (path "/412a327d-1ee3-473e-bc00-1545004b7edf"
-          (reference "C?") (unit 1)
+          (reference "C6") (unit 1)
         )
       )
@@
   (symbol (lib_id "GPAD_SCH_LIB:DFPlayermini_241116") (at -173.99 138.43 0) (unit 1)
     (in_bom yes) (on_board yes) (dnp no) (fields_autoplaced)
-    (property "Reference" "J?" (at -163.83 124.46 0)
+    (property "Reference" "J1" (at -163.83 124.46 0)
       (effects (font (size 1.27 1.27)))
     )
@@
       (effects (font (size 1.27 1.27)))
     )
-    (property "Footprint" "" (at -173.99 138.43 0)
+    (property "Footprint" "GeneralPurposeAlarmDevicePCB:DFPlayer_mini_20241116" (at -173.99 138.43 0)
       (effects (font (size 1.27 1.27)) hide)
     )
@@
       (project "PCBa_KRAKE"
         (path "/412a327d-1ee3-473e-bc00-1545004b7edf"
-          (reference "J?") (unit 1)
+          (reference "J1") (unit 1)
         )
       )
@@
   (symbol (lib_id "Device:C_Polarized") (at -185.42 52.07 0) (unit 1)
     (in_bom yes) (on_board yes) (dnp no)
-    (property "Reference" "C?" (at -182.4228 50.9016 0)
+    (property "Reference" "C1" (at -182.4228 50.9016 0)
       (effects (font (size 1.27 1.27)) (justify left))
     )
@@
       (project "PCBa_KRAKE"
         (path "/412a327d-1ee3-473e-bc00-1545004b7edf"
-          (reference "C?") (unit 1)
+          (reference "C1") (unit 1)
         )
       )
@@
   (symbol (lib_id "Device:C_Polarized") (at -158.75 97.79 0) (unit 1)
     (in_bom yes) (on_board yes) (dnp no)
-    (property "Reference" "C?" (at -155.7528 96.6216 0)
+    (property "Reference" "C4" (at -155.7528 96.6216 0)
       (effects (font (size 1.27 1.27)) (justify left))
     )
@@
       (project "PCBa_KRAKE"
         (path "/412a327d-1ee3-473e-bc00-1545004b7edf"
-          (reference "C?") (unit 1)
+          (reference "C4") (unit 1)
         )
       )
@@
   (symbol (lib_id "Device:C") (at -172.72 97.79 0) (unit 1)
     (in_bom yes) (on_board yes) (dnp no)
-    (property "Reference" "C?" (at -169.799 96.6216 0)
+    (property "Reference" "C2" (at -169.799 96.6216 0)
       (effects (font (size 1.27 1.27)) (justify left))
     )
@@
       (project "PCBa_KRAKE"
         (path "/412a327d-1ee3-473e-bc00-1545004b7edf"
-          (reference "C?") (unit 1)
+          (reference "C2") (unit 1)
         )
       )
@@
   (symbol (lib_id "Device:C") (at -151.13 48.26 0) (unit 1)
     (in_bom yes) (on_board yes) (dnp no)
-    (property "Reference" "C?" (at -148.209 47.0916 0)
+    (property "Reference" "C5" (at -148.209 47.0916 0)
       (effects (font (size 1.27 1.27)) (justify left))
     )
@@
       (project "PCBa_KRAKE"
         (path "/412a327d-1ee3-473e-bc00-1545004b7edf"
-          (reference "C?") (unit 1)
+          (reference "C5") (unit 1)
         )
       )
@@
   (symbol (lib_id "Device:C") (at -171.45 53.34 0) (unit 1)
     (in_bom yes) (on_board yes) (dnp no)
-    (property "Reference" "C?" (at -168.529 52.1716 0)
+    (property "Reference" "C3" (at -168.529 52.1716 0)
       (effects (font (size 1.27 1.27)) (justify left))
     )
@@
       (project "PCBa_KRAKE"
         (path "/412a327d-1ee3-473e-bc00-1545004b7edf"
-          (reference "C?") (unit 1)
+          (reference "C3") (unit 1)
         )
       )
@@
   (symbol (lib_id "Device:R") (at -165.1 88.9 270) (unit 1)
     (in_bom yes) (on_board yes) (dnp no)
-    (property "Reference" "R?" (at -166.37 83.82 90)
+    (property "Reference" "R1" (at -166.37 83.82 90)
       (effects (font (size 1.27 1.27)))
     )
@@
       (project "PCBa_KRAKE"
         (path "/412a327d-1ee3-473e-bc00-1545004b7edf"
-          (reference "R?") (unit 1)
-        )
-      )
+          (reference "R1") (unit 1)
+        )
+      )

Commit message: Adding boot to load circuit, connected th DF player schematic symbol with the esp32, and editted the electric type of the module pins.
Parts:
- added LS?: Speaker, symbol Device:Speaker
- added Q998, Q999: MMBT2222ALT1G, symbol Simulation_SPICE:NPN
- added R505 (x2): 10K, Resistor_SMD:R_0603_1608Metric_Pad0.98x0.95mm_HandSolder, symbol Device:R
Connections:
- net +5V: now also J1.1 (VCC)
- net ControllerRX: now also J1.3 (TX)
- net ControllerTX: now also J1.2 (RX)
- net GND: now also J1.10 (GND), J1.7 (GND)
- net at J1.6 (SPK_1): now also LS?.2
- net at J1.8 (SPK_2): now also LS?.1
- new net: Q998.2 (B), R505.2
- new net: Q998.3 (E), R505.1
- new net: Q999.2 (B), R505.2
- new net: Q999.3 (E), R505.1
- no-connect marks 4 -> 3
Other:
- moved on the sheet: J1

Commit message: Connecting the boot circuit to the UART and move it into the UART page.
Parts:
- removed Q998, Q999: MMBT2222ALT1G, symbol Simulation_SPICE:NPN
- removed R505 (x2): 10K, Resistor_SMD:R_0603_1608Metric_Pad0.98x0.95mm_HandSolder, symbol Device:R
- added S?: SWITCH_TACTILE_SPST-NO_0.05A_24V, GeneralPurposeAlarmDevicePCB:Switch_Tactile_THT_6x6mm, symbol GPAD_SCH_LIB:SWITCH_TACTILE_SPST-NO_0.05A_24V
Connections:
- net GPIO0: now reaches U999.25 (IO0)
Other:
- sheet USB_UART ports: added GPIO0, nRESET; removed none

Commit message: Updating ESP32 schematic symbol and added the df player into the audio schematic.
Connections:
- net Busy: now reaches U999.7 (IO35)
Other:
- sheet AlarmAudio ports: added Busy, ControllerRX, ControllerTX; removed none
Changed lines of the file:
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@@
     (stroke (width 0) (type default))
   )
-  (wire (pts (xy 236.22 101.6) (xy 243.84 101.6))
+  (wire (pts (xy 236.22 107.95) (xy 243.84 107.95))
     (stroke (width 0) (type default))
   )
@@
     (stroke (width 0) (type default))
   )
+  (wire (pts (xy -127 102.87) (xy -115.57 102.87))
+    (stroke (width 0) (type default))
+  )
   (wire (pts (xy 29.21 21.59) (xy 31.75 21.59))
     (stroke (width 0) (type default))
@@
     (stroke (width 0) (type default))
   )
-  (wire (pts (xy 236.22 107.95) (xy 243.84 107.95))
+  (wire (pts (xy 236.22 114.3) (xy 243.84 114.3))
     (stroke (width 0) (type default))
   )
@@
     (stroke (width 0) (type default))
   )
+  (wire (pts (xy 241.3 101.6) (xy 243.84 101.6))
+    (stroke (width 0) (type default))
+  )
   (wire (pts (xy 71.12 104.14) (xy 64.77 104.14))
     (stroke (width 0) (type default))
@@
     (stroke (width 0) (type default))
   )
+  (wire (pts (xy 241.3 96.52) (xy 243.84 96.52))
+    (stroke (width 0) (type default))
+  )
   (wire (pts (xy 130.81 92.71) (xy 130.81 96.52))
     (stroke (width 0) (type default))
@@
     (stroke (width 0) (type default))
   )
+  (wire (pts (xy 241.3 99.06) (xy 243.84 99.06))
+    (stroke (width 0) (type default))
+  )
   (wire (pts (xy 204.47 143.51) (xy 207.01 143.51))
     (stroke (width 0) (type default))
@@
     )
   )
+  (global_label "Busy" (shape output) (at 241.3 101.6 180) (fields_autoplaced)
+    (effects (font (size 1.27 1.27)) (justify right))
+    (property "Intersheetrefs" "${INTERSHEET_REFS}" (at 234.6337 101.6 0)
+      (effects (font (size 1.27 1.27)) (justify right) hide)
+    )
+  )
+  (global_label "ControllerRX" (shape output) (at 241.3 99.06 180) (fields_autoplaced)
+    (effects (font (size 1.27 1.27)) (justify right))
+    (property "Intersheetrefs" "${INTERSHEET_REFS}" (at 227.1348 99.06 0)
+      (effects (font (size 1.27 1.27)) (justify right) hide)
+    )
+  )
   (global_label "SCL" (shape input) (at 142.24 88.9 0) (fields_autoplaced)
     (effects (font (size 1.27 1.27)) (justify left))
@@
     )
   )
-  (global_label "Tone" (shape output) (at 236.22 107.95 180) (fields_autoplaced)
+  (global_label "Tone" (shape output) (at 236.22 114.3 180) (fields_autoplaced)
     (effects (font (size 1.27 1.27)) (justify right))
-    (property "Intersheetrefs" "${INTERSHEET_REFS}" (at 229.6142 107.95 0)
+    (property "Intersheetrefs" "${INTERSHEET_REFS}" (at 229.6142 114.3 0)
       (effects (font (size 1.27 1.27)) (justify right) hide)
     )
@@
     )
   )
+  (global_label "Busy" (shape input) (at -127 102.87 180) (fields_autoplaced)
+    (effects (font (size 1.27 1.27)) (justify right))
+    (property "Intersheetrefs" "${INTERSHEET_REFS}" (at -133.6663 102.87 0)
+      (effects (font (size 1.27 1.27)) (justify right) hide)
+    )
+  )
   (global_label "PC3" (shape bidirectional) (at 220.98 140.97 0) (fields_autoplaced)
     (effects (font (size 1.27 1.27)) (justify left))
@@
     )
   )
-  (global_label "Attenuate" (shape output) (at 236.22 101.6 180) (fields_autoplaced)
+  (global_label "Attenuate" (shape output) (at 236.22 107.95 180) (fields_autoplaced)
     (effects (font (size 1.27 1.27)) (justify right))
-    (property "Intersheetrefs" "${INTERSHEET_REFS}" (at 225.0785 101.6 0)
+    (property "Intersheetrefs" "${INTERSHEET_REFS}" (at 225.0785 107.95 0)
       (effects (font (size 1.27 1.27)) (justify right) hide)
     )
@@
     )
   )
+  (global_label "ControllerTX" (shape input) (at 241.3 96.52 180) (fields_autoplaced)
+    (effects (font (size 1.27 1.27)) (justify right))
+    (property "Intersheetrefs" "${INTERSHEET_REFS}" (at 227.4372 96.52 0)
+      (effects (font (size 1.27 1.27)) (justify right) hide)
+    )
+  )
   (global_label "Light0" (shape output) (at 236.22 139.7 180) (fields_autoplaced)
     (effects (font (size 1.27 1.27)) (justify right))
@@
       (effects (font (size 1.27 1.27)) (justify left top))
     )
-    (pin "Tone" input (at 243.84 107.95 180)
+    (pin "Tone" input (at 243.84 114.3 180)
       (effects (font (size 1.27 1.27)) (justify left))
     )
@@
       (effects (font (size 1.27 1.27)) (justify left))
     )
-    (pin "Attenuate" input (at 243.84 101.6 180)
+    (pin "Attenuate" input (at 243.84 107.95 180)
+      (effects (font (size 1.27 1.27)) (justify left))
+    )
+    (pin "ControllerTX" input (at 243.84 96.52 180)
+      (effects (font (size 1.27 1.27)) (justify left))
+    )
+    (pin "ControllerRX" output (at 243.84 99.06 180)
+      (effects (font (size 1.27 1.27)) (justify left))
+    )
+    (pin "Busy" output (at 243.84 101.6 180)
       (effects (font (size 1.27 1.27)) (justify left))
     )

Commit message: Deleted a duplicate DFplayer, connected the UART2 to the DFplayer, added and connected a boot switch.
Parts:
- removed J1: Conn_01x08, GeneralPurposeAlarmDevicePCB:DFPlayer_mini_20241116, symbol GPAD_SCH_LIB:DFPlayermini_241116
- removed LS?: Speaker, symbol Device:Speaker
Connections:
- net GND: now also S?.3, S?.4
- net GPIO0: now also S?.1, S?.2
- net ControllerRX2: now reaches U999.27 (RX2/GPIO16)
- net ControllerTX2: now reaches U999.28 (TX2/GPIO17)
Other:
- note added: "nRESET"
- moved on the sheet: S?

Commit message: Wiring up the Rotary Encoder.
Parts:
- added R? (x3): 10K, Resistor_SMD:R_0603_1608Metric_Pad0.98x0.95mm_HandSolder, symbol Device:R
- added SW?: RotaryEncoder_Switch, Rotary_Encoder:RotaryEncoder_Alps_EC12E-Switch_Vertical_H20mm, symbol Device:RotaryEncoder_Switch
Connections:
- net GND: now also SW?.C, SW?.S2
- net at U999.12 (GPIO27): now also R?.1, SW?.S1
- net 3v3Controller: now reaches C2.1, C4.1, R1.1, U999.2 (VDD)
- net 3v3Controller: now also R?.2, R?.2, R?.2
- net at U999.4 (GPIO36_VP): now also R?.1, SW?.B
- net at U999.5 (GPIO39_VN): now also R?.1, SW?.A
Other:
- note added: "DT"
- note added: "clk"
- moved on the sheet: C2, C4, R1

Commit message: Added the built in LED.
Parts:
- added D106: RED 0603, LED_SMD:LED_0603_1608Metric_Pad1.05x0.95mm_HandSolder, symbol Device:LED
- added R112: 330R, Resistor_SMD:R_0603_1608Metric_Pad0.98x0.95mm_HandSolder, symbol Device:R
Connections:
- net GND: now also D106.1 (K)
- net at U999.24 (GPIO2): now also R112.2
- new net: D106.2 (A), R112.1
Changed lines of the file:
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@@
     (stroke (width 0) (type default))
   )
+  (wire (pts (xy -66.04 171.45) (xy -66.04 170.18))
+    (stroke (width 0) (type default))
+  )
   (wire (pts (xy -125.73 100.33) (xy -115.57 100.33))
     (stroke (width 0) (type default))
@@
     (stroke (width 0) (type default))
   )
+  (wire (pts (xy -66.04 162.56) (xy -66.04 154.94))
+    (stroke (width 0) (type default))
+  )
   (wire (pts (xy 219.71 113.03) (xy 218.44 113.03))
     (stroke (width 0) (type default))
@@
     (stroke (width 0) (type default))
   )
+  (wire (pts (xy -82.55 154.94) (xy -66.04 154.94))
+    (stroke (width 0) (type default))
+  )
   (wire (pts (xy 74.93 109.22) (xy 71.12 109.22))
     (stroke (width 0) (type default))
@@
     (stroke (width 0) (type default))
   )
+  (wire (pts (xy -82.55 134.62) (xy -82.55 154.94))
+    (stroke (width 0) (type default))
+  )
   (wire (pts (xy 237.49 119.38) (xy 243.84 119.38))
     (stroke (width 0) (type default))
@@
     (stroke (width 0) (type default))
   )
+  (wire (pts (xy -66.04 179.07) (xy -66.04 181.61))
+    (stroke (width 0) (type default))
+  )
   (wire (pts (xy 58.42 24.13) (xy 58.42 29.21))
     (stroke (width 0) (type default))
@@
     )
   )
+  (symbol (lib_id "Device:R") (at -66.04 166.37 180) (unit 1)
+    (in_bom yes) (on_board yes) (dnp no)
+    (property "Reference" "R112" (at -60.96 165.1 90)
+      (effects (font (size 1.27 1.27)))
+    )
+    (property "Value" "330R" (at -63.5 166.37 90)
+      (effects (font (size 1.27 1.27)))
+    )
+    (property "Footprint" "Resistor_SMD:R_0603_1608Metric_Pad0.98x0.95mm_HandSolder" (at -64.262 166.37 90)
+      (effects (font (size 1.27 1.27)) hide)
+    )
+    (property "Datasheet" "~" (at -66.04 166.37 0)
+      (effects (font (size 1.27 1.27)) hide)
+    )
+    (property "Distributor 1" "JLCPCB" (at -66.04 166.37 90)
+      (effects (font (size 1.27 1.27)) hide)
+    )
+    (property "Distributor 1 PN" "C269711" (at -66.04 166.37 90)
+      (effects (font (size 1.27 1.27)) hide)
+    )
+    (property "Manufacturer" "TyoHM" (at -66.04 166.37 90)
+      (effects (font (size 1.27 1.27)) hide)
+    )
+    (property "MPN" "RMC06033301%N" (at -66.04 166.37 90)
+      (effects (font (size 1.27 1.27)) hide)
+    )
+    (property "Description" "0.1W ±1% 330Ω 0603 Chip Resistor - Surface Mount ROHS" (at -66.04 166.37 0)
+      (effects (font (size 1.27 1.27)) hide)
+    )
+    (property "AssemblyType" "SMT" (at -66.04 166.37 0)
+      (effects (font (size 1.27 1.27)) hide)
+    )
+    (property "Cost" "0.0015" (at -66.04 166.37 0)
+      (effects (font (size 1.27 1.27)) hide)
+    )
+    (pin "1")
+    (pin "2")
+    (instances
+      (project "PCBa_KRAKE"
+        (path "/412a327d-1ee3-473e-bc00-1545004b7edf"
+          (reference "R112") (unit 1)
+        )
+      )
+    )
+  )
   (symbol (lib_id "power:+3.3V") (at -220.98 87.63 0) (unit 1)
     (in_bom yes) (on_board yes) (dnp no) (fields_autoplaced)
@@
     )
   )
+  (symbol (lib_id "Device:LED") (at -66.04 175.26 90) (unit 1)
+    (in_bom yes) (on_board yes) (dnp no)
+    (property "Reference" "D106" (at -60.96 175.26 90)
+      (effects (font (size 1.524 1.524)))
+    )
+    (property "Value" "RED 0603" (at -57.15 177.8 90)
+      (effects (font (size 1.524 1.524)))
+    )
+    (property "Footprint" "LED_SMD:LED_0603_1608Metric_Pad1.05x0.95mm_HandSolder" (at -66.04 175.26 0)
+      (effects (font (size 1.27 1.27)) hide)
+    )
+    (property "Datasheet" "~" (at -66.04 175.26 0)
+      (effects (font (size 1.27 1.27)) hide)
+    )
+    (property "Distributor 1" "JLCPCB" (at -66.04 175.26 0)
+      (effects (font (size 1.27 1.27)) hide)
+    )
+    (property "Distributor 1 PN" "C2286" (at -76.2 170.18 0)
+      (effects (font (size 1.524 1.524)) (justify left) hide)
+    )
+    (property "MPN" "LTST-C171KRKT" (at -78.74 170.18 0)
+      (effects (font (size 1.524 1.524)) (justify left) hide)
+    )
+    (property "Category" "Optoelectronics" (at -81.28 170.18 0)
+      (effects (font (size 1.524 1.524)) (justify left) hide)
+    )
+    (property "Family" "LED Indication - Discrete" (at -83.82 170.18 0)
+      (effects (font (size 1.524 1.524)) (justify left) hide)
+    )
+    (property "Description" "LED RED CLEAR SMD" (at -91.44 170.18 0)
+      (effects (font (size 1.524 1.524)) (justify left) hide)
+    )
+    (property "Manufacturer" "Lite-On Inc." (at -93.98 170.18 0)
+      (effects (font (size 1.524 1.524)) (justify left) hide)
+    )
+    (property "Status" "Active" (at -96.52 170.18 0)
+      (effects (font (size 1.524 1.524)) (justify left) hide)
+    )
+    (property "DK_Datasheet_Link" "http://optoelectronics.liteon.com/upload/download/DS22-2000-109/LTST-C171KRKT.pdf" (at 49.53 309.88 0)
+      (effects (font (size 1.27 1.27)) hide)
+    )
+    (property "DK_Detail_Page" "/product-detail/en/lite-on-inc/LTST-C171KRKT/160-1427-1-ND/386800" (at 49.53 309.88 0)
+      (effects (font (size 1.27 1.27)) hide)
+    )
+    (property "Digi-Key_PN" "160-1427-1-ND" (at 49.53 309.88 0)
+      (effects (font (size 1.27 1.27)) hide)
+    )
+    (property "AssemblyType" "HAND" (at -66.04 175.26 0)
+      (effects (font (size 1.27 1.27)) hide)
+    )
+    (property "Cost" "0.0054" (at -66.04 175.26 0)
+      (effects (font (size 1.27 1.27)) hide)
+    )
+    (pin "1")
+    (pin "2")
+    (instances
+      (project "PCBa_KRAKE"
+        (path "/412a327d-1ee3-473e-bc00-1545004b7edf"
+          (reference "D106") (unit 1)
+        )
+      )
+    )
+  )
   (symbol (lib_id "power:PWR_FLAG") (at -201.93 86.36 0) (unit 1)
     (in_bom yes) (on_board yes) (dnp no)
@@
         )
       )
+    )
+  )
+  (symbol (lib_id "power:GND") (at -66.04 181.61 0) (unit 1)
+    (in_bom yes) (on_board yes) (dnp no)
+    (property "Reference" "#PWR020" (at -66.04 187.96 0)
+      (effects (font (size 1.27 1.27)) hide)
+    )
+    (property "Value" "GND" (at -65.913 186.0042 0)
+      (effects (font (size 1.27 1.27)))
+    )
+    (property "Footprint" "" (at -66.04 181.61 0)
+      (effects (font (size 1.27 1.27)) hide)
+    )
+    (property "Datasheet" "" (at -66.04 181.61 0)
+      (effects (font (size 1.27 1.27)) hide)
+    )
+    (pin "1")
+    (instances
+      (project "PCBa_KRAKE"
+        (path "/412a327d-1ee3-473e-bc00-1545004b7edf"
+          (reference "#PWR020") (unit 1)
+        )
+      )

Commit message: Adding the I2C level shifter circuit for LCD.Added test points for 5V I2C.
Other:
- sheet LCD And I2C Interface ports: added 3V3Raw; removed none
Changed lines of the file:
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@@
     (stroke (width 0) (type default))
   )
+  (wire (pts (xy 213.36 26.67) (xy 229.87 26.67))
+    (stroke (width 0) (type default))
+  )
   (wire (pts (xy 113.03 24.13) (xy 124.46 24.13))
     (stroke (width 0) (type default))
@@
     (stroke (width 0) (type default))
   )
+  (wire (pts (xy 213.36 25.4) (xy 213.36 26.67))
+    (stroke (width 0) (type default))
+  )
   (wire (pts (xy 123.19 76.2) (xy 123.19 80.01))
     (stroke (width 0) (type default))
@@
     )
   )
+  (symbol (lib_id "power:+3.3V") (at 213.36 25.4 0) (unit 1)
+    (in_bom yes) (on_board yes) (dnp no) (fields_autoplaced)
+    (property "Reference" "#PWR017" (at 213.36 29.21 0)
+      (effects (font (size 1.27 1.27)) hide)
+    )
+    (property "Value" "+3.3V" (at 213.36 20.32 0)
+      (effects (font (size 1.27 1.27)))
+    )
+    (property "Footprint" "" (at 213.36 25.4 0)
+      (effects (font (size 1.27 1.27)) hide)
+    )
+    (property "Datasheet" "" (at 213.36 25.4 0)
+      (effects (font (size 1.27 1.27)) hide)
+    )
+    (pin "1")
+    (instances
+      (project "PCBa_KRAKE"
+        (path "/412a327d-1ee3-473e-bc00-1545004b7edf"
+          (reference "#PWR017") (unit 1)
+        )
+      )
+    )
+  )
   (symbol (lib_id "Device:C") (at 228.6 74.93 0) (unit 1)
     (in_bom yes) (on_board yes) (dnp no)
@@
       (effects (font (size 1.27 1.27)) (justify left))
     )
+    (pin "3V3Raw" input (at 229.87 26.67 180)
+      (effects (font (size 1.27 1.27)) (justify left))
+    )
