File: PCBa_KRAKE/PCBa_KRAKE.kicad_pcb (KiCad board)
At the start: 2 copper layers, 137.2 x 83.8 mm, 140 parts, among them J101 Barrel_Jack_Switch_SMT, J102 0.100_2Pin, J103 0.100_2Pin, J105 S04B-XASK-1(LF)(SN)Rev2, J401 RJ12_6P6C_HORZ, J501 USB_B_Micro_Local, J601 22-23-2021, J602 22-23-2021, Q201 MMBT2222A-7-F, Q202 MMBT2222A-7-F, Q203 MMBT2222A-7-F, Q204 MMBT2222A-7-F, Q205 MMBT2222A-7-F, Q301 BSS138, Q601 BSS138, Q602 DNI, T1 JLC_ToolingHole_0576mm, T2 JLC_ToolingHole_0576mm, T3 JLC_ToolingHole_0576mm, U101 LM7805_TO220, U102 PI_ATMEGA328P-AU-InOrder, U301 PCF8574AT_3_518, U302 LCD_20x4_Character-GPAD_SCH_L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, U501 CH340E

Commit message: Deleted the 16mhz quarts crystal, deleted the sheild footprint.
Parts:
- added U999: ESP32-WROOM-32D, RF_Module:ESP32-WROOM-32D, F.Cu at (110.1, 152.5)
- BZ601: value Buzzer_Adafruit_P1536A -> BUZZER MAGNETIC 5V 12MM TH
- R103: value 1K -> DNI

Commit message: PCBa_KRAKE schematic fix input output pin connections to ESP32.
Parts:
- removed A101: Arduino_UNO_R3_Shield, GeneralPurposeAlarmDevicePCB:Arduino_UNO_R3_NoMountingHoles3D

Commit message: Added the datasheet for the DFPlayer.
Parts:
- added C1: 47uF 16V, Capacitor_SMD:CP_Elec_5x5.4, F.Cu at (51.7, 140.4)
- added C2: 100nF, Capacitor_SMD:C_0603_1608Metric_Pad1.08x0.95mm_HandSolder, F.Cu at (61.7, 138.2)
- added C3: 100nF, Capacitor_SMD:C_0603_1608Metric_Pad1.08x0.95mm_HandSolder, F.Cu at (61.7, 140.7)
- added C4: 47uF 16V, Capacitor_SMD:CP_Elec_5x5.4, F.Cu at (51.7, 147.2)
- added C5: 100nF, Capacitor_SMD:C_0603_1608Metric_Pad1.08x0.95mm_HandSolder, F.Cu at (61.7, 143.2)
- added C6: 47uF 16V, Capacitor_SMD:CP_Elec_5x5.4, F.Cu at (51.7, 154.1)
- added J1: Conn_01x08, GeneralPurposeAlarmDevicePCB:DFPlayer_mini_20241116, F.Cu at (70.6, 157.0)
- added R1: 1R0, Resistor_SMD:R_0603_1608Metric_Pad0.98x0.95mm_HandSolder, F.Cu at (61.7, 145.7)
- added U1: AMS1117-3.3, Package_TO_SOT_SMD:SOT-223-3_TabPin2, F.Cu at (61.1, 151.1)
Connections:
- TP105 pad 1: Net-(A101-3V3) -> unconnected-(TP105-Pad1)
- U102 pad 7: Net-(U102-XTAL1/PB6) -> unconnected-(U102-XTAL1/PB6-Pad7)
- U102 pad 8: Net-(U102-XTAL2/PB7) -> unconnected-(U102-XTAL2/PB7-Pad8)
- U999 pad 1: unconnected-(U999-GND-Pad1) -> GND
- U999 pad 10: unconnected-(U999-IO25-Pad10) -> SPI_SCK
- U999 pad 11: unconnected-(U999-IO26-Pad11) -> COPI
- U999 pad 15: unconnected-(U999-GND-Pad15) -> GND
- U999 pad 2: unconnected-(U999-VDD-Pad2) -> Net-(U999-VDD)
- U999 pad 23: unconnected-(U999-IO15-Pad23) -> Light0
- U999 pad 26: unconnected-(U999-IO4-Pad26) -> Light1
- U999 pad 29: unconnected-(U999-IO5-Pad29) -> Light2
- U999 pad 3: unconnected-(U999-EN-Pad3) -> nRESET
- U999 pad 30: unconnected-(U999-IO18-Pad30) -> Light3
- U999 pad 31: unconnected-(U999-IO19-Pad31) -> Light4
- U999 pad 33: unconnected-(U999-IO21-Pad33) -> SDA
- U999 pad 34: unconnected-(U999-RXD0/IO3-Pad34) -> ControllerRX
- U999 pad 35: unconnected-(U999-TXD0/IO1-Pad35) -> ControllerTX
- U999 pad 36: unconnected-(U999-IO22-Pad36) -> SCL
- U999 pad 38: unconnected-(U999-GND-Pad38) -> GND
- U999 pad 39: unconnected-(U999-GND-Pad39) -> GND
- U999 pad 6: unconnected-(U999-IO34-Pad6) -> Switch_Mute
- U999 pad 8: unconnected-(U999-IO32-Pad8) -> CIPO
- U999 pad 9: unconnected-(U999-IO33-Pad9) -> nCS
Routing:
- net unconnected-(TP105-Pad1): track 0.00 -> 5.19 mm
- net Net-(A101-3V3): track 5.19 -> 0.00 mm

Commit message: Updating ESP32 schematic symbol and added the df player into the audio schematic.
Parts:
- removed J1: Conn_01x08, GeneralPurposeAlarmDevicePCB:DFPlayer_mini_20241116
- added J2: Conn_01x08_Pin, Connector_PinHeader_2.54mm:PinHeader_1x08_P2.54mm_Vertical, F.Cu at (57.9, 138.5)

Commit message: Rewired the Rotary Encoder and Rewired the DF Player Busy signal, changed the pin connection of the mute buttom from GPIO34 to GPIO35.
Parts:
- moved U999 153.4 mm to (89.2, 0.59)
Changed lines of the file:
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@@
   )
   (footprint "RF_Module:ESP32-WROOM-32D" (layer "F.Cu")
-    (at 110.096 152.522)
+    (at 89.154 0.593)
     (descr "2.4 GHz Wi-Fi and Bluetooth module, https://www.espressif.com/sites/default/files/documentation/esp32-wroom-32d_esp32-wroom-32u_datasheet_en.pdf")
     (tags "2.4 GHz Wi-Fi and Bluetooth module ESP32-D0WD Espressif ESP32-WROOM-32E")
@@
       (polygon
         (pts
-          (xy 86.096 142.972)
-          (xy 134.096 142.972)
-          (xy 134.096 121.782)
-          (xy 86.096 121.782)
+          (xy 65.154 -8.957)
+          (xy 113.154 -8.957)
+          (xy 113.154 -30.147)
+          (xy 65.154 -30.147)
         )
       )
