File: PCBa_KRAKE/PCBa_KRAKE.kicad_pcb (KiCad board)
At the start: 2 copper layers, 137.2 x 83.8 mm, 190 parts, among them J101 Barrel_Jack_Switch_SMT, J102 0.100_2Pin, J103 0.100_2Pin, J104 Conn_01x14 1mm, J106 Conn_01x14 1mm, J107 Conn_01x10 1mm, J401 RJ12_6P6C_HORZ, J501 USB_C_Receptacle_USB2.0, J601 1X2P 1.27 mm Header, J602 22-23-2021, J603 DFPlayermini, J701 DE9_Receptacle_MountingHoles, Q201 MMBT2222A-7-F, Q202 MMBT2222A-7-F, Q203 MMBT2222A-7-F, Q204 MMBT2222A-7-F, Q205 MMBT2222A-7-F, Q206 MMBT2222A-7-F, Q207 MMBT2222A-7-F, Q301 BSS138, Q302 BSS138, Q303 BSS138, Q304 BSS138, Q305 BSS138, Q401 BSS138, Q402 BSS138, SW101 RotaryEncoder_Switch, U101 LM7805_TO220, U102 ESP32-WROOM-32D, U103 AMS1117-3.3, U301 PCF8574AT_3_518, U302 LCD_20x4_Character-GPAD_SCH_L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, U501 CH340T, U701 MAX3232

Commit message: Adding Rotary encoder step file, And placed it in the PCB.
Parts:
- BZ601: moved to F.Cu
- SW101: moved to B.Cu
- moved SW101 168.4 mm to (78.4, 83.9), turned to 180 degrees
- moved BZ601 27.5 mm to (102.4, 84.1), turned to 0 degrees

Commit message: PLacing and routing, Added new EMC resistors at the output of the microcoontroller.
Parts:
- added R113: 39R, Resistor_SMD:R_0603_1608Metric_Pad0.98x0.95mm_HandSolder, F.Cu at (122.9, 29.0)
- added R114: 39R, Resistor_SMD:R_0603_1608Metric_Pad0.98x0.95mm_HandSolder, F.Cu at (122.9, 36.1)
- added R115: 39R, Resistor_SMD:R_0603_1608Metric_Pad0.98x0.95mm_HandSolder, F.Cu at (122.9, 37.6)
- added R116: 39R, Resistor_SMD:R_0603_1608Metric_Pad0.98x0.95mm_HandSolder, F.Cu at (122.9, 39.4)
- moved R702 212.6 mm to (113.5, 49.2), turned to -90 degrees
- moved R703 189.0 mm to (93.8, 35.1), turned to 180 degrees
- moved C106 114.8 mm to (90.9, 29.0), turned to 90 degrees
- moved C103 111.8 mm to (94.7, 28.2), turned to 90 degrees
- moved J104 6.10 mm to (97.0, 28.0)
- moved J106 6.10 mm to (119.6, 40.9)
- moved J107 6.10 mm to (104.4, 45.8)
- moved U102 6.10 mm to (108.5, 34.2)
- moved R503 6.04 mm to (122.9, 31.2)
- moved D106 5.03 mm to (106.4, 50.1)
- moved R112 5.03 mm to (106.3, 48.3)
Connections:
- J106 pad 13: COPI -> Net-(J106-Pin_13)
- J106 pad 4: ControllerTX2 -> Net-(J106-Pin_4)
- J106 pad 5: nCS -> Net-(J106-Pin_5)
- J106 pad 6: SPI_SCK -> Net-(J106-Pin_6)
- U102 pad 28: ControllerTX2 -> Net-(J106-Pin_4)
- U102 pad 29: nCS -> Net-(J106-Pin_5)
- U102 pad 30: SPI_SCK -> Net-(J106-Pin_6)
- U102 pad 37: COPI -> Net-(J106-Pin_13)

Commit message: Routing and connecting and level shifter.
Parts:
- moved R511 344.0 mm to (255.5, 121.9)
- moved D502 343.8 mm to (251.9, 123.4)
- moved R513 338.2 mm to (251.5, 120.4), turned to 180 degrees
- moved C505 331.1 mm to (224.3, 127.0), turned to 180 degrees
- moved C504 318.8 mm to (225.1, 123.2), turned to 180 degrees
- moved R512 313.8 mm to (224.8, 120.1)
- moved R510 312.8 mm to (221.8, 120.3), turned to 90 degrees
- moved J603 310.2 mm to (230.1, 123.2)
- moved J701 266.5 mm to (92.9, 175.9)
- moved C701 259.6 mm to (80.5, 152.9), turned to -90 degrees
- moved C702 259.5 mm to (80.5, 156.4), turned to -90 degrees
- moved R708 257.5 mm to (91.8, 171.6), turned to -90 degrees
- moved C703 257.2 mm to (88.9, 147.3), turned to 180 degrees
- moved U701 254.6 mm to (87.0, 156.3)
- moved R705 253.8 mm to (90.0, 171.6), turned to -90 degrees
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Routing:
- net +5V: track 270.3 -> 257.6 mm
- net Net-(Q401-D): track 12.8 -> 4.60 mm
- net Net-(Q402-D): track 11.0 -> 5.98 mm
- net /LCD And I2C Interface/Vcc_LCD: track 119.4 -> 122.5 mm
Other:
- board text added: "BOOT"
- board text added: "CIPO"
- board text added: "locked"
- board text removed: "Reset"

Commit message: Routing and connecting, shifted U101 up.
Parts:
- moved Q302 272.0 mm to (170.4, 68.1)
- moved R313 272.0 mm to (173.2, 68.1)
- moved R315 272.0 mm to (167.4, 68.1)
- moved R314 272.0 mm to (170.4, 70.6)
- moved Q303 263.5 mm to (170.2, 59.5)
- moved R316 263.5 mm to (173.2, 59.4)
- moved R317 263.5 mm to (170.7, 62.2)
- moved R318 263.5 mm to (167.1, 59.7)
- moved Q304 257.2 mm to (159.3, 59.7)
- moved R319 257.2 mm to (162.1, 59.8)
- moved R320 257.2 mm to (159.6, 62.2)
- moved R322 257.2 mm to (156.3, 59.8)
- moved R323 255.5 mm to (159.8, 70.8)
- moved Q305 255.5 mm to (159.4, 68.1)
- moved R321 255.5 mm to (162.6, 68.3)
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Routing:
- net GND: track 91.5 -> 93.1 mm
- net Vin: track 39.9 -> 41.5 mm
- net +5V: track 257.6 -> 256.2 mm

Commit message: Routed and connected USB diff signals amd more.
Parts:
- removed H105: MountingHole_Pad_3.5mm, GeneralPurposeAlarmDevicePCB:MountingHole_3.5mm_Pad_Via
- moved TP203 108.7 mm to (50.8, 133.6)
- moved J501 104.7 mm to (47.4, 154.4)
- moved R211 104.7 mm to (54.9, 151.2)
- moved R212 104.6 mm to (41.2, 151.5)
- moved R213 103.3 mm to (41.8, 147.3)
- moved C501 103.2 mm to (40.4, 143.2)
- moved C502 103.2 mm to (36.6, 143.3)
- moved R504 103.2 mm to (50.6, 137.0)
- moved U501 103.2 mm to (46.6, 143.8)
- moved Q206 103.1 mm to (43.5, 128.6)
- moved Q207 103.1 mm to (38.2, 128.0)
- moved D501 102.8 mm to (46.8, 134.4), turned to 180 degrees
- moved R216 102.8 mm to (36.6, 137.4), turned to -90 degrees
- moved R501 102.7 mm to (47.0, 137.7)
- moved R214 102.4 mm to (44.2, 136.9)
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Connections:
- F401 pad 1: ControllerVcc -> /SPI Peripherial/ControllerVcc
- J401 pad 4: SPI_SCK -> /SPI Peripherial/SCK
- J501 pad A4: VBus -> /USB_UART/VBus
- J501 pad A9: VBus -> /USB_UART/VBus
- J501 pad B4: VBus -> /USB_UART/VBus
- J501 pad B9: VBus -> /USB_UART/VBus
- Q206 pad 3: nRESET -> /USB_UART/nRESET
- Q207 pad 2: GPIO0 -> /USB_UART/GPIO0
- Q304 pad 2: COPI -> /SPI Peripherial/COPI
- Q305 pad 2: SPI_SCK -> /SPI Peripherial/SCK
- R1009 pad 1: /SPI Peripherial/5VRaw -> unconnected-(R1009-Pad1)
- R201 pad 2: Light0 -> /AlarmLights5/Light0
- R203 pad 2: Light1 -> /AlarmLights5/Light1
- R205 pad 2: Light2 -> /AlarmLights5/Light2
- R207 pad 2: Light3 -> /AlarmLights5/Light3
- R209 pad 2: Light4 -> /AlarmLights5/Light4
- R320 pad 2: COPI -> /SPI Peripherial/COPI
- R322 pad 1: COPI -> /SPI Peripherial/COPI
- R323 pad 2: SPI_SCK -> /SPI Peripherial/SCK
- R324 pad 1: SPI_SCK -> /SPI Peripherial/SCK
- R402 pad 2: SPI_SCK -> /SPI Peripherial/SCK
- R502 pad 1: ControllerRX -> /USB_UART/ControllerRX
- R702 pad 1: TX1 -> /RS232/TX1
- R704 pad 1: CTS1 -> /RS232/CTS1
- TP201 pad 1: VBus -> /USB_UART/VBus
Routing:
- net Net-(Q201-B): track 2.19 -> 64.9 mm, vias 0 -> 2
- net Light0: track 62.7 -> 0.00 mm, vias 2 -> 0
- net Light4: track 49.2 -> 0.00 mm, vias 4 -> 0
- net /AlarmLights5/Light4: track 0.00 -> 49.2 mm, vias 0 -> 4
- net Light1: track 44.7 -> 0.00 mm, vias 3 -> 0
- net /AlarmLights5/Light1: track 0.00 -> 44.7 mm, vias 0 -> 3
- net Net-(U501-VCC): track 0.00 -> 28.0 mm
- net Net-(U501-RXD): track 0.00 -> 16.8 mm, vias 0 -> 2
- net Light3: track 15.2 -> 0.00 mm, vias 2 -> 0
- net /AlarmLights5/Light3: track 0.00 -> 15.2 mm, vias 0 -> 2
- net GND: track 93.1 -> 108.3 mm
- net +5V: track 256.2 -> 270.1 mm
- net Net-(U501-TXD): track 0.00 -> 13.8 mm, vias 0 -> 2
- net /USB_UART/VBus: track 0.00 -> 11.5 mm
- net Net-(U501-V3): track 0.00 -> 9.31 mm
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- added copper zone on F.Cu, net Net-(U501-VCC)

Commit message: Moved the USB C circuit to the board, in exact place of old USB B.
Parts:
- added REF**: RJ45_Amphenol_54602-x08_Horizontal, Connector_RJ:RJ45_Amphenol_54602-x08_Horizontal, F.Cu at (71.7, 152.9)
- added REF**: DSUB-9_Female_Vertical_P2.77x2.84mm_MountingHoles, Connector_Dsub:DSUB-9_Female_Vertical_P2.77x2.84mm_MountingHoles, B.Cu at (99.8, 158.6)
- moved C502 83.9 mm to (99.7, 87.9)
- moved D501 83.9 mm to (109.9, 79.0)
- moved R212 83.9 mm to (104.2, 96.1)
- moved R214 83.9 mm to (107.3, 81.5)
- moved R501 83.9 mm to (110.1, 82.3)
- moved R502 83.9 mm to (115.4, 85.3)
- moved TP202 83.9 mm to (118.2, 90.9)
- moved TP203 83.9 mm to (113.9, 78.2)
- moved U501 83.9 mm to (109.7, 88.4)
- moved C501 83.9 mm to (103.5, 87.8)
- moved C503 83.9 mm to (114.4, 88.9)
- moved J501 83.9 mm to (110.5, 99.1)
- moved Q206 83.9 mm to (106.6, 73.2)
- moved Q207 83.9 mm to (101.3, 72.6)
- moved R211 83.9 mm to (118.0, 95.8)
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