File: PCBa_KRAKE/PCBa_KRAKE.kicad_pcb (KiCad board)
At the start: 2 copper layers, 137.2 x 83.8 mm, 192 parts, among them J101 Barrel_Jack_Switch_SMT, J102 0.100_2Pin, J103 0.100_2Pin, J104 Conn_01x14 1mm, J106 Conn_01x14 1mm, J107 Conn_01x10 1mm, J401 RJ12_6P6C_HORZ, J501 USB_C_Receptacle_USB2.0, J601 1X2P 1.27 mm Header, J602 22-23-2021, J603 DFPlayermini, J701 DE9_Receptacle_MountingHoles, Q201 MMBT2222A-7-F, Q202 MMBT2222A-7-F, Q203 MMBT2222A-7-F, Q204 MMBT2222A-7-F, Q205 MMBT2222A-7-F, Q206 MMBT2222A-7-F, Q207 MMBT2222A-7-F, Q301 BSS138, Q302 BSS138, Q303 BSS138, Q304 BSS138, Q305 BSS138, Q401 BSS138, Q402 BSS138, SW101 RotaryEncoder_Switch, U101 LM7805_TO220, U102 ESP32-WROOM-32D, U103 AMS1117-3.3, U301 PCF8574AT_3_518, U302 LCD_20x4_Character-GPAD_SCH_L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, U501 CH340T, U701 MAX3232

Commit message: Got rid of ERC spoke errors by providing more ground vias and ground fills.
Routing:
- net GND: vias 107 -> 111
Changed lines of the file:
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@@
   (via (at 161.204 44.196) (size 0.8) (drill 0.4) (layers "F.Cu" "B.Cu") (net 1))
   (via (at 78.72736 99.095) (size 0.8) (drill 0.4) (layers "F.Cu" "B.Cu") (free) (net 1))
+  (via (at 71.12 91.694) (size 0.8) (drill 0.4) (layers "F.Cu" "B.Cu") (net 1))
   (via (at 67.31 31.75) (size 0.8) (drill 0.4) (layers "F.Cu" "B.Cu") (net 1))
   (via (at 153.67 80.01) (size 0.8) (drill 0.4) (layers "F.Cu" "B.Cu") (net 1))
@@
   (via (at 138.938 30.988) (size 0.8) (drill 0.4) (layers "F.Cu" "B.Cu") (net 1))
   (via (at 164.338 68.326) (size 0.8) (drill 0.4) (layers "F.Cu" "B.Cu") (net 1))
+  (via (at 136.906 72.644) (size 0.8) (drill 0.4) (layers "F.Cu" "B.Cu") (net 1))
   (via (at 79.502 61.468) (size 0.8) (drill 0.4) (layers "F.Cu" "B.Cu") (net 1))
   (via (at 121.412 27.432) (size 0.8) (drill 0.4) (layers "F.Cu" "B.Cu") (net 1))
@@
   (via (at 151.13 70.358) (size 0.8) (drill 0.4) (layers "F.Cu" "B.Cu") (net 1))
   (via (at 157.209545 42.417661) (size 0.8) (drill 0.4) (layers "F.Cu" "B.Cu") (net 1))
+  (via (at 70.104 96.012) (size 0.8) (drill 0.4) (layers "F.Cu" "B.Cu") (net 1))
   (via (at 67.818 88.392) (size 0.8) (drill 0.4) (layers "F.Cu" "B.Cu") (net 1))
   (via (at 102.362 98.806) (size 0.8) (drill 0.4) (layers "F.Cu" "B.Cu") (free) (net 1))
@@
   (via (at 66.548 68.326) (size 0.8) (drill 0.4) (layers "F.Cu" "B.Cu") (net 1))
   (via (at 146.685 29.845) (size 0.8) (drill 0.4) (layers "F.Cu" "B.Cu") (net 1))
+  (via (at 136.398 69.342) (size 0.8) (drill 0.4) (layers "F.Cu" "B.Cu") (net 1))
   (via (at 139.446 39.624) (size 0.8) (drill 0.4) (layers "F.Cu" "B.Cu") (net 1))
   (segment (start 93.98 93.9) (end 96.6 96.52) (width 0.25) (layer "B.Cu") (net 1))
@@
   (segment (start 104.297 44.958) (end 105.008265 44.958) (width 0.25) (layer "F.Cu") (net 109))
   (segment (start 112.394 45.768) (end 112.394 48.398995) (width 0.25) (layer "F.Cu") (net 110))
+  (segment (start 131.9325 74.448574) (end 131.9325 61.8695) (width 0.25) (layer "F.Cu") (net 110))
   (segment (start 129.286 55.626) (end 132.334 52.578) (width 0.25) (layer "F.Cu") (net 110))
-  (segment (start 131.9325 61.8695) (end 132.334 61.468) (width 0.25) (layer "F.Cu") (net 110))
   (segment (start 112.908 43.679) (end 112.908 44.679) (width 0.25) (layer "F.Cu") (net 110))
   (segment (start 112.394 48.398995) (end 113.267505 49.2725) (width 0.25) (layer "F.Cu") (net 110))
@@
   (segment (start 112.394 45.193) (end 112.394 45.768) (width 0.25) (layer "F.Cu") (net 110))
   (segment (start 112.908 44.679) (end 112.394 45.193) (width 0.25) (layer "F.Cu") (net 110))
-  (segment (start 137.922 76.962) (end 135.971 75.011) (width 0.25) (layer "F.Cu") (net 110))
-  (segment (start 131.9325 74.448574) (end 131.9325 61.8695) (width 0.25) (layer "F.Cu") (net 110))
+  (segment (start 135.717 75.011) (end 132.494926 75.011) (width 0.25) (layer "F.Cu") (net 110))
   (segment (start 114.86976 49.2725) (end 121.22326 55.626) (width 0.25) (layer "F.Cu") (net 110))
+  (segment (start 137.922 76.962) (end 137.668 76.962) (width 0.25) (layer "F.Cu") (net 110))
   (segment (start 113.267505 49.2725) (end 114.86976 49.2725) (width 0.25) (layer "F.Cu") (net 110))
-  (segment (start 135.971 75.011) (end 132.494926 75.011) (width 0.25) (layer "F.Cu") (net 110))
+  (segment (start 131.9325 61.8695) (end 132.334 61.468) (width 0.25) (layer "F.Cu") (net 110))
   (segment (start 132.494926 75.011) (end 131.9325 74.448574) (width 0.25) (layer "F.Cu") (net 110))
+  (segment (start 137.668 76.962) (end 135.717 75.011) (width 0.25) (layer "F.Cu") (net 110))
   (via (at 132.334 52.578) (size 0.8) (drill 0.4) (layers "F.Cu" "B.Cu") (net 110))
   (via (at 132.334 61.468) (size 0.8) (drill 0.4) (layers "F.Cu" "B.Cu") (net 110))
@@
   (segment (start 138.1985 80.691) (end 133.279 80.691) (width 0.25) (layer "F.Cu") (net 140))
   (segment (start 139.5495 82.042) (end 138.1985 80.691) (width 0.25) (layer "F.Cu") (net 140))
-  (segment (start 140.462 77.978) (end 136.825 74.341) (width 0.25) (layer "F.Cu") (net 141))
+  (segment (start 137.16 85.344) (end 140.208 85.344) (width 0.25) (layer "F.Cu") (net 141))
+  (segment (start 134.7705 86.106) (end 136.398 86.106) (width 0.25) (layer "F.Cu") (net 141))
+  (segment (start 136.571 74.341) (end 133.279 74.341) (width 0.25) (layer "F.Cu") (net 141))
+  (segment (start 140.462 85.09) (end 140.462 78.232) (width 0.25) (layer "F.Cu") (net 141))
+  (segment (start 140.462 78.232) (end 136.571 74.341) (width 0.25) (layer "F.Cu") (net 141))
   (segment (start 136.398 86.106) (end 137.16 85.344) (width 0.25) (layer "F.Cu") (net 141))
-  (segment (start 136.825 74.341) (end 133.279 74.341) (width 0.25) (layer "F.Cu") (net 141))
   (segment (start 140.208 85.344) (end 140.462 85.09) (width 0.25) (layer "F.Cu") (net 141))
-  (segment (start 140.462 85.09) (end 140.462 77.978) (width 0.25) (layer "F.Cu") (net 141))
-  (segment (start 134.7705 86.106) (end 136.398 86.106) (width 0.25) (layer "F.Cu") (net 141))
-  (segment (start 137.16 85.344) (end 140.208 85.344) (width 0.25) (layer "F.Cu") (net 141))
   (segment (start 131.164 78.078) (end 129.54 76.454) (width 0.25) (layer "F.Cu") (net 142))
   (segment (start 130.383 75.611) (end 133.279 75.611) (width 0.25) (layer "F.Cu") (net 142))

Commit message: Cleared DRC warning by changing the min Silkscreen hieght to 0.75 mm. Note this violates JLCPCB 1.0 mm requirements.
Parts:
- moved G*** 103.0 mm to (117.1, 67.1)
- moved J601 14.8 mm to (125.2, 67.1)
Routing:
- net Net-(J603-SPK_2): track 5.60 -> 21.6 mm, vias 0 -> 2
- net Net-(J603-SPK_1): track 7.19 -> 22.8 mm, vias 0 -> 2
- net ControllerRX: track 60.8 -> 62.3 mm
- net GPIO0: track 53.1 -> 52.3 mm
- net Net-(U501-RXD): track 80.9 -> 81.5 mm
Other:
- board text added: "Public Invention, Krake Rev 1.0 20250111"
- board text removed: "General Purpouse Alarm Device, Public Invention, Rev 2.0 20230228"

Commit message: Cleared all DRC issues and Warnings.
Parts:
- added TP405: Vcontrast, TestPoint:TestPoint_Loop_D2.54mm_Drill1.5mm_Beaded, F.Cu at (180.1, 32.8)
- moved S102 0.72 mm to (119.7, 46.3)
- moved S101 0.51 mm to (90.0, 46.3)
Routing:
- net SCL: track 30.6 -> 49.2 mm
- net /LCD And I2C Interface/Vcc_LCD: track 152.3 -> 137.5 mm
- net ControllerRX: track 62.3 -> 69.9 mm
- net COPI: track 59.1 -> 66.4 mm
- net GPIO0: track 52.3 -> 58.7 mm
- net SDA: track 34.4 -> 40.8 mm
- net nCS: track 61.0 -> 66.5 mm
- net Net-(U301-P3): track 38.1 -> 33.8 mm
- net Net-(U302-VO): track 40.6 -> 44.6 mm
- net Net-(U701-T1IN): track 63.1 -> 59.6 mm
- net CIPO: track 79.4 -> 82.5 mm
- net GND: track 191.6 -> 194.4 mm, vias 111 -> 113
- net Net-(J603-TX): track 57.2 -> 54.9 mm
- net ControllerTX2: track 62.1 -> 60.0 mm
- net RX1: track 58.4 -> 56.4 mm
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Other:
- board text added: "MP3 Player"
- board text added: "Power from SPI"
- board text removed: "Power by Controller_Vcc"

Commit message: Removed micro vias, And provided ground USB UART interface.
Routing:
- net Net-(Q207-B): track 20.6 -> 18.2 mm
- net Net-(U501-V3): track 28.6 -> 30.4 mm
- net Net-(J603-SPK_2): track 20.4 -> 18.6 mm
- net Net-(U501-VCC): track 35.6 -> 34.3 mm
- net ControllerRX: track 69.9 -> 70.5 mm
- net GND: vias 113 -> 116
