File: PCBa_KRAKE/SPI Peripherial.kicad_sch (KiCad schematic)
At the start: 6 parts, among them J401 RJ12_6P6C_HORZ

Commit message: Adding cooments in the title block, page setting of PCBa_Krake.
Other:
- title: GeneralPurposeAlarmDevicePCB -> KRAKE_PCB
Changed lines of the file:
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@@
   (paper "USLetter")
   (title_block
-    (title "GeneralPurposeAlarmDevicePCB")
-    (date "2023-04-25")
-    (rev "2.2")
+    (title "KRAKE_PCB")
+    (date "2024-11-23")
+    (rev "1")
     (company "PublicInvention")
     (comment 1 "GNU Affero General Public License v3.0")
-    (comment 2 "DrawnBy: (Forrest) Lee Erickson")
+    (comment 2 "DrawnBy: (Forrest) Lee Erickson, Nagham Kheir")
+    (comment 3 "https://github.com/PubInv/krake")
+    (comment 4 "Inherited from the GPAD")
   )
   (wire (pts (xy 189.23 102.87) (xy 198.12 102.87))

Commit message: Adding a level shifter to the SPI bus.
Parts:
- added Q? (x4): BSS138, Package_TO_SOT_SMD:SOT-23, symbol Transistor_FET:BSS138
- added R? (x8): 4K7, Resistor_SMD:R_0603_1608Metric_Pad0.98x0.95mm_HandSolder, symbol Device:R
- added R? (x4): DNI, Resistor_SMD:R_0603_1608Metric_Pad0.98x0.95mm_HandSolder, symbol Device:R
Connections:
- net CIPO: now also Q?.2 (S), R?.1, R?.2; no longer R401.1
- net COPI: now also Q?.2 (S), R?.1, R?.2; no longer R403.1
- net SCK: now also J401.4, R402.2, Q?.2 (S), R?.1, R?.2; no longer R402.1
- net nCS: now also Q?.2 (S), R?.1, R?.2; no longer R404.1
- net MISO: now reaches J401.6, R401.2
- net MOSI: now reaches J401.2, R403.2
- net SS: now reaches J401.1, R404.2
- new net: Q?.3 (D), R401.1, R?.1, R?.1
- new net: Q?.3 (D), R402.1, R?.1, R?.1
- new net: Q?.3 (D), R403.1, R?.1, R?.1
- new net: Q?.3 (D), R404.1, R?.1, R?.1
- new net +5V: R?.2, R?.2, R?.2, R?.2
- new net 3V3Raw: Q?.1 (G), Q?.1 (G), Q?.1 (G), Q?.1 (G), R?.2, R?.2, R?.2, R?.2
Other:
- note added: "At this interface we have a 5v logic levels."
- note added: "these are 3v3 logic levels"
- moved on the sheet: F401, J401, R401, R402, R403, R404

Commit message: Added 5V to 3v3 level shifters to SPI bus.Added but not wired a USBc connector.
Connections:
- net +5V: no longer R?.2, R?.2
- new net 5VRaw: R?.2
Changed lines of the file:
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@@
-    (stroke (width 0) (type default))
-  )
-  (wire (pts (xy 135.89 61.595) (xy 125.73 61.595))
     (stroke (width 0) (type default))
   )
@@
   )
   (text "Note: Check that pin 1 is on the left when viewing the connector on layout."
-    (at -32.385 128.905 0)
+    (at 29.845 128.27 0)
     (effects (font (size 1.27 1.27)) (justify left bottom))
   )
@@
   )
   (hierarchical_label "3V3Raw" (shape input) (at 170.18 57.785 0) (fields_autoplaced)
+    (effects (font (size 1.27 1.27)) (justify left))
+  )
+  (hierarchical_label "5VRaw" (shape input) (at 136.525 57.785 90) (fields_autoplaced)
     (effects (font (size 1.27 1.27)) (justify left))
   )
@@
     )
   )
-  (symbol (lib_id "power:+5V") (at 195.58 66.675 0) (mirror y) (unit 1)
-    (in_bom yes) (on_board yes) (dnp no)
-    (property "Reference" "#PWR0303" (at 195.58 70.485 0)
-      (effects (font (size 1.27 1.27)) hide)
-    )
-    (property "Value" "+5V" (at 195.199 62.2808 0)
-      (effects (font (size 1.27 1.27)))
-    )
-    (property "Footprint" "" (at 195.58 66.675 0)
-      (effects (font (size 1.27 1.27)) hide)
-    )
-    (property "Datasheet" "" (at 195.58 66.675 0)
-      (effects (font (size 1.27 1.27)) hide)
-    )
-    (pin "1")
-    (instances
-      (project "PCBa_KRAKE"
-        (path "/412a327d-1ee3-473e-bc00-1545004b7edf/00000000-0000-0000-0000-000062b871ee"
-          (reference "#PWR0303") (unit 1)
-        )
-        (path "/412a327d-1ee3-473e-bc00-1545004b7edf/00000000-0000-0000-0000-000062b93801"
-          (reference "#PWR035") (unit 1)
-        )
-      )
-    )
-  )
   (symbol (lib_id "Device:R") (at 126.365 180.34 0) (mirror x) (unit 1)
     (in_bom yes) (on_board yes) (dnp no)
@@
         )
       )
-    )
-  )
-  (symbol (lib_id "power:+5V") (at 136.525 57.785 0) (mirror y) (unit 1)
-    (in_bom yes) (on_board yes) (dnp no)
-    (property "Reference" "#PWR0303" (at 136.525 61.595 0)
-      (effects (font (size 1.27 1.27)) hide)
-    )
-    (property "Value" "+5V" (at 136.144 53.3908 0)
-      (effects (font (size 1.27 1.27)))
-    )
-    (property "Footprint" "" (at 136.525 57.785 0)
-      (effects (font (size 1.27 1.27)) hide)
-    )
-    (property "Datasheet" "" (at 136.525 57.785 0)
-      (effects (font (size 1.27 1.27)) hide)
-    )
-    (pin "1")
-    (instances
-      (project "PCBa_KRAKE"
-        (path "/412a327d-1ee3-473e-bc00-1545004b7edf/00000000-0000-0000-0000-000062b871ee"
-          (reference "#PWR0303") (unit 1)
-        )
-        (path "/412a327d-1ee3-473e-bc00-1545004b7edf/00000000-0000-0000-0000-000062b93801"
-          (reference "#PWR034") (unit 1)
-        )
-      )

Commit message: Added ESD protection to the level shifter of the SPI bus.
Parts:
- added D? (x4): BAT54S, Package_TO_SOT_SMD:SOT-23, symbol Diode:BAT54S
Connections:
- net +5V is gone; now on net 5VRaw: R?.2, R?.2
- net 5VRaw: now also R?.2, D?.2 (K), D?.2 (K), D?.2 (K), D?.2 (K)
- net GND: now also D?.1 (A), D?.1 (A), D?.1 (A), D?.1 (A)
- net at Q?.3 (D), R401.1, R?.1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: now also D?.3 (COM)
- net at Q?.3 (D), R402.1, R?.1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: now also D?.3 (COM)
- net at Q?.3 (D), R403.1, R?.1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: now also D?.3 (COM)
- net at Q?.3 (D), R404.1, R?.1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: now also D?.3 (COM)
Other:
- moved on the sheet: F401, J401, Q?, R401, R402, R403, R404, R?

Commit message: Cleanup schematic component placement.
Other:
- note removed: "/* Hardware Notes Peripheral SPI Line Pin in Arduino, IO setup MOSI 11 or ICSP-4 Input, ATmegaPin BP3, 17 MISO 12 or ICSP-1 Output, ATmegaPin BP4, 18 SCK 13 or ICSP-3 Input, ATmegaPin BP5, 19 SS 10 Input, ATmegaPin BP2, 16 */"
- note removed: "Note: Check that pin 1 is on the left when viewing the connector on layout."
- moved on the sheet: D?, F401, Q?, R401, R402, R?

Commit message: Schematic changes 20241209.
Parts:
- added C103: 100nF, Capacitor_SMD:C_0603_1608Metric_Pad1.08x0.95mm_HandSolder, symbol Device:C
Connections:
- net 5VRaw: now also C103.2
- net GND: now also C103.1
Other:
- note added: "3v3 to 5v level shifter"
- note added: "5v to 3v3level shifter"
- note added: "ESD protection circuit"
- note added: "Place near Clamp Diodes"
Changed lines of the file:
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@@
   (junction (at 191.135 78.105) (diameter 0) (color 0 0 0 0)
   )
+  (junction (at 210.82 27.305) (diameter 0) (color 0 0 0 0)
+  )
   (junction (at 130.175 129.54) (diameter 0) (color 0 0 0 0)
   )
@@
     (stroke (width 0) (type default))
   )
-  (wire (pts (xy 210.82 29.845) (xy 210.82 40.005))
+  (wire (pts (xy 210.82 26.67) (xy 210.82 27.305))
     (stroke (width 0) (type default))
   )
@@
     (stroke (width 0) (type default))
   )
+  (wire (pts (xy 205.105 27.305) (xy 210.82 27.305))
+    (stroke (width 0) (type default))
+  )
   (wire (pts (xy 93.345 123.825) (xy 94.615 123.825))
     (stroke (width 0) (type default))
@@
     (stroke (width 0) (type default))
   )
-  (wire (pts (xy 244.475 29.845) (xy 210.82 29.845))
+  (wire (pts (xy 244.475 26.67) (xy 210.82 26.67))
     (stroke (width 0) (type default))
   )
@@
   )
   (wire (pts (xy 154.305 47.625) (xy 155.575 47.625))
+    (stroke (width 0) (type default))
+  )
+  (wire (pts (xy 210.82 27.305) (xy 210.82 40.005))
     (stroke (width 0) (type default))
   )
@@
     )
   )
+  (text "3v3 to 5v level shifter" (at 127 60.325 0)
+    (effects (font (size 1.27 1.27)) (justify left bottom))
+  )
   (text "At this interface we have a 5v logic levels." (at 18.415 69.215 0)
     (effects (font (size 1.27 1.27)) (justify left bottom))
   )
+  (text "Place near Clamp Diodes" (at 188.595 25.4 0)
+    (effects (font (size 1.27 1.27)) (justify left bottom))
+  )
+  (text "  5v to 3v3level shifter" (at 179.705 142.24 0)
+    (effects (font (size 1.27 1.27)) (justify left bottom))
+  )
+  (text "  5v to 3v3level shifter" (at 97.79 141.605 0)
+    (effects (font (size 1.27 1.27)) (justify left bottom))
+  )
   (text "SPI Peripherial Interface" (at 18.415 23.495 0)
     (effects (font (size 2.54 2.54)) (justify left bottom))
@@
     (effects (font (size 1.27 1.27)) (justify left bottom))
   )
+  (text "ESD protection circuit" (at 177.165 41.275 0)
+    (effects (font (size 1.27 1.27)) (justify left bottom))
+  )
+  (text "  5v to 3v3level shifter" (at 201.295 60.325 0)
+    (effects (font (size 1.27 1.27)) (justify left bottom))
+  )
   (label "SS" (at 43.815 86.995 0) (fields_autoplaced)
     (effects (font (size 1.27 1.27)) (justify left bottom))
@@
     (effects (font (size 1.27 1.27)) (justify left))
   )
-  (hierarchical_label "5VRaw" (shape input) (at 244.475 29.845 0) (fields_autoplaced)
+  (hierarchical_label "5VRaw" (shape input) (at 244.475 26.67 0) (fields_autoplaced)
     (effects (font (size 1.27 1.27)) (justify left))
   )
@@
     )
   )
+  (symbol (lib_id "power:GND") (at 205.105 34.925 0) (unit 1)
+    (in_bom yes) (on_board yes) (dnp no)
+    (property "Reference" "#PWR038" (at 205.105 41.275 0)
+      (effects (font (size 1.27 1.27)) hide)
+    )
+    (property "Value" "GND" (at 205.74 33.655 0)
+      (effects (font (size 1.27 1.27)))
+    )
+    (property "Footprint" "" (at 205.105 34.925 0)
+      (effects (font (size 1.27 1.27)) hide)
+    )
+    (property "Datasheet" "" (at 205.105 34.925 0)
+      (effects (font (size 1.27 1.27)) hide)
+    )
+    (pin "1")
+    (instances
+      (project "PCBa_KRAKE"
+        (path "/412a327d-1ee3-473e-bc00-1545004b7edf/00000000-0000-0000-0000-000062b93801"
+          (reference "#PWR038") (unit 1)
+        )
+      )
+    )
+  )
   (symbol (lib_id "Transistor_FET:BSS138") (at 226.695 45.72 90) (mirror x) (unit 1)
     (in_bom yes) (on_board yes) (dnp no)
@@
         )
       )
+    )
+  )
+  (symbol (lib_id "Device:C") (at 205.105 31.115 180) (unit 1)
+    (in_bom yes) (on_board yes) (dnp no)
+    (property "Reference" "C103" (at 202.184 32.2834 0)
+      (effects (font (size 1.27 1.27)) (justify left))
+    )
+    (property "Value" "100nF" (at 202.184 29.972 0)
+      (effects (font (size 1.27 1.27)) (justify left))
+    )
+    (property "Footprint" "Capacitor_SMD:C_0603_1608Metric_Pad1.08x0.95mm_HandSolder" (at 204.1398 27.305 0)
+      (effects (font (size 1.27 1.27)) hide)
+    )
+    (property "Datasheet" "~" (at 205.105 31.115 0)
+      (effects (font (size 1.27 1.27)) hide)
+    )
+    (property "Distributor 1" "JLCPCB" (at 205.105 31.115 0)
+      (effects (font (size 1.27 1.27)) hide)
+    )
+    (property "Distributor 1 PN" "C14663" (at 205.105 31.115 0)
+      (effects (font (size 1.27 1.27)) hide)
+    )
+    (property "Manufacturer" "YAGEO" (at 205.105 31.115 0)
+      (effects (font (size 1.27 1.27)) hide)
+    )
+    (property "MPN" "CC0603KRX7R9BB104" (at 205.105 31.115 0)
+      (effects (font (size 1.27 1.27)) hide)
+    )
+    (property "Description" "50V 100nF X7R ±10% 0603 Multilayer Ceramic Capacitors MLCC - SMD/SMT ROHS" (at 205.105 31.115 0)
+      (effects (font (size 1.27 1.27)) hide)
+    )
+    (property "AssemblyType" "SMT" (at 205.105 31.115 0)
+      (effects (font (size 1.27 1.27)) hide)
+    )
+    (property "Cost" "0.0021" (at 205.105 31.115 0)
+      (effects (font (size 1.27 1.27)) hide)
+    )
+    (pin "1")
+    (pin "2")
+    (instances
+      (project "PCBa_KRAKE"
+        (path "/412a327d-1ee3-473e-bc00-1545004b7edf"
+          (reference "C103") (unit 1)
+        )
+        (path "/412a327d-1ee3-473e-bc00-1545004b7edf/00000000-0000-0000-0000-000062b93801"
+          (reference "C?") (unit 1)
+        )
+      )
