File: PCBa_KRAKE/SPI Peripherial.kicad_sch (KiCad schematic)
At the start: 27 parts, among them J401 RJ12_6P6C_HORZ

Commit message: Renames UART1 GPIO pins of ESP32. Relocated internal LED. And asthetic changes.
Other:
- moved on the sheet: F401, R401, R402, R403

Commit message: ERC Okay, waved warnings on symbol issues.
Connections:
- net +12in: now also F401.2, J401.5
Changed lines of the file:
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@@
+    (stroke (width 0) (type default))
+  )
+  (wire (pts (xy 43.815 75.565) (xy 71.12 75.565))
     (stroke (width 0) (type default))
   )
@@
   )
   (wire (pts (xy 203.2 114.935) (xy 203.2 122.555))
-    (stroke (width 0) (type default))
-  )
-  (wire (pts (xy 71.12 75.565) (xy 43.815 75.565))
     (stroke (width 0) (type default))
   )
@@
     (effects (font (size 1.27 1.27)) (justify left bottom))
   )
-  (label "+12in" (at 43.18 75.565 0) (fields_autoplaced)
-    (effects (font (size 1.27 1.27)) (justify left bottom))
-  )
+  (label "+12in" (at 43.815 75.565 0) (fields_autoplaced)
+    (effects (font (size 1.27 1.27)) (justify left bottom))
+  )

Commit message: Corrected the voltage connection for the mute switch, from 5V to 3V3. Rerouted and reconnected the tracks for R603.
Other:
- moved on the sheet: C103, D?, F401, J401, Q?, R403, R404, R?

Commit message: Found missing part numbers. ESP32.
Parts:
- D? (x4): Cost (none) -> 0.0098; Distributor 1 (none) -> JLCPCB; Distributor 1 PN (none) -> C47546; MPN (none) -> BAT54S,215; Manufacturer (none) -> Nexperia
Changed lines of the file:
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@@
+      (effects (font (size 1.27 1.27)) hide)
+    )
+    (property "Distributor 1 PN" "C47546" (at 168.91 127 0)
+      (effects (font (size 1.27 1.27)) hide)
+    )
+    (property "Cost" "0.0098" (at 168.91 127 0)
+      (effects (font (size 1.27 1.27)) hide)
+    )
+    (property "Description" "30V 1 pair in series 800mV@100mA 200mA SOT-23 Schottky Diodes ROHS" (at 168.91 127 0)
+      (effects (font (size 1.27 1.27)) hide)
+    )
+    (property "Distributor 1" "JLCPCB" (at 168.91 127 0)
+      (effects (font (size 1.27 1.27)) hide)
+    )
+    (property "MPN" "BAT54S,215" (at 168.91 127 0)
+      (effects (font (size 1.27 1.27)) hide)
+    )
+    (property "Manufacturer" "Nexperia" (at 168.91 127 0)
       (effects (font (size 1.27 1.27)) hide)
     )
@@
       (effects (font (size 1.27 1.27)) hide)
     )
+    (property "Distributor 1 PN" "C47546" (at 86.36 124.46 0)
+      (effects (font (size 1.27 1.27)) hide)
+    )
+    (property "Cost" "0.0098" (at 86.36 124.46 0)
+      (effects (font (size 1.27 1.27)) hide)
+    )
+    (property "Description" "30V 1 pair in series 800mV@100mA 200mA SOT-23 Schottky Diodes ROHS" (at 86.36 124.46 0)
+      (effects (font (size 1.27 1.27)) hide)
+    )
+    (property "Distributor 1" "JLCPCB" (at 86.36 124.46 0)
+      (effects (font (size 1.27 1.27)) hide)
+    )
+    (property "MPN" "BAT54S,215" (at 86.36 124.46 0)
+      (effects (font (size 1.27 1.27)) hide)
+    )
+    (property "Manufacturer" "Nexperia" (at 86.36 124.46 0)
+      (effects (font (size 1.27 1.27)) hide)
+    )
     (pin "1")
     (pin "2")
@@
       (effects (font (size 1.27 1.27)) hide)
     )
+    (property "Distributor 1 PN" "C47546" (at 116.84 48.26 0)
+      (effects (font (size 1.27 1.27)) hide)
+    )
+    (property "Cost" "0.0098" (at 116.84 48.26 0)
+      (effects (font (size 1.27 1.27)) hide)
+    )
+    (property "Description" "30V 1 pair in series 800mV@100mA 200mA SOT-23 Schottky Diodes ROHS" (at 116.84 48.26 0)
+      (effects (font (size 1.27 1.27)) hide)
+    )
+    (property "Distributor 1" "JLCPCB" (at 116.84 48.26 0)
+      (effects (font (size 1.27 1.27)) hide)
+    )
+    (property "MPN" "BAT54S,215" (at 116.84 48.26 0)
+      (effects (font (size 1.27 1.27)) hide)
+    )
+    (property "Manufacturer" "Nexperia" (at 116.84 48.26 0)
+      (effects (font (size 1.27 1.27)) hide)
+    )
     (pin "1")
     (pin "2")
@@
       (effects (font (size 1.27 1.27)) hide)
     )
+    (property "Distributor 1 PN" "C47546" (at 191.77 49.53 0)
+      (effects (font (size 1.27 1.27)) hide)
+    )
+    (property "Cost" "0.0098" (at 191.77 49.53 0)
+      (effects (font (size 1.27 1.27)) hide)
+    )
+    (property "Description" "30V 1 pair in series 800mV@100mA 200mA SOT-23 Schottky Diodes ROHS" (at 191.77 49.53 0)
+      (effects (font (size 1.27 1.27)) hide)
+    )
+    (property "Distributor 1" "JLCPCB" (at 191.77 49.53 0)
+      (effects (font (size 1.27 1.27)) hide)
+    )
+    (property "MPN" "BAT54S,215" (at 191.77 49.53 0)
+      (effects (font (size 1.27 1.27)) hide)
+    )
+    (property "Manufacturer" "Nexperia" (at 191.77 49.53 0)
+      (effects (font (size 1.27 1.27)) hide)
+    )

Commit message: Adding component information. Deleted a redundant LED from the schematic.
Parts:
- D? (x4): AssemblyType (none) -> SMT
- F401: value Polyfuse_Small -> Polyfuse_Small_1A
Changed lines of the file:
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@@
       (effects (font (size 1.27 1.27)))
     )
-    (property "Value" "Polyfuse_Small" (at 83.82 69.215 90)
+    (property "Value" "Polyfuse_Small_1A" (at 83.82 69.215 90)
       (effects (font (size 1.27 1.27)))
     )
@@
       (effects (font (size 1.27 1.27)) hide)
     )
+    (property "AssemblyType" "SMT" (at 168.91 127 0)
+      (effects (font (size 1.27 1.27)) hide)
+    )
     (pin "1")
     (pin "2")
@@
       (effects (font (size 1.27 1.27)) hide)
     )
+    (property "AssemblyType" "SMT" (at 86.36 124.46 0)
+      (effects (font (size 1.27 1.27)) hide)
+    )
     (pin "1")
     (pin "2")
@@
       (effects (font (size 1.27 1.27)) hide)
     )
+    (property "AssemblyType" "SMT" (at 116.84 48.26 0)
+      (effects (font (size 1.27 1.27)) hide)
+    )
     (pin "1")
     (pin "2")
@@
       (effects (font (size 1.27 1.27)) hide)
     )
+    (property "AssemblyType" "SMT" (at 191.77 49.53 0)
+      (effects (font (size 1.27 1.27)) hide)
+    )
