File: PCBa_KRAKE/AlarmAudio.kicad_sch (KiCad schematic)
At the start: 18 parts, among them J601 22-23-2021, J602 22-23-2021, Q601 BSS138, Q602 DNI

Commit message: Updating ESP32 schematic symbol and added the df player into the audio schematic.
Parts:
- added J1: Conn_01x08, GeneralPurposeAlarmDevicePCB:DFPlayer_mini_20241116, symbol GPAD_SCH_LIB:DFPlayermini_241116
- added LS?: Speaker, symbol Device:Speaker
- added R502 (x2), R503: 330R, Resistor_SMD:R_0603_1608Metric_Pad0.98x0.95mm_HandSolder, symbol Device:R
Connections:
- net +5V: now also J1.1 (VCC)
- net GND: now also J1.10 (GND), J1.7 (GND)
- new net: J1.2 (RX), R502.1
- new net: J1.8 (SPK_2), LS?.1
- new net: J1.6 (SPK_1), LS?.2
- new net: J1.3 (TX), R503.1
- new net: J1.16 (BUSY), R502.1
- new net Busy: R502.2
- new net ControllerRX: R503.2
- new net ControllerTX: R502.2
Other:
- note added: "NULL MODEM"
- note added: "Place R503 near uControler TX pin."

Commit message: Fixed the DFPlayer schematic symbol, for pin electrical type and symbol name.
Parts:
- J1: value Conn_01x08 -> DFPlayermini
Changed lines of the file:
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@@
       (effects (font (size 1.27 1.27)))
     )
-    (property "Value" "Conn_01x08" (at 223.52 121.92 0)
+    (property "Value" "DFPlayermini" (at 223.52 121.92 0)
       (effects (font (size 1.27 1.27)))
     )
@@
       (effects (font (size 1.27 1.27)) hide)
     )
-    (property "Datasheet" "~" (at 213.36 133.35 0)
+    (property "Datasheet" "https://image.dfrobot.com/image/data/DFR0299/DFPlayer%20Mini%20Manul.pdf" (at 213.36 133.35 0)
       (effects (font (size 1.27 1.27)) hide)
     )

Commit message: Added a decoupling power supply to the DFPlayer and added an LED to the Busy pin.
Parts:
- added C2: 100nF, Capacitor_SMD:C_0603_1608Metric_Pad1.08x0.95mm_HandSolder, symbol Device:C
- added C4: 47uF 16V, Capacitor_SMD:CP_Elec_5x5.4, symbol Device:C_Polarized
- added D106: RED 0603, LED_SMD:LED_0603_1608Metric_Pad1.05x0.95mm_HandSolder, symbol Device:LED
- added R1: 1R0, Resistor_SMD:R_0603_1608Metric_Pad0.98x0.95mm_HandSolder, symbol Device:R
- added R112: 330R, Resistor_SMD:R_0603_1608Metric_Pad0.98x0.95mm_HandSolder, symbol Device:R
Connections:
- net +5V: now also R1.2; no longer J1.1 (VCC)
- net GND: now also C2.2, C4.2
- net at J1.16 (BUSY), R502.1: now also D106.1 (K)
- new net: D106.2 (A), R112.1
- new net 5VDFP: C2.1, C4.1, J1.1 (VCC), R1.1, R112.2

Commit message: Adding cooments in the title block, page setting of PCBa_Krake.
Other:
- title: GeneralPurposeAlarmDevicePCB -> KRAKE_PCB
Changed lines of the file:
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@@
   (paper "USLetter")
   (title_block
-    (title "GeneralPurposeAlarmDevicePCB")
-    (date "2023-04-25")
-    (rev "2.2")
+    (title "KRAKE_PCB")
+    (date "2024-11-23")
+    (rev "1")
     (company "PublicInvention")
     (comment 1 "GNU Affero General Public License v3.0")
-    (comment 2 "DrawnBy: (Forrest) Lee Erickson")
+    (comment 2 "DrawnBy: (Forrest) Lee Erickson, Nagham Kheir")
+    (comment 3 "https://github.com/PubInv/krake")
+    (comment 4 "Inherited from the GPAD")
   )
   (junction (at 95.25 123.19) (diameter 0) (color 0 0 0 0)

Commit message: Added a connector for external speaker.
Parts:
- added J?: 22-23-2021, Connector_Molex:Molex_KK-254_AE-6410-02A_1x02_P2.54mm_Vertical, symbol GPAD_SCH_LIB:22-23-2021
Changed lines of the file:
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@@
     (effects (font (size 1.27 1.27)) (justify left bottom))
+  )
+  (text "For external \"speaker\"." (at 171.45 146.05 0)
+    (effects (font (size 1.27 1.27)) (justify right bottom))
   )
   (label "5VDFP" (at 238.76 87.63 0) (fields_autoplaced)
@@
         )
       )
+    )
+  )
+  (symbol (lib_id "GPAD_SCH_LIB:22-23-2021") (at 170.18 151.13 270) (unit 1)
+    (in_bom yes) (on_board yes) (dnp no)
+    (property "Reference" "J?" (at 166.37 148.59 90)
+      (effects (font (size 1.27 1.27)) (justify right))
+    )
+    (property "Value" "22-23-2021" (at 173.99 157.48 90)
+      (effects (font (size 1.27 1.27)) (justify right))
+    )
+    (property "Footprint" "Connector_Molex:Molex_KK-254_AE-6410-02A_1x02_P2.54mm_Vertical" (at 175.26 156.21 0)
+      (effects (font (size 1.524 1.524)) (justify left) hide)
+    )
+    (property "Datasheet" "https://media.digikey.com/pdf/Data%20Sheets/Molex%20PDFs/A-6373-N_Series_Dwg_2010-12-03.pdf" (at 177.8 156.21 0)
+      (effects (font (size 1.524 1.524)) (justify left) hide)
+    )
+    (property "Digi-Key_PN" "WM4200-ND" (at 180.34 156.21 0)
+      (effects (font (size 1.524 1.524)) (justify left) hide)
+    )
+    (property "MPN" "22-23-2021" (at 182.88 156.21 0)
+      (effects (font (size 1.524 1.524)) (justify left) hide)
+    )
+    (property "Category" "Connectors, Interconnects" (at 185.42 156.21 0)
+      (effects (font (size 1.524 1.524)) (justify left) hide)
+    )
+    (property "Family" "Rectangular Connectors - Headers, Male Pins" (at 187.96 156.21 0)
+      (effects (font (size 1.524 1.524)) (justify left) hide)
+    )
+    (property "DK_Datasheet_Link" "https://media.digikey.com/pdf/Data%20Sheets/Molex%20PDFs/A-6373-N_Series_Dwg_2010-12-03.pdf" (at 190.5 156.21 0)
+      (effects (font (size 1.524 1.524)) (justify left) hide)
+    )
+    (property "DK_Detail_Page" "/product-detail/en/molex/22-23-2021/WM4200-ND/26667" (at 193.04 156.21 0)
+      (effects (font (size 1.524 1.524)) (justify left) hide)
+    )
+    (property "Description" "CONN HEADER VERT 2POS 2.54MM" (at 195.58 156.21 0)
+      (effects (font (size 1.524 1.524)) (justify left) hide)
+    )
+    (property "Manufacturer" "Molex" (at 198.12 156.21 0)
+      (effects (font (size 1.524 1.524)) (justify left) hide)
+    )
+    (property "Status" "Active" (at 200.66 156.21 0)
+      (effects (font (size 1.524 1.524)) (justify left) hide)
+    )
+    (property "Assembly Type" "" (at 58.42 -43.18 0)
+      (effects (font (size 1.27 1.27)) hide)
+    )
+    (property "AssemblyType" "HAND" (at 170.18 151.13 0)
+      (effects (font (size 1.27 1.27)) hide)
+    )
+    (property "Cost" "0.22000" (at 170.18 151.13 0)
+      (effects (font (size 1.27 1.27)) hide)
+    )
+    (property "Distributor 1" "DigiKey" (at 170.18 151.13 0)
+      (effects (font (size 1.27 1.27)) hide)
+    )
+    (property "Distributor 1 PN" "900-0022232021-ND" (at 170.18 151.13 0)
+      (effects (font (size 1.27 1.27)) hide)
+    )
+    (pin "1")
+    (pin "2")
+    (instances
+      (project "PCBa_KRAKE"
+        (path "/412a327d-1ee3-473e-bc00-1545004b7edf/00000000-0000-0000-0000-000062dd8e5f"
+          (reference "J?") (unit 1)
+        )
+        (path "/412a327d-1ee3-473e-bc00-1545004b7edf"
+          (reference "J?") (unit 1)
+        )
+      )

Commit message: Working in a new brnach to do PCBa edits.
Parts:
- gave numbers to parts that had none: 1
Changed lines of the file:
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@@
   (symbol (lib_id "GPAD_SCH_LIB:22-23-2021") (at 170.18 151.13 270) (unit 1)
     (in_bom yes) (on_board yes) (dnp no)
-    (property "Reference" "J?" (at 166.37 148.59 90)
+    (property "Reference" "J502" (at 166.37 148.59 90)
       (effects (font (size 1.27 1.27)) (justify right))
     )
@@
       (project "PCBa_KRAKE"
         (path "/412a327d-1ee3-473e-bc00-1545004b7edf/00000000-0000-0000-0000-000062dd8e5f"
-          (reference "J?") (unit 1)
+          (reference "J502") (unit 1)
         )
         (path "/412a327d-1ee3-473e-bc00-1545004b7edf"
