File: PCBa_KRAKE/AlarmAudio.kicad_sch (KiCad schematic)
At the start: 29 parts, among them J1 DFPlayermini, J502 22-23-2021, J601 22-23-2021, J602 22-23-2021, Q601 BSS138, Q602 DNI

Commit message: Adding speaker pin header and a speaker 3D model footprint.
Parts:
- J601: renamed from J502; value 22-23-2021 -> 1X2P 1.27 mm Header; footprint Connector_Molex:Molex_KK-254_AE-6410-02A_1x02_P2.54mm_Vertical -> Connector_PinHeader_1.27mm:PinHeader_1x02_P1.27mm_Vertical; AssemblyType HAND -> (none); Category Connectors, Interconnects -> (none); Cost 0.22000 -> (none); DK_Datasheet_Link https://media.digikey.com/pdf/Data%20Sheets/Molex%20PDFs/A-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 -> (none); DK_Detail_Page /product-detail/en/molex/22-23-2021/WM4200-ND/26667 -> (none); Digi-Key_PN WM4200-ND -> (none); Distributor 1 DigiKey -> JLCPCB; Distributor 1 PN 900-0022232021-ND -> C7496728; Family Rectangular Connectors - Headers, Male Pins -> (none); MPN 22-23-2021 -> (none); Manufacturer Molex -> (none); Status Active -> (none)
- LS?: footprint (none) -> GeneralPurposeAlarmDevicePCB:Speaker2w_Buzzer_12x9.5RM7.6
Connections:
- net at J601.1: now also J1.8 (SPK_2), LS?.1
- net at J601.2: now also J1.6 (SPK_1), LS?.2
Other:
- moved on the sheet: J601, LS?
Changed lines of the file:
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@@
   (junction (at 182.88 40.64) (diameter 0) (color 0 0 0 0)
   )
+  (junction (at 196.85 148.59) (diameter 0) (color 0 0 0 0)
+  )
   (junction (at 72.39 48.26) (diameter 0) (color 0 0 0 0)
   )
@@
   (junction (at 177.8 48.26) (diameter 0) (color 0 0 0 0)
   )
+  (junction (at 201.93 151.13) (diameter 0) (color 0 0 0 0)
+  )
   (junction (at 137.16 68.58) (diameter 0) (color 0 0 0 0)
   )
@@
     (stroke (width 0) (type default))
   )
-  (wire (pts (xy 201.93 151.13) (xy 201.93 143.51))
+  (wire (pts (xy 201.93 143.51) (xy 201.93 151.13))
     (stroke (width 0) (type default))
   )
@@
     (stroke (width 0) (type default))
   )
+  (wire (pts (xy 194.31 151.13) (xy 201.93 151.13))
+    (stroke (width 0) (type default))
+  )
   (wire (pts (xy 177.8 130.81) (xy 165.1 130.81))
     (stroke (width 0) (type default))
@@
     (stroke (width 0) (type default))
   )
+  (wire (pts (xy 189.865 159.385) (xy 201.93 159.385))
+    (stroke (width 0) (type default))
+  )
   (wire (pts (xy 110.49 97.79) (xy 116.84 97.79))
     (stroke (width 0) (type default))
@@
     (stroke (width 0) (type default))
   )
+  (wire (pts (xy 189.865 156.845) (xy 196.85 156.845))
+    (stroke (width 0) (type default))
+  )
   (wire (pts (xy 95.25 118.11) (xy 95.25 123.19))
     (stroke (width 0) (type default))
@@
     (stroke (width 0) (type default))
   )
+  (wire (pts (xy 196.85 156.845) (xy 196.85 148.59))
+    (stroke (width 0) (type default))
+  )
   (wire (pts (xy 160.02 68.58) (xy 161.29 68.58))
     (stroke (width 0) (type default))
   )
-  (wire (pts (xy 194.31 151.13) (xy 201.93 151.13))
-    (stroke (width 0) (type default))
-  )
   (wire (pts (xy 62.23 134.62) (xy 62.23 137.16))
     (stroke (width 0) (type default))
@@
     (stroke (width 0) (type default))
   )
+  (wire (pts (xy 201.93 151.13) (xy 201.93 159.385))
+    (stroke (width 0) (type default))
+  )
   (wire (pts (xy 83.82 123.19) (xy 81.28 123.19))
     (stroke (width 0) (type default))
@@
     (stroke (width 0) (type default))
   )
+  (wire (pts (xy 123.19 71.12) (xy 123.19 77.47))
+    (stroke (width 0) (type default))
+  )
+  (wire (pts (xy 81.28 118.11) (xy 83.82 118.11))
+    (stroke (width 0) (type default))
+  )
+  (wire (pts (xy 223.52 87.63) (xy 227.33 87.63))
+    (stroke (width 0) (type default))
+  )
+  (wire (pts (xy 50.8 118.11) (xy 40.64 118.11))
+    (stroke (width 0) (type default))
+  )
   (wire (pts (xy 194.31 148.59) (xy 196.85 148.59))
-    (stroke (width 0) (type default))
-  )
-  (wire (pts (xy 123.19 71.12) (xy 123.19 77.47))
-    (stroke (width 0) (type default))
-  )
-  (wire (pts (xy 81.28 118.11) (xy 83.82 118.11))
-    (stroke (width 0) (type default))
-  )
-  (wire (pts (xy 223.52 87.63) (xy 227.33 87.63))
-    (stroke (width 0) (type default))
-  )
-  (wire (pts (xy 50.8 118.11) (xy 40.64 118.11))
     (stroke (width 0) (type default))
   )
@@
     )
   )
-  (symbol (lib_id "GPAD_SCH_LIB:22-23-2021") (at 170.18 151.13 270) (unit 1)
-    (in_bom yes) (on_board yes) (dnp no)
-    (property "Reference" "J502" (at 166.37 148.59 90)
+  (symbol (lib_id "GPAD_SCH_LIB:22-23-2021") (at 191.77 151.13 270) (mirror x) (unit 1)
+    (in_bom yes) (on_board yes) (dnp no)
+    (property "Reference" "J601" (at 196.85 152.4 90)
       (effects (font (size 1.27 1.27)) (justify right))
     )
-    (property "Value" "22-23-2021" (at 173.99 157.48 90)
+    (property "Value" "1X2P 1.27 mm Header" (at 195.58 144.78 90)
       (effects (font (size 1.27 1.27)) (justify right))
     )
-    (property "Footprint" "Connector_Molex:Molex_KK-254_AE-6410-02A_1x02_P2.54mm_Vertical" (at 175.26 156.21 0)
-      (effects (font (size 1.524 1.524)) (justify left) hide)
-    )
-    (property "Datasheet" "https://media.digikey.com/pdf/Data%20Sheets/Molex%20PDFs/A-6373-N_Series_Dwg_2010-12-03.pdf" (at 177.8 156.21 0)
-      (effects (font (size 1.524 1.524)) (justify left) hide)
-    )
-    (property "Digi-Key_PN" "WM4200-ND" (at 180.34 156.21 0)
-      (effects (font (size 1.524 1.524)) (justify left) hide)
-    )
-    (property "MPN" "22-23-2021" (at 182.88 156.21 0)
-      (effects (font (size 1.524 1.524)) (justify left) hide)
-    )
-    (property "Category" "Connectors, Interconnects" (at 185.42 156.21 0)
-      (effects (font (size 1.524 1.524)) (justify left) hide)
-    )
-    (property "Family" "Rectangular Connectors - Headers, Male Pins" (at 187.96 156.21 0)
-      (effects (font (size 1.524 1.524)) (justify left) hide)
-    )
-    (property "DK_Datasheet_Link" "https://media.digikey.com/pdf/Data%20Sheets/Molex%20PDFs/A-6373-N_Series_Dwg_2010-12-03.pdf" (at 190.5 156.21 0)
-      (effects (font (size 1.524 1.524)) (justify left) hide)
-    )
-    (property "DK_Detail_Page" "/product-detail/en/molex/22-23-2021/WM4200-ND/26667" (at 193.04 156.21 0)
-      (effects (font (size 1.524 1.524)) (justify left) hide)
-    )
-    (property "Description" "CONN HEADER VERT 2POS 2.54MM" (at 195.58 156.21 0)
-      (effects (font (size 1.524 1.524)) (justify left) hide)
-    )
-    (property "Manufacturer" "Molex" (at 198.12 156.21 0)
-      (effects (font (size 1.524 1.524)) (justify left) hide)
-    )
-    (property "Status" "Active" (at 200.66 156.21 0)
-      (effects (font (size 1.524 1.524)) (justify left) hide)
-    )
-    (property "Assembly Type" "" (at 58.42 -43.18 0)
-      (effects (font (size 1.27 1.27)) hide)
-    )
-    (property "AssemblyType" "HAND" (at 170.18 151.13 0)
-      (effects (font (size 1.27 1.27)) hide)
-    )
-    (property "Cost" "0.22000" (at 170.18 151.13 0)
-      (effects (font (size 1.27 1.27)) hide)
-    )
-    (property "Distributor 1" "DigiKey" (at 170.18 151.13 0)
-      (effects (font (size 1.27 1.27)) hide)
-    )
-    (property "Distributor 1 PN" "900-0022232021-ND" (at 170.18 151.13 0)
+    (property "Footprint" "Connector_PinHeader_1.27mm:PinHeader_1x02_P1.27mm_Vertical" (at 196.85 146.05 0)
+      (effects (font (size 1.524 1.524)) (justify left) hide)
+    )
+    (property "Datasheet" " " (at 199.39 146.05 0)
+      (effects (font (size 1.524 1.524)) (justify left) hide)
+    )
+    (property "Digi-Key_PN" " " (at 201.93 146.05 0)
+      (effects (font (size 1.524 1.524)) (justify left) hide)
+    )
+    (property "MPN" " " (at 204.47 146.05 0)
+      (effects (font (size 1.524 1.524)) (justify left) hide)
+    )
+    (property "Category" " " (at 207.01 146.05 0)
+      (effects (font (size 1.524 1.524)) (justify left) hide)
+    )
+    (property "Family" " " (at 209.55 146.05 0)
+      (effects (font (size 1.524 1.524)) (justify left) hide)
+    )
+    (property "DK_Datasheet_Link" " " (at 212.09 146.05 0)
+      (effects (font (size 1.524 1.524)) (justify left) hide)
+    )
+    (property "DK_Detail_Page" "" (at 214.63 146.05 0)
+      (effects (font (size 1.524 1.524)) (justify left) hide)
+    )
+    (property "Description" "Direct Insert 2P 1.5mm Single Row 1x2P Plugin,P=1.5mm Pin Headers ROHS" (at 217.17 146.05 0)
+      (effects (font (size 1.524 1.524)) (justify left) hide)
+    )
+    (property "Manufacturer" "" (at 219.71 146.05 0)
+      (effects (font (size 1.524 1.524)) (justify left) hide)
+    )
+    (property "Status" "" (at 222.25 146.05 0)
+      (effects (font (size 1.524 1.524)) (justify left) hide)
+    )
+    (property "Assembly Type" "" (at 80.01 345.44 0)
+      (effects (font (size 1.27 1.27)) hide)
+    )
+    (property "AssemblyType" "" (at 191.77 151.13 0)
+      (effects (font (size 1.27 1.27)) hide)
+    )
+    (property "Cost" "" (at 191.77 151.13 0)
+      (effects (font (size 1.27 1.27)) hide)
+    )
+    (property "Distributor 1" "JLCPCB" (at 191.77 151.13 0)
+      (effects (font (size 1.27 1.27)) hide)
+    )
+    (property "Distributor 1 PN" "C7496728" (at 191.77 151.13 0)
       (effects (font (size 1.27 1.27)) hide)
     )
@@
       (project "PCBa_KRAKE"
         (path "/412a327d-1ee3-473e-bc00-1545004b7edf/00000000-0000-0000-0000-000062dd8e5f"
-          (reference "J502") (unit 1)
+          (reference "J601") (unit 1)
         )
         (path "/412a327d-1ee3-473e-bc00-1545004b7edf"
@@
     )
   )
-  (symbol (lib_id "Device:Speaker") (at 189.23 151.13 180) (unit 1)
+  (symbol (lib_id "Device:Speaker") (at 184.785 159.385 180) (unit 1)
     (in_bom yes) (on_board yes) (dnp no) (fields_autoplaced)
-    (property "Reference" "LS?" (at 188.722 139.7 0)
-      (effects (font (size 1.27 1.27)))
-    )
-    (property "Value" "Speaker" (at 188.722 142.24 0)
-      (effects (font (size 1.27 1.27)))
-    )
-    (property "Footprint" "" (at 189.23 146.05 0)
-      (effects (font (size 1.27 1.27)) hide)
-    )
-    (property "Datasheet" "~" (at 189.484 149.86 0)
+    (property "Reference" "LS?" (at 184.277 148.59 0)
+      (effects (font (size 1.27 1.27)))
+    )
+    (property "Value" "Speaker" (at 184.277 151.13 0)
+      (effects (font (size 1.27 1.27)))
+    )
+    (property "Footprint" "GeneralPurposeAlarmDevicePCB:Speaker2w_Buzzer_12x9.5RM7.6" (at 184.785 154.305 0)
+      (effects (font (size 1.27 1.27)) hide)
+    )
+    (property "Datasheet" "~" (at 185.039 158.115 0)
       (effects (font (size 1.27 1.27)) hide)
     )
@@
         )
         (path "/412a327d-1ee3-473e-bc00-1545004b7edf/00000000-0000-0000-0000-000062dd8e5f"
-          (reference "LS501") (unit 1)
-        )
-      )
+          (reference "BZ601") (unit 1)
+        )
+      )

Commit message: ERC Okay, waved warnings on symbol issues.
Parts:
- removed BZ601: BUZZER MAGNETIC 5V 12MM TH, GeneralPurposeAlarmDevicePCB:Buzzer_12.2mm_9.7mm_7.62mm, symbol GPAD_SCH_LIB:Buzzer_Adafruit_P1536A
- removed C601: 47uF 16V, Capacitor_SMD:CP_Elec_5x5.4, symbol Device:C_Polarized
- removed J601: 22-23-2021, Connector_Molex:Molex_KK-254_AE-6410-02A_1x02_P2.54mm_Vertical, symbol GPAD_SCH_LIB:22-23-2021
- removed Q601: BSS138, Package_TO_SOT_SMD:SOT-23, symbol Transistor_FET:BSS138
- removed Q602: DNI, digikey-footprints:SOT-23-3, symbol Device:Q_PNP_BEC
- removed R505: 10K, Resistor_SMD:R_0603_1608Metric_Pad0.98x0.95mm_HandSolder, symbol Device:R
- removed R506, R604: DNI, Resistor_SMD:R_0603_1608Metric_Pad0.98x0.95mm_HandSolder, symbol Device:R
- removed R507, R508, R601: 1R, Resistor_SMD:R_0603_1608Metric_Pad0.98x0.95mm_HandSolder, symbol Device:R
- removed R602: 1K, Resistor_SMD:R_0603_1608Metric_Pad0.98x0.95mm_HandSolder, symbol Device:R
- removed R605: 330R, Resistor_SMD:R_0603_1608Metric_Pad0.98x0.95mm_HandSolder, symbol Device:R
- removed TP501: VccBuzzer, TestPoint:TestPoint_Loop_D2.54mm_Drill1.5mm_Beaded, symbol Connector:TestPoint
Connections:
- no-connect marks 0 -> 8
Other:
- note added: "Notes on DFPayer USA1 has a low cost(TD5580A) which is not the DFROBOT MockingKrake has the DFROBOT"
- note removed: "Notes on Buzzer vendors Units assembled with these two parts are similar in performance but not identical. Assemble SN 22, 23, 24 and 25 with Digikey number 433-WST-1210T-ND. Assemble SN 26, 27, 28 , 29 and 30 with Digikey number 102-CMI-1295-0585T-ND. And Assemble SN ?16, 17, 18 , and 19? with Adafruit part."
- moved on the sheet: C2, C4, C602, D106, J1, J601, J602, LS?, R1, R112, R502, R503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

Commit message: Fixing annotations.
Changed lines of the file:
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@@
   (symbol (lib_id "GPAD_SCH_LIB:DFPlayermini_241116") (at 198.755 112.395 0) (unit 1)
     (in_bom yes) (on_board yes) (dnp no) (fields_autoplaced)
-    (property "Reference" "J1" (at 208.915 98.425 0)
+    (property "Reference" "J1" (at 208.915 99.06 0)
       (effects (font (size 1.27 1.27)))
     )
-    (property "Value" "DFPlayermini" (at 208.915 100.965 0)
+    (property "Value" "DFPlayermini" (at 208.915 101.6 0)
       (effects (font (size 1.27 1.27)))
     )
@@
         )
         (path "/412a327d-1ee3-473e-bc00-1545004b7edf/00000000-0000-0000-0000-000062dd8e5f"
-          (reference "J501") (unit 1)
+          (reference "J603") (unit 1)
         )
       )

Commit message: Rotating and connecting the rotary encoder.
Connections:
- net +5V: no longer R603.2
- new net 3v3: R603.2
Other:
- moved on the sheet: C2, C4, C602, D106, J1, J601, J602, R1, R112, R502, R503, R603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

Commit message: Fixed Hardware, PCB of 20250114, J601 Interferes with DFPlayer SD Card Egress/Ingress #137
Other:
- note added: "The speaker is not mounted directly onto the board"
Changed lines of the file:
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@@
     )
+  )
+  (text "The speaker is not mounted directly onto the board"
+    (at 170.18 144.78 0)
+    (effects (font (size 1.27 1.27)) (justify left bottom))
   )
   (text "Notes on DFPayer\n\nUSA1 has a low cost(TD5580A) which is not the DFROBOT\nMockingKrake has the DFROBOT"
