File: PCBa_KRAKE/AlarmAudio.kicad_sch (KiCad schematic)
At the start: 15 parts, among them J1 DFPlayermini, J601 1X2P 1.27 mm Header, J602 22-23-2021

Commit message: Adding component information. Deleted a redundant LED from the schematic.
Parts:
- removed D106: RED 0603, LED_SMD:LED_0603_1608Metric_Pad1.05x0.95mm_HandSolder, symbol Device:LED
- removed R112: 330R, Resistor_SMD:R_0603_1608Metric_Pad0.98x0.95mm_HandSolder, symbol Device:R
- J601: Cost (none) -> 0.0183
- J602: value 22-23-2021 -> 0.100_2Pin; footprint Connector_Molex:Molex_KK-254_AE-6410-02A_1x02_P2.54mm_Vertical -> Connector_PinHeader_2.54mm:PinHeader_1x02_P2.54mm_Vertical; Cost 0.22000 -> 0.1458; Distributor 1 DigiKey -> JLCPCB; Distributor 1 PN 900-0022232021-ND -> C168673; MPN 22-23-2021 -> 68000-102HLF; Manufacturer Molex -> Amphenol ICC
Changed lines of the file:
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@@
   (junction (at 212.09 71.12) (diameter 0) (color 0 0 0 0)
   )
-  (junction (at 217.17 67.31) (diameter 0) (color 0 0 0 0)
-  )
   (junction (at 198.12 71.12) (diameter 0) (color 0 0 0 0)
   )
   (junction (at 66.04 81.28) (diameter 0) (color 0 0 0 0)
-  )
-  (junction (at 224.79 105.41) (diameter 0) (color 0 0 0 0)
   )
   (junction (at 187.96 130.81) (diameter 0) (color 0 0 0 0)
@@
     (stroke (width 0) (type default))
   )
-  (wire (pts (xy 231.14 102.87) (xy 231.14 105.41))
-    (stroke (width 0) (type default))
-  )
   (wire (pts (xy 194.31 67.31) (xy 201.93 67.31))
     (stroke (width 0) (type default))
@@
     (stroke (width 0) (type default))
   )
-  (wire (pts (xy 224.79 105.41) (xy 231.14 105.41))
-    (stroke (width 0) (type default))
-  )
   (wire (pts (xy 68.58 66.04) (xy 68.58 81.28))
     (stroke (width 0) (type default))
@@
     (stroke (width 0) (type default))
   )
-  (wire (pts (xy 231.14 95.25) (xy 231.14 93.98))
-    (stroke (width 0) (type default))
-  )
   (wire (pts (xy 78.74 102.87) (xy 78.74 105.41))
     (stroke (width 0) (type default))
@@
     (stroke (width 0) (type default))
   )
-  (wire (pts (xy 217.17 67.31) (xy 231.14 67.31))
-    (stroke (width 0) (type default))
-  )
   (wire (pts (xy 187.96 130.81) (xy 187.96 138.43))
     (stroke (width 0) (type default))
@@
   )
   (wire (pts (xy 187.96 123.19) (xy 194.31 123.19))
-    (stroke (width 0) (type default))
-  )
-  (wire (pts (xy 231.14 67.31) (xy 231.14 86.36))
     (stroke (width 0) (type default))
   )
@@
     (effects (font (size 1.27 1.27)) (justify right bottom))
   )
-  (label "5VDFP" (at 224.79 67.31 0) (fields_autoplaced)
+  (label "5VDFP" (at 217.17 68.58 0) (fields_autoplaced)
     (effects (font (size 1.27 1.27)) (justify left bottom))
   )
@@
       (effects (font (size 1.27 1.27)) hide)
     )
-    (property "Cost" "" (at 177.8 130.81 0)
+    (property "Cost" "0.0183" (at 177.8 130.81 0)
       (effects (font (size 1.27 1.27)) hide)
     )
@@
         (path "/412a327d-1ee3-473e-bc00-1545004b7edf/00000000-0000-0000-0000-000062dd8e5f"
           (reference "BZ601") (unit 1)
-        )
-      )
-    )
-  )
-  (symbol (lib_id "Device:LED") (at 231.14 99.06 90) (unit 1)
-    (in_bom yes) (on_board yes) (dnp no)
-    (property "Reference" "D106" (at 236.22 99.06 90)
-      (effects (font (size 1.524 1.524)))
-    )
-    (property "Value" "RED 0603" (at 240.03 101.6 90)
-      (effects (font (size 1.524 1.524)))
-    )
-    (property "Footprint" "LED_SMD:LED_0603_1608Metric_Pad1.05x0.95mm_HandSolder" (at 231.14 99.06 0)
-      (effects (font (size 1.27 1.27)) hide)
-    )
-    (property "Datasheet" "~" (at 231.14 99.06 0)
-      (effects (font (size 1.27 1.27)) hide)
-    )
-    (property "Distributor 1" "JLCPCB" (at 231.14 99.06 0)
-      (effects (font (size 1.27 1.27)) hide)
-    )
-    (property "Distributor 1 PN" "C2286" (at 220.98 93.98 0)
-      (effects (font (size 1.524 1.524)) (justify left) hide)
-    )
-    (property "MPN" "LTST-C171KRKT" (at 218.44 93.98 0)
-      (effects (font (size 1.524 1.524)) (justify left) hide)
-    )
-    (property "Category" "Optoelectronics" (at 215.9 93.98 0)
-      (effects (font (size 1.524 1.524)) (justify left) hide)
-    )
-    (property "Family" "LED Indication - Discrete" (at 213.36 93.98 0)
-      (effects (font (size 1.524 1.524)) (justify left) hide)
-    )
-    (property "Description" "LED RED CLEAR SMD" (at 205.74 93.98 0)
-      (effects (font (size 1.524 1.524)) (justify left) hide)
-    )
-    (property "Manufacturer" "Lite-On Inc." (at 203.2 93.98 0)
-      (effects (font (size 1.524 1.524)) (justify left) hide)
-    )
-    (property "Status" "Active" (at 200.66 93.98 0)
-      (effects (font (size 1.524 1.524)) (justify left) hide)
-    )
-    (property "DK_Datasheet_Link" "http://optoelectronics.liteon.com/upload/download/DS22-2000-109/LTST-C171KRKT.pdf" (at 346.71 233.68 0)
-      (effects (font (size 1.27 1.27)) hide)
-    )
-    (property "DK_Detail_Page" "/product-detail/en/lite-on-inc/LTST-C171KRKT/160-1427-1-ND/386800" (at 346.71 233.68 0)
-      (effects (font (size 1.27 1.27)) hide)
-    )
-    (property "Digi-Key_PN" "160-1427-1-ND" (at 346.71 233.68 0)
-      (effects (font (size 1.27 1.27)) hide)
-    )
-    (property "AssemblyType" "HAND" (at 231.14 99.06 0)
-      (effects (font (size 1.27 1.27)) hide)
-    )
-    (property "Cost" "0.0054" (at 231.14 99.06 0)
-      (effects (font (size 1.27 1.27)) hide)
-    )
-    (pin "1")
-    (pin "2")
-    (instances
-      (project "PCBa_KRAKE"
-        (path "/412a327d-1ee3-473e-bc00-1545004b7edf"
-          (reference "D106") (unit 1)
-        )
-        (path "/412a327d-1ee3-473e-bc00-1545004b7edf/00000000-0000-0000-0000-000062dd8e5f"
-          (reference "D502") (unit 1)
         )
       )
@@
       (effects (font (size 1.27 1.27)) hide)
     )
+    (property "Description" "47uF 16V 33mA@120Hz ±20% SMD,D5xL5.4mm Aluminum Electrolytic Capacitors - SMD ROHS" (at 212.09 76.2 0)
+      (effects (font (size 1.27 1.27)) hide)
+    )
     (pin "1")
     (pin "2")
@@
       (effects (font (size 1.27 1.27)) (justify right))
     )
-    (property "Value" "22-23-2021" (at 80.01 106.68 90)
+    (property "Value" "0.100_2Pin" (at 80.01 106.68 90)
       (effects (font (size 1.27 1.27)) (justify right))
     )
-    (property "Footprint" "Connector_Molex:Molex_KK-254_AE-6410-02A_1x02_P2.54mm_Vertical" (at 78.74 105.41 0)
+    (property "Footprint" "Connector_PinHeader_2.54mm:PinHeader_1x02_P2.54mm_Vertical" (at 78.74 105.41 0)
       (effects (font (size 1.524 1.524)) (justify left) hide)
     )
@@
       (effects (font (size 1.524 1.524)) (justify left) hide)
     )
-    (property "MPN" "22-23-2021" (at 71.12 105.41 0)
+    (property "MPN" "68000-102HLF" (at 71.12 105.41 0)
       (effects (font (size 1.524 1.524)) (justify left) hide)
     )
@@
       (effects (font (size 1.524 1.524)) (justify left) hide)
     )
-    (property "Description" "CONN HEADER VERT 2POS 2.54MM" (at 58.42 105.41 0)
-      (effects (font (size 1.524 1.524)) (justify left) hide)
-    )
-    (property "Manufacturer" "Molex" (at 55.88 105.41 0)
+    (property "Description" "HEADER VERT 2POS 2.54MM" (at 58.42 105.41 0)
+      (effects (font (size 1.524 1.524)) (justify left) hide)
+    )
+    (property "Manufacturer" "Amphenol ICC" (at 55.88 105.41 0)
       (effects (font (size 1.524 1.524)) (justify left) hide)
     )
@@
       (effects (font (size 1.27 1.27)) hide)
     )
-    (property "Cost" "0.22000" (at 83.82 100.33 0)
-      (effects (font (size 1.27 1.27)) hide)
-    )
-    (property "Distributor 1" "DigiKey" (at 83.82 100.33 0)
-      (effects (font (size 1.27 1.27)) hide)
-    )
-    (property "Distributor 1 PN" "900-0022232021-ND" (at 83.82 100.33 0)
+    (property "Cost" "0.1458" (at 83.82 100.33 0)
+      (effects (font (size 1.27 1.27)) hide)
+    )
+    (property "Distributor 1" "JLCPCB" (at 83.82 100.33 0)
+      (effects (font (size 1.27 1.27)) hide)
+    )
+    (property "Distributor 1 PN" "C168673" (at 83.82 100.33 0)
       (effects (font (size 1.27 1.27)) hide)
     )
@@
         )
       )
-    )
-  )
-  (symbol (lib_id "Device:R") (at 231.14 90.17 180) (unit 1)
-    (in_bom yes) (on_board yes) (dnp no)
-    (property "Reference" "R112" (at 236.22 88.9 90)
-      (effects (font (size 1.27 1.27)))
-    )
-    (property "Value" "330R" (at 233.68 90.17 90)
-      (effects (font (size 1.27 1.27)))
-    )
-    (property "Footprint" "Resistor_SMD:R_0603_1608Metric_Pad0.98x0.95mm_HandSolder" (at 232.918 90.17 90)
-      (effects (font (size 1.27 1.27)) hide)
-    )
-    (property "Datasheet" "~" (at 231.14 90.17 0)
-      (effects (font (size 1.27 1.27)) hide)
-    )
-    (property "Distributor 1" "JLCPCB" (at 231.14 90.17 90)
-      (effects (font (size 1.27 1.27)) hide)
-    )
-    (property "Distributor 1 PN" "C269711" (at 231.14 90.17 90)
-      (effects (font (size 1.27 1.27)) hide)
-    )
-    (property "Manufacturer" "TyoHM" (at 231.14 90.17 90)
-      (effects (font (size 1.27 1.27)) hide)
-    )
-    (property "MPN" "RMC06033301%N" (at 231.14 90.17 90)
-      (effects (font (size 1.27 1.27)) hide)
-    )
-    (property "Description" "0.1W ±1% 330Ω 0603 Chip Resistor - Surface Mount ROHS" (at 231.14 90.17 0)
-      (effects (font (size 1.27 1.27)) hide)
-    )
-    (property "AssemblyType" "SMT" (at 231.14 90.17 0)
-      (effects (font (size 1.27 1.27)) hide)
-    )
-    (property "Cost" "0.0015" (at 231.14 90.17 0)
-      (effects (font (size 1.27 1.27)) hide)
-    )
-    (pin "1")
-    (pin "2")
-    (instances
-      (project "PCBa_KRAKE"
-        (path "/412a327d-1ee3-473e-bc00-1545004b7edf"
-          (reference "R112") (unit 1)
-        )
-        (path "/412a327d-1ee3-473e-bc00-1545004b7edf/00000000-0000-0000-0000-000062dd8e5f"
-          (reference "R513") (unit 1)
-        )
-      )

Commit message: Editting missing feilds in the builk editor, And added a pin header for the LCD.
Connections:
- net at J1.8 (SPK_2), J601.1: no longer LS?.1
- net at J1.6 (SPK_1), J601.2: no longer LS?.2
- no-connect marks 8 -> 10
Changed lines of the file:
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@@
   (junction (at 213.36 67.31) (diameter 0) (color 0 0 0 0)
-  )
-  (junction (at 182.88 128.27) (diameter 0) (color 0 0 0 0)
   )
   (junction (at 68.58 81.28) (diameter 0) (color 0 0 0 0)
@@
   (junction (at 66.04 81.28) (diameter 0) (color 0 0 0 0)
   )
-  (junction (at 187.96 130.81) (diameter 0) (color 0 0 0 0)
-  )
   (junction (at 78.74 81.28) (diameter 0) (color 0 0 0 0)
   )
+  (no_connect (at 175.26 135.89))
   (no_connect (at 224.79 110.49))
+  (no_connect (at 175.26 138.43))
   (no_connect (at 224.79 113.03))
   (no_connect (at 224.79 107.95))
@@
     (stroke (width 0) (type default))
   )
-  (wire (pts (xy 175.26 138.43) (xy 187.96 138.43))
-    (stroke (width 0) (type default))
-  )
   (wire (pts (xy 163.83 93.98) (xy 172.72 93.98))
     (stroke (width 0) (type default))
@@
   )
   (wire (pts (xy 44.45 81.28) (xy 44.45 77.47))
-    (stroke (width 0) (type default))
-  )
-  (wire (pts (xy 175.26 135.89) (xy 182.88 135.89))
     (stroke (width 0) (type default))
   )
@@
     (stroke (width 0) (type default))
   )
-  (wire (pts (xy 182.88 135.89) (xy 182.88 128.27))
-    (stroke (width 0) (type default))
-  )
   (wire (pts (xy 66.04 97.79) (xy 66.04 100.33))
     (stroke (width 0) (type default))
@@
     (stroke (width 0) (type default))
   )
-  (wire (pts (xy 187.96 130.81) (xy 187.96 138.43))
-    (stroke (width 0) (type default))
-  )

Commit message: Editting bulk editor feilds.
Parts:
- J1: AssemblyType (none) -> HAND; Cost (none) -> 3.33; Distributor 1 (none) -> Amazon; Distributor 1 PN (none) -> Amazon; MPN (none) -> https://www.amazon.com/dp/B089D5NLW1; Manufacturer (none) -> DFROBOT
- J601: AssemblyType (none) -> HAND; MPN (none) -> PZ150V-02P; Manufacturer (none) -> XFCN
- LS?: Cost (none) -> 1; Distributor 1 (none) -> Amazon; Distributor 1 PN (none) -> https://www.amazon.com/dp/B0DCTL83H6; MPN (none) -> ZGW-1; Manufacturer (none) -> YFUSET
Changed lines of the file:
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@@
+      (effects (font (size 1.27 1.27)) hide)
+    )
+    (property "MPN 2" "" (at 58.42 81.28 0)
+      (effects (font (size 1.27 1.27)) hide)
+    )
+    (property "Manufacturer 2" "" (at 58.42 81.28 0)
       (effects (font (size 1.27 1.27)) hide)
     )
@@
       (effects (font (size 1.27 1.27)) hide)
     )
+    (property "MPN 2" "" (at 66.04 93.98 0)
+      (effects (font (size 1.27 1.27)) hide)
+    )
+    (property "Manufacturer 2" "" (at 66.04 93.98 0)
+      (effects (font (size 1.27 1.27)) hide)
+    )
     (pin "1")
     (pin "2")
@@
       (effects (font (size 1.524 1.524)) (justify left) hide)
     )
-    (property "MPN" " " (at 190.5 125.73 0)
+    (property "MPN" "PZ150V-02P" (at 190.5 125.73 0)
       (effects (font (size 1.524 1.524)) (justify left) hide)
     )
@@
       (effects (font (size 1.524 1.524)) (justify left) hide)
     )
-    (property "Manufacturer" "" (at 205.74 125.73 0)
+    (property "Manufacturer" "XFCN" (at 205.74 125.73 0)
       (effects (font (size 1.524 1.524)) (justify left) hide)
     )
@@
       (effects (font (size 1.27 1.27)) hide)
     )
-    (property "AssemblyType" "" (at 177.8 130.81 0)
+    (property "AssemblyType" "HAND" (at 177.8 130.81 0)
       (effects (font (size 1.27 1.27)) hide)
     )
@@
       (effects (font (size 1.27 1.27)) hide)
     )
+    (property "MPN 2" "" (at 177.8 130.81 0)
+      (effects (font (size 1.27 1.27)) hide)
+    )
+    (property "Manufacturer 2" "" (at 177.8 130.81 0)
+      (effects (font (size 1.27 1.27)) hide)
+    )
     (pin "1")
     (pin "2")
@@
     )
     (property "Cost" "0.0015" (at 171.45 105.41 0)
+      (effects (font (size 1.27 1.27)) hide)
+    )
+    (property "MPN 2" "" (at 171.45 105.41 0)
+      (effects (font (size 1.27 1.27)) hide)
+    )
+    (property "Manufacturer 2" "" (at 171.45 105.41 0)
       (effects (font (size 1.27 1.27)) hide)
     )
@@
     )
     (property "Cost" "0.0015" (at 205.74 67.31 0)
+      (effects (font (size 1.27 1.27)) hide)
+    )
+    (property "MPN 2" "" (at 205.74 67.31 0)
+      (effects (font (size 1.27 1.27)) hide)
+    )
+    (property "Manufacturer 2" "" (at 205.74 67.31 0)
       (effects (font (size 1.27 1.27)) hide)
     )
@@
       (effects (font (size 1.27 1.27)) hide)
     )
+    (property "Cost" "1" (at 170.18 138.43 0)
+      (effects (font (size 1.27 1.27)) hide)
+    )
+    (property "Description" "8 Ohm 2W Speaker 8ohm Round 28mm Loud Speakers Compatible with Small Loudspeaker Audio MP3 MP4 Player Speaker (with Terminal)" (at 170.18 138.43 0)
+      (effects (font (size 1.27 1.27)) hide)
+    )
+    (property "Distributor 1" "Amazon" (at 170.18 138.43 0)
+      (effects (font (size 1.27 1.27)) hide)
+    )
+    (property "Distributor 1 PN" "https://www.amazon.com/dp/B0DCTL83H6" (at 170.18 138.43 0)
+      (effects (font (size 1.27 1.27)) hide)
+    )
+    (property "MPN" "ZGW-1" (at 170.18 138.43 0)
+      (effects (font (size 1.27 1.27)) hide)
+    )
+    (property "Manufacturer" "	YFUSET" (at 170.18 138.43 0)
+      (effects (font (size 1.27 1.27)) hide)
+    )
+    (property "MPN 2" "" (at 170.18 138.43 0)
+      (effects (font (size 1.27 1.27)) hide)
+    )
+    (property "Manufacturer 2" "" (at 170.18 138.43 0)
+      (effects (font (size 1.27 1.27)) hide)
+    )
     (pin "1")
     (pin "2")
@@
     )
     (property "Cost" "0.0015" (at 167.64 113.03 0)
+      (effects (font (size 1.27 1.27)) hide)
+    )
+    (property "MPN 2" "" (at 167.64 113.03 0)
+      (effects (font (size 1.27 1.27)) hide)
+    )
+    (property "Manufacturer 2" "" (at 167.64 113.03 0)
       (effects (font (size 1.27 1.27)) hide)
     )
@@
       (effects (font (size 1.27 1.27)) hide)
     )
+    (property "MPN 2" "" (at 92.71 83.82 0)
+      (effects (font (size 1.27 1.27)) hide)
+    )
+    (property "Manufacturer 2" "" (at 92.71 83.82 0)
+      (effects (font (size 1.27 1.27)) hide)
+    )
     (pin "1")
     (pin "2")
@@
       (effects (font (size 1.27 1.27)) hide)
     )
+    (property "MPN 2" "" (at 212.09 76.2 0)
+      (effects (font (size 1.27 1.27)) hide)
+    )
+    (property "Manufacturer 2" "" (at 212.09 76.2 0)
+      (effects (font (size 1.27 1.27)) hide)
+    )
     (pin "1")
     (pin "2")
@@
       (effects (font (size 1.27 1.27)) hide)
     )
+    (property "MPN 2" "" (at 198.12 76.2 0)
+      (effects (font (size 1.27 1.27)) hide)
+    )
+    (property "Manufacturer 2" "" (at 198.12 76.2 0)
+      (effects (font (size 1.27 1.27)) hide)
+    )
     (pin "1")
     (pin "2")
@@
       (effects (font (size 1.27 1.27)) hide)
     )
+    (property "MPN 2" "" (at 83.82 100.33 0)
+      (effects (font (size 1.27 1.27)) hide)
+    )
+    (property "Manufacturer 2" "" (at 83.82 100.33 0)
+      (effects (font (size 1.27 1.27)) hide)
+    )
     (pin "1")
     (pin "2")
@@
     )
     (property "Cost" "0.0015" (at 176.53 93.98 0)
+      (effects (font (size 1.27 1.27)) hide)
+    )
+    (property "MPN 2" "" (at 176.53 93.98 0)
+      (effects (font (size 1.27 1.27)) hide)
+    )
+    (property "Manufacturer 2" "" (at 176.53 93.98 0)
       (effects (font (size 1.27 1.27)) hide)
     )
@@
       (effects (font (size 1.27 1.27)) hide)
     )
+    (property "AssemblyType" "HAND" (at 199.39 113.03 0)
+      (effects (font (size 1.27 1.27)) hide)
+    )
+    (property "Cost" "3.33" (at 199.39 113.03 0)
+      (effects (font (size 1.27 1.27)) hide)
+    )
+    (property "Description" "Mini MP3 Player" (at 199.39 113.03 0)
+      (effects (font (size 1.27 1.27)) hide)
+    )
+    (property "Distributor 1" "Amazon" (at 199.39 113.03 0)
+      (effects (font (size 1.27 1.27)) hide)
+    )
+    (property "Distributor 1 PN" "Amazon" (at 199.39 113.03 0)
+      (effects (font (size 1.27 1.27)) hide)
+    )
+    (property "MPN" "https://www.amazon.com/dp/B089D5NLW1" (at 199.39 113.03 0)
+      (effects (font (size 1.27 1.27)) hide)
+    )
+    (property "MPN 2" "" (at 199.39 113.03 0)
+      (effects (font (size 1.27 1.27)) hide)
+    )
+    (property "Manufacturer" "DFROBOT" (at 199.39 113.03 0)
+      (effects (font (size 1.27 1.27)) hide)
+    )
+    (property "Manufacturer 2" "" (at 199.39 113.03 0)
+      (effects (font (size 1.27 1.27)) hide)
+    )

Commit message: Initial commit for the BOM list. And added an SD card schematic symbol.
Parts:
- added SD601: Micro_SD_Card_16GB_DFPLAYER, symbol GPAD_SCH_LIB:Micro_SD_Card_16GB_DFPLAYER
- LS?: AssemblyType (none) -> HAND
Other:
- note added: "MP3 file are added on this card for DFplayer"
Changed lines of the file:
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@@
     (effects (font (size 1.27 1.27)) (justify right bottom))
+  )
+  (text "MP3 file are added on this card for DFplayer" (at 73.66 162.56 0)
+    (effects (font (size 2.54 2.54)) (justify left bottom))
   )
   (label "5VDFP" (at 217.17 68.58 0) (fields_autoplaced)
@@
     )
     (property "Manufacturer 2" "" (at 170.18 138.43 0)
+      (effects (font (size 1.27 1.27)) hide)
+    )
+    (property "AssemblyType" "HAND" (at 170.18 138.43 0)
       (effects (font (size 1.27 1.27)) hide)
     )
@@
         )
       )
+    )
+  )
+  (symbol (lib_id "GPAD_SCH_LIB:Micro_SD_Card_16GB_DFPLAYER") (at 83.82 177.8 0) (unit 1)
+    (in_bom yes) (on_board no) (dnp no) (fields_autoplaced)
+    (property "Reference" "SD601" (at 105.41 175.895 0)
+      (effects (font (size 1.27 1.27)) (justify left))
+    )
+    (property "Value" "Micro_SD_Card_16GB_DFPLAYER" (at 105.41 178.435 0)
+      (effects (font (size 1.27 1.27)) (justify left))
+    )
+    (property "Footprint" "" (at 113.03 170.18 0)
+      (effects (font (size 1.27 1.27)) hide)
+    )
+    (property "Datasheet" "" (at 90.17 177.8 0)
+      (effects (font (size 1.27 1.27)) hide)
+    )
+    (property "AssemblyType" "HAND" (at 83.82 177.8 0)
+      (effects (font (size 1.27 1.27)) hide)
+    )
+    (property "Cost" "7.11" (at 83.82 177.8 0)
+      (effects (font (size 1.27 1.27)) hide)
+    )
+    (property "Description" "SanDisk Flash 16 GB SDHC Flash Memory Card SDSDB-016G " (at 83.82 177.8 0)
+      (effects (font (size 1.27 1.27)) hide)
+    )
+    (property "Distributor 1" "Amazon" (at 83.82 177.8 0)
+      (effects (font (size 1.27 1.27)) hide)
+    )
+    (property "Distributor 1 PN" "https://www.amazon.com/SanDisk-Flash-Memory-SDSDB-016G-Change/dp/B001W1BSM0" (at 83.82 177.8 0)
+      (effects (font (size 1.27 1.27)) hide)
+    )
+    (property "MPN" "SDSDB-016G-E11" (at 83.82 177.8 0)
+      (effects (font (size 1.27 1.27)) hide)
+    )
+    (property "Manufacturer" "	SanDisk" (at 83.82 177.8 0)
+      (effects (font (size 1.27 1.27)) hide)
+    )
+    (instances
+      (project "PCBa_KRAKE"
+        (path "/412a327d-1ee3-473e-bc00-1545004b7edf/00000000-0000-0000-0000-000062dd8e5f"
+          (reference "SD601") (unit 1)
+        )
+      )

Commit message: AlarmAudio.kicad_sch, replaced the J601 part by a Molex part and updated the footprint.
Parts:
- J601: value 1X2P 1.27 mm Header -> 1X2P 1.25 mm Header; footprint Connector_PinHeader_1.27mm:PinHeader_1x02_P1.27mm_Vertical -> Connector_Molex:Molex_PicoBlade_53047-0210_1x02_P1.25mm_Vertical; Distributor 1 PN C7496728 -> C114130; MPN PZ150V-02P -> 530470210; Manufacturer XFCN -> MOLEX
Changed lines of the file:
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@@
       (effects (font (size 1.27 1.27)) (justify right))
     )
-    (property "Value" "1X2P 1.27 mm Header" (at 181.61 124.46 90)
+    (property "Value" "1X2P 1.25 mm Header" (at 181.61 124.46 90)
       (effects (font (size 1.27 1.27)) (justify right))
     )
-    (property "Footprint" "Connector_PinHeader_1.27mm:PinHeader_1x02_P1.27mm_Vertical" (at 182.88 125.73 0)
+    (property "Footprint" "Connector_Molex:Molex_PicoBlade_53047-0210_1x02_P1.25mm_Vertical" (at 182.88 125.73 0)
       (effects (font (size 1.524 1.524)) (justify left) hide)
     )
@@
       (effects (font (size 1.524 1.524)) (justify left) hide)
     )
-    (property "MPN" "PZ150V-02P" (at 190.5 125.73 0)
+    (property "MPN" "530470210" (at 190.5 125.73 0)
       (effects (font (size 1.524 1.524)) (justify left) hide)
     )
@@
       (effects (font (size 1.524 1.524)) (justify left) hide)
     )
-    (property "Description" "Direct Insert 2P 1.5mm Single Row 1x2P Plugin,P=1.5mm Pin Headers ROHS" (at 203.2 125.73 0)
+    (property "Description" "1.25mm 1x2P 2 2P 3.2mm 4.25mm 4.2mm PA Phosphor Bronze PicoBlade(MX 1.25) " (at 203.2 125.73 0)
       (effects (font (size 1.524 1.524)) (justify left) hide)
     )
-    (property "Manufacturer" "XFCN" (at 205.74 125.73 0)
+    (property "Manufacturer" "MOLEX" (at 205.74 125.73 0)
       (effects (font (size 1.524 1.524)) (justify left) hide)
     )
@@
       (effects (font (size 1.27 1.27)) hide)
     )
-    (property "Distributor 1 PN" "C7496728" (at 177.8 130.81 0)
+    (property "Distributor 1 PN" "C114130" (at 177.8 130.81 0)
       (effects (font (size 1.27 1.27)) hide)
     )
