File: PCBa_KRAKE/USB_UART.kicad_sch (KiCad schematic)
At the start: 19 parts, among them J501 USB_B_Micro_Local, Q998 MMBT2222ALT1G, Q999 MMBT2222ALT1G, U501 CH340T

Commit message: Added 5V to 3v3 level shifters to SPI bus.Added but not wired a USBc connector.
Parts:
- added J?: USB_C_Receptacle_USB2.0, symbol Connector:USB_C_Receptacle_USB2.0
Connections:
- new net: J?.A1 (GND), J?.A12 (GND), J?.B1 (GND), J?.B12 (GND)
- new net: J?.A4 (VBUS), J?.A9 (VBUS), J?.B4 (VBUS), J?.B9 (VBUS)
Changed lines of the file:
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@@
+    )
+  )
+  (symbol (lib_id "Connector:USB_C_Receptacle_USB2.0") (at 53.34 96.52 0) (unit 1)
+    (in_bom yes) (on_board yes) (dnp no) (fields_autoplaced)
+    (property "Reference" "J?" (at 53.34 75.565 0)
+      (effects (font (size 1.27 1.27)))
+    )
+    (property "Value" "USB_C_Receptacle_USB2.0" (at 53.34 78.105 0)
+      (effects (font (size 1.27 1.27)))
+    )
+    (property "Footprint" "" (at 57.15 96.52 0)
+      (effects (font (size 1.27 1.27)) hide)
+    )
+    (property "Datasheet" "https://www.usb.org/sites/default/files/documents/usb_type-c.zip" (at 57.15 96.52 0)
+      (effects (font (size 1.27 1.27)) hide)
+    )
+    (pin "A1")
+    (pin "A12")
+    (pin "A4")
+    (pin "A5")
+    (pin "A6")
+    (pin "A7")
+    (pin "A8")
+    (pin "A9")
+    (pin "B1")
+    (pin "B12")
+    (pin "B4")
+    (pin "B5")
+    (pin "B6")
+    (pin "B7")
+    (pin "B8")
+    (pin "B9")
+    (pin "S1")
+    (instances
+      (project "PCBa_KRAKE"
+        (path "/412a327d-1ee3-473e-bc00-1545004b7edf"
+          (reference "J?") (unit 1)
+        )
+        (path "/412a327d-1ee3-473e-bc00-1545004b7edf/00000000-0000-0000-0000-000062bc4e7e"
+          (reference "J?") (unit 1)
+        )
+      )
     )
   )

Commit message: Editted USB C schematic symbol. Replaced the USB B with the USB C.
Parts:
- removed J501: USB_B_Micro_Local, GeneralPurposeAlarmDevicePCB:USB_Micro-B_Amphenol_10118194_Horizontal, symbol GPAD_SCH_LIB:USB_B_Micro_Local
- removed J?: USB_C_Receptacle_USB2.0, symbol Connector:USB_C_Receptacle_USB2.0
- added J?: USB_C_Receptacle_USB2.0, symbol Connector:USB_C_Receptacle_USB2.0
- added J?: USB_C_Receptacle_USB2.0, symbol GPAD_SCH_LIB:USB_C_Receptacle_USB2.0_GPAD
- added R? (x2): 5K1, Resistor_SMD:R_0603_1608Metric_Pad0.98x0.95mm_HandSolder, symbol Device:R
Connections:
- net GND: now also J?.A1 (GND), J?.A12 (GND), J?.B1 (GND), J?.B12 (GND), J?.S1 (SHIELD), R?.1, R?.1
- net VBus: now also J?.A4 (VBUS), J?.A9 (VBUS), J?.B4 (VBUS), J?.B9 (VBUS)
- net at U501.7 (UD-): now also J?.A7 (D-), J?.B7 (D-)
- net at U501.6 (UD+): now also J?.A6 (D+), J?.B6 (D+)
- new net: J?.A1 (GND), J?.A12 (GND), J?.B1 (GND), J?.B12 (GND)
- new net: J?.A4 (VBUS), J?.A9 (VBUS), J?.B4 (VBUS), J?.B9 (VBUS)
- new net: J?.A5 (CC1), R?.2
- new net: J?.B5 (CC2), R?.2
- no-connect marks 1 -> 0
Other:
- moved on the sheet: R1, TP201

Commit message: Replaced USB B with USB C connector.
Parts:
- removed J?: USB_C_Receptacle_USB2.0, symbol Connector:USB_C_Receptacle_USB2.0
Changed lines of the file:
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@@
-    )
-  )
-  (symbol (lib_id "Connector:USB_C_Receptacle_USB2.0") (at 24.13 102.87 0) (unit 1)
-    (in_bom yes) (on_board yes) (dnp no) (fields_autoplaced)
-    (property "Reference" "J?" (at 24.13 80.01 0)
-      (effects (font (size 1.27 1.27)))
-    )
-    (property "Value" "USB_C_Receptacle_USB2.0" (at 24.13 82.55 0)
-      (effects (font (size 1.27 1.27)))
-    )
-    (property "Footprint" "" (at 27.94 102.87 0)
-      (effects (font (size 1.27 1.27)) hide)
-    )
-    (property "Datasheet" "https://www.usb.org/sites/default/files/documents/usb_type-c.zip" (at 27.94 102.87 0)
-      (effects (font (size 1.27 1.27)) hide)
-    )
-    (pin "A1")
-    (pin "A12")
-    (pin "A4")
-    (pin "A5")
-    (pin "A6")
-    (pin "A7")
-    (pin "A8")
-    (pin "A9")
-    (pin "B1")
-    (pin "B12")
-    (pin "B4")
-    (pin "B5")
-    (pin "B6")
-    (pin "B7")
-    (pin "B8")
-    (pin "B9")
-    (pin "S1")
-    (instances
-      (project "PCBa_KRAKE"
-        (path "/412a327d-1ee3-473e-bc00-1545004b7edf/00000000-0000-0000-0000-000062bc4e7e"
-          (reference "J?") (unit 1)
-        )
-      )
     )
   )

Commit message: Annotated the new parts.
Parts:
- gave numbers to parts that had none: 3
Changed lines of the file:
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@@
         )
         (path "/412a327d-1ee3-473e-bc00-1545004b7edf/00000000-0000-0000-0000-000062bc4e7e"
-          (reference "R?") (unit 1)
+          (reference "R216") (unit 1)
         )
       )
@@
         )
         (path "/412a327d-1ee3-473e-bc00-1545004b7edf/00000000-0000-0000-0000-000062bc4e7e"
-          (reference "R?") (unit 1)
+          (reference "R213") (unit 1)
         )
       )
@@
         )
         (path "/412a327d-1ee3-473e-bc00-1545004b7edf/00000000-0000-0000-0000-000062bc4e7e"
-          (reference "R?") (unit 1)
+          (reference "R214") (unit 1)
         )
       )
@@
   (symbol (lib_id "Device:R") (at 100.33 110.49 180) (unit 1)
     (in_bom yes) (on_board yes) (dnp no)
-    (property "Reference" "R?" (at 104.14 109.22 0)
+    (property "Reference" "R212" (at 104.14 109.22 0)
       (effects (font (size 1.27 1.27)))
     )
@@
       (project "PCBa_KRAKE"
         (path "/412a327d-1ee3-473e-bc00-1545004b7edf/00000000-0000-0000-0000-000062bc4e7e"
-          (reference "R?") (unit 1)
+          (reference "R212") (unit 1)
         )
       )
@@
   (symbol (lib_id "GPAD_SCH_LIB:USB_C_Receptacle_USB2.0_GPAD") (at 71.12 102.87 0) (unit 1)
     (in_bom yes) (on_board yes) (dnp no) (fields_autoplaced)
-    (property "Reference" "J?" (at 71.12 80.01 0)
+    (property "Reference" "J201" (at 71.12 80.01 0)
       (effects (font (size 1.27 1.27)))
     )
@@
       (project "PCBa_KRAKE"
         (path "/412a327d-1ee3-473e-bc00-1545004b7edf/00000000-0000-0000-0000-000062bc4e7e"
-          (reference "J?") (unit 1)
+          (reference "J201") (unit 1)
         )
       )
@@
         )
         (path "/412a327d-1ee3-473e-bc00-1545004b7edf/00000000-0000-0000-0000-000062bc4e7e"
-          (reference "Q?") (unit 1)
+          (reference "Q206") (unit 1)
         )
       )
@@
   (symbol (lib_id "Device:R") (at 92.71 113.03 180) (unit 1)
     (in_bom yes) (on_board yes) (dnp no)
-    (property "Reference" "R?" (at 96.52 111.76 0)
+    (property "Reference" "R211" (at 96.52 111.76 0)
       (effects (font (size 1.27 1.27)))
     )
@@
       (project "PCBa_KRAKE"
         (path "/412a327d-1ee3-473e-bc00-1545004b7edf/00000000-0000-0000-0000-000062bc4e7e"
-          (reference "R?") (unit 1)
+          (reference "R211") (unit 1)
         )
       )
@@
         )
         (path "/412a327d-1ee3-473e-bc00-1545004b7edf/00000000-0000-0000-0000-000062bc4e7e"
-          (reference "Q?") (unit 1)
+          (reference "Q207") (unit 1)
         )
       )
@@
         )
         (path "/412a327d-1ee3-473e-bc00-1545004b7edf/00000000-0000-0000-0000-000062bc4e7e"
-          (reference "R?") (unit 1)
-        )
-      )
+          (reference "R215") (unit 1)
+        )
+      )

Commit message: Adding footprints for USB type C.
Parts:
- removed Q998, Q999: MMBT2222ALT1G, symbol Simulation_SPICE:NPN
- added Q205 (x2): MMBT2222A-7-F, Package_TO_SOT_SMD:SOT-23, symbol GPAD_SCH_LIB:MMBT2222A-7-F
- J201: footprint (none) -> GeneralPurposeAlarmDevicePCB:USB_C_Receptacle_HRO_TYPE-C-31-M-12; Cost (none) -> 0.1529; Distributor 1 (none) -> JLCPCB; Distributor 1 PN (none) -> C165948
Connections:
- net GPIO0: now also Q205.2 (E)
- net nRESET: now also Q205.3 (C)
- net at R505.1, U501.15 (~{DTR}): now also Q205.3 (C)
- net at R505.2: now also Q205.1 (B) (x2)
- net at R505.1, U501.16 (~{RTS}): now also Q205.2 (E)
Changed lines of the file:
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@@
+    )
+  )
+  (symbol (lib_id "GPAD_SCH_LIB:MMBT2222A-7-F") (at 208.28 125.73 0) (unit 1)
+    (in_bom yes) (on_board yes) (dnp no)
+    (property "Reference" "Q205" (at 213.0552 124.3838 0)
+      (effects (font (size 1.524 1.524)) (justify left))
+    )
+    (property "Value" "MMBT2222A-7-F" (at 213.0552 127.0762 0)
+      (effects (font (size 1.524 1.524)) (justify left))
+    )
+    (property "Footprint" "Package_TO_SOT_SMD:SOT-23" (at 213.36 120.65 0)
+      (effects (font (size 1.524 1.524)) (justify left) hide)
+    )
+    (property "Datasheet" "https://www.diodes.com/assets/Datasheets/ds30041.pdf" (at 213.36 118.11 0)
+      (effects (font (size 1.524 1.524)) (justify left) hide)
+    )
+    (property "Digi-Key_PN" "MMBT2222A-FDICT-ND" (at 213.36 115.57 0)
+      (effects (font (size 1.524 1.524)) (justify left) hide)
+    )
+    (property "MPN" "MMBT2222A-7-F" (at 213.36 113.03 0)
+      (effects (font (size 1.524 1.524)) (justify left) hide)
+    )
+    (property "Category" "Discrete Semiconductor Products" (at 213.36 110.49 0)
+      (effects (font (size 1.524 1.524)) (justify left) hide)
+    )
+    (property "Family" "Transistors - Bipolar (BJT) - Single" (at 213.36 107.95 0)
+      (effects (font (size 1.524 1.524)) (justify left) hide)
+    )
+    (property "DK_Datasheet_Link" "https://www.diodes.com/assets/Datasheets/ds30041.pdf" (at 213.36 105.41 0)
+      (effects (font (size 1.524 1.524)) (justify left) hide)
+    )
+    (property "DK_Detail_Page" "/product-detail/en/diodes-incorporated/MMBT2222A-7-F/MMBT2222A-FDICT-ND/815723" (at 213.36 102.87 0)
+      (effects (font (size 1.524 1.524)) (justify left) hide)
+    )
+    (property "Description" "TRANS NPN 40V 0.6A SMD SOT23-3" (at 213.36 100.33 0)
+      (effects (font (size 1.524 1.524)) (justify left) hide)
+    )
+    (property "Manufacturer" "Diodes Incorporated" (at 213.36 97.79 0)
+      (effects (font (size 1.524 1.524)) (justify left) hide)
+    )
+    (property "Status" "Active" (at 213.36 95.25 0)
+      (effects (font (size 1.524 1.524)) (justify left) hide)
+    )
+    (property "AssemblyType" "SMT" (at 208.28 125.73 0)
+      (effects (font (size 1.27 1.27)) hide)
+    )
+    (property "Distributor 1" "JLCPCB" (at 208.28 125.73 0)
+      (effects (font (size 1.27 1.27)) hide)
+    )
+    (property "Distributor 1 PN" "C94515" (at 208.28 125.73 0)
+      (effects (font (size 1.27 1.27)) hide)
+    )
+    (property "Cost" "0.0475" (at 208.28 125.73 0)
+      (effects (font (size 1.27 1.27)) hide)
+    )
+    (pin "1")
+    (pin "2")
+    (pin "3")
+    (instances
+      (project "PCBa_KRAKE"
+        (path "/412a327d-1ee3-473e-bc00-1545004b7edf/00000000-0000-0000-0000-000062b3ac2f"
+          (reference "Q205") (unit 1)
+        )
+        (path "/412a327d-1ee3-473e-bc00-1545004b7edf/00000000-0000-0000-0000-000062bc4e7e"
+          (reference "Q206") (unit 1)
+        )
+      )
+    )
+  )
+  (symbol (lib_id "GPAD_SCH_LIB:MMBT2222A-7-F") (at 208.28 142.24 0) (unit 1)
+    (in_bom yes) (on_board yes) (dnp no)
+    (property "Reference" "Q205" (at 213.0552 140.8938 0)
+      (effects (font (size 1.524 1.524)) (justify left))
+    )
+    (property "Value" "MMBT2222A-7-F" (at 213.0552 143.5862 0)
+      (effects (font (size 1.524 1.524)) (justify left))
+    )
+    (property "Footprint" "Package_TO_SOT_SMD:SOT-23" (at 213.36 137.16 0)
+      (effects (font (size 1.524 1.524)) (justify left) hide)
+    )
+    (property "Datasheet" "https://www.diodes.com/assets/Datasheets/ds30041.pdf" (at 213.36 134.62 0)
+      (effects (font (size 1.524 1.524)) (justify left) hide)
+    )
+    (property "Digi-Key_PN" "MMBT2222A-FDICT-ND" (at 213.36 132.08 0)
+      (effects (font (size 1.524 1.524)) (justify left) hide)
+    )
+    (property "MPN" "MMBT2222A-7-F" (at 213.36 129.54 0)
+      (effects (font (size 1.524 1.524)) (justify left) hide)
+    )
+    (property "Category" "Discrete Semiconductor Products" (at 213.36 127 0)
+      (effects (font (size 1.524 1.524)) (justify left) hide)
+    )
+    (property "Family" "Transistors - Bipolar (BJT) - Single" (at 213.36 124.46 0)
+      (effects (font (size 1.524 1.524)) (justify left) hide)
+    )
+    (property "DK_Datasheet_Link" "https://www.diodes.com/assets/Datasheets/ds30041.pdf" (at 213.36 121.92 0)
+      (effects (font (size 1.524 1.524)) (justify left) hide)
+    )
+    (property "DK_Detail_Page" "/product-detail/en/diodes-incorporated/MMBT2222A-7-F/MMBT2222A-FDICT-ND/815723" (at 213.36 119.38 0)
+      (effects (font (size 1.524 1.524)) (justify left) hide)
+    )
+    (property "Description" "TRANS NPN 40V 0.6A SMD SOT23-3" (at 213.36 116.84 0)
+      (effects (font (size 1.524 1.524)) (justify left) hide)
+    )
+    (property "Manufacturer" "Diodes Incorporated" (at 213.36 114.3 0)
+      (effects (font (size 1.524 1.524)) (justify left) hide)
+    )
+    (property "Status" "Active" (at 213.36 111.76 0)
+      (effects (font (size 1.524 1.524)) (justify left) hide)
+    )
+    (property "AssemblyType" "SMT" (at 208.28 142.24 0)
+      (effects (font (size 1.27 1.27)) hide)
+    )
+    (property "Distributor 1" "JLCPCB" (at 208.28 142.24 0)
+      (effects (font (size 1.27 1.27)) hide)
+    )
+    (property "Distributor 1 PN" "C94515" (at 208.28 142.24 0)
+      (effects (font (size 1.27 1.27)) hide)
+    )
+    (property "Cost" "0.0475" (at 208.28 142.24 0)
+      (effects (font (size 1.27 1.27)) hide)
+    )
+    (pin "1")
+    (pin "2")
+    (pin "3")
+    (instances
+      (project "PCBa_KRAKE"
+        (path "/412a327d-1ee3-473e-bc00-1545004b7edf/00000000-0000-0000-0000-000062b3ac2f"
+          (reference "Q205") (unit 1)
+        )
+        (path "/412a327d-1ee3-473e-bc00-1545004b7edf/00000000-0000-0000-0000-000062bc4e7e"
+          (reference "Q207") (unit 1)
+        )
+      )
     )
   )
@@
       (effects (font (size 1.27 1.27)))
     )
-    (property "Footprint" "" (at 74.93 102.87 0)
+    (property "Footprint" "GeneralPurposeAlarmDevicePCB:USB_C_Receptacle_HRO_TYPE-C-31-M-12" (at 74.93 102.87 0)
       (effects (font (size 1.27 1.27)) hide)
     )
     (property "Datasheet" "https://www.usb.org/sites/default/files/documents/usb_type-c.zip" (at 74.93 102.87 0)
+      (effects (font (size 1.27 1.27)) hide)
+    )
+    (property "Distributor 1" "JLCPCB" (at 71.12 102.87 0)
+      (effects (font (size 1.27 1.27)) hide)
+    )
+    (property "Distributor 1 PN" "C165948" (at 71.12 102.87 0)
+      (effects (font (size 1.27 1.27)) hide)
+    )
+    (property "Cost" "0.1529" (at 71.12 102.87 0)
       (effects (font (size 1.27 1.27)) hide)
     )
@@
     )
   )
-  (symbol (lib_id "Simulation_SPICE:NPN") (at 208.28 125.73 0) (unit 1)
-    (in_bom yes) (on_board yes) (dnp no)
-    (property "Reference" "Q999" (at 212.09 127 0)
-      (effects (font (size 1.27 1.27)) (justify left))
-    )
-    (property "Value" "MMBT2222ALT1G" (at 212.09 124.46 0)
-      (effects (font (size 1.27 1.27)) (justify left))
-    )
-    (property "Footprint" "" (at 271.78 125.73 0)
-      (effects (font (size 1.27 1.27)) hide)
-    )
-    (property "Datasheet" "~" (at 271.78 125.73 0)
-      (effects (font (size 1.27 1.27)) hide)
-    )
-    (pin "1")
-    (pin "2")
-    (pin "3")
-    (instances
-      (project "PCBa_KRAKE"
-        (path "/412a327d-1ee3-473e-bc00-1545004b7edf"
-          (reference "Q999") (unit 1)
-        )
-        (path "/412a327d-1ee3-473e-bc00-1545004b7edf/00000000-0000-0000-0000-000062bc4e7e"
-          (reference "Q206") (unit 1)
-        )
-      )
-    )
-  )
   (symbol (lib_id "Device:R") (at 92.71 113.03 180) (unit 1)
     (in_bom yes) (on_board yes) (dnp no)
@@
         )
       )
-    )
-  )
-  (symbol (lib_id "Simulation_SPICE:NPN") (at 208.28 142.24 0) (mirror x) (unit 1)
-    (in_bom yes) (on_board yes) (dnp no)
-    (property "Reference" "Q998" (at 212.09 140.97 0)
-      (effects (font (size 1.27 1.27)) (justify left))
-    )
-    (property "Value" "MMBT2222ALT1G" (at 212.09 143.51 0)
-      (effects (font (size 1.27 1.27)) (justify left))
-    )
-    (property "Footprint" "" (at 271.78 142.24 0)
-      (effects (font (size 1.27 1.27)) hide)
-    )
-    (property "Datasheet" "~" (at 271.78 142.24 0)
-      (effects (font (size 1.27 1.27)) hide)
-    )
-    (pin "1")
-    (pin "2")
-    (pin "3")
-    (instances
-      (project "PCBa_KRAKE"
-        (path "/412a327d-1ee3-473e-bc00-1545004b7edf"
-          (reference "Q998") (unit 1)
-        )
-        (path "/412a327d-1ee3-473e-bc00-1545004b7edf/00000000-0000-0000-0000-000062bc4e7e"
-          (reference "Q207") (unit 1)
-        )
-      )

Commit message: ERC Okay, waved warnings on symbol issues.
Connections:
- no-connect marks 0 -> 11
Changed lines of the file:
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@@
   (junction (at 86.36 95.25) (diameter 0) (color 0 0 0 0)
   )
+  (junction (at 160.655 76.2) (diameter 0) (color 0 0 0 0)
+  )
   (junction (at 175.26 105.41) (diameter 0) (color 0 0 0 0)
   )
@@
   (junction (at 102.87 72.39) (diameter 0) (color 0 0 0 0)
   )
+  (no_connect (at 165.1 102.87))
+  (no_connect (at 165.1 97.79))
+  (no_connect (at 165.1 115.57))
+  (no_connect (at 144.78 102.87))
+  (no_connect (at 165.1 100.33))
+  (no_connect (at 144.78 107.95))
+  (no_connect (at 165.1 113.03))
+  (no_connect (at 86.36 115.57))
+  (no_connect (at 86.36 118.11))
+  (no_connect (at 144.78 90.17))
+  (no_connect (at 165.1 120.65))
   (wire (pts (xy 106.68 76.2) (xy 120.65 76.2))
     (stroke (width 0) (type default))
@@
     (stroke (width 0) (type default))
   )
+  (wire (pts (xy 160.655 74.295) (xy 160.655 76.2))
+    (stroke (width 0) (type default))
+  )
   (wire (pts (xy 165.1 87.63) (xy 168.91 87.63))
     (stroke (width 0) (type default))
@@
     (stroke (width 0) (type default))
   )
+  (wire (pts (xy 160.655 76.2) (xy 198.12 76.2))
+    (stroke (width 0) (type default))
+  )
   (wire (pts (xy 114.3 121.92) (xy 114.3 123.19))
     (stroke (width 0) (type default))
   )
-  (wire (pts (xy 154.94 76.2) (xy 198.12 76.2))
+  (wire (pts (xy 154.94 76.2) (xy 160.655 76.2))
     (stroke (width 0) (type default))
   )
@@
         )
       )
+    )
+  )
+  (symbol (lib_id "power:PWR_FLAG") (at 160.655 74.295 0) (unit 1)
+    (in_bom yes) (on_board yes) (dnp no)
+    (property "Reference" "#FLG0101" (at 160.655 72.39 0)
+      (effects (font (size 1.27 1.27)) hide)
+    )
+    (property "Value" "PWR_FLAG" (at 158.115 69.215 0)
+      (effects (font (size 1.27 1.27)))
+    )
+    (property "Footprint" "" (at 160.655 74.295 0)
+      (effects (font (size 1.27 1.27)) hide)
+    )
+    (property "Datasheet" "~" (at 160.655 74.295 0)
+      (effects (font (size 1.27 1.27)) hide)
+    )
+    (pin "1")
+    (instances
+      (project "PCBa_KRAKE"
+        (path "/412a327d-1ee3-473e-bc00-1545004b7edf"
+          (reference "#FLG0101") (unit 1)
+        )
+        (path "/412a327d-1ee3-473e-bc00-1545004b7edf/00000000-0000-0000-0000-000062bc4e7e"
+          (reference "#FLG0201") (unit 1)
+        )
+      )

Commit message: Fixing annotations.
Parts:
- renumbered J201 to J501
Changed lines of the file:
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@@
   (symbol (lib_id "GPAD_SCH_LIB:USB_C_Receptacle_USB2.0_GPAD") (at 71.12 102.87 0) (unit 1)
     (in_bom yes) (on_board yes) (dnp no) (fields_autoplaced)
-    (property "Reference" "J201" (at 71.12 80.01 0)
+    (property "Reference" "J501" (at 71.12 80.01 0)
       (effects (font (size 1.27 1.27)))
     )
@@
       (project "PCBa_KRAKE"
         (path "/412a327d-1ee3-473e-bc00-1545004b7edf/00000000-0000-0000-0000-000062bc4e7e"
-          (reference "J201") (unit 1)
+          (reference "J501") (unit 1)
         )
       )
