File: PCBa_KRAKE/USB_UART.kicad_sch (KiCad schematic)
At the start: 21 parts, among them J501 USB_C_Receptacle_USB2.0, Q205 MMBT2222A-7-F, U501 CH340T

Commit message: Filing and updating.
Other:
- note added: "Caution: the USB to UART does not work, U501 is missing a crystal and two capacitors Q207 emitter and collector are interchanged."
Changed lines of the file:
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@@
     (stroke (width 0) (type default))
   )
-  (image (at 243.84 180.34) (scale 0.75)
+  (image (at 251.46 173.99) (scale 0.75)
     (data
       iVBORw0KGgoAAAANSUhEUgAAASAAAAEgCAYAAAAUg66AAAAABHNCSVQICAgIfAhkiAAAAAlwSFlz
@@
     (effects (font (size 1.27 1.27)) (justify left bottom))
   )
+  (text "Caution: the USB to UART does not work,\nU501 is missing a crystal and two capacitors \nQ207 emitter and collector are interchanged. "
+    (at 58.42 57.15 0)
+    (effects (font (face "Arial") (size 5.08 5.08) (thickness 1.016) bold (color 255 24 53 1)) (justify left bottom))
+  )
   (hierarchical_label "nRESET" (shape passive) (at 214.63 118.11 0) (fields_autoplaced)

Commit message: USB_UART.kicad_sch, replaced CH340T with CH340B. New schematic symbol CH340B.
Parts:
- removed U501: CH340T, GeneralPurposeAlarmDevicePCB:SSOP-20_5.3x7.2mm_P0.65mm_CH340T, symbol GPAD_SCH_LIB:CH340T
- added TP204: nRST, TestPoint:TestPoint_Loop_D2.54mm_Drill1.5mm_Beaded, symbol Connector:TestPoint
- added U501: CH340B, Package_SO:SOIC-16_3.9x9.9mm_P1.27mm, symbol GPAD_SCH_LIB:CH340B
Connections:
- net GND: now also U501.1 (GND)
- net at R502.2: now also U501.2 (TXD)
- net at R503.2: now also U501.3 (RXD)
- net at C503.1, R1.1, TP202.1: now also U501.4 (V3)
- net at C501.1, C502.1, R1.1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: now also U501.16 (VCC)
- net at R501.1: now also U501.15 (TNOW)
- net at R504.2, TP203.1: now also U501.9 (~{CTS})
- net at Q205.3 (C), R505.1: now also U501.13 (~{DTR})
- net at Q205.2 (E), R505.1: now also U501.14 (~{RTS})
- net at J501.A6 (D+), J501.B6 (D+): now also U501.5 (UD+)
- net at J501.A7 (D-), J501.B7 (D-): now also U501.6 (UD-)
- new net: TP204.1, U501.7 (RST#)
- no-connect marks 11 -> 5
Other:
- note added: "The DTR# pin of CH340 is used as a configuration input pin before the USB configuration is complete. An external 4.7KΩ pull-down resistor can be connected with this pin to generate default low level during USB enumeration, apply larger supply current to the USB bus via the configuration descriptor."

Commit message: USB_UART.kicad_sch, flipped the emmiter and the collctor for Q207. Added NC symbols for U303.
Connections:
- net GPIO0: now also Q205.3 (C); no longer Q205.2 (E)
- net at R505.1, U501.13 (~{DTR}): now also Q205.2 (E); no longer Q205.3 (C)
Changed lines of the file:
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@@
     )
   )
-  (symbol (lib_id "GPAD_SCH_LIB:MMBT2222A-7-F") (at 208.28 142.24 0) (unit 1)
+  (symbol (lib_id "GPAD_SCH_LIB:MMBT2222A-7-F") (at 208.28 142.24 0) (mirror x) (unit 1)
     (in_bom yes) (on_board yes) (dnp no)
-    (property "Reference" "Q205" (at 213.0552 140.8938 0)
+    (property "Reference" "Q205" (at 213.0552 143.5862 0)
       (effects (font (size 1.524 1.524)) (justify left))
     )
-    (property "Value" "MMBT2222A-7-F" (at 213.0552 143.5862 0)
+    (property "Value" "MMBT2222A-7-F" (at 213.0552 140.8938 0)
       (effects (font (size 1.524 1.524)) (justify left))
     )
-    (property "Footprint" "Package_TO_SOT_SMD:SOT-23" (at 213.36 137.16 0)
+    (property "Footprint" "Package_TO_SOT_SMD:SOT-23" (at 213.36 147.32 0)
       (effects (font (size 1.524 1.524)) (justify left) hide)
     )
-    (property "Datasheet" "https://www.diodes.com/assets/Datasheets/ds30041.pdf" (at 213.36 134.62 0)
+    (property "Datasheet" "https://www.diodes.com/assets/Datasheets/ds30041.pdf" (at 213.36 149.86 0)
       (effects (font (size 1.524 1.524)) (justify left) hide)
     )
-    (property "Digi-Key_PN" "MMBT2222A-FDICT-ND" (at 213.36 132.08 0)
+    (property "Digi-Key_PN" "MMBT2222A-FDICT-ND" (at 213.36 152.4 0)
       (effects (font (size 1.524 1.524)) (justify left) hide)
     )
-    (property "MPN" "MMBT2222A-7-F" (at 213.36 129.54 0)
+    (property "MPN" "MMBT2222A-7-F" (at 213.36 154.94 0)
       (effects (font (size 1.524 1.524)) (justify left) hide)
     )
-    (property "Category" "Discrete Semiconductor Products" (at 213.36 127 0)
+    (property "Category" "Discrete Semiconductor Products" (at 213.36 157.48 0)
       (effects (font (size 1.524 1.524)) (justify left) hide)
     )
-    (property "Family" "Transistors - Bipolar (BJT) - Single" (at 213.36 124.46 0)
+    (property "Family" "Transistors - Bipolar (BJT) - Single" (at 213.36 160.02 0)
       (effects (font (size 1.524 1.524)) (justify left) hide)
     )
-    (property "DK_Datasheet_Link" "https://www.diodes.com/assets/Datasheets/ds30041.pdf" (at 213.36 121.92 0)
+    (property "DK_Datasheet_Link" "https://www.diodes.com/assets/Datasheets/ds30041.pdf" (at 213.36 162.56 0)
       (effects (font (size 1.524 1.524)) (justify left) hide)
     )
-    (property "DK_Detail_Page" "/product-detail/en/diodes-incorporated/MMBT2222A-7-F/MMBT2222A-FDICT-ND/815723" (at 213.36 119.38 0)
+    (property "DK_Detail_Page" "/product-detail/en/diodes-incorporated/MMBT2222A-7-F/MMBT2222A-FDICT-ND/815723" (at 213.36 165.1 0)
       (effects (font (size 1.524 1.524)) (justify left) hide)
     )
-    (property "Description" "TRANS NPN 40V 0.6A SMD SOT23-3" (at 213.36 116.84 0)
+    (property "Description" "TRANS NPN 40V 0.6A SMD SOT23-3" (at 213.36 167.64 0)
       (effects (font (size 1.524 1.524)) (justify left) hide)
     )
-    (property "Manufacturer" "Diodes Incorporated" (at 213.36 114.3 0)
+    (property "Manufacturer" "Diodes Incorporated" (at 213.36 170.18 0)
       (effects (font (size 1.524 1.524)) (justify left) hide)
     )
-    (property "Status" "Active" (at 213.36 111.76 0)
+    (property "Status" "Active" (at 213.36 172.72 0)
       (effects (font (size 1.524 1.524)) (justify left) hide)
     )

Commit message: USB_UART.kicad_sch, Added a discription for D501 functionality.
Parts:
- added R217: 4K7, Resistor_SMD:R_0603_1608Metric_Pad0.98x0.95mm_HandSolder, symbol Device:R
Connections:
- net GND: now also R217.1
- net at Q205.2 (E), R505.1, U501.13 (~{DTR}): now also R217.2
Other:
- note added: "D501 indicates when data is transmitted. The serial port sends ongoing status indication, high level is active."
- note added: "The DTR# pin of CH340 is used as a configuration input pin before the USB configuration is complete. An external 4.7KΩ pull-down resistor (R217) can be connected with this pin to generate default low level during USB enumeration, apply larger supply current to the USB bus via the configuration descriptor."
- note removed: "The DTR# pin of CH340 is used as a configuration input pin before the USB configuration is complete. An external 4.7KΩ pull-down resistor can be connected with this pin to generate default low level during USB enumeration, apply larger supply current to the USB bus via the configuration descriptor."
- moved on the sheet: R504, TP203

Commit message: Fixed the previous PWA_REV_2 file by added the changes of the USB UART. PCBa_krake is reverted to when no changes done to the schem.
Parts:
- removed R217: 4K7, Resistor_SMD:R_0603_1608Metric_Pad0.98x0.95mm_HandSolder, symbol Device:R
- removed TP204: nRST, TestPoint:TestPoint_Loop_D2.54mm_Drill1.5mm_Beaded, symbol Connector:TestPoint
- removed U501: CH340B, Package_SO:SOIC-16_3.9x9.9mm_P1.27mm, symbol GPAD_SCH_LIB:CH340B
- added U501: CH340T, GeneralPurposeAlarmDevicePCB:SSOP-20_5.3x7.2mm_P0.65mm_CH340T, symbol GPAD_SCH_LIB:CH340T
Connections:
- net GND: now also U501.8 (GND)
- net GPIO0: now also Q205.2 (E); no longer Q205.3 (C)
- net at R502.2: now also U501.3 (TXD)
- net at R503.2: now also U501.4 (RXD)
- net at C503.1, R1.1, TP202.1: now also U501.5 (V3)
- net at C501.1, C502.1, R1.1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: now also U501.19 (VCC)
- net at R501.1: now also U501.17 (TNOW)
- net at R504.2, TP203.1: now also U501.11 (~{CTS})
- net at R505.1: now also Q205.3 (C), U501.15 (~{DTR}); no longer Q205.2 (E)
- net at Q205.2 (E), R505.1: now also U501.16 (~{RTS})
- net at J501.A6 (D+), J501.B6 (D+): now also U501.6 (UD+)
- net at J501.A7 (D-), J501.B7 (D-): now also U501.7 (UD-)
- no-connect marks 5 -> 11
Other:
- note removed: "D501 indicates when data is transmitted. The serial port sends ongoing status indication, high level is active."
- note removed: "The DTR# pin of CH340 is used as a configuration input pin before the USB configuration is complete. An external 4.7KΩ pull-down resistor (R217) can be connected with this pin to generate default low level during USB enumeration, apply larger supply current to the USB bus via the configuration descriptor."
- moved on the sheet: R504, TP203
