File: PCBa_KRAKE/LCD And I2C Interface.kicad_sch (KiCad schematic)
At the start: 32 parts, among them Q301 BSS138, U301 PCF8574AT_3_518, U302 LCD_20x4_Character-GPAD_SCH_L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

Commit message: Adding the I2C level shifter circuit for LCD.Added test points for 5V I2C.
Parts:
- added Q? (x2): BSS138, Package_TO_SOT_SMD:SOT-23, symbol Transistor_FET:BSS138
- added R? (x4): 4K7, Resistor_SMD:R_0603_1608Metric_Pad0.98x0.95mm_HandSolder, symbol Device:R
- added R? (x2): DNI, Resistor_SMD:R_0603_1608Metric_Pad0.98x0.95mm_HandSolder, symbol Device:R
- added TP?: SDA, TestPoint:TestPoint_Loop_D2.54mm_Drill1.5mm_Beaded, symbol Connector:TestPoint
- added TP?: SCL, TestPoint:TestPoint_Loop_D2.54mm_Drill1.5mm_Beaded, symbol Connector:TestPoint
Connections:
- net SCL: now also Q?.2 (S), R?.1, R?.2; no longer U301.14 (SCL)
- net SDA: now also Q?.2 (S), R?.1, R?.2; no longer U301.15 (SDA)
- net Vcc_LCD: now also R?.2, R?.2
- new net: Q?.3 (D), R?.1, R?.1, TP?.1, U301.14 (SCL)
- new net: Q?.3 (D), R?.1, R?.1, TP?.1, U301.15 (SDA)
- new net 3V3Raw: Q?.1 (G), Q?.1 (G), R?.2, R?.2

Commit message: Adding cooments in the title block, page setting of PCBa_Krake.
Other:
- title: GeneralPurposeAlarmDevicePCB -> KRAKE_PCB
Changed lines of the file:
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@@
   (paper "USLetter")
   (title_block
-    (title "GeneralPurposeAlarmDevicePCB")
-    (date "2023-04-25")
-    (rev "2.2")
+    (title "KRAKE_PCB")
+    (date "2024-11-23")
+    (rev "1")
     (company "PublicInvention")
     (comment 1 "GNU Affero General Public License v3.0")
-    (comment 2 "DrawnBy: (Forrest) Lee Erickson")
+    (comment 2 "DrawnBy: (Forrest) Lee Erickson, Nagham Kheir")
+    (comment 3 "https://github.com/PubInv/krake")
+    (comment 4 "Inherited from the GPAD")
   )
   (junction (at 173.99 80.01) (diameter 0) (color 0 0 0 0)

Commit message: Annotated the new parts.
Parts:
- gave numbers to parts that had none: 10
Changed lines of the file:
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@@
   (symbol (lib_id "Device:R") (at 78.74 63.5 180) (unit 1)
     (in_bom yes) (on_board yes) (dnp no)
-    (property "Reference" "R?" (at 81.28 59.69 0)
+    (property "Reference" "R410" (at 81.28 59.69 0)
       (effects (font (size 1.27 1.27)))
     )
@@
       (project "PCBa_KRAKE"
         (path "/412a327d-1ee3-473e-bc00-1545004b7edf/00000000-0000-0000-0000-000062b871ee"
-          (reference "R?") (unit 1)
+          (reference "R410") (unit 1)
         )
       )
@@
   (symbol (lib_id "Transistor_FET:BSS138") (at 53.34 72.39 270) (unit 1)
     (in_bom yes) (on_board yes) (dnp no)
-    (property "Reference" "Q?" (at 55.88 71.12 90)
+    (property "Reference" "Q401" (at 55.88 71.12 90)
       (effects (font (size 1.27 1.27)) (justify left))
     )
@@
       (project "PCBa_KRAKE"
         (path "/412a327d-1ee3-473e-bc00-1545004b7edf/00000000-0000-0000-0000-000062b871ee"
-          (reference "Q?") (unit 1)
+          (reference "Q401") (unit 1)
         )
       )
@@
   (symbol (lib_id "Device:R") (at 69.85 63.5 180) (unit 1)
     (in_bom yes) (on_board yes) (dnp no)
-    (property "Reference" "R?" (at 72.39 59.69 0)
+    (property "Reference" "R409" (at 72.39 59.69 0)
       (effects (font (size 1.27 1.27)))
     )
@@
       (project "PCBa_KRAKE"
         (path "/412a327d-1ee3-473e-bc00-1545004b7edf/00000000-0000-0000-0000-000062b871ee"
-          (reference "R?") (unit 1)
+          (reference "R409") (unit 1)
         )
       )
@@
   (symbol (lib_id "Device:R") (at 31.75 63.5 180) (unit 1)
     (in_bom yes) (on_board yes) (dnp no)
-    (property "Reference" "R?" (at 34.29 59.69 0)
+    (property "Reference" "R405" (at 34.29 59.69 0)
       (effects (font (size 1.27 1.27)))
     )
@@
       (project "PCBa_KRAKE"
         (path "/412a327d-1ee3-473e-bc00-1545004b7edf/00000000-0000-0000-0000-000062b871ee"
-          (reference "R?") (unit 1)
+          (reference "R405") (unit 1)
         )
       )
@@
   (symbol (lib_id "Device:R") (at 40.64 63.5 180) (unit 1)
     (in_bom yes) (on_board yes) (dnp no)
-    (property "Reference" "R?" (at 43.18 59.69 0)
+    (property "Reference" "R406" (at 43.18 59.69 0)
       (effects (font (size 1.27 1.27)))
     )
@@
       (project "PCBa_KRAKE"
         (path "/412a327d-1ee3-473e-bc00-1545004b7edf/00000000-0000-0000-0000-000062b871ee"
-          (reference "R?") (unit 1)
+          (reference "R406") (unit 1)
         )
       )
@@
   (symbol (lib_id "Device:R") (at 50.8 82.55 270) (unit 1)
     (in_bom no) (on_board yes) (dnp no)
-    (property "Reference" "R?" (at 46.99 80.01 90)
+    (property "Reference" "R407" (at 46.99 80.01 90)
       (effects (font (size 1.27 1.27)))
     )
@@
       (project "PCBa_KRAKE"
         (path "/412a327d-1ee3-473e-bc00-1545004b7edf/00000000-0000-0000-0000-000062b871ee"
-          (reference "R?") (unit 1)
+          (reference "R407") (unit 1)
         )
       )
@@
   (symbol (lib_id "Device:R") (at 62.23 93.98 270) (unit 1)
     (in_bom no) (on_board yes) (dnp no)
-    (property "Reference" "R?" (at 58.42 91.44 90)
+    (property "Reference" "R408" (at 58.42 91.44 90)
       (effects (font (size 1.27 1.27)))
     )
@@
       (project "PCBa_KRAKE"
         (path "/412a327d-1ee3-473e-bc00-1545004b7edf/00000000-0000-0000-0000-000062b871ee"
-          (reference "R?") (unit 1)
+          (reference "R408") (unit 1)
         )
       )
@@
   (symbol (lib_id "Transistor_FET:BSS138") (at 63.5 83.82 270) (unit 1)
     (in_bom yes) (on_board yes) (dnp no)
-    (property "Reference" "Q?" (at 66.04 82.55 90)
+    (property "Reference" "Q402" (at 66.04 82.55 90)
       (effects (font (size 1.27 1.27)) (justify left))
     )
@@
       (project "PCBa_KRAKE"
         (path "/412a327d-1ee3-473e-bc00-1545004b7edf/00000000-0000-0000-0000-000062b871ee"
-          (reference "Q?") (unit 1)
+          (reference "Q402") (unit 1)
         )
       )
@@
   (symbol (lib_id "Connector:TestPoint") (at 134.62 67.31 0) (unit 1)
     (in_bom yes) (on_board yes) (dnp no)
-    (property "Reference" "TP?" (at 130.81 62.23 0)
+    (property "Reference" "TP404" (at 130.81 62.23 0)
       (effects (font (size 1.27 1.27)) (justify left))
     )
@@
       (project "PCBa_KRAKE"
         (path "/412a327d-1ee3-473e-bc00-1545004b7edf/00000000-0000-0000-0000-000062b871ee"
-          (reference "TP?") (unit 1)
+          (reference "TP404") (unit 1)
         )
       )
@@
   (symbol (lib_id "Connector:TestPoint") (at 129.54 71.12 0) (unit 1)
     (in_bom yes) (on_board yes) (dnp no)
-    (property "Reference" "TP?" (at 125.73 66.04 0)
+    (property "Reference" "TP403" (at 125.73 66.04 0)
       (effects (font (size 1.27 1.27)) (justify left))
     )
@@
       (project "PCBa_KRAKE"
         (path "/412a327d-1ee3-473e-bc00-1545004b7edf/00000000-0000-0000-0000-000062b871ee"
-          (reference "TP?") (unit 1)
-        )
-      )
+          (reference "TP403") (unit 1)
+        )
+      )

Commit message: Cleared all DRC issues and Warnings.
Parts:
- added TP102: Vcontrast, TestPoint:TestPoint_Loop_D2.54mm_Drill1.5mm_Beaded, symbol Connector:TestPoint
Connections:
- net at R306.1, R308.2, RV301.2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: now also TP102.1
Changed lines of the file:
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@@
   (junction (at 125.73 85.09) (diameter 0) (color 0 0 0 0)
   )
+  (junction (at 214.63 62.23) (diameter 0) (color 0 0 0 0)
+  )
   (junction (at 97.79 52.07) (diameter 0) (color 0 0 0 0)
   )
@@
     (stroke (width 0) (type default))
   )
+  (wire (pts (xy 214.63 62.23) (xy 220.98 62.23))
+    (stroke (width 0) (type default))
+  )
   (wire (pts (xy 20.32 86.36) (xy 31.75 86.36))
     (stroke (width 0) (type default))
@@
     (stroke (width 0) (type default))
   )
-  (wire (pts (xy 198.12 62.23) (xy 220.98 62.23))
+  (wire (pts (xy 198.12 62.23) (xy 214.63 62.23))
     (stroke (width 0) (type default))
   )
@@
   )
   (wire (pts (xy 88.9 59.69) (xy 88.9 52.07))
+    (stroke (width 0) (type default))
+  )
+  (wire (pts (xy 214.63 60.96) (xy 214.63 62.23))
     (stroke (width 0) (type default))
   )
@@
       (effects (font (size 1.27 1.27)) hide)
     )
-    (property "Value" "GND" (at 216.027 53.9242 0)
+    (property "Value" "GND" (at 219.71 50.8 0)
       (effects (font (size 1.27 1.27)))
     )
@@
     )
   )
+  (symbol (lib_id "Connector:TestPoint") (at 214.63 60.96 0) (unit 1)
+    (in_bom yes) (on_board yes) (dnp no)
+    (property "Reference" "TP102" (at 210.82 54.61 0)
+      (effects (font (size 1.27 1.27)) (justify left))
+    )
+    (property "Value" "Vcontrast" (at 210.82 55.88 0)
+      (effects (font (size 1.27 1.27)) (justify left))
+    )
+    (property "Footprint" "TestPoint:TestPoint_Loop_D2.54mm_Drill1.5mm_Beaded" (at 219.71 60.96 0)
+      (effects (font (size 1.27 1.27)) hide)
+    )
+    (property "Datasheet" "~" (at 219.71 60.96 0)
+      (effects (font (size 1.27 1.27)) hide)
+    )
+    (property "AssemblyType" "HAND" (at 214.63 60.96 0)
+      (effects (font (size 1.27 1.27)) hide)
+    )
+    (pin "1")
+    (instances
+      (project "PCBa_KRAKE"
+        (path "/412a327d-1ee3-473e-bc00-1545004b7edf"
+          (reference "TP102") (unit 1)
+        )
+        (path "/412a327d-1ee3-473e-bc00-1545004b7edf/00000000-0000-0000-0000-000062b871ee"
+          (reference "TP405") (unit 1)
+        )
+      )
+    )
+  )
   (symbol (lib_id "power:GND") (at 199.39 76.2 0) (unit 1)
     (in_bom yes) (on_board yes) (dnp no)
@@
   (symbol (lib_id "Connector:TestPoint") (at 134.62 67.31 0) (unit 1)
     (in_bom yes) (on_board yes) (dnp no)
-    (property "Reference" "TP404" (at 130.81 62.23 0)
-      (effects (font (size 1.27 1.27)) (justify left))
-    )
-    (property "Value" "SDA" (at 130.81 66.04 0)
+    (property "Reference" "TP404" (at 134.62 60.96 0)
+      (effects (font (size 1.27 1.27)) (justify left))
+    )
+    (property "Value" "SDA" (at 135.89 63.5 0)
       (effects (font (size 1.27 1.27)) (justify left))
     )
@@
   (symbol (lib_id "Connector:TestPoint") (at 129.54 71.12 0) (unit 1)
     (in_bom yes) (on_board yes) (dnp no)
-    (property "Reference" "TP403" (at 125.73 66.04 0)
-      (effects (font (size 1.27 1.27)) (justify left))
-    )
-    (property "Value" "SCL" (at 125.73 69.85 0)
-      (effects (font (size 1.27 1.27)) (justify left))
-    )
+    (property "Reference" "TP403" (at 124.46 64.77 0)
+      (effects (font (size 1.27 1.27)) (justify left))
+    )
+    (property "Value" "SCL" (at 124.46 67.31 0)
+      (effects (font (size 1.27 1.27)) (justify left))
+    )

Commit message: Found missing part numbers. ESP32.
Parts:
- TP102, TP401: Distributor 1 (none) -> JLCPCB; Distributor 1 PN (none) -> C5277086
- TP402, TP403, TP404: Distributor 1 (none) -> JLCPCB; Distributor 1 PN (none) -> C5199804
Changed lines of the file:
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@@
+      (effects (font (size 1.27 1.27)) hide)
+    )
+    (property "Distributor 1" "JLCPCB" (at 139.7 106.68 0)
+      (effects (font (size 1.27 1.27)) hide)
+    )
+    (property "Description" "Test Points/Test Rings ROHS yellow" (at 139.7 106.68 0)
+      (effects (font (size 1.27 1.27)) hide)
+    )
+    (property "Distributor 1 PN" "C5199804" (at 139.7 106.68 0)
       (effects (font (size 1.27 1.27)) hide)
     )
@@
       (effects (font (size 1.27 1.27)) hide)
     )
+    (property "Distributor 1" "JLCPCB" (at 214.63 60.96 0)
+      (effects (font (size 1.27 1.27)) hide)
+    )
+    (property "Description" "Test Points/Test Rings ROHS red" (at 214.63 60.96 0)
+      (effects (font (size 1.27 1.27)) hide)
+    )
+    (property "Distributor 1 PN" "C5277086" (at 214.63 60.96 0)
+      (effects (font (size 1.27 1.27)) hide)
+    )
     (pin "1")
     (instances
@@
       (effects (font (size 1.27 1.27)) hide)
     )
+    (property "Distributor 1" "JLCPCB" (at 134.62 67.31 0)
+      (effects (font (size 1.27 1.27)) hide)
+    )
+    (property "Description" "Test Points/Test Rings ROHS yellow" (at 134.62 67.31 0)
+      (effects (font (size 1.27 1.27)) hide)
+    )
+    (property "Distributor 1 PN" "C5199804" (at 134.62 67.31 0)
+      (effects (font (size 1.27 1.27)) hide)
+    )
     (pin "1")
     (instances
@@
     )
     (property "AssemblyType" "HAND" (at 223.52 35.56 0)
+      (effects (font (size 1.27 1.27)) hide)
+    )
+    (property "Description" "Test Points/Test Rings ROHS red" (at 223.52 35.56 0)
+      (effects (font (size 1.27 1.27)) hide)
+    )
+    (property "Distributor 1" "JLCPCB" (at 223.52 35.56 0)
+      (effects (font (size 1.27 1.27)) hide)
+    )
+    (property "Distributor 1 PN" "C5277086" (at 223.52 35.56 0)
       (effects (font (size 1.27 1.27)) hide)
     )
@@
       (effects (font (size 1.27 1.27)) hide)
     )
+    (property "Distributor 1" "JLCPCB" (at 129.54 71.12 0)
+      (effects (font (size 1.27 1.27)) hide)
+    )
+    (property "Description" "Test Points/Test Rings ROHS yellow" (at 129.54 71.12 0)
+      (effects (font (size 1.27 1.27)) hide)
+    )
+    (property "Distributor 1 PN" "C5199804" (at 129.54 71.12 0)
+      (effects (font (size 1.27 1.27)) hide)
+    )
