File: PCBa_KRAKE/LCD And I2C Interface.kicad_sch (KiCad schematic)
At the start: 43 parts, among them Q301 BSS138, Q401 BSS138, Q402 BSS138, U301 PCF8574AT_3_518, U302 LCD_20x4_Character-GPAD_SCH_L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

Commit message: Adding component information. Deleted a redundant LED from the schematic.
Parts:
- TP102, TP401: Cost (none) -> 0.0717; MPN (none) -> RH-5000; Manufacturer (none) -> ronghe
- TP402, TP403, TP404: Cost (none) -> 0.0800; MPN (none) -> RH-5004; Manufacturer (none) -> ronghe
Changed lines of the file:
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@@
+      (effects (font (size 1.27 1.27)) hide)
+    )
+    (property "Description" "47uF 16V 33mA@120Hz ±20% SMD,D5xL5.4mm Aluminum Electrolytic Capacitors - SMD ROHS" (at 215.9 44.45 0)
       (effects (font (size 1.27 1.27)) hide)
     )
@@
     )
     (property "Distributor 1 PN" "C5199804" (at 139.7 106.68 0)
+      (effects (font (size 1.27 1.27)) hide)
+    )
+    (property "MPN" "RH-5004" (at 139.7 106.68 0)
+      (effects (font (size 1.27 1.27)) hide)
+    )
+    (property "Manufacturer" "ronghe" (at 139.7 106.68 0)
+      (effects (font (size 1.27 1.27)) hide)
+    )
+    (property "Cost" "0.0800" (at 139.7 106.68 0)
       (effects (font (size 1.27 1.27)) hide)
     )
@@
       (effects (font (size 1.27 1.27)) hide)
     )
+    (property "MPN" "RH-5000" (at 214.63 60.96 0)
+      (effects (font (size 1.27 1.27)) hide)
+    )
+    (property "Manufacturer" "ronghe" (at 214.63 60.96 0)
+      (effects (font (size 1.27 1.27)) hide)
+    )
+    (property "Cost" "0.0717" (at 214.63 60.96 0)
+      (effects (font (size 1.27 1.27)) hide)
+    )
     (pin "1")
     (instances
@@
       (effects (font (size 1.27 1.27)) hide)
     )
+    (property "MPN" "RH-5004" (at 134.62 67.31 0)
+      (effects (font (size 1.27 1.27)) hide)
+    )
+    (property "Manufacturer" "ronghe" (at 134.62 67.31 0)
+      (effects (font (size 1.27 1.27)) hide)
+    )
+    (property "Cost" "0.0800" (at 134.62 67.31 0)
+      (effects (font (size 1.27 1.27)) hide)
+    )
     (pin "1")
     (instances
@@
     )
     (property "Distributor 1 PN" "C5277086" (at 223.52 35.56 0)
+      (effects (font (size 1.27 1.27)) hide)
+    )
+    (property "MPN" "RH-5000" (at 223.52 35.56 0)
+      (effects (font (size 1.27 1.27)) hide)
+    )
+    (property "Manufacturer" "ronghe" (at 223.52 35.56 0)
+      (effects (font (size 1.27 1.27)) hide)
+    )
+    (property "Cost" "0.0717" (at 223.52 35.56 0)
       (effects (font (size 1.27 1.27)) hide)
     )
@@
       (effects (font (size 1.27 1.27)) hide)
     )
+    (property "MPN" "RH-5004" (at 129.54 71.12 0)
+      (effects (font (size 1.27 1.27)) hide)
+    )
+    (property "Manufacturer" "ronghe" (at 129.54 71.12 0)
+      (effects (font (size 1.27 1.27)) hide)
+    )
+    (property "Cost" "0.0800" (at 129.54 71.12 0)
+      (effects (font (size 1.27 1.27)) hide)
+    )

Commit message: Editting missing feilds in the builk editor, And added a pin header for the LCD.
Parts:
- added U303: LCD20X4, Connector_PinHeader_2.54mm:PinHeader_1x16_P2.54mm_Vertical, symbol Connector_Generic:Conn_01x16
Changed lines of the file:
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@@
+    )
+  )
+  (symbol (lib_id "Connector_Generic:Conn_01x16") (at 252.73 81.28 0) (unit 1)
+    (in_bom yes) (on_board yes) (dnp no) (fields_autoplaced)
+    (property "Reference" "U303" (at 255.27 81.28 0)
+      (effects (font (size 1.27 1.27)) (justify left))
+    )
+    (property "Value" "LCD20X4" (at 255.27 83.82 0)
+      (effects (font (size 1.27 1.27)) (justify left))
+    )
+    (property "Footprint" "Connector_PinHeader_2.54mm:PinHeader_1x16_P2.54mm_Vertical" (at 252.73 81.28 0)
+      (effects (font (size 1.27 1.27)) hide)
+    )
+    (property "Datasheet" "~" (at 252.73 81.28 0)
+      (effects (font (size 1.27 1.27)) hide)
+    )
+    (property "Distributor 1" "JLCPCB" (at 252.73 81.28 0)
+      (effects (font (size 1.27 1.27)) hide)
+    )
+    (property "Distributor 1 PN" "C22465876" (at 252.73 81.28 0)
+      (effects (font (size 1.27 1.27)) hide)
+    )
+    (property "MPN" "PZ254V-11-16P" (at 252.73 81.28 0)
+      (effects (font (size 1.27 1.27)) hide)
+    )
+    (property "Manufacturer" "XFCN" (at 252.73 81.28 0)
+      (effects (font (size 1.27 1.27)) hide)
+    )
+    (property "Cost" "0.09" (at 252.73 81.28 0)
+      (effects (font (size 1.27 1.27)) hide)
+    )
+    (property "Description" "Plugin,P=2.54mm Pin Headers ROHS" (at 252.73 81.28 0)
+      (effects (font (size 1.27 1.27)) hide)
+    )
+    (pin "1")
+    (pin "10")
+    (pin "11")
+    (pin "12")
+    (pin "13")
+    (pin "14")
+    (pin "15")
+    (pin "16")
+    (pin "2")
+    (pin "3")
+    (pin "4")
+    (pin "5")
+    (pin "6")
+    (pin "7")
+    (pin "8")
+    (pin "9")
+    (instances
+      (project "PCBa_KRAKE"
+        (path "/412a327d-1ee3-473e-bc00-1545004b7edf/00000000-0000-0000-0000-000062b871ee"
+          (reference "U303") (unit 1)
+        )
+      )
     )
   )

Commit message: Editting bulk editor feilds.
Parts:
- MF403, MF406, MF409, MF412: AssemblyType (none) -> HAND
- U301: Manufacturer (none) -> NXP Semicon
- U302: MPN (none) -> https://www.ebay.com/itm/403534100457; Manufacturer (none) -> NA
- U303: value LCD20X4 -> Conn_01x16; AssemblyType (none) -> HAND

Commit message: Updating schematic title block and MPN in the bulk editor.
Parts:
- MF401, MF404, MF407, MF410: MPN (none) -> 90272A108; Manufacturer (none) -> McMaster-Carr
- MF402, MF405, MF408, MF411: MPN (none) -> 94639A702; Manufacturer (none) -> McMaster-Carr
- MF403, MF406, MF409, MF412: MPN (none) -> 4694; Manufacturer (none) -> Keystone Electronics
Changed lines of the file:
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@@
 (kicad_sch (version 20230121) (generator eeschema)
-  (paper "USLetter")
+  (paper "A4")
   (title_block
     (title "KRAKE_PCB")
     (date "2024-11-23")
-    (rev "1")
+    (rev "1.0")
     (company "PublicInvention")
     (comment 1 "GNU Affero General Public License v3.0")
@@
       (effects (font (size 1.27 1.27)) hide)
     )
+    (property "MPN" "4694" (at 18.415 154.305 0)
+      (effects (font (size 1.27 1.27)) hide)
+    )
+    (property "Manufacturer" "Keystone Electronics" (at 18.415 154.305 0)
+      (effects (font (size 1.27 1.27)) hide)
+    )
+    (property "Description" "#4-40 Hex Nut 0.187\" (4.75mm) 3/16\" Steel" (at 18.415 154.305 0)
+      (effects (font (size 1.27 1.27)) hide)
+    )
     (instances
       (project "PCBa_KRAKE"
@@
       (effects (font (size 1.27 1.27)) hide)
     )
+    (property "MPN" "94639A702" (at 90.17 139.7 0)
+      (effects (font (size 1.27 1.27)) hide)
+    )
+    (property "Manufacturer" "McMaster-Carr" (at 90.17 139.7 0)
+      (effects (font (size 1.27 1.27)) hide)
+    )
     (instances
       (project "PCBa_KRAKE"
@@
       (effects (font (size 1.27 1.27)) hide)
     )
+    (property "MPN" "4694" (at 125.73 154.94 0)
+      (effects (font (size 1.27 1.27)) hide)
+    )
+    (property "Manufacturer" "Keystone Electronics" (at 125.73 154.94 0)
+      (effects (font (size 1.27 1.27)) hide)
+    )
+    (property "Description" "#4-40 Hex Nut 0.187\" (4.75mm) 3/16\" Steel" (at 125.73 154.94 0)
+      (effects (font (size 1.27 1.27)) hide)
+    )
     (instances
       (project "PCBa_KRAKE"
@@
       (effects (font (size 1.27 1.27)) hide)
     )
+    (property "MPN" "4694" (at 90.17 155.575 0)
+      (effects (font (size 1.27 1.27)) hide)
+    )
+    (property "Manufacturer" "Keystone Electronics" (at 90.17 155.575 0)
+      (effects (font (size 1.27 1.27)) hide)
+    )
+    (property "Description" "#4-40 Hex Nut 0.187\" (4.75mm) 3/16\" Steel" (at 90.17 155.575 0)
+      (effects (font (size 1.27 1.27)) hide)
+    )
     (instances
       (project "PCBa_KRAKE"
@@
       (effects (font (size 1.27 1.27)) hide)
     )
+    (property "MPN" "90272A108" (at 55.88 123.19 0)
+      (effects (font (size 1.27 1.27)) hide)
+    )
+    (property "Manufacturer" "McMaster-Carr" (at 55.88 123.19 0)
+      (effects (font (size 1.27 1.27)) hide)
+    )
     (instances
       (project "PCBa_KRAKE"
@@
       (effects (font (size 1.27 1.27)) hide)
     )
+    (property "MPN" "94639A702" (at 19.05 138.43 0)
+      (effects (font (size 1.27 1.27)) hide)
+    )
+    (property "Manufacturer" "McMaster-Carr" (at 19.05 138.43 0)
+      (effects (font (size 1.27 1.27)) hide)
+    )
     (instances
       (project "PCBa_KRAKE"
@@
       (effects (font (size 1.27 1.27)) hide)
     )
+    (property "MPN" "90272A108" (at 90.17 123.19 0)
+      (effects (font (size 1.27 1.27)) hide)
+    )
+    (property "Manufacturer" "McMaster-Carr" (at 90.17 123.19 0)
+      (effects (font (size 1.27 1.27)) hide)
+    )
     (instances
       (project "PCBa_KRAKE"
@@
       (effects (font (size 1.27 1.27)) hide)
     )
+    (property "MPN" "90272A108" (at 124.46 123.19 0)
+      (effects (font (size 1.27 1.27)) hide)
+    )
+    (property "Manufacturer" "McMaster-Carr" (at 124.46 123.19 0)
+      (effects (font (size 1.27 1.27)) hide)
+    )
     (instances
       (project "PCBa_KRAKE"
@@
       (effects (font (size 1.27 1.27)) hide)
     )
+    (property "MPN" "94639A702" (at 55.88 138.43 0)
+      (effects (font (size 1.27 1.27)) hide)
+    )
+    (property "Manufacturer" "McMaster-Carr" (at 55.88 138.43 0)
+      (effects (font (size 1.27 1.27)) hide)
+    )
     (instances
       (project "PCBa_KRAKE"
@@
       (effects (font (size 1.27 1.27)) hide)
     )
+    (property "MPN" "4694" (at 55.245 154.305 0)
+      (effects (font (size 1.27 1.27)) hide)
+    )
+    (property "Manufacturer" "Keystone Electronics" (at 55.245 154.305 0)
+      (effects (font (size 1.27 1.27)) hide)
+    )
+    (property "Description" "#4-40 Hex Nut 0.187\" (4.75mm) 3/16\" Steel" (at 55.245 154.305 0)
+      (effects (font (size 1.27 1.27)) hide)
+    )
     (instances
       (project "PCBa_KRAKE"
@@
       (effects (font (size 1.27 1.27)) hide)
     )
+    (property "MPN" "94639A702" (at 125.73 138.43 0)
+      (effects (font (size 1.27 1.27)) hide)
+    )
+    (property "Manufacturer" "McMaster-Carr" (at 125.73 138.43 0)
+      (effects (font (size 1.27 1.27)) hide)
+    )
     (instances
       (project "PCBa_KRAKE"
@@
       (effects (font (size 1.27 1.27)) hide)
     )
+    (property "MPN" "90272A108" (at 19.05 123.19 0)
+      (effects (font (size 1.27 1.27)) hide)
+    )
+    (property "Manufacturer" "McMaster-Carr" (at 19.05 123.19 0)
+      (effects (font (size 1.27 1.27)) hide)
+    )

Commit message: Generating and plotting gerbers and BOM and CPL.
Parts:
- MF401, MF402, MF404, MF405, MF407, MF408, MF410, MF411: footprint NA -> (none)
Changed lines of the file:
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@@
       (effects (font (size 1.27 1.27)) (justify left))
     )
-    (property "Footprint" "NA" (at 90.17 139.7 0)
+    (property "Footprint" "" (at 90.17 139.7 0)
       (effects (font (size 1.27 1.27)) hide)
     )
@@
       (effects (font (size 1.27 1.27)) (justify left))
     )
-    (property "Footprint" "NA" (at 55.88 123.19 0)
+    (property "Footprint" "" (at 55.88 123.19 0)
       (effects (font (size 1.27 1.27)) hide)
     )
@@
       (effects (font (size 1.27 1.27)) (justify left))
     )
-    (property "Footprint" "NA" (at 19.05 138.43 0)
+    (property "Footprint" "" (at 19.05 138.43 0)
       (effects (font (size 1.27 1.27)) hide)
     )
@@
       (effects (font (size 1.27 1.27)) (justify left))
     )
-    (property "Footprint" "NA" (at 90.17 123.19 0)
+    (property "Footprint" "" (at 90.17 123.19 0)
       (effects (font (size 1.27 1.27)) hide)
     )
@@
       (effects (font (size 1.27 1.27)) (justify left))
     )
-    (property "Footprint" "NA" (at 124.46 123.19 0)
+    (property "Footprint" "" (at 124.46 123.19 0)
       (effects (font (size 1.27 1.27)) hide)
     )
@@
       (effects (font (size 1.27 1.27)) (justify left))
     )
-    (property "Footprint" "NA" (at 55.88 138.43 0)
+    (property "Footprint" "" (at 55.88 138.43 0)
       (effects (font (size 1.27 1.27)) hide)
     )
@@
       (effects (font (size 1.27 1.27)) (justify left))
     )
-    (property "Footprint" "NA" (at 125.73 138.43 0)
+    (property "Footprint" "" (at 125.73 138.43 0)
       (effects (font (size 1.27 1.27)) hide)
     )
@@
       (effects (font (size 1.27 1.27)) (justify left))
     )
-    (property "Footprint" "NA" (at 19.05 123.19 0)
-      (effects (font (size 1.27 1.27)) hide)
-    )
+    (property "Footprint" "" (at 19.05 123.19 0)
+      (effects (font (size 1.27 1.27)) hide)
+    )

Commit message: USB_UART.kicad_sch, flipped the emmiter and the collctor for Q207. Added NC symbols for U303.
Connections:
- no-connect marks 0 -> 16
Changed lines of the file:
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@@
   (junction (at 167.64 52.07) (diameter 0) (color 0 0 0 0)
   )
+  (no_connect (at 247.65 81.28))
+  (no_connect (at 247.65 86.36))
+  (no_connect (at 247.65 91.44))
+  (no_connect (at 247.65 68.58))
+  (no_connect (at 247.65 76.2))
+  (no_connect (at 247.65 73.66))
+  (no_connect (at 247.65 63.5))
+  (no_connect (at 247.65 93.98))
+  (no_connect (at 247.65 88.9))
+  (no_connect (at 247.65 99.06))
+  (no_connect (at 247.65 101.6))
+  (no_connect (at 247.65 66.04))
+  (no_connect (at 247.65 71.12))
+  (no_connect (at 247.65 78.74))
+  (no_connect (at 247.65 96.52))
+  (no_connect (at 247.65 83.82))
   (wire (pts (xy 175.26 77.47) (xy 173.99 77.47))
     (stroke (width 0) (type default))
@@
   )
   (symbol (lib_id "Connector_Generic:Conn_01x16") (at 252.73 81.28 0) (unit 1)
-    (in_bom yes) (on_board yes) (dnp no) (fields_autoplaced)
+    (in_bom yes) (on_board no) (dnp no) (fields_autoplaced)
     (property "Reference" "U303" (at 255.27 81.28 0)
       (effects (font (size 1.27 1.27)) (justify left))

Commit message: Fixed the previous PWA_REV_2 file by added the changes of the USB UART. PCBa_krake is reverted to when no changes done to the schem.
Connections:
- no-connect marks 16 -> 0
Changed lines of the file:
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@@
   (junction (at 167.64 52.07) (diameter 0) (color 0 0 0 0)
   )
-  (no_connect (at 247.65 81.28))
-  (no_connect (at 247.65 86.36))
-  (no_connect (at 247.65 91.44))
-  (no_connect (at 247.65 68.58))
-  (no_connect (at 247.65 76.2))
-  (no_connect (at 247.65 73.66))
-  (no_connect (at 247.65 63.5))
-  (no_connect (at 247.65 93.98))
-  (no_connect (at 247.65 88.9))
-  (no_connect (at 247.65 99.06))
-  (no_connect (at 247.65 101.6))
-  (no_connect (at 247.65 66.04))
-  (no_connect (at 247.65 71.12))
-  (no_connect (at 247.65 78.74))
-  (no_connect (at 247.65 96.52))
-  (no_connect (at 247.65 83.82))
   (wire (pts (xy 175.26 77.47) (xy 173.99 77.47))
     (stroke (width 0) (type default))
@@
   )
   (symbol (lib_id "Connector_Generic:Conn_01x16") (at 252.73 81.28 0) (unit 1)
-    (in_bom yes) (on_board no) (dnp no) (fields_autoplaced)
+    (in_bom yes) (on_board yes) (dnp no) (fields_autoplaced)
     (property "Reference" "U303" (at 255.27 81.28 0)
       (effects (font (size 1.27 1.27)) (justify left))
