File: PCBa_KRAKE/RS232.kicad_sch (KiCad schematic)
At the start: 19 parts

Commit message: Editting bulk editor feilds.
Parts:
- J?: AssemblyType (none) -> SMT; Cost (none) -> 0.5; Distributor 1 (none) -> Amazon; Distributor 1 PN (none) -> Amazon; MPN (none) -> https://www.amazon.com/Pc-Accessories-Connectors-Connector-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; Manufacturer (none) -> Connectors Pro
- U?: AssemblyType (none) -> SMT; Cost (none) -> 1.6050; MPN (none) -> MAX3232ID; Manufacturer (none) -> Texas Instruments
Changed lines of the file:
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@@
+      (effects (font (size 1.27 1.27)) hide)
+    )
+    (property "MPN 2" "" (at 132.08 46.99 0)
+      (effects (font (size 1.27 1.27)) hide)
+    )
+    (property "Manufacturer 2" "" (at 132.08 46.99 0)
       (effects (font (size 1.27 1.27)) hide)
     )
@@
     )
     (property "Datasheet" " ~" (at 195.58 127 0)
+      (effects (font (size 1.27 1.27)) hide)
+    )
+    (property "MPN 2" "" (at 195.58 127 0)
+      (effects (font (size 1.27 1.27)) hide)
+    )
+    (property "Manufacturer 2" "" (at 195.58 127 0)
+      (effects (font (size 1.27 1.27)) hide)
+    )
+    (property "AssemblyType" "SMT" (at 195.58 127 0)
+      (effects (font (size 1.27 1.27)) hide)
+    )
+    (property "Cost" "0.5" (at 195.58 127 0)
+      (effects (font (size 1.27 1.27)) hide)
+    )
+    (property "Description" "DB9 Male and Female D-Sub Solder Type Connector" (at 195.58 127 0)
+      (effects (font (size 1.27 1.27)) hide)
+    )
+    (property "Distributor 1" "Amazon" (at 195.58 127 0)
+      (effects (font (size 1.27 1.27)) hide)
+    )
+    (property "Distributor 1 PN" "Amazon" (at 195.58 127 0)
+      (effects (font (size 1.27 1.27)) hide)
+    )
+    (property "MPN" "https://www.amazon.com/Pc-Accessories-Connectors-Connector-20-Pack/dp/B014IVD7L0/ref=sr_1_1" (at 195.58 127 0)
+      (effects (font (size 1.27 1.27)) hide)
+    )
+    (property "Manufacturer" "Connectors Pro" (at 195.58 127 0)
       (effects (font (size 1.27 1.27)) hide)
     )
@@
       (effects (font (size 1.27 1.27)) hide)
     )
+    (property "MPN 2" "" (at 104.14 106.68 0)
+      (effects (font (size 1.27 1.27)) hide)
+    )
+    (property "Manufacturer 2" "" (at 104.14 106.68 0)
+      (effects (font (size 1.27 1.27)) hide)
+    )
+    (property "AssemblyType" "SMT" (at 104.14 106.68 0)
+      (effects (font (size 1.27 1.27)) hide)
+    )
+    (property "Cost" "1.6050" (at 104.14 106.68 0)
+      (effects (font (size 1.27 1.27)) hide)
+    )
+    (property "Description" "250Kbps Transceiver 2/2 SOIC-16 RS232 ICs ROHS" (at 104.14 106.68 0)
+      (effects (font (size 1.27 1.27)) hide)
+    )
+    (property "MPN" "MAX3232ID" (at 104.14 106.68 0)
+      (effects (font (size 1.27 1.27)) hide)
+    )
+    (property "Manufacturer" "Texas Instruments" (at 104.14 106.68 0)
+      (effects (font (size 1.27 1.27)) hide)
+    )
     (pin "1")
     (pin "10")
@@
       (effects (font (size 1.27 1.27)) hide)
     )
+    (property "MPN 2" "" (at 165.1 132.08 0)
+      (effects (font (size 1.27 1.27)) hide)
+    )
+    (property "Manufacturer 2" "" (at 165.1 132.08 0)
+      (effects (font (size 1.27 1.27)) hide)
+    )
     (pin "1")
     (pin "2")
@@
       (effects (font (size 1.27 1.27)) hide)
     )
+    (property "MPN 2" "" (at 176.53 83.82 0)
+      (effects (font (size 1.27 1.27)) hide)
+    )
+    (property "Manufacturer 2" "" (at 176.53 83.82 0)
+      (effects (font (size 1.27 1.27)) hide)
+    )
     (pin "1")
     (pin "2")
@@
     )
     (property "Cost" "0.0015" (at 165.1 149.86 0)
+      (effects (font (size 1.27 1.27)) hide)
+    )
+    (property "MPN 2" "" (at 165.1 149.86 0)
+      (effects (font (size 1.27 1.27)) hide)
+    )
+    (property "Manufacturer 2" "" (at 165.1 149.86 0)
       (effects (font (size 1.27 1.27)) hide)
     )
@@
       (effects (font (size 1.27 1.27)) hide)
     )
+    (property "MPN 2" "" (at 190.5 83.82 0)
+      (effects (font (size 1.27 1.27)) hide)
+    )
+    (property "Manufacturer 2" "" (at 190.5 83.82 0)
+      (effects (font (size 1.27 1.27)) hide)
+    )
     (pin "1")
     (pin "2")
@@
     )
     (property "Cost" "0.0015" (at 138.43 46.99 0)
+      (effects (font (size 1.27 1.27)) hide)
+    )
+    (property "MPN 2" "" (at 138.43 46.99 0)
+      (effects (font (size 1.27 1.27)) hide)
+    )
+    (property "Manufacturer 2" "" (at 138.43 46.99 0)
       (effects (font (size 1.27 1.27)) hide)
     )
@@
       (effects (font (size 1.27 1.27)) hide)
     )
+    (property "MPN 2" "" (at 55.88 86.36 0)
+      (effects (font (size 1.27 1.27)) hide)
+    )
+    (property "Manufacturer 2" "" (at 55.88 86.36 0)
+      (effects (font (size 1.27 1.27)) hide)
+    )
     (pin "1")
     (pin "2")
@@
       (effects (font (size 1.27 1.27)) hide)
     )
+    (property "MPN 2" "" (at 55.88 101.6 0)
+      (effects (font (size 1.27 1.27)) hide)
+    )
+    (property "Manufacturer 2" "" (at 55.88 101.6 0)
+      (effects (font (size 1.27 1.27)) hide)
+    )
     (pin "1")
     (pin "2")
@@
     )
     (property "Cost" "0.0015" (at 143.51 46.99 0)
+      (effects (font (size 1.27 1.27)) hide)
+    )
+    (property "MPN 2" "" (at 143.51 46.99 0)
+      (effects (font (size 1.27 1.27)) hide)
+    )
+    (property "Manufacturer 2" "" (at 143.51 46.99 0)
       (effects (font (size 1.27 1.27)) hide)
     )
@@
       (effects (font (size 1.27 1.27)) hide)
     )
+    (property "MPN 2" "" (at 163.83 127 0)
+      (effects (font (size 1.27 1.27)) hide)
+    )
+    (property "Manufacturer 2" "" (at 163.83 127 0)
+      (effects (font (size 1.27 1.27)) hide)
+    )
     (pin "1")
     (pin "2")
@@
       (effects (font (size 1.27 1.27)) hide)
     )
+    (property "MPN 2" "" (at 182.88 74.93 0)
+      (effects (font (size 1.27 1.27)) hide)
+    )
+    (property "Manufacturer 2" "" (at 182.88 74.93 0)
+      (effects (font (size 1.27 1.27)) hide)
+    )
     (pin "1")
     (pin "2")
@@
     )
     (property "Cost" "0.0015" (at 165.1 142.24 0)
+      (effects (font (size 1.27 1.27)) hide)
+    )
+    (property "MPN 2" "" (at 165.1 142.24 0)
+      (effects (font (size 1.27 1.27)) hide)
+    )
+    (property "Manufacturer 2" "" (at 165.1 142.24 0)
       (effects (font (size 1.27 1.27)) hide)
     )
@@
       (effects (font (size 1.27 1.27)) hide)
     )
+    (property "MPN 2" "" (at 165.1 137.16 0)
+      (effects (font (size 1.27 1.27)) hide)
+    )
+    (property "Manufacturer 2" "" (at 165.1 137.16 0)
+      (effects (font (size 1.27 1.27)) hide)
+    )
     (pin "1")
     (pin "2")
@@
       (effects (font (size 1.27 1.27)) hide)
     )
+    (property "MPN 2" "" (at 80.01 120.65 0)
+      (effects (font (size 1.27 1.27)) hide)
+    )
+    (property "Manufacturer 2" "" (at 80.01 120.65 0)
+      (effects (font (size 1.27 1.27)) hide)
+    )
     (pin "1")
     (pin "2")
@@
     )
     (property "Cost" "0.0015" (at 127 46.99 0)
+      (effects (font (size 1.27 1.27)) hide)
+    )
+    (property "MPN 2" "" (at 127 46.99 0)
+      (effects (font (size 1.27 1.27)) hide)
+    )
+    (property "Manufacturer 2" "" (at 127 46.99 0)
       (effects (font (size 1.27 1.27)) hide)
     )
@@
       (effects (font (size 1.27 1.27)) hide)
     )
+    (property "MPN 2" "" (at 163.83 121.92 0)
+      (effects (font (size 1.27 1.27)) hide)
+    )
+    (property "Manufacturer 2" "" (at 163.83 121.92 0)
+      (effects (font (size 1.27 1.27)) hide)
+    )
     (pin "1")
     (pin "2")
@@
       (effects (font (size 1.27 1.27)) hide)
     )
+    (property "MPN 2" "" (at 80.01 76.2 0)
+      (effects (font (size 1.27 1.27)) hide)
+    )
+    (property "Manufacturer 2" "" (at 80.01 76.2 0)
+      (effects (font (size 1.27 1.27)) hide)
+    )

Commit message: Updating schematic title block and MPN in the bulk editor.
Parts:
- U?: Distributor 1 PN (none) -> C354119
Changed lines of the file:
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@@
     (title "KRAKE_PCB")
     (date "2024-11-23")
-    (rev "1")
+    (rev "1.0")
     (company "PublicInvention")
     (comment 1 "GNU Affero General Public License v3.0")
@@
       (effects (font (size 1.27 1.27)) hide)
     )
+    (property "Distributor 1 PN" "C354119" (at 104.14 106.68 0)
+      (effects (font (size 1.27 1.27)) hide)
+    )

Commit message: enclosure/U_Box_V105_Krake_RevB.scad, implementing changes to accomdate KRAKE.
Parts:
- J?: Distributor 1 Amazon -> DigiKey; Distributor 1 PN Amazon -> 609-5189-ND; MPN 2 (none) -> LD09S13A4GX00LF; Manufacturer 2 (none) -> Amphenol ICC (FCI)
Changed lines of the file:
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@@
       (effects (font (size 1.27 1.27)) hide)
     )
-    (property "MPN 2" "" (at 195.58 127 0)
+    (property "MPN 2" "LD09S13A4GX00LF" (at 195.58 127 0)
       (effects (font (size 1.27 1.27)) hide)
     )
-    (property "Manufacturer 2" "" (at 195.58 127 0)
+    (property "Manufacturer 2" "Amphenol ICC (FCI)" (at 195.58 127 0)
       (effects (font (size 1.27 1.27)) hide)
     )
@@
       (effects (font (size 1.27 1.27)) hide)
     )
-    (property "Distributor 1" "Amazon" (at 195.58 127 0)
+    (property "Distributor 1" "DigiKey" (at 195.58 127 0)
       (effects (font (size 1.27 1.27)) hide)
     )
-    (property "Distributor 1 PN" "Amazon" (at 195.58 127 0)
+    (property "Distributor 1 PN" "609-5189-ND" (at 195.58 127 0)
       (effects (font (size 1.27 1.27)) hide)
     )
