File: PCBa_KRAKE/AlarmLights5.kicad_sch (KiCad schematic)
At the start: 25 parts, among them Q201 MMBT2222A-7-F, Q202 MMBT2222A-7-F, Q203 MMBT2222A-7-F, Q204 MMBT2222A-7-F, Q205 MMBT2222A-7-F

Commit message: Adding cooments in the title block, page setting of PCBa_Krake.
Other:
- title: GeneralPurposeAlarmDevicePCB -> KRAKE_PCB
Changed lines of the file:
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@@
   (paper "USLetter")
   (title_block
-    (title "GeneralPurposeAlarmDevicePCB")
-    (date "2023-04-25")
-    (rev "2.2")
+    (title "KRAKE_PCB")
+    (date "2024-11-23")
+    (rev "1")
     (company "PublicInvention")
     (comment 1 "GNU Affero General Public License v3.0")
-    (comment 2 "DrawnBy: (Forrest) Lee Erickson")
+    (comment 2 "DrawnBy: (Forrest) Lee Erickson, Nagham Kheir")
+    (comment 3 "https://github.com/PubInv/krake")
+    (comment 4 "Inherited from the GPAD")
   )
   (junction (at 119.38 71.12) (diameter 0) (color 0 0 0 0)

Commit message: routing and connecting.
Other:
- note added: "currect setting resistor, Base"
- note added: "currect setting resistor, LED"
- note added: "current sink transistor"
Changed lines of the file:
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@@
     )
+  )
+  (text "currect setting \nresistor, Base" (at 77.47 95.25 0)
+    (effects (font (size 0.762 0.762)) (justify left bottom))
+  )
+  (text "currect setting \nresistor, LED" (at 90.17 80.01 0)
+    (effects (font (size 0.762 0.762)) (justify left bottom))
+  )
+  (text "current sink\ntransistor" (at 91.44 105.41 0)
+    (effects (font (size 0.762 0.762)) (justify left bottom))
   )
   (text "Alarm lights, 5 Levels" (at 128.27 69.85 0)
@@
   (symbol (lib_id "Device:R") (at 76.2 93.98 180) (unit 1)
     (in_bom yes) (on_board yes) (dnp no)
-    (property "Reference" "R201" (at 81.28 92.71 0)
+    (property "Reference" "R201" (at 78.74 88.9 0)
       (effects (font (size 1.27 1.27)))
     )
-    (property "Value" "4K7" (at 80.01 95.25 0)
+    (property "Value" "4K7" (at 80.01 91.44 0)
       (effects (font (size 1.27 1.27)))
     )
@@
   (symbol (lib_id "Device:R") (at 88.9 78.74 180) (unit 1)
     (in_bom yes) (on_board yes) (dnp no)
-    (property "Reference" "R202" (at 91.44 74.93 0)
+    (property "Reference" "R202" (at 91.44 73.66 0)
       (effects (font (size 1.27 1.27)))
     )
-    (property "Value" "330R" (at 92.71 80.01 0)
+    (property "Value" "330R" (at 92.71 76.2 0)
       (effects (font (size 1.27 1.27)))
     )

Commit message: Editting bulk editor feilds.
Parts:
- MF601, MF602, MF603, MF604, MF605: AssemblyType (none) -> HAND; Cost (none) -> NA; Distributor 1 (none) -> NA; Distributor 1 PN (none) -> NA; MPN (none) -> NA; Manufacturer (none) -> NA
