File: PCBa_KRAKE/Enclosure.kicad_sch (KiCad schematic)
At the start: 2 parts

Commit message: Editting bulk editor feilds.
Parts:
- MF102: footprint (none) -> NA; AssemblyType (none) -> HAND; MPN (none) -> NA; Manufacturer (none) -> NA
Changed lines of the file:
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@@
       (effects (font (size 1.27 1.27)) (justify left))
     )
-    (property "Footprint" "" (at 118.11 65.405 0)
+    (property "Footprint" "NA" (at 118.11 65.405 0)
       (effects (font (size 1.27 1.27)) hide)
     )
@@
     )
     (property "Distributor 2 PN" "" (at 118.11 65.405 0)
+      (effects (font (size 1.27 1.27)) hide)
+    )
+    (property "MPN 2" "" (at 118.11 65.405 0)
+      (effects (font (size 1.27 1.27)) hide)
+    )
+    (property "Manufacturer 2" "" (at 118.11 65.405 0)
+      (effects (font (size 1.27 1.27)) hide)
+    )
+    (property "AssemblyType" "HAND" (at 118.11 65.405 0)
+      (effects (font (size 1.27 1.27)) hide)
+    )
+    (property "Description" "NA" (at 118.11 65.405 0)
+      (effects (font (size 1.27 1.27)) hide)
+    )
+    (property "MPN" "NA" (at 118.11 65.405 0)
+      (effects (font (size 1.27 1.27)) hide)
+    )
+    (property "Manufacturer" "NA" (at 118.11 65.405 0)
       (effects (font (size 1.27 1.27)) hide)
     )
@@
       (effects (font (size 1.27 1.27)) hide)
     )
+    (property "MPN 2" "" (at 160.02 64.135 0)
+      (effects (font (size 1.27 1.27)) hide)
+    )
+    (property "Manufacturer 2" "" (at 160.02 64.135 0)
+      (effects (font (size 1.27 1.27)) hide)
+    )

Commit message: Updating schematic title block and MPN in the bulk editor.
Parts:
- MF101: value PCB_GPAD_VER2 -> PCB_KRAKE_VER1; footprint NA -> (none); Distributor 1 PN PCB_GPAD_V1 -> PCB_KRAKE_V1; MPN PCB_GPAD_V1 -> Gerbers2501181555.zip
- MF102: value ENCLOSURE_GPAD_VER1 -> ENCLOSURE_KRAKE_VER1; Distributor 1 PN ENCLOSURE_GPAD_VER1 -> ENCLOSURE_KRAKE_VER1
Other:
- company: (none) -> PublicInvention
- title: (none) -> KRAKE_PCB
Changed lines of the file:
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@@
 (kicad_sch (version 20230121) (generator eeschema)
   (paper "A4")
+  (title_block
+    (title "KRAKE_PCB")
+    (date "2024-11-23")
+    (rev "1.0")
+    (company "PublicInvention")
+    (comment 1 "GNU Affero General Public License v3.0")
+    (comment 2 "DrawnBy: (Forrest) Lee Erickson, Nagham Kheir")
+    (comment 3 "https://github.com/PubInv/krake")
+    (comment 4 "Inherited from the GPAD")
+  )
   (symbol (lib_id "GPAD_SCH_LIB:ENCLOSURE_GPAD_VER1") (at 118.11 65.405 0) (unit 1)
     (in_bom yes) (on_board no) (dnp no)
@@
       (effects (font (size 1.27 1.27)) (justify left))
     )
-    (property "Value" "ENCLOSURE_GPAD_VER1" (at 107.95 62.865 0)
+    (property "Value" "ENCLOSURE_KRAKE_VER1" (at 107.95 62.865 0)
       (effects (font (size 1.27 1.27)) (justify left))
     )
@@
       (effects (font (size 1.27 1.27)) hide)
     )
-    (property "Datasheet" "https://www.mcmaster.com/catalog/128/3306" (at 118.11 65.405 0)
+    (property "Datasheet" "" (at 118.11 65.405 0)
       (effects (font (size 1.27 1.27)) hide)
     )
@@
       (effects (font (size 1.27 1.27)) hide)
     )
-    (property "Distributor 1 PN" "ENCLOSURE_GPAD_VER1" (at 118.11 65.405 0)
+    (property "Distributor 1 PN" "ENCLOSURE_KRAKE_VER1" (at 118.11 65.405 0)
       (effects (font (size 1.27 1.27)) hide)
     )
@@
       (effects (font (size 1.27 1.27)) (justify left))
     )
-    (property "Value" "PCB_GPAD_VER2" (at 153.67 62.865 0)
+    (property "Value" "PCB_KRAKE_VER1" (at 153.67 62.865 0)
       (effects (font (size 1.27 1.27)) (justify left))
     )
-    (property "Footprint" "NA" (at 160.02 64.135 0)
+    (property "Footprint" "" (at 160.02 64.135 0)
       (effects (font (size 1.27 1.27)) hide)
     )
-    (property "Datasheet" "https://www.mcmaster.com/catalog/128/3306" (at 160.02 64.135 0)
+    (property "Datasheet" "Gerbers2501181555.zip" (at 160.02 64.135 0)
       (effects (font (size 1.27 1.27)) hide)
     )
@@
       (effects (font (size 1.27 1.27)) hide)
     )
-    (property "Distributor 1 PN" "PCB_GPAD_V1" (at 160.02 64.135 0)
+    (property "Distributor 1 PN" "PCB_KRAKE_V1" (at 160.02 64.135 0)
       (effects (font (size 1.27 1.27)) hide)
     )
@@
       (effects (font (size 1.27 1.27)) hide)
     )
-    (property "Description" "PCB for GPAD Version 1" (at 160.02 64.135 0)
+    (property "Description" "PCB for KRAKE Version 1" (at 160.02 64.135 0)
       (effects (font (size 1.27 1.27)) hide)
     )
-    (property "MPN" "PCB_GPAD_V1" (at 160.02 64.135 0)
+    (property "MPN" "Gerbers2501181555.zip" (at 160.02 64.135 0)
       (effects (font (size 1.27 1.27)) hide)
     )

Commit message: Generating and plotting gerbers and BOM and CPL.
Parts:
- MF102: footprint NA -> (none)
Changed lines of the file:
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@@
       (effects (font (size 1.27 1.27)) (justify left))
     )
-    (property "Footprint" "NA" (at 118.11 65.405 0)
+    (property "Footprint" "" (at 118.11 65.405 0)
       (effects (font (size 1.27 1.27)) hide)
     )
