File: PWA_REV2/PWA_REV2.kicad_sch (KiCad schematic)
At the start: 58 parts, among them J101 Barrel_Jack_Switch_SMT, J102 0.100_2Pin, J103 0.100_2Pin, J104 Conn_01x14 1mm, J106 Conn_01x14 1mm, J107 Conn_01x10 1mm, SW101 RotaryEncoder_Switch, T101 ToolingHole_Pad_1.152mm, T102 ToolingHole_Pad_1.152mm, T103 ToolingHole_Pad_1.152mm, U101 LM7805_TO220, U102 ESP32-WROOM-32E-N4, U103 AMS1117-3.3

Commit message: Fixed the previous PWA_REV_2 file by added the changes of the USB UART. PCBa_krake is reverted to when no changes done to the schem.
Other:
- title: Krake Rev2 -> KRAKE_PCB
- moved on the sheet: MF103

Commit message: PWA_REV2, changed TP101 to be Test Points/Test Rings 1.25 mm Green, RH-5116.
Parts:
- TP101: Cost 0.2018 -> 0.4; Distributor 1 PN C7589090 -> C5199806; MPN RH-5121 -> RH-5116
Changed lines of the file:
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@@
       (effects (font (size 1.27 1.27)) hide)
     )
-    (property "Datasheet" "~" (at 31.75 44.45 0)
+    (property "Datasheet" "https://lcsc.com/datasheet/lcsc_datasheet_2504101957_ronghe-RH-5116_C5199806.pdf" (at 31.75 44.45 0)
       (effects (font (size 1.27 1.27)) hide)
     )
@@
       (effects (font (size 1.27 1.27)) hide)
     )
-    (property "Description" "Test Points/Test Rings ROHS green" (at 26.67 44.45 0)
+    (property "Description" "Test Points/Test Rings 1.25 mm Green" (at 26.67 44.45 0)
       (effects (font (size 1.27 1.27)) hide)
     )
@@
       (effects (font (size 1.27 1.27)) hide)
     )
-    (property "Distributor 1 PN" "C7589090" (at 26.67 44.45 0)
+    (property "Distributor 1 PN" "C5199806" (at 26.67 44.45 0)
       (effects (font (size 1.27 1.27)) hide)
     )
-    (property "MPN" "RH-5121" (at 26.67 44.45 0)
+    (property "MPN" "RH-5116" (at 26.67 44.45 0)
       (effects (font (size 1.27 1.27)) hide)
     )
@@
       (effects (font (size 1.27 1.27)) hide)
     )
-    (property "Cost" "0.2018" (at 26.67 44.45 0)
+    (property "Cost" "0.4" (at 26.67 44.45 0)
       (effects (font (size 1.27 1.27)) hide)
     )

Commit message: PWA_REV2.kicad_sch, updated the footptint of the testpoint to 1mm hole and corrected description.
Parts:
- TP101, TP102, TP103: footprint TestPoint:TestPoint_Loop_D2.54mm_Drill1.5mm_Beaded -> TestPoint:TestPoint_Loop_D1.80mm_Drill1.0mm_Beaded
Changed lines of the file:
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@@
       (effects (font (size 1.27 1.27)) (justify left))
     )
-    (property "Footprint" "TestPoint:TestPoint_Loop_D2.54mm_Drill1.5mm_Beaded" (at 66.04 24.13 0)
+    (property "Footprint" "TestPoint:TestPoint_Loop_D1.80mm_Drill1.0mm_Beaded" (at 66.04 24.13 0)
       (effects (font (size 1.27 1.27)) hide)
     )
@@
       (effects (font (size 1.27 1.27)) hide)
     )
-    (property "Description" "Test Points/Test Rings ROHS red" (at 60.96 24.13 0)
+    (property "Description" "Test Points/Test Rings 1.25 mm Red" (at 60.96 24.13 0)
       (effects (font (size 1.27 1.27)) hide)
     )
@@
       (effects (font (size 1.27 1.27)) (justify left))
     )
-    (property "Footprint" "TestPoint:TestPoint_Loop_D2.54mm_Drill1.5mm_Beaded" (at 31.75 44.45 0)
+    (property "Footprint" "TestPoint:TestPoint_Loop_D1.80mm_Drill1.0mm_Beaded" (at 31.75 44.45 0)
       (effects (font (size 1.27 1.27)) hide)
     )
@@
       (effects (font (size 1.27 1.27)) (justify left))
     )
-    (property "Footprint" "TestPoint:TestPoint_Loop_D2.54mm_Drill1.5mm_Beaded" (at 127 27.94 0)
+    (property "Footprint" "TestPoint:TestPoint_Loop_D1.80mm_Drill1.0mm_Beaded" (at 127 27.94 0)
       (effects (font (size 1.27 1.27)) hide)
     )
@@
       (effects (font (size 1.27 1.27)) hide)
     )
-    (property "Description" "Test Points/Test Rings ROHS red" (at 121.92 27.94 0)
-      (effects (font (size 1.27 1.27)) hide)
-    )
+    (property "Description" "Test Points/Test Rings 1.25 mm Red" (at 121.92 27.94 0)
+      (effects (font (size 1.27 1.27)) hide)
+    )

Commit message: PWA_REV2.kicad, Adding test points, GND, SPI, and UART0. Filed a keystone datasheet.
Parts:
- added TP100: TP+3.3V, TestPoint:TestPoint_Loop_D2.54mm_Drill1.5mm_Beaded, symbol Connector:TestPoint
- added TP104, TP105, TP106: TP_GND, TestPoint:TestPoint_Loop_D1.80mm_Drill1.0mm_Beaded, symbol Connector:TestPoint
- added TP404: U0_RX, TestPoint:TestPoint_Loop_D1.80mm_Drill1.0mm_Beaded, symbol Connector:TestPoint
- added TP404: U0_TX, TestPoint:TestPoint_Loop_D1.80mm_Drill1.0mm_Beaded, symbol Connector:TestPoint
Connections:
- net +3.3V: now also TP100.1
- net ControllerRX: now also TP404.1
- net ControllerTX: now also TP404.1
- net GND: now also TP104.1, TP105.1, TP106.1

Commit message: PWA_REV2.kicad, Adding test points for the decoupling 5v resistors.
Parts:
- added TP?: 3v3Controller, TestPoint:TestPoint_Loop_D2.54mm_Drill1.5mm_Beaded, symbol Connector:TestPoint
Connections:
- net 3v3Controller: now also TP?.1
Changed lines of the file:
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@@
   (junction (at 210.82 139.7) (diameter 0) (color 0 0 0 0)
   )
+  (junction (at 33.02 88.9) (diameter 0) (color 0 0 0 0)
+  )
   (junction (at 121.92 27.94) (diameter 0) (color 0 0 0 0)
   )
@@
     (stroke (width 0) (type default))
   )
+  (wire (pts (xy 33.02 80.01) (xy 33.02 88.9))
+    (stroke (width 0) (type default))
+  )
   (wire (pts (xy 62.23 27.94) (xy 62.23 33.02))
     (stroke (width 0) (type default))
@@
     )
   )
+  (symbol (lib_id "Connector:TestPoint") (at 33.02 80.01 0) (unit 1)
+    (in_bom yes) (on_board yes) (dnp no)
+    (property "Reference" "TP?" (at 22.86 72.39 0)
+      (effects (font (size 1.27 1.27)) (justify left))
+    )
+    (property "Value" "3v3Controller" (at 22.86 74.93 0)
+      (effects (font (size 1.27 1.27)) (justify left))
+    )
+    (property "Footprint" "TestPoint:TestPoint_Loop_D2.54mm_Drill1.5mm_Beaded" (at 38.1 80.01 0)
+      (effects (font (size 1.27 1.27)) hide)
+    )
+    (property "Datasheet" "~" (at 38.1 80.01 0)
+      (effects (font (size 1.27 1.27)) hide)
+    )
+    (property "AssemblyType" "HAND" (at 33.02 80.01 0)
+      (effects (font (size 1.27 1.27)) hide)
+    )
+    (property "Description" "Test Points/Test Rings ROHS red" (at 33.02 80.01 0)
+      (effects (font (size 1.27 1.27)) hide)
+    )
+    (property "Distributor 1" "JLCPCB" (at 33.02 80.01 0)
+      (effects (font (size 1.27 1.27)) hide)
+    )
+    (property "Distributor 1 PN" "C5277086" (at 33.02 80.01 0)
+      (effects (font (size 1.27 1.27)) hide)
+    )
+    (property "MPN" "RH-5000" (at 33.02 80.01 0)
+      (effects (font (size 1.27 1.27)) hide)
+    )
+    (property "Manufacturer" "ronghe" (at 33.02 80.01 0)
+      (effects (font (size 1.27 1.27)) hide)
+    )
+    (property "Cost" "0.0717" (at 33.02 80.01 0)
+      (effects (font (size 1.27 1.27)) hide)
+    )
+    (property "MPN 2" "" (at 33.02 80.01 0)
+      (effects (font (size 1.27 1.27)) hide)
+    )
+    (property "Manufacturer 2" "" (at 33.02 80.01 0)
+      (effects (font (size 1.27 1.27)) hide)
+    )
+    (pin "1")
+    (instances
+      (project "PWA_REV2"
+        (path "/412a327d-1ee3-473e-bc00-1545004b7edf"
+          (reference "TP?") (unit 1)
+        )
+      )
+    )
+  )
   (symbol (lib_id "Connector:TestPoint") (at 121.92 27.94 0) (unit 1)
     (in_bom yes) (on_board yes) (dnp no)
@@
       (effects (font (size 1.27 1.27)) hide)
     )
-    (property "Value" "PWR_FLAG" (at 36.83 83.2358 0)
+    (property "Value" "PWR_FLAG" (at 39.37 83.82 0)
       (effects (font (size 1.27 1.27)))
     )

Commit message: PWA_REV2.kicad, Adding test points for the decoupling 3v3 resistors and for the VCC USB.
Parts:
- gave numbers to parts that had none: 1
Changed lines of the file:
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@@
   (symbol (lib_id "Connector:TestPoint") (at 33.02 80.01 0) (unit 1)
     (in_bom yes) (on_board yes) (dnp no)
-    (property "Reference" "TP?" (at 22.86 72.39 0)
+    (property "Reference" "TP109" (at 22.86 72.39 0)
       (effects (font (size 1.27 1.27)) (justify left))
     )
@@
       (project "PWA_REV2"
         (path "/412a327d-1ee3-473e-bc00-1545004b7edf"
-          (reference "TP?") (unit 1)
+          (reference "TP109") (unit 1)
         )
       )
