File: PWA_REV2/PWA_REV2.kicad_sch (KiCad schematic)
At the start: 65 parts, among them J101 Barrel_Jack_Switch_SMT, J102 0.100_2Pin, J103 0.100_2Pin, J104 Conn_01x14 1mm, J106 Conn_01x14 1mm, J107 Conn_01x10 1mm, SW101 RotaryEncoder_Switch, T101 ToolingHole_Pad_1.152mm, T102 ToolingHole_Pad_1.152mm, T103 ToolingHole_Pad_1.152mm, U101 LM7805_TO220, U102 ESP32-WROOM-32E-N4, U103 AMS1117-3.3

Commit message: PWA_REV2, Made a new Footprint, saved it in the GeneralPurposeAlarmDevicePCB, with the name D_SMB_POLARITY. Updated the schematic with the Diode Footprint. Issue 237.
Parts:
- D101, D103, D104: footprint Diode_SMD:D_SMB -> GeneralPurposeAlarmDevicePCB:D_SMB_POLARITY
Changed lines of the file:
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@@
       (effects (font (size 1.27 1.27)))
     )
-    (property "Footprint" "Diode_SMD:D_SMB" (at 53.34 27.94 0)
+    (property "Footprint" "GeneralPurposeAlarmDevicePCB:D_SMB_POLARITY" (at 53.34 27.94 0)
       (effects (font (size 1.27 1.27)) hide)
     )
@@
       (effects (font (size 1.27 1.27)))
     )
-    (property "Footprint" "Diode_SMD:D_SMB" (at 180.34 31.75 0)
+    (property "Footprint" "GeneralPurposeAlarmDevicePCB:D_SMB_POLARITY" (at 180.34 31.75 0)
       (effects (font (size 1.27 1.27)) hide)
     )
@@
       (effects (font (size 1.27 1.27)))
     )
-    (property "Footprint" "Diode_SMD:D_SMB" (at 92.71 63.5 0)
-      (effects (font (size 1.27 1.27)) hide)
-    )
+    (property "Footprint" "GeneralPurposeAlarmDevicePCB:D_SMB_POLARITY" (at 92.71 63.5 0)
+      (effects (font (size 1.27 1.27)) hide)
+    )

Commit message: PWA_REV2, Customised the rotary encoder schematic and footprint for mounting pad pins, issue 252.
Parts:
- SW101: footprint Rotary_Encoder:RotaryEncoder_Alps_EC12E-Switch_Vertical_H20mm -> GeneralPurposeAlarmDevicePCB:RotaryEncoder_Alps_EC12E-Switch_Vertical_H20mm_MP1_MP2; symbol Device:RotaryEncoder_Switch -> GPAD_SCH_LIB:RotaryEncoder_Switch_MP
Connections:
- net GND: now also SW101.MP1 (A), SW101.MP2 (A)
Changed lines of the file:
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@@
     (stroke (width 0) (type default))
   )
+  (wire (pts (xy 46.99 129.54) (xy 46.99 132.08))
+    (stroke (width 0) (type default))
+  )
   (wire (pts (xy 111.76 121.92) (xy 114.3 121.92))
     (stroke (width 0) (type default))
@@
     (stroke (width 0) (type default))
   )
+  (wire (pts (xy 63.5 129.54) (xy 46.99 129.54))
+    (stroke (width 0) (type default))
+  )
   (wire (pts (xy 171.45 87.63) (xy 171.45 88.9))
     (stroke (width 0) (type default))
@@
     )
   )
+  (symbol (lib_id "power:GND") (at 63.5 144.78 0) (unit 1)
+    (in_bom yes) (on_board yes) (dnp no)
+    (property "Reference" "#PWR0104" (at 63.5 151.13 0)
+      (effects (font (size 1.27 1.27)) hide)
+    )
+    (property "Value" "GND" (at 63.627 149.1742 0)
+      (effects (font (size 1.27 1.27)))
+    )
+    (property "Footprint" "" (at 63.5 144.78 0)
+      (effects (font (size 1.27 1.27)) hide)
+    )
+    (property "Datasheet" "" (at 63.5 144.78 0)
+      (effects (font (size 1.27 1.27)) hide)
+    )
+    (pin "1")
+    (instances
+      (project "PWA_REV2"
+        (path "/412a327d-1ee3-473e-bc00-1545004b7edf"
+          (reference "#PWR0104") (unit 1)
+        )
+      )
+    )
+  )
   (symbol (lib_id "Device:R") (at 182.88 114.3 270) (unit 1)
     (in_bom yes) (on_board yes) (dnp no)
@@
     )
   )
-  (symbol (lib_id "Device:RotaryEncoder_Switch") (at 63.5 137.16 0) (unit 1)
+  (symbol (lib_id "GPAD_SCH_LIB:RotaryEncoder_Switch_MP") (at 63.5 137.16 0) (unit 1)
     (in_bom yes) (on_board yes) (dnp no) (fields_autoplaced)
     (property "Reference" "SW101" (at 63.5 127 0)
@@
       (effects (font (size 1.27 1.27)))
     )
-    (property "Footprint" "Rotary_Encoder:RotaryEncoder_Alps_EC12E-Switch_Vertical_H20mm" (at 59.69 133.096 0)
+    (property "Footprint" "GeneralPurposeAlarmDevicePCB:RotaryEncoder_Alps_EC12E-Switch_Vertical_H20mm_MP1_MP2" (at 59.69 133.096 0)
       (effects (font (size 1.27 1.27)) hide)
     )
@@
     (pin "B")
     (pin "C")
+    (pin "MP1")
+    (pin "MP2")
     (pin "S1")
     (pin "S2")
@@
         )
       )
+    )
+  )
+  (symbol (lib_id "power:GND") (at 46.99 132.08 0) (unit 1)
+    (in_bom yes) (on_board yes) (dnp no)
+    (property "Reference" "#PWR0105" (at 46.99 138.43 0)
+      (effects (font (size 1.27 1.27)) hide)
+    )
+    (property "Value" "GND" (at 47.117 136.4742 0)
+      (effects (font (size 1.27 1.27)))
+    )
+    (property "Footprint" "" (at 46.99 132.08 0)
+      (effects (font (size 1.27 1.27)) hide)
+    )
+    (property "Datasheet" "" (at 46.99 132.08 0)
+      (effects (font (size 1.27 1.27)) hide)
+    )
+    (pin "1")
+    (instances
+      (project "PWA_REV2"
+        (path "/412a327d-1ee3-473e-bc00-1545004b7edf"
+          (reference "#PWR0105") (unit 1)
+        )
+      )

Commit message: USB_UART, moving the RX test point closer to where the tx of USB is.
Parts:
- removed TP404: U0_RX, TestPoint:TestPoint_Loop_D1.80mm_Drill1.0mm_Beaded, symbol Connector:TestPoint
Changed lines of the file:
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@@
   (junction (at 147.32 138.43) (diameter 0) (color 0 0 0 0)
   )
-  (junction (at 171.45 99.06) (diameter 0) (color 0 0 0 0)
-  )
   (junction (at 210.82 139.7) (diameter 0) (color 0 0 0 0)
   )
@@
     (stroke (width 0) (type default))
   )
-  (wire (pts (xy 171.45 97.79) (xy 171.45 99.06))
-    (stroke (width 0) (type default))
-  )
   (wire (pts (xy 67.31 19.05) (xy 175.26 19.05))
     (stroke (width 0) (type default))
@@
     (stroke (width 0) (type default))
   )
-  (wire (pts (xy 209.55 96.52) (xy 209.55 97.79))
-    (stroke (width 0) (type default))
-  )
   (wire (pts (xy 101.6 93.98) (xy 111.76 93.98))
     (stroke (width 0) (type default))
@@
     (stroke (width 0) (type default))
   )
-  (wire (pts (xy 161.29 99.06) (xy 171.45 99.06))
+  (wire (pts (xy 161.29 99.06) (xy 175.26 99.06))
     (stroke (width 0) (type default))
   )
@@
     (stroke (width 0) (type default))
   )
-  (wire (pts (xy 209.55 97.79) (xy 171.45 97.79))
-    (stroke (width 0) (type default))
-  )
   (wire (pts (xy 105.41 72.39) (xy 101.6 72.39))
     (stroke (width 0) (type default))
@@
     (stroke (width 0) (type default))
   )
-  (wire (pts (xy 171.45 99.06) (xy 175.26 99.06))
-    (stroke (width 0) (type default))
-  )
   (wire (pts (xy 111.76 111.76) (xy 114.3 111.76))
     (stroke (width 0) (type default))
@@
         )
       )
-    )
-  )
-  (symbol (lib_id "Connector:TestPoint") (at 209.55 96.52 0) (unit 1)
-    (in_bom yes) (on_board yes) (dnp no)
-    (property "Reference" "TP404" (at 209.55 90.17 0)
-      (effects (font (size 1.27 1.27)) (justify left))
-    )
-    (property "Value" "U0_RX" (at 210.82 92.71 0)
-      (effects (font (size 1.27 1.27)) (justify left))
-    )
-    (property "Footprint" "TestPoint:TestPoint_Loop_D1.80mm_Drill1.0mm_Beaded" (at 214.63 96.52 0)
-      (effects (font (size 1.27 1.27)) hide)
-    )
-    (property "Datasheet" "~" (at 214.63 96.52 0)
-      (effects (font (size 1.27 1.27)) hide)
-    )
-    (property "AssemblyType" "HAND" (at 209.55 96.52 0)
-      (effects (font (size 1.27 1.27)) hide)
-    )
-    (property "Distributor 1" "JLCPCB" (at 209.55 96.52 0)
-      (effects (font (size 1.27 1.27)) hide)
-    )
-    (property "Description" "Test Points/Test Rings 1.25 mm Yellow" (at 209.55 96.52 0)
-      (effects (font (size 1.27 1.27)) hide)
-    )
-    (property "Distributor 1 PN" "C5199804" (at 209.55 96.52 0)
-      (effects (font (size 1.27 1.27)) hide)
-    )
-    (property "MPN" "RH-5004" (at 209.55 96.52 0)
-      (effects (font (size 1.27 1.27)) hide)
-    )
-    (property "Manufacturer" "ronghe" (at 209.55 96.52 0)
-      (effects (font (size 1.27 1.27)) hide)
-    )
-    (property "Cost" "0.0800" (at 209.55 96.52 0)
-      (effects (font (size 1.27 1.27)) hide)
-    )
-    (property "MPN 2" "" (at 209.55 96.52 0)
-      (effects (font (size 1.27 1.27)) hide)
-    )
-    (property "Manufacturer 2" "" (at 209.55 96.52 0)
-      (effects (font (size 1.27 1.27)) hide)
-    )
-    (pin "1")
-    (instances
-      (project "PWA_REV2"
-        (path "/412a327d-1ee3-473e-bc00-1545004b7edf/00000000-0000-0000-0000-000062b871ee"
-          (reference "TP404") (unit 1)
-        )
-        (path "/412a327d-1ee3-473e-bc00-1545004b7edf"
-          (reference "TP108") (unit 1)
-        )
-      )

Commit message: USB_UART, moving the RX test point closer to where the tx of USB is.
Parts:
- TP404: value U0_TX -> U0_RX
Connections:
- net ControllerRX: now also TP404.1
- net ControllerTX: no longer TP404.1
Changed lines of the file:
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@@
   (junction (at 147.32 138.43) (diameter 0) (color 0 0 0 0)
   )
+  (junction (at 171.45 99.06) (diameter 0) (color 0 0 0 0)
+  )
   (junction (at 210.82 139.7) (diameter 0) (color 0 0 0 0)
   )
@@
   (junction (at 163.83 27.94) (diameter 0) (color 0 0 0 0)
   )
-  (junction (at 187.96 96.52) (diameter 0) (color 0 0 0 0)
-  )
   (junction (at 238.76 34.29) (diameter 0) (color 0 0 0 0)
   )
@@
     (stroke (width 0) (type default))
   )
+  (wire (pts (xy 171.45 97.79) (xy 171.45 99.06))
+    (stroke (width 0) (type default))
+  )
   (wire (pts (xy 67.31 19.05) (xy 175.26 19.05))
     (stroke (width 0) (type default))
@@
     (stroke (width 0) (type default))
   )
-  (wire (pts (xy 187.96 93.98) (xy 187.96 96.52))
-    (stroke (width 0) (type default))
-  )
   (wire (pts (xy 173.99 121.92) (xy 181.61 121.92))
     (stroke (width 0) (type default))
@@
     (stroke (width 0) (type default))
   )
+  (wire (pts (xy 209.55 96.52) (xy 209.55 97.79))
+    (stroke (width 0) (type default))
+  )
   (wire (pts (xy 101.6 93.98) (xy 111.76 93.98))
     (stroke (width 0) (type default))
@@
     (stroke (width 0) (type default))
   )
-  (wire (pts (xy 203.2 91.44) (xy 203.2 93.98))
-    (stroke (width 0) (type default))
-  )
   (wire (pts (xy 40.64 27.94) (xy 39.37 27.94))
     (stroke (width 0) (type default))
@@
     (stroke (width 0) (type default))
   )
-  (wire (pts (xy 203.2 93.98) (xy 187.96 93.98))
-    (stroke (width 0) (type default))
-  )
   (wire (pts (xy 129.54 135.89) (xy 129.54 138.43))
     (stroke (width 0) (type default))
@@
     (stroke (width 0) (type default))
   )
-  (wire (pts (xy 161.29 99.06) (xy 175.26 99.06))
+  (wire (pts (xy 161.29 99.06) (xy 171.45 99.06))
     (stroke (width 0) (type default))
   )
@@
     (stroke (width 0) (type default))
   )
+  (wire (pts (xy 209.55 97.79) (xy 171.45 97.79))
+    (stroke (width 0) (type default))
+  )
   (wire (pts (xy 105.41 72.39) (xy 101.6 72.39))
     (stroke (width 0) (type default))
@@
     (stroke (width 0) (type default))
   )
+  (wire (pts (xy 171.45 99.06) (xy 175.26 99.06))
+    (stroke (width 0) (type default))
+  )
   (wire (pts (xy 111.76 111.76) (xy 114.3 111.76))
     (stroke (width 0) (type default))
@@
     (stroke (width 0) (type default))
   )
-  (wire (pts (xy 187.96 96.52) (xy 191.77 96.52))
-    (stroke (width 0) (type default))
-  )
   (wire (pts (xy 111.76 116.84) (xy 114.3 116.84))
     (stroke (width 0) (type default))
@@
     (stroke (width 0) (type default))
   )
-  (wire (pts (xy 161.29 96.52) (xy 187.96 96.52))
+  (wire (pts (xy 161.29 96.52) (xy 191.77 96.52))
     (stroke (width 0) (type default))
   )
@@
     )
   )
+  (symbol (lib_id "Connector:TestPoint") (at 209.55 96.52 0) (unit 1)
+    (in_bom yes) (on_board yes) (dnp no)
+    (property "Reference" "TP404" (at 209.55 90.17 0)
+      (effects (font (size 1.27 1.27)) (justify left))
+    )
+    (property "Value" "U0_RX" (at 210.82 92.71 0)
+      (effects (font (size 1.27 1.27)) (justify left))
+    )
+    (property "Footprint" "TestPoint:TestPoint_Loop_D1.80mm_Drill1.0mm_Beaded" (at 214.63 96.52 0)
+      (effects (font (size 1.27 1.27)) hide)
+    )
+    (property "Datasheet" "~" (at 214.63 96.52 0)
+      (effects (font (size 1.27 1.27)) hide)
+    )
+    (property "AssemblyType" "HAND" (at 209.55 96.52 0)
+      (effects (font (size 1.27 1.27)) hide)
+    )
+    (property "Distributor 1" "JLCPCB" (at 209.55 96.52 0)
+      (effects (font (size 1.27 1.27)) hide)
+    )
+    (property "Description" "Test Points/Test Rings 1.25 mm Yellow" (at 209.55 96.52 0)
+      (effects (font (size 1.27 1.27)) hide)
+    )
+    (property "Distributor 1 PN" "C5199804" (at 209.55 96.52 0)
+      (effects (font (size 1.27 1.27)) hide)
+    )
+    (property "MPN" "RH-5004" (at 209.55 96.52 0)
+      (effects (font (size 1.27 1.27)) hide)
+    )
+    (property "Manufacturer" "ronghe" (at 209.55 96.52 0)
+      (effects (font (size 1.27 1.27)) hide)
+    )
+    (property "Cost" "0.0800" (at 209.55 96.52 0)
+      (effects (font (size 1.27 1.27)) hide)
+    )
+    (property "MPN 2" "" (at 209.55 96.52 0)
+      (effects (font (size 1.27 1.27)) hide)
+    )
+    (property "Manufacturer 2" "" (at 209.55 96.52 0)
+      (effects (font (size 1.27 1.27)) hide)
+    )
+    (pin "1")
+    (instances
+      (project "PWA_REV2"
+        (path "/412a327d-1ee3-473e-bc00-1545004b7edf/00000000-0000-0000-0000-000062b871ee"
+          (reference "TP404") (unit 1)
+        )
+        (path "/412a327d-1ee3-473e-bc00-1545004b7edf"
+          (reference "TP108") (unit 1)
+        )
+      )
+    )
+  )
   (symbol (lib_id "Regulator_Linear:AMS1117-3.3") (at 251.46 34.29 0) (unit 1)
     (in_bom yes) (on_board yes) (dnp no) (fields_autoplaced)
@@
         )
       )
-    )
-  )
-  (symbol (lib_id "Connector:TestPoint") (at 203.2 91.44 0) (unit 1)
-    (in_bom yes) (on_board yes) (dnp no)
-    (property "Reference" "TP404" (at 203.2 85.09 0)
-      (effects (font (size 1.27 1.27)) (justify left))
-    )
-    (property "Value" "U0_TX" (at 204.47 87.63 0)
-      (effects (font (size 1.27 1.27)) (justify left))
-    )
-    (property "Footprint" "TestPoint:TestPoint_Loop_D1.80mm_Drill1.0mm_Beaded" (at 208.28 91.44 0)
-      (effects (font (size 1.27 1.27)) hide)
-    )
-    (property "Datasheet" "~" (at 208.28 91.44 0)
-      (effects (font (size 1.27 1.27)) hide)
-    )
-    (property "AssemblyType" "HAND" (at 203.2 91.44 0)
-      (effects (font (size 1.27 1.27)) hide)
-    )
-    (property "Distributor 1" "JLCPCB" (at 203.2 91.44 0)
-      (effects (font (size 1.27 1.27)) hide)
-    )
-    (property "Description" "Test Points/Test Rings 1.25 mm Yellow" (at 203.2 91.44 0)
-      (effects (font (size 1.27 1.27)) hide)
-    )
-    (property "Distributor 1 PN" "C5199804" (at 203.2 91.44 0)
-      (effects (font (size 1.27 1.27)) hide)
-    )
-    (property "MPN" "RH-5004" (at 203.2 91.44 0)
-      (effects (font (size 1.27 1.27)) hide)
-    )
-    (property "Manufacturer" "ronghe" (at 203.2 91.44 0)
-      (effects (font (size 1.27 1.27)) hide)
-    )
-    (property "Cost" "0.0800" (at 203.2 91.44 0)
-      (effects (font (size 1.27 1.27)) hide)
-    )
-    (property "MPN 2" "" (at 203.2 91.44 0)
-      (effects (font (size 1.27 1.27)) hide)
-    )
-    (property "Manufacturer 2" "" (at 203.2 91.44 0)
-      (effects (font (size 1.27 1.27)) hide)
-    )
-    (pin "1")
-    (instances
-      (project "PWA_REV2"
-        (path "/412a327d-1ee3-473e-bc00-1545004b7edf/00000000-0000-0000-0000-000062b871ee"
-          (reference "TP404") (unit 1)
-        )
-        (path "/412a327d-1ee3-473e-bc00-1545004b7edf"
-          (reference "TP107") (unit 1)
-        )
-      )

Commit message: PWA_REV2, Corrected test points footprints.
Parts:
- TP100, TP109: footprint TestPoint:TestPoint_Loop_D2.54mm_Drill1.5mm_Beaded -> TestPoint:TestPoint_Loop_D1.80mm_Drill1.0mm_Beaded
Changed lines of the file:
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@@
       (effects (font (size 1.27 1.27)) (justify left))
     )
-    (property "Footprint" "TestPoint:TestPoint_Loop_D2.54mm_Drill1.5mm_Beaded" (at 280.67 30.48 0)
+    (property "Footprint" "TestPoint:TestPoint_Loop_D1.80mm_Drill1.0mm_Beaded" (at 280.67 30.48 0)
       (effects (font (size 1.27 1.27)) hide)
     )
@@
       (effects (font (size 1.27 1.27)) (justify left))
     )
-    (property "Footprint" "TestPoint:TestPoint_Loop_D2.54mm_Drill1.5mm_Beaded" (at 38.1 80.01 0)
-      (effects (font (size 1.27 1.27)) hide)
-    )
+    (property "Footprint" "TestPoint:TestPoint_Loop_D1.80mm_Drill1.0mm_Beaded" (at 38.1 80.01 0)
+      (effects (font (size 1.27 1.27)) hide)
+    )

Commit message: PWA_REV2, Placed testpoint and routed it. Changed the settings of some Values of old testpoints to be on silkscreen.
Parts:
- +5esp32: footprint TestPoint:TestPoint_Loop_D2.54mm_Drill1.5mm_Beaded -> TestPoint:TestPoint_Loop_D1.80mm_Drill1.0mm_Beaded
Changed lines of the file:
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@@
       (effects (font (size 1.27 1.27)) (justify left))
     )
-    (property "Footprint" "TestPoint:TestPoint_Loop_D2.54mm_Drill1.5mm_Beaded" (at 241.3 29.21 0)
+    (property "Footprint" "TestPoint:TestPoint_Loop_D1.80mm_Drill1.0mm_Beaded" (at 241.3 29.21 0)
       (effects (font (size 1.27 1.27)) hide)
     )
