File: PWA_REV2/PWA_REV2.kicad_sch (KiCad schematic)
At the start: 66 parts, among them J101 Barrel_Jack_Switch_SMT, J102 0.100_2Pin, J103 0.100_2Pin, J104 Conn_01x14 1mm, J106 Conn_01x14 1mm, J107 Conn_01x10 1mm, SW101 RotaryEncoder_Switch, T101 ToolingHole_Pad_1.152mm, T102 ToolingHole_Pad_1.152mm, T103 ToolingHole_Pad_1.152mm, U101 LM7805_TO220, U102 ESP32-WROOM-32E-N4, U103 AMS1117-3.3

Commit message: gerbers, generated and submitted files to PCPWAY to place an order, PWA_Rev, corrected and fixed the MPN and description of components.
Parts:
- D106: DK_Datasheet_Link http://optoelectronics.liteon.com/upload/download/DS22-2000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 -> (none); DK_Detail_Page /product-detail/en/lite-on-inc/LTST-C171KRKT/160-1427-1-ND/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 -> (none); Digi-Key_PN 160-1427-1-ND -> (none); MPN LTST-C171KRKT -> KT-0603R; Manufacturer Lite-On Inc. -> Hubei KENTO Elec
- J101: MPN DC-005-5A-2.0-SMT / 54-00164 -> DC-005-5A-2.0-SMT; MPN 2 (none) -> 54-00164; Manufacturer XKB Connectivity / Tensility International Corp -> XKB Connectivity; Manufacturer 2 (none) -> Tensility International Corp
- S101: value SWITCH_TACTILE_SPST-NO_0.05A_24V -> SWITCH_TACTILE_FLAT_6mmx6mm_SPST-NO_0.05A_24V; MPN TE Connectivity 1825910-7, Dongguan Guangzhu Industrial C13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 -> TE Connectivity 1825910-7, Dongguan Guangzhu Industrial; MPN 2 (none) -> TS6685H-250gf; Manufacturer 2 (none) -> YE
- SYM101, SYM102: AssemblyType (none) -> NA
Changed lines of the file:
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@@
       (effects (font (size 1.27 1.27)) hide)
     )
-    (property "Datasheet" "https://tensility.s3.amazonaws.com/uploads/pdffiles/54-00164.pdf" (at 26.67 31.496 0)
+    (property "Datasheet" "https://www.lcsc.com/datasheet/C319134.pdf   , https://tensility.s3.amazonaws.com/uploads/pdffiles/54-00164.pdf" (at 26.67 31.496 0)
       (effects (font (size 1.27 1.27)) hide)
     )
@@
       (effects (font (size 1.27 1.27)) hide)
     )
-    (property "Manufacturer" "XKB Connectivity / Tensility International Corp" (at 25.4 30.48 0)
+    (property "Manufacturer" "XKB Connectivity " (at 25.4 30.48 0)
       (effects (font (size 1.27 1.27)) hide)
     )
-    (property "MPN" "DC-005-5A-2.0-SMT / 54-00164" (at 25.4 30.48 0)
+    (property "MPN" "DC-005-5A-2.0-SMT" (at 25.4 30.48 0)
       (effects (font (size 1.27 1.27)) hide)
     )
@@
       (effects (font (size 1.27 1.27)) hide)
     )
-    (property "MPN 2" "" (at 25.4 30.48 0)
+    (property "MPN 2" "54-00164" (at 25.4 30.48 0)
       (effects (font (size 1.27 1.27)) hide)
     )
-    (property "Manufacturer 2" "" (at 25.4 30.48 0)
+    (property "Manufacturer 2" "Tensility International Corp" (at 25.4 30.48 0)
       (effects (font (size 1.27 1.27)) hide)
     )
@@
       (effects (font (size 1.524 1.524)))
     )
-    (property "Value" "SWITCH_TACTILE_SPST-NO_0.05A_24V" (at 62.23 67.945 0)
+    (property "Value" "SWITCH_TACTILE_FLAT_6mmx6mm_SPST-NO_0.05A_24V   " (at 62.23 67.945 0)
       (effects (font (size 1.524 1.524)))
     )
@@
       (effects (font (size 1.524 1.524)) (justify left) hide)
     )
-    (property "MPN" "TE Connectivity 1825910-7,   Dongguan Guangzhu Industrial C13828" (at 45.72 50.8 0)
+    (property "MPN" "TE Connectivity 1825910-7,   Dongguan Guangzhu Industrial " (at 45.72 50.8 0)
       (effects (font (size 1.524 1.524)) (justify left) hide)
     )
@@
       (effects (font (size 1.27 1.27)) hide)
     )
-    (property "MPN 2" "" (at 50.8 63.5 0)
+    (property "MPN 2" "TS6685H-250gf" (at 50.8 63.5 0)
       (effects (font (size 1.27 1.27)) hide)
     )
-    (property "Manufacturer 2" "" (at 50.8 63.5 0)
+    (property "Manufacturer 2" "YE" (at 50.8 63.5 0)
       (effects (font (size 1.27 1.27)) hide)
     )
@@
       (effects (font (size 1.27 1.27)) hide)
     )
+    (property "AssemblyType" "NA" (at 26.67 20.32 0)
+      (effects (font (size 1.27 1.27)) hide)
+    )
     (instances
       (project "PWA_REV2"
@@
       (effects (font (size 1.27 1.27)) hide)
     )
-    (property "Datasheet" "~" (at 119.38 162.56 0)
+    (property "Datasheet" "https://jlcpcb.com/api/file/downloadByFileSystemAccessId/8550723991833485312" (at 119.38 162.56 0)
       (effects (font (size 1.27 1.27)) hide)
     )
@@
       (effects (font (size 1.524 1.524)) (justify left) hide)
     )
-    (property "MPN" "LTST-C171KRKT" (at 132.08 157.48 0)
+    (property "MPN" "KT-0603R" (at 132.08 157.48 0)
       (effects (font (size 1.524 1.524)) (justify left) hide)
     )
@@
       (effects (font (size 1.524 1.524)) (justify left) hide)
     )
-    (property "Manufacturer" "Lite-On Inc." (at 147.32 157.48 0)
+    (property "Manufacturer" "Hubei KENTO Elec" (at 147.32 157.48 0)
       (effects (font (size 1.524 1.524)) (justify left) hide)
     )
@@
       (effects (font (size 1.524 1.524)) (justify left) hide)
     )
-    (property "DK_Datasheet_Link" "http://optoelectronics.liteon.com/upload/download/DS22-2000-109/LTST-C171KRKT.pdf" (at 3.81 297.18 0)
+    (property "DK_Datasheet_Link" "" (at 3.81 297.18 0)
       (effects (font (size 1.27 1.27)) hide)
     )
-    (property "DK_Detail_Page" "/product-detail/en/lite-on-inc/LTST-C171KRKT/160-1427-1-ND/386800" (at 3.81 297.18 0)
+    (property "DK_Detail_Page" "" (at 3.81 297.18 0)
       (effects (font (size 1.27 1.27)) hide)
     )
-    (property "Digi-Key_PN" "160-1427-1-ND" (at 3.81 297.18 0)
+    (property "Digi-Key_PN" "" (at 3.81 297.18 0)
       (effects (font (size 1.27 1.27)) hide)
     )
@@
       (effects (font (size 1.27 1.27)) hide)
     )
+    (property "AssemblyType" "NA" (at 266.7 173.99 0)
+      (effects (font (size 1.27 1.27)) hide)
+    )

Commit message: PWA_REV2.kicad_sch, Change mounting holes for exclude from BOM.
Parts:
- H101, H102, H103, H104: now left out of the parts list
Changed lines of the file:
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@@
   )
   (symbol (lib_id "GPAD_SCH_LIB:MountingHole_Pad_3.5mm") (at 217.17 147.32 0) (unit 1)
-    (in_bom yes) (on_board yes) (dnp no)
+    (in_bom no) (on_board yes) (dnp no)
     (property "Reference" "H104" (at 219.71 146.0754 0)
       (effects (font (size 1.27 1.27)) (justify left))
@@
   )
   (symbol (lib_id "GPAD_SCH_LIB:MountingHole_Pad_3.5mm") (at 217.17 139.7 0) (unit 1)
-    (in_bom yes) (on_board yes) (dnp no)
+    (in_bom no) (on_board yes) (dnp no)
     (property "Reference" "H103" (at 219.71 138.4554 0)
       (effects (font (size 1.27 1.27)) (justify left))
@@
   )
   (symbol (lib_id "GPAD_SCH_LIB:MountingHole_Pad_3.5mm") (at 217.17 132.08 0) (unit 1)
-    (in_bom yes) (on_board yes) (dnp no)
+    (in_bom no) (on_board yes) (dnp no)
     (property "Reference" "H102" (at 219.71 130.8354 0)
       (effects (font (size 1.27 1.27)) (justify left))
@@
   )
   (symbol (lib_id "GPAD_SCH_LIB:MountingHole_Pad_3.5mm") (at 217.17 124.46 0) (unit 1)
-    (in_bom yes) (on_board yes) (dnp no)
+    (in_bom no) (on_board yes) (dnp no)
     (property "Reference" "H101" (at 219.71 123.2154 0)
       (effects (font (size 1.27 1.27)) (justify left))

Commit message: PWA_REV2.kicad_sch, Change tooling holes for exclude from BOM.
Parts:
- T101, T102, T103: now left out of the parts list
Changed lines of the file:
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@@
   )
   (symbol (lib_id "GPAD_SCH_LIB:ToolingHole_Pad_1.152mm") (at 212.09 109.22 0) (unit 1)
-    (in_bom yes) (on_board yes) (dnp no) (fields_autoplaced)
+    (in_bom no) (on_board yes) (dnp no) (fields_autoplaced)
     (property "Reference" "T102" (at 214.63 107.95 0)
       (effects (font (size 1.27 1.27)) (justify left))
@@
   )
   (symbol (lib_id "GPAD_SCH_LIB:ToolingHole_Pad_1.152mm") (at 212.09 114.3 0) (unit 1)
-    (in_bom yes) (on_board yes) (dnp no) (fields_autoplaced)
+    (in_bom no) (on_board yes) (dnp no) (fields_autoplaced)
     (property "Reference" "T103" (at 214.63 113.03 0)
       (effects (font (size 1.27 1.27)) (justify left))
@@
   )
   (symbol (lib_id "GPAD_SCH_LIB:ToolingHole_Pad_1.152mm") (at 212.09 104.14 0) (unit 1)
-    (in_bom yes) (on_board yes) (dnp no) (fields_autoplaced)
+    (in_bom no) (on_board yes) (dnp no) (fields_autoplaced)
     (property "Reference" "T101" (at 214.63 102.87 0)
       (effects (font (size 1.27 1.27)) (justify left))

Commit message: PWA_REV2.kicad_sch, Change open hardware logo for exclude from BOM.
Parts:
- SYM101: now left out of the parts list
Changed lines of the file:
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@@
   )
   (symbol (lib_id "Graphic:Logo_Open_Hardware_Small") (at 266.7 173.99 0) (unit 1)
-    (in_bom yes) (on_board yes) (dnp no) (fields_autoplaced)
+    (in_bom no) (on_board yes) (dnp no) (fields_autoplaced)
     (property "Reference" "SYM101" (at 266.7 167.005 0)
       (effects (font (size 1.27 1.27)))

Commit message: PWA_REV2.kicad_sch, Change four DNI resistors to Do not populate for exclude from BOM.
Parts:
- R106, R107: now not fitted
Connections:
- net +5V: no longer R106.2
- net VBus: no longer R106.1
Changed lines of the file:
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@@
     )
   )
-  (symbol (lib_id "Device:R") (at 157.48 35.56 270) (unit 1)
-    (in_bom yes) (on_board yes) (dnp no)
-    (property "Reference" "R106" (at 156.21 30.48 90)
+  (symbol (lib_id "Device:R") (at 157.48 35.56 0) (unit 1)
+    (in_bom yes) (on_board yes) (dnp yes)
+    (property "Reference" "R106" (at 152.4 36.83 90)
       (effects (font (size 1.27 1.27)))
     )
-    (property "Value" "DNI" (at 157.48 33.02 90)
+    (property "Value" "DNI" (at 154.94 35.56 90)
       (effects (font (size 1.27 1.27)))
     )
-    (property "Footprint" "Resistor_SMD:R_0603_1608Metric_Pad0.98x0.95mm_HandSolder" (at 157.48 33.782 90)
+    (property "Footprint" "Resistor_SMD:R_0603_1608Metric_Pad0.98x0.95mm_HandSolder" (at 155.702 35.56 90)
       (effects (font (size 1.27 1.27)) hide)
     )
@@
   )
   (symbol (lib_id "Device:R") (at 189.23 38.1 270) (unit 1)
-    (in_bom yes) (on_board yes) (dnp no)
+    (in_bom yes) (on_board yes) (dnp yes)
     (property "Reference" "R107" (at 187.96 33.02 90)
       (effects (font (size 1.27 1.27)))
