File: PWA_REV2/AlarmAudio.kicad_sch (KiCad schematic)
At the start: 14 parts, among them J1 DFPlayermini, J601 1X2P 1.27 mm Header, J602 0.100_2Pin

Commit message: Fixed the previous PWA_REV_2 file by added the changes of the USB UART. PCBa_krake is reverted to when no changes done to the schem.
Other:
- title: Krake Rev2 -> KRAKE_PCB
Changed lines of the file:
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@@
   (paper "A4")
   (title_block
-    (title "Krake Rev2")
-    (date "2025-07-16")
-    (rev "2.0")
+    (title "KRAKE_PCB")
+    (date "2024-11-23")
+    (rev "1.0")
     (company "PublicInvention")
     (comment 1 "GNU Affero General Public License v3.0")
@@
     (pin "1")
     (instances
-      (project "PWA_REV2"
+      (project "PCBa_KRAKE"
         (path "/412a327d-1ee3-473e-bc00-1545004b7edf/00000000-0000-0000-0000-000062dd8e5f"
           (reference "#PWR0606") (unit 1)
@@
     (pin "2")
     (instances
-      (project "PWA_REV2"
+      (project "PCBa_KRAKE"
         (path "/412a327d-1ee3-473e-bc00-1545004b7edf/00000000-0000-0000-0000-000062dd8e5f"
           (reference "R603") (unit 1)
@@
     (pin "2")
     (instances
-      (project "PWA_REV2"
+      (project "PCBa_KRAKE"
         (path "/412a327d-1ee3-473e-bc00-1545004b7edf/00000000-0000-0000-0000-000062dd8e5f"
           (reference "C602") (unit 1)
@@
     (pin "1")
     (instances
-      (project "PWA_REV2"
+      (project "PCBa_KRAKE"
         (path "/412a327d-1ee3-473e-bc00-1545004b7edf/00000000-0000-0000-0000-000062dd8e5f"
           (reference "#PWR0607") (unit 1)
@@
     (pin "1")
     (instances
-      (project "PWA_REV2"
+      (project "PCBa_KRAKE"
         (path "/412a327d-1ee3-473e-bc00-1545004b7edf"
           (reference "#FLG01") (unit 1)
@@
     (pin "2")
     (instances
-      (project "PWA_REV2"
+      (project "PCBa_KRAKE"
         (path "/412a327d-1ee3-473e-bc00-1545004b7edf/00000000-0000-0000-0000-000062dd8e5f"
           (reference "J601") (unit 1)
@@
     (pin "1")
     (instances
-      (project "PWA_REV2"
+      (project "PCBa_KRAKE"
         (path "/412a327d-1ee3-473e-bc00-1545004b7edf/00000000-0000-0000-0000-000062dd8e5f"
           (reference "#PWR0118") (unit 1)
@@
     (pin "2")
     (instances
-      (project "PWA_REV2"
+      (project "PCBa_KRAKE"
         (path "/412a327d-1ee3-473e-bc00-1545004b7edf/00000000-0000-0000-0000-000062bc4e7e"
           (reference "R502") (unit 1)
@@
     (pin "2")
     (instances
-      (project "PWA_REV2"
+      (project "PCBa_KRAKE"
         (path "/412a327d-1ee3-473e-bc00-1545004b7edf"
           (reference "R1") (unit 1)
@@
     (pin "1")
     (instances
-      (project "PWA_REV2"
+      (project "PCBa_KRAKE"
         (path "/412a327d-1ee3-473e-bc00-1545004b7edf"
           (reference "#PWR011") (unit 1)
@@
     (pin "2")
     (instances
-      (project "PWA_REV2"
+      (project "PCBa_KRAKE"
         (path "/412a327d-1ee3-473e-bc00-1545004b7edf"
           (reference "LS?") (unit 1)
@@
     (pin "1")
     (instances
-      (project "PWA_REV2"
+      (project "PCBa_KRAKE"
         (path "/412a327d-1ee3-473e-bc00-1545004b7edf"
           (reference "#PWR012") (unit 1)
@@
     (pin "2")
     (instances
-      (project "PWA_REV2"
+      (project "PCBa_KRAKE"
         (path "/412a327d-1ee3-473e-bc00-1545004b7edf/00000000-0000-0000-0000-000062bc4e7e"
           (reference "R503") (unit 1)
@@
     (pin "4")
     (instances
-      (project "PWA_REV2"
+      (project "PCBa_KRAKE"
         (path "/412a327d-1ee3-473e-bc00-1545004b7edf/00000000-0000-0000-0000-000062dd8e5f"
           (reference "S601") (unit 1)
@@
     (pin "2")
     (instances
-      (project "PWA_REV2"
+      (project "PCBa_KRAKE"
         (path "/412a327d-1ee3-473e-bc00-1545004b7edf"
           (reference "C4") (unit 1)
@@
     (pin "2")
     (instances
-      (project "PWA_REV2"
+      (project "PCBa_KRAKE"
         (path "/412a327d-1ee3-473e-bc00-1545004b7edf"
           (reference "C2") (unit 1)
@@
     (pin "2")
     (instances
-      (project "PWA_REV2"
+      (project "PCBa_KRAKE"
         (path "/412a327d-1ee3-473e-bc00-1545004b7edf/00000000-0000-0000-0000-000062dd8e5f"
           (reference "J602") (unit 1)
@@
     )
     (instances
-      (project "PWA_REV2"
+      (project "PCBa_KRAKE"
         (path "/412a327d-1ee3-473e-bc00-1545004b7edf/00000000-0000-0000-0000-000062dd8e5f"
           (reference "SD601") (unit 1)
@@
     (pin "2")
     (instances
-      (project "PWA_REV2"
+      (project "PCBa_KRAKE"
         (path "/412a327d-1ee3-473e-bc00-1545004b7edf/00000000-0000-0000-0000-000062bc4e7e"
           (reference "R502") (unit 1)
@@
     (pin "1")
     (instances
-      (project "PWA_REV2"
+      (project "PCBa_KRAKE"
         (path "/412a327d-1ee3-473e-bc00-1545004b7edf"
           (reference "#PWR08") (unit 1)
@@
     (pin "1")
     (instances
-      (project "PWA_REV2"
+      (project "PCBa_KRAKE"
         (path "/412a327d-1ee3-473e-bc00-1545004b7edf"
           (reference "#PWR016") (unit 1)
@@
     (pin "1")
     (instances
-      (project "PWA_REV2"
+      (project "PCBa_KRAKE"
         (path "/412a327d-1ee3-473e-bc00-1545004b7edf"
           (reference "#PWR07") (unit 1)
@@
     (pin "8")
     (instances
-      (project "PWA_REV2"
+      (project "PCBa_KRAKE"
         (path "/412a327d-1ee3-473e-bc00-1545004b7edf"
           (reference "J1") (unit 1)

Commit message: PWA_REV2.kicad, Adding test points for the decoupling 5v resistors.
Parts:
- added TP?: 5VDFP, TestPoint:TestPoint_Loop_D2.54mm_Drill1.5mm_Beaded, symbol Connector:TestPoint
Connections:
- net 5VDFP: now also TP?.1
Other:
- note added: "Bypass capacitors"
- note added: "Decoupling Resistor"
Changed lines of the file:
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@@
   (junction (at 78.74 81.28) (diameter 0) (color 0 0 0 0)
+  )
+  (junction (at 218.44 67.31) (diameter 0) (color 0 0 0 0)
   )
   (no_connect (at 175.26 135.89))
@@
     (stroke (width 0) (type default))
   )
+  (wire (pts (xy 218.44 67.31) (xy 220.98 67.31))
+    (stroke (width 0) (type default))
+  )
   (wire (pts (xy 66.04 97.79) (xy 66.04 100.33))
     (stroke (width 0) (type default))
@@
     (stroke (width 0) (type default))
   )
-  (wire (pts (xy 212.09 71.12) (xy 217.17 71.12))
+  (wire (pts (xy 212.09 71.12) (xy 220.98 71.12))
     (stroke (width 0) (type default))
   )
@@
     (stroke (width 0) (type default))
   )
-  (wire (pts (xy 217.17 71.12) (xy 217.17 67.31))
+  (wire (pts (xy 220.98 71.12) (xy 220.98 67.31))
     (stroke (width 0) (type default))
   )
@@
     (stroke (width 0) (type default))
   )
-  (wire (pts (xy 213.36 67.31) (xy 217.17 67.31))
+  (wire (pts (xy 213.36 67.31) (xy 218.44 67.31))
     (stroke (width 0) (type default))
   )
@@
   )
   (wire (pts (xy 198.12 82.55) (xy 198.12 80.01))
+    (stroke (width 0) (type default))
+  )
+  (wire (pts (xy 218.44 58.42) (xy 218.44 67.31))
     (stroke (width 0) (type default))
   )
@@
     (effects (font (size 1.27 1.27)) (justify right bottom))
   )
+  (text "Bypass capacitors" (at 215.9 82.55 0)
+    (effects (font (size 1.27 1.27)) (justify left bottom))
+  )
+  (text "Decoupling Resistor " (at 189.23 60.96 0)
+    (effects (font (size 1.27 1.27)) (justify left bottom))
+  )
   (text "MP3 file are added on this card for DFplayer" (at 73.66 162.56 0)
     (effects (font (size 2.54 2.54)) (justify left bottom))
   )
-  (label "5VDFP" (at 217.17 68.58 0) (fields_autoplaced)
+  (label "5VDFP" (at 220.98 68.58 0) (fields_autoplaced)
     (effects (font (size 1.27 1.27)) (justify left bottom))
   )
@@
       (effects (font (size 1.27 1.27)) hide)
     )
-    (property "Value" "PWR_FLAG" (at 213.36 61.6458 0)
+    (property "Value" "PWR_FLAG" (at 212.09 62.23 0)
       (effects (font (size 1.27 1.27)))
     )
@@
   (symbol (lib_id "Device:R") (at 205.74 67.31 270) (unit 1)
     (in_bom yes) (on_board yes) (dnp no)
-    (property "Reference" "R1" (at 204.47 62.23 90)
+    (property "Reference" "R1" (at 203.2 62.23 90)
       (effects (font (size 1.27 1.27)))
     )
@@
         )
       )
+    )
+  )
+  (symbol (lib_id "Connector:TestPoint") (at 218.44 58.42 0) (unit 1)
+    (in_bom yes) (on_board yes) (dnp no)
+    (property "Reference" "TP?" (at 208.28 50.8 0)
+      (effects (font (size 1.27 1.27)) (justify left))
+    )
+    (property "Value" "5VDFP" (at 208.28 53.34 0)
+      (effects (font (size 1.27 1.27)) (justify left))
+    )
+    (property "Footprint" "TestPoint:TestPoint_Loop_D2.54mm_Drill1.5mm_Beaded" (at 223.52 58.42 0)
+      (effects (font (size 1.27 1.27)) hide)
+    )
+    (property "Datasheet" "~" (at 223.52 58.42 0)
+      (effects (font (size 1.27 1.27)) hide)
+    )
+    (property "AssemblyType" "HAND" (at 218.44 58.42 0)
+      (effects (font (size 1.27 1.27)) hide)
+    )
+    (property "Description" "Test Points/Test Rings ROHS red" (at 218.44 58.42 0)
+      (effects (font (size 1.27 1.27)) hide)
+    )
+    (property "Distributor 1" "JLCPCB" (at 218.44 58.42 0)
+      (effects (font (size 1.27 1.27)) hide)
+    )
+    (property "Distributor 1 PN" "C5277086" (at 218.44 58.42 0)
+      (effects (font (size 1.27 1.27)) hide)
+    )
+    (property "MPN" "RH-5000" (at 218.44 58.42 0)
+      (effects (font (size 1.27 1.27)) hide)
+    )
+    (property "Manufacturer" "ronghe" (at 218.44 58.42 0)
+      (effects (font (size 1.27 1.27)) hide)
+    )
+    (property "Cost" "0.0717" (at 218.44 58.42 0)
+      (effects (font (size 1.27 1.27)) hide)
+    )
+    (property "MPN 2" "" (at 218.44 58.42 0)
+      (effects (font (size 1.27 1.27)) hide)
+    )
+    (property "Manufacturer 2" "" (at 218.44 58.42 0)
+      (effects (font (size 1.27 1.27)) hide)
+    )
+    (pin "1")
+    (instances
+      (project "PWA_REV2"
+        (path "/412a327d-1ee3-473e-bc00-1545004b7edf"
+          (reference "TP?") (unit 1)
+        )
+        (path "/412a327d-1ee3-473e-bc00-1545004b7edf/00000000-0000-0000-0000-000062dd8e5f"
+          (reference "TP?") (unit 1)
+        )
+      )

Commit message: AlarmAudio.kicad_sch, issue 176, Adding a 2mm JST 2pin header speaker connector.
Parts:
- added J603: 2mm_2Pin, Connector_JST:JST_PH_B2B-PH-K_1x02_P2.00mm_Vertical, symbol GPAD_SCH_LIB:22-23-2021
- J601: value 1X2P 1.27 mm Header -> 1X2P 1.25 mm Header; footprint Connector_PinHeader_1.27mm:PinHeader_1x02_P1.27mm_Vertical -> Connector_Molex:Molex_PicoBlade_53047-0210_1x02_P1.25mm_Vertical; Distributor 1 PN C7496728 -> C114130; MPN PZ150V-02P -> 530470210; Manufacturer XFCN -> MOLEX
Connections:
- net at J1.8 (SPK_2), J601.1: now also J603.1
- net at J1.6 (SPK_1), J601.2: now also J603.2
Changed lines of the file:
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@@
   (junction (at 68.58 81.28) (diameter 0) (color 0 0 0 0)
   )
+  (junction (at 182.88 128.27) (diameter 0) (color 0 0 0 0)
+  )
   (junction (at 85.09 81.28) (diameter 0) (color 0 0 0 0)
+  )
+  (junction (at 186.69 130.81) (diameter 0) (color 0 0 0 0)
   )
   (junction (at 212.09 71.12) (diameter 0) (color 0 0 0 0)
@@
     (stroke (width 0) (type default))
   )
-  (wire (pts (xy 180.34 130.81) (xy 187.96 130.81))
+  (wire (pts (xy 182.88 135.89) (xy 182.88 128.27))
+    (stroke (width 0) (type default))
+  )
+  (wire (pts (xy 187.96 135.89) (xy 182.88 135.89))
+    (stroke (width 0) (type default))
+  )
+  (wire (pts (xy 180.34 130.81) (xy 186.69 130.81))
     (stroke (width 0) (type default))
   )
@@
   )
   (wire (pts (xy 212.09 72.39) (xy 212.09 71.12))
+    (stroke (width 0) (type default))
+  )
+  (wire (pts (xy 186.69 133.35) (xy 186.69 130.81))
+    (stroke (width 0) (type default))
+  )
+  (wire (pts (xy 186.69 130.81) (xy 187.96 130.81))
+    (stroke (width 0) (type default))
+  )
+  (wire (pts (xy 187.96 133.35) (xy 186.69 133.35))
     (stroke (width 0) (type default))
   )
@@
     )
   )
-  (symbol (lib_id "power:PWR_FLAG") (at 213.36 66.04 0) (unit 1)
-    (in_bom yes) (on_board yes) (dnp no)
-    (property "Reference" "#FLG01" (at 213.36 64.135 0)
-      (effects (font (size 1.27 1.27)) hide)
-    )
-    (property "Value" "PWR_FLAG" (at 212.09 62.23 0)
-      (effects (font (size 1.27 1.27)))
-    )
-    (property "Footprint" "" (at 213.36 66.04 0)
-      (effects (font (size 1.27 1.27)) hide)
-    )
-    (property "Datasheet" "~" (at 213.36 66.04 0)
-      (effects (font (size 1.27 1.27)) hide)
-    )
-    (pin "1")
-    (instances
-      (project "PWA_REV2"
-        (path "/412a327d-1ee3-473e-bc00-1545004b7edf"
-          (reference "#FLG01") (unit 1)
-        )
-        (path "/412a327d-1ee3-473e-bc00-1545004b7edf/00000000-0000-0000-0000-000062dd8e5f"
-          (reference "#FLG02") (unit 1)
-        )
-      )
-    )
-  )
   (symbol (lib_id "GPAD_SCH_LIB:22-23-2021") (at 177.8 130.81 270) (mirror x) (unit 1)
     (in_bom yes) (on_board yes) (dnp no)
@@
       (effects (font (size 1.27 1.27)) (justify right))
     )
-    (property "Value" "1X2P 1.27 mm Header" (at 181.61 124.46 90)
+    (property "Value" "1X2P 1.25 mm Header" (at 181.61 124.46 90)
       (effects (font (size 1.27 1.27)) (justify right))
     )
-    (property "Footprint" "Connector_PinHeader_1.27mm:PinHeader_1x02_P1.27mm_Vertical" (at 182.88 125.73 0)
+    (property "Footprint" "Connector_Molex:Molex_PicoBlade_53047-0210_1x02_P1.25mm_Vertical" (at 182.88 125.73 0)
       (effects (font (size 1.524 1.524)) (justify left) hide)
     )
@@
       (effects (font (size 1.524 1.524)) (justify left) hide)
     )
-    (property "MPN" "PZ150V-02P" (at 190.5 125.73 0)
+    (property "MPN" "530470210" (at 190.5 125.73 0)
       (effects (font (size 1.524 1.524)) (justify left) hide)
     )
@@
       (effects (font (size 1.524 1.524)) (justify left) hide)
     )
-    (property "Description" "Direct Insert 2P 1.5mm Single Row 1x2P Plugin,P=1.5mm Pin Headers ROHS" (at 203.2 125.73 0)
-      (effects (font (size 1.524 1.524)) (justify left) hide)
-    )
-    (property "Manufacturer" "XFCN" (at 205.74 125.73 0)
+    (property "Description" "1.25mm 1x2P 2 2P 3.2mm 4.25mm 4.2mm PA Phosphor Bronze PicoBlade(MX 1.25) " (at 203.2 125.73 0)
+      (effects (font (size 1.524 1.524)) (justify left) hide)
+    )
+    (property "Manufacturer" "MOLEX" (at 205.74 125.73 0)
       (effects (font (size 1.524 1.524)) (justify left) hide)
     )
@@
       (effects (font (size 1.27 1.27)) hide)
     )
-    (property "Distributor 1 PN" "C7496728" (at 177.8 130.81 0)
+    (property "Distributor 1 PN" "C114130" (at 177.8 130.81 0)
       (effects (font (size 1.27 1.27)) hide)
     )
@@
         (path "/412a327d-1ee3-473e-bc00-1545004b7edf"
           (reference "J?") (unit 1)
+        )
+      )
+    )
+  )
+  (symbol (lib_id "power:PWR_FLAG") (at 213.36 66.04 0) (unit 1)
+    (in_bom yes) (on_board yes) (dnp no)
+    (property "Reference" "#FLG01" (at 213.36 64.135 0)
+      (effects (font (size 1.27 1.27)) hide)
+    )
+    (property "Value" "PWR_FLAG" (at 212.09 62.23 0)
+      (effects (font (size 1.27 1.27)))
+    )
+    (property "Footprint" "" (at 213.36 66.04 0)
+      (effects (font (size 1.27 1.27)) hide)
+    )
+    (property "Datasheet" "~" (at 213.36 66.04 0)
+      (effects (font (size 1.27 1.27)) hide)
+    )
+    (pin "1")
+    (instances
+      (project "PWA_REV2"
+        (path "/412a327d-1ee3-473e-bc00-1545004b7edf"
+          (reference "#FLG01") (unit 1)
+        )
+        (path "/412a327d-1ee3-473e-bc00-1545004b7edf/00000000-0000-0000-0000-000062dd8e5f"
+          (reference "#FLG02") (unit 1)
         )
       )
@@
         )
       )
+    )
+  )
+  (symbol (lib_id "GPAD_SCH_LIB:22-23-2021") (at 190.5 133.35 90) (mirror x) (unit 1)
+    (in_bom yes) (on_board yes) (dnp no)
+    (property "Reference" "J603" (at 194.31 130.81 90)
+      (effects (font (size 1.27 1.27)) (justify right))
+    )
+    (property "Value" "2mm_2Pin" (at 186.69 139.7 90)
+      (effects (font (size 1.27 1.27)) (justify right))
+    )
+    (property "Footprint" "Connector_JST:JST_PH_B2B-PH-K_1x02_P2.00mm_Vertical" (at 185.42 138.43 0)
+      (effects (font (size 1.524 1.524)) (justify left) hide)
+    )
+    (property "Datasheet" "https://jlcpcb.com/api/file/downloadByFileSystemAccessId/8588889744620572672" (at 182.88 138.43 0)
+      (effects (font (size 1.524 1.524)) (justify left) hide)
+    )
+    (property "Digi-Key_PN" "B2B-PH-K-S" (at 180.34 138.43 0)
+      (effects (font (size 1.524 1.524)) (justify left) hide)
+    )
+    (property "MPN" "B2B-PH-K-S(LF)(SN)" (at 177.8 138.43 0)
+      (effects (font (size 1.524 1.524)) (justify left) hide)
+    )
+    (property "Category" "Connectors, Interconnects" (at 175.26 138.43 0)
+      (effects (font (size 1.524 1.524)) (justify left) hide)
+    )
+    (property "Description" "HEADER VERT 2POS 2MM" (at 165.1 138.43 0)
+      (effects (font (size 1.524 1.524)) (justify left) hide)
+    )
+    (property "Manufacturer" "JST" (at 162.56 138.43 0)
+      (effects (font (size 1.524 1.524)) (justify left) hide)
+    )
+    (property "Status" "Active" (at 160.02 138.43 0)
+      (effects (font (size 1.524 1.524)) (justify left) hide)
+    )
+    (property "Cost" "0.0306" (at 190.5 133.35 0)
+      (effects (font (size 1.27 1.27)) hide)
+    )
+    (property "Distributor 1" "JLCPCB" (at 190.5 133.35 0)
+      (effects (font (size 1.27 1.27)) hide)
+    )
+    (property "Distributor 1 PN" "C131337" (at 190.5 133.35 0)
+      (effects (font (size 1.27 1.27)) hide)
+    )
+    (property "MPN 2" "" (at 190.5 133.35 0)
+      (effects (font (size 1.27 1.27)) hide)
+    )
+    (property "Manufacturer 2" "" (at 190.5 133.35 0)
+      (effects (font (size 1.27 1.27)) hide)
+    )
+    (pin "1")
+    (pin "2")
+    (instances
+      (project "PWA_REV2"
+        (path "/412a327d-1ee3-473e-bc00-1545004b7edf/00000000-0000-0000-0000-000062dd8e5f"
+          (reference "J603") (unit 1)
+        )
+      )

Commit message: AlarmAudio.kicad_sch, Renamed j603 to clear duplicate ERC error.
Parts:
- renumbered J603 to J604
Changed lines of the file:
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@@
   (symbol (lib_id "GPAD_SCH_LIB:22-23-2021") (at 190.5 133.35 90) (mirror x) (unit 1)
     (in_bom yes) (on_board yes) (dnp no)
-    (property "Reference" "J603" (at 194.31 130.81 90)
+    (property "Reference" "J604" (at 194.31 130.81 90)
       (effects (font (size 1.27 1.27)) (justify right))
     )
@@
       (project "PWA_REV2"
         (path "/412a327d-1ee3-473e-bc00-1545004b7edf/00000000-0000-0000-0000-000062dd8e5f"
-          (reference "J603") (unit 1)
+          (reference "J604") (unit 1)
         )
       )
