File: PWA_REV2/AlarmAudio.kicad_sch (KiCad schematic)
At the start: 16 parts, among them J1 DFPlayermini, J601 1X2P 1.25 mm Header, J602 0.100_2Pin, J604 2mm_2Pin

Commit message: PWA_REV2, Corrected test points footprints.
Parts:
- TP?: footprint TestPoint:TestPoint_Loop_D2.54mm_Drill1.5mm_Beaded -> TestPoint:TestPoint_Loop_D1.80mm_Drill1.0mm_Beaded
Changed lines of the file:
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@@
       (effects (font (size 1.27 1.27)) (justify left))
     )
-    (property "Footprint" "TestPoint:TestPoint_Loop_D2.54mm_Drill1.5mm_Beaded" (at 223.52 58.42 0)
+    (property "Footprint" "TestPoint:TestPoint_Loop_D1.80mm_Drill1.0mm_Beaded" (at 223.52 58.42 0)
       (effects (font (size 1.27 1.27)) hide)
     )

Commit message: PWA_REV2, solved issue 239, added functionality discription to D106, and similarly we corrected Schematic and PCB text for MENU BOOT RESET MUTE CONTRAST POWER.
Other:
- note added: "MUTE"
Changed lines of the file:
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@@
     (effects (font (size 1.27 1.27)) (justify left bottom))
+  )
+  (text "MUTE" (at 86.36 91.44 0)
+    (effects (font (size 2.54 2.54)) (justify left bottom))
   )
   (text "Place R503 near uControler TX pin." (at 128.905 108.585 0)
@@
   )
   (symbol (lib_id "GPAD_SCH_LIB:SWITCH_TACTILE_12mmx12mm_SPST-NO_0.05A_24V") (at 92.71 83.82 0) (unit 1)
-    (in_bom yes) (on_board yes) (dnp no) (fields_autoplaced)
+    (in_bom yes) (on_board yes) (dnp no)
     (property "Reference" "S601" (at 92.71 74.93 0)
       (effects (font (size 1.524 1.524)))

Commit message: PWA_REV2, resolved issue 255, added several 3d models.
Parts:
- J601: footprint Connector_Molex:Molex_PicoBlade_53047-0210_1x02_P1.25mm_Vertical -> GeneralPurposeAlarmDevicePCB:Molex_PicoBlade_53047-0210_1x02_P1.25mm_Vertical
Changed lines of the file:
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@@
       (effects (font (size 1.27 1.27)) (justify right))
     )
-    (property "Footprint" "Connector_Molex:Molex_PicoBlade_53047-0210_1x02_P1.25mm_Vertical" (at 182.88 125.73 0)
+    (property "Footprint" "GeneralPurposeAlarmDevicePCB:Molex_PicoBlade_53047-0210_1x02_P1.25mm_Vertical" (at 182.88 125.73 0)
       (effects (font (size 1.524 1.524)) (justify left) hide)
     )
