File: PWA_REV2/AlarmAudio.kicad_sch (KiCad schematic)
At the start: 16 parts, among them J1 DFPlayermini, J601 1X2P 1.25 mm Header, J602 0.100_2Pin, J604 2mm_2Pin

Commit message: PWA_REV2, We corrected Assembly Type for some components, and we added the JLCPCB PN for the DB9 and the CH340B.
Parts:
- J604: AssemblyType (none) -> HAND
Changed lines of the file:
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@@
+      (effects (font (size 1.27 1.27)) hide)
+    )
+    (property "AssemblyType" "HAND" (at 190.5 133.35 0)
       (effects (font (size 1.27 1.27)) hide)
     )

Commit message: Adding files to preserve while fixing merge conflicts.
Parts:
- S601: value SWITCH_TACTILE_12mmx12mm_SPST-NO_0.05A_24V -> SWITCH_TACTILE_Projected_12mmx12mm_7.3mm_SPST-NO_0.05A_24V
Changed lines of the file:
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@@
       (effects (font (size 1.524 1.524)))
     )
-    (property "Value" "SWITCH_TACTILE_12mmx12mm_SPST-NO_0.05A_24V" (at 92.71 78.74 0)
+    (property "Value" " SWITCH_TACTILE_Projected_12mmx12mm_7.3mm_SPST-NO_0.05A_24V" (at 92.71 78.74 0)
       (effects (font (size 1.524 1.524)))
     )
@@
       (effects (font (size 1.524 1.524)) (justify left) hide)
     )
-    (property "Datasheet" "" (at 97.79 76.2 0)
+    (property "Datasheet" "https://eu.mouser.com/datasheet/3/39/1/en-b3f.pdf" (at 97.79 76.2 0)
       (effects (font (size 1.524 1.524)) (justify left) hide)
     )
@@
       (effects (font (size 1.524 1.524)) (justify left) hide)
     )
-    (property "Description" "SWITCH_TACTILE_12mmx12mm_SPST-NO_0.05A_24V" (at 97.79 58.42 0)
+    (property "Description" " SWITCH_TACTILE_Projected_12mmx12mm_7.3mm_SPST-NO_0.05A_24V" (at 97.79 58.42 0)
       (effects (font (size 1.524 1.524)) (justify left) hide)
     )

Commit message: PWA_REV2/PWA_REV2.kicad_pcb, Update for the actualy Mute key cap. Fixed MAX3232 part number.
Parts:
- S601: footprint GeneralPurposeAlarmDevicePCB:SW_PUSH-12mm_WithCap_Green -> GeneralPurposeAlarmDevicePCB:SW_PUSH-12mm_WithGPAD_KeyCap
Changed lines of the file:
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@@
       (effects (font (size 1.524 1.524)))
     )
-    (property "Footprint" "GeneralPurposeAlarmDevicePCB:SW_PUSH-12mm_WithCap_Green" (at 97.79 78.74 0)
+    (property "Footprint" "GeneralPurposeAlarmDevicePCB:SW_PUSH-12mm_WithGPAD_KeyCap" (at 97.79 78.74 0)
       (effects (font (size 1.524 1.524)) (justify left) hide)
     )

Commit message: Hardware, PWA, Add a Jumper to BOM for J102 so that USB Connector Can Power Krake, issue 312.
:q
q
Parts:
- S601: value SWITCH_TACTILE_Projected_12mmx12mm_7.3mm_SPST-NO_0.05A_24V -> SWITCH_TACTILE_Projected_12mmx12mm_7.3mm_SPST-NO_0.05A_24V
- gave numbers to parts that had none: 2
- renumbered C2 to C504, C4 to C505, J1 to J603, R503 to R509, R502 to R510, R502 to R511, R1 to R512

Commit message: Revert "Hardware, PWA, Add a Jumper to BOM for J102 so that USB Connector Can Power Krake, issue 312."
This reverts commit c2819b8ee4999f733f52d823f88f6aefd6456fcc.
Parts:
- S601: value SWITCH_TACTILE_Projected_12mmx12mm_7.3mm_SPST-NO_0.05A_24V -> SWITCH_TACTILE_Projected_12mmx12mm_7.3mm_SPST-NO_0.05A_24V
- renumbered C504 to C2, C505 to C4, J603 to J1, BZ601 to LS?, R512 to R1, R510 to R502, R511 to R502, R509 to R503, TP501 to TP?
