File: PWA_REV2/AlarmLights5.kicad_sch (KiCad schematic)
At the start: 25 parts, among them Q201 MMBT2222A-7-F, Q202 MMBT2222A-7-F, Q203 MMBT2222A-7-F, Q204 MMBT2222A-7-F, Q205 MMBT2222A-7-F

Commit message: Fixed the previous PWA_REV_2 file by added the changes of the USB UART. PCBa_krake is reverted to when no changes done to the schem.
Other:
- title: Krake Rev2 -> KRAKE_PCB
Changed lines of the file:
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@@
   (paper "A4")
   (title_block
-    (title "Krake Rev2")
-    (date "2025-07-16")
-    (rev "2.0")
+    (title "KRAKE_PCB")
+    (date "2024-11-23")
+    (rev "1.0")
     (company "PublicInvention")
     (comment 1 "GNU Affero General Public License v3.0")
@@
     (pin "2")
     (instances
-      (project "PWA_REV2"
+      (project "PCBa_KRAKE"
         (path "/412a327d-1ee3-473e-bc00-1545004b7edf/00000000-0000-0000-0000-000062b3ac2f"
           (reference "R201") (unit 1)
@@
     (pin "1")
     (instances
-      (project "PWA_REV2"
+      (project "PCBa_KRAKE"
         (path "/412a327d-1ee3-473e-bc00-1545004b7edf/00000000-0000-0000-0000-000062b3ac2f"
           (reference "#PWR0202") (unit 1)
@@
     (pin "2")
     (instances
-      (project "PWA_REV2"
+      (project "PCBa_KRAKE"
         (path "/412a327d-1ee3-473e-bc00-1545004b7edf/00000000-0000-0000-0000-000062b3ac2f"
           (reference "R202") (unit 1)
@@
     (pin "2")
     (instances
-      (project "PWA_REV2"
+      (project "PCBa_KRAKE"
         (path "/412a327d-1ee3-473e-bc00-1545004b7edf/00000000-0000-0000-0000-000062b3ac2f"
           (reference "R203") (unit 1)
@@
     (pin "1")
     (instances
-      (project "PWA_REV2"
+      (project "PCBa_KRAKE"
         (path "/412a327d-1ee3-473e-bc00-1545004b7edf/00000000-0000-0000-0000-000062b3ac2f"
           (reference "#PWR0203") (unit 1)
@@
     (pin "2")
     (instances
-      (project "PWA_REV2"
+      (project "PCBa_KRAKE"
         (path "/412a327d-1ee3-473e-bc00-1545004b7edf/00000000-0000-0000-0000-000062b3ac2f"
           (reference "R204") (unit 1)
@@
     (pin "2")
     (instances
-      (project "PWA_REV2"
+      (project "PCBa_KRAKE"
         (path "/412a327d-1ee3-473e-bc00-1545004b7edf/00000000-0000-0000-0000-000062b3ac2f"
           (reference "R205") (unit 1)
@@
     (pin "1")
     (instances
-      (project "PWA_REV2"
+      (project "PCBa_KRAKE"
         (path "/412a327d-1ee3-473e-bc00-1545004b7edf/00000000-0000-0000-0000-000062b3ac2f"
           (reference "#PWR0204") (unit 1)
@@
     (pin "2")
     (instances
-      (project "PWA_REV2"
+      (project "PCBa_KRAKE"
         (path "/412a327d-1ee3-473e-bc00-1545004b7edf/00000000-0000-0000-0000-000062b3ac2f"
           (reference "R206") (unit 1)
@@
     (pin "2")
     (instances
-      (project "PWA_REV2"
+      (project "PCBa_KRAKE"
         (path "/412a327d-1ee3-473e-bc00-1545004b7edf/00000000-0000-0000-0000-000062b3ac2f"
           (reference "R207") (unit 1)
@@
     (pin "1")
     (instances
-      (project "PWA_REV2"
+      (project "PCBa_KRAKE"
         (path "/412a327d-1ee3-473e-bc00-1545004b7edf/00000000-0000-0000-0000-000062b3ac2f"
           (reference "#PWR0205") (unit 1)
@@
     (pin "2")
     (instances
-      (project "PWA_REV2"
+      (project "PCBa_KRAKE"
         (path "/412a327d-1ee3-473e-bc00-1545004b7edf/00000000-0000-0000-0000-000062b3ac2f"
           (reference "R208") (unit 1)
@@
     (pin "2")
     (instances
-      (project "PWA_REV2"
+      (project "PCBa_KRAKE"
         (path "/412a327d-1ee3-473e-bc00-1545004b7edf/00000000-0000-0000-0000-000062b3ac2f"
           (reference "R209") (unit 1)
@@
     (pin "1")
     (instances
-      (project "PWA_REV2"
+      (project "PCBa_KRAKE"
         (path "/412a327d-1ee3-473e-bc00-1545004b7edf/00000000-0000-0000-0000-000062b3ac2f"
           (reference "#PWR0206") (unit 1)
@@
     (pin "2")
     (instances
-      (project "PWA_REV2"
+      (project "PCBa_KRAKE"
         (path "/412a327d-1ee3-473e-bc00-1545004b7edf/00000000-0000-0000-0000-000062b3ac2f"
           (reference "R210") (unit 1)
@@
     (pin "2")
     (instances
-      (project "PWA_REV2"
+      (project "PCBa_KRAKE"
         (path "/412a327d-1ee3-473e-bc00-1545004b7edf/00000000-0000-0000-0000-000062b3ac2f"
           (reference "D202") (unit 1)
@@
     (pin "2")
     (instances
-      (project "PWA_REV2"
+      (project "PCBa_KRAKE"
         (path "/412a327d-1ee3-473e-bc00-1545004b7edf/00000000-0000-0000-0000-000062b3ac2f"
           (reference "D203") (unit 1)
@@
     (pin "2")
     (instances
-      (project "PWA_REV2"
+      (project "PCBa_KRAKE"
         (path "/412a327d-1ee3-473e-bc00-1545004b7edf/00000000-0000-0000-0000-000062b3ac2f"
           (reference "D204") (unit 1)
@@
     (pin "2")
     (instances
-      (project "PWA_REV2"
+      (project "PCBa_KRAKE"
         (path "/412a327d-1ee3-473e-bc00-1545004b7edf/00000000-0000-0000-0000-000062b3ac2f"
           (reference "D205") (unit 1)
@@
     (pin "2")
     (instances
-      (project "PWA_REV2"
+      (project "PCBa_KRAKE"
         (path "/412a327d-1ee3-473e-bc00-1545004b7edf/00000000-0000-0000-0000-000062b3ac2f"
           (reference "D201") (unit 1)
@@
     (pin "1")
     (instances
-      (project "PWA_REV2"
+      (project "PCBa_KRAKE"
         (path "/412a327d-1ee3-473e-bc00-1545004b7edf/00000000-0000-0000-0000-000062b3ac2f"
           (reference "#PWR0201") (unit 1)
@@
     (pin "3")
     (instances
-      (project "PWA_REV2"
+      (project "PCBa_KRAKE"
         (path "/412a327d-1ee3-473e-bc00-1545004b7edf/00000000-0000-0000-0000-000062b3ac2f"
           (reference "Q201") (unit 1)
@@
     (pin "3")
     (instances
-      (project "PWA_REV2"
+      (project "PCBa_KRAKE"
         (path "/412a327d-1ee3-473e-bc00-1545004b7edf/00000000-0000-0000-0000-000062b3ac2f"
           (reference "Q205") (unit 1)
@@
     (pin "3")
     (instances
-      (project "PWA_REV2"
+      (project "PCBa_KRAKE"
         (path "/412a327d-1ee3-473e-bc00-1545004b7edf/00000000-0000-0000-0000-000062b3ac2f"
           (reference "Q204") (unit 1)
@@
     (pin "3")
     (instances
-      (project "PWA_REV2"
+      (project "PCBa_KRAKE"
         (path "/412a327d-1ee3-473e-bc00-1545004b7edf/00000000-0000-0000-0000-000062b3ac2f"
           (reference "Q203") (unit 1)
@@
     (pin "3")
     (instances
-      (project "PWA_REV2"
+      (project "PCBa_KRAKE"
         (path "/412a327d-1ee3-473e-bc00-1545004b7edf/00000000-0000-0000-0000-000062b3ac2f"
           (reference "Q202") (unit 1)
@@
     )
     (instances
-      (project "PWA_REV2"
+      (project "PCBa_KRAKE"
         (path "/412a327d-1ee3-473e-bc00-1545004b7edf/00000000-0000-0000-0000-000062b3ac2f"
           (reference "MF605") (unit 1)
@@
     )
     (instances
-      (project "PWA_REV2"
+      (project "PCBa_KRAKE"
         (path "/412a327d-1ee3-473e-bc00-1545004b7edf/00000000-0000-0000-0000-000062b3ac2f"
           (reference "MF604") (unit 1)
@@
     )
     (instances
-      (project "PWA_REV2"
+      (project "PCBa_KRAKE"
         (path "/412a327d-1ee3-473e-bc00-1545004b7edf/00000000-0000-0000-0000-000062b3ac2f"
           (reference "MF603") (unit 1)
@@
     )
     (instances
-      (project "PWA_REV2"
+      (project "PCBa_KRAKE"
         (path "/412a327d-1ee3-473e-bc00-1545004b7edf/00000000-0000-0000-0000-000062b3ac2f"
           (reference "MF602") (unit 1)
@@
     )
     (instances
-      (project "PWA_REV2"
+      (project "PCBa_KRAKE"
         (path "/412a327d-1ee3-473e-bc00-1545004b7edf/00000000-0000-0000-0000-000062b3ac2f"
           (reference "MF601") (unit 1)
