File: PWA_REV2/RS232.kicad_sch (KiCad schematic)
At the start: 19 parts

Commit message: Fixed the previous PWA_REV_2 file by added the changes of the USB UART. PCBa_krake is reverted to when no changes done to the schem.
Other:
- title: Krake Rev2 -> KRAKE_PCB
Changed lines of the file:
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@@
   (paper "A4")
   (title_block
-    (title "Krake Rev2")
-    (date "2025-07-16")
-    (rev "2.0")
+    (title "KRAKE_PCB")
+    (date "2024-11-23")
+    (rev "1.0")
     (company "PublicInvention")
     (comment 1 "GNU Affero General Public License v3.0")
@@
     (pin "1")
     (instances
-      (project "PWA_REV2"
+      (project "PCBa_KRAKE"
         (path "/412a327d-1ee3-473e-bc00-1545004b7edf"
           (reference "#PWR028") (unit 1)
@@
     (pin "2")
     (instances
-      (project "PWA_REV2"
+      (project "PCBa_KRAKE"
         (path "/412a327d-1ee3-473e-bc00-1545004b7edf/00000000-0000-0000-0000-000062bc4e7e"
           (reference "R503") (unit 1)
@@
     (pin "9")
     (instances
-      (project "PWA_REV2"
+      (project "PCBa_KRAKE"
         (path "/412a327d-1ee3-473e-bc00-1545004b7edf"
           (reference "J?") (unit 1)
@@
     (pin "1")
     (instances
-      (project "PWA_REV2"
+      (project "PCBa_KRAKE"
         (path "/412a327d-1ee3-473e-bc00-1545004b7edf"
           (reference "#PWR031") (unit 1)
@@
     (pin "9")
     (instances
-      (project "PWA_REV2"
+      (project "PCBa_KRAKE"
         (path "/412a327d-1ee3-473e-bc00-1545004b7edf"
           (reference "U?") (unit 1)
@@
     (pin "2")
     (instances
-      (project "PWA_REV2"
+      (project "PCBa_KRAKE"
         (path "/412a327d-1ee3-473e-bc00-1545004b7edf/00000000-0000-0000-0000-000062bc4e7e"
           (reference "R503") (unit 1)
@@
     (pin "1")
     (instances
-      (project "PWA_REV2"
+      (project "PCBa_KRAKE"
         (path "/412a327d-1ee3-473e-bc00-1545004b7edf"
           (reference "#PWR032") (unit 1)
@@
     (pin "2")
     (instances
-      (project "PWA_REV2"
+      (project "PCBa_KRAKE"
         (path "/412a327d-1ee3-473e-bc00-1545004b7edf"
           (reference "C?") (unit 1)
@@
     (pin "1")
     (instances
-      (project "PWA_REV2"
+      (project "PCBa_KRAKE"
         (path "/412a327d-1ee3-473e-bc00-1545004b7edf"
           (reference "#FLG03") (unit 1)
@@
     (pin "2")
     (instances
-      (project "PWA_REV2"
+      (project "PCBa_KRAKE"
         (path "/412a327d-1ee3-473e-bc00-1545004b7edf/00000000-0000-0000-0000-000062bc4e7e"
           (reference "R503") (unit 1)
@@
     (pin "2")
     (instances
-      (project "PWA_REV2"
+      (project "PCBa_KRAKE"
         (path "/412a327d-1ee3-473e-bc00-1545004b7edf"
           (reference "C?") (unit 1)
@@
     (pin "2")
     (instances
-      (project "PWA_REV2"
+      (project "PCBa_KRAKE"
         (path "/412a327d-1ee3-473e-bc00-1545004b7edf/00000000-0000-0000-0000-000062bc4e7e"
           (reference "R503") (unit 1)
@@
     (pin "2")
     (instances
-      (project "PWA_REV2"
+      (project "PCBa_KRAKE"
         (path "/412a327d-1ee3-473e-bc00-1545004b7edf"
           (reference "C?") (unit 1)
@@
     (pin "2")
     (instances
-      (project "PWA_REV2"
+      (project "PCBa_KRAKE"
         (path "/412a327d-1ee3-473e-bc00-1545004b7edf"
           (reference "C?") (unit 1)
@@
     (pin "2")
     (instances
-      (project "PWA_REV2"
+      (project "PCBa_KRAKE"
         (path "/412a327d-1ee3-473e-bc00-1545004b7edf/00000000-0000-0000-0000-000062bc4e7e"
           (reference "R503") (unit 1)
@@
     (pin "2")
     (instances
-      (project "PWA_REV2"
+      (project "PCBa_KRAKE"
         (path "/412a327d-1ee3-473e-bc00-1545004b7edf/00000000-0000-0000-0000-000062bc4e7e"
           (reference "R503") (unit 1)
@@
     (pin "2")
     (instances
-      (project "PWA_REV2"
+      (project "PCBa_KRAKE"
         (path "/412a327d-1ee3-473e-bc00-1545004b7edf"
           (reference "R?") (unit 1)
@@
     (pin "2")
     (instances
-      (project "PWA_REV2"
+      (project "PCBa_KRAKE"
         (path "/412a327d-1ee3-473e-bc00-1545004b7edf/00000000-0000-0000-0000-000062bc4e7e"
           (reference "R503") (unit 1)
@@
     (pin "2")
     (instances
-      (project "PWA_REV2"
+      (project "PCBa_KRAKE"
         (path "/412a327d-1ee3-473e-bc00-1545004b7edf/00000000-0000-0000-0000-000062bc4e7e"
           (reference "R503") (unit 1)
@@
     (pin "1")
     (instances
-      (project "PWA_REV2"
+      (project "PCBa_KRAKE"
         (path "/412a327d-1ee3-473e-bc00-1545004b7edf"
           (reference "#PWR030") (unit 1)
@@
     (pin "1")
     (instances
-      (project "PWA_REV2"
+      (project "PCBa_KRAKE"
         (path "/412a327d-1ee3-473e-bc00-1545004b7edf"
           (reference "#PWR026") (unit 1)
@@
     (pin "2")
     (instances
-      (project "PWA_REV2"
+      (project "PCBa_KRAKE"
         (path "/412a327d-1ee3-473e-bc00-1545004b7edf"
           (reference "C?") (unit 1)
@@
     (pin "2")
     (instances
-      (project "PWA_REV2"
+      (project "PCBa_KRAKE"
         (path "/412a327d-1ee3-473e-bc00-1545004b7edf/00000000-0000-0000-0000-000062bc4e7e"
           (reference "R503") (unit 1)
@@
     (pin "1")
     (instances
-      (project "PWA_REV2"
+      (project "PCBa_KRAKE"
         (path "/412a327d-1ee3-473e-bc00-1545004b7edf"
           (reference "#PWR027") (unit 1)
@@
     (pin "2")
     (instances
-      (project "PWA_REV2"
+      (project "PCBa_KRAKE"
         (path "/412a327d-1ee3-473e-bc00-1545004b7edf/00000000-0000-0000-0000-000062bc4e7e"
           (reference "R503") (unit 1)
@@
     (pin "2")
     (instances
-      (project "PWA_REV2"
+      (project "PCBa_KRAKE"
         (path "/412a327d-1ee3-473e-bc00-1545004b7edf"
           (reference "C?") (unit 1)
