File: PWA_REV2/RS232.kicad_sch (KiCad schematic)
At the start: 19 parts

Commit message: PWA_REV2, We corrected Assembly Type for some components, and we added the JLCPCB PN for the DB9 and the CH340B.
Parts:
- J?: AssemblyType SMT -> HAND; Distributor 1 DigiKey -> JLCPCB; Distributor 1 PN 609-5189-ND -> C3013509; Distributor 2 (none) -> DigiKey; Distributor 2 PN (none) -> 609-5189-ND
Changed lines of the file:
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@@
       (effects (font (size 1.27 1.27)) hide)
     )
-    (property "AssemblyType" "SMT" (at 195.58 127 0)
+    (property "AssemblyType" "HAND" (at 195.58 127 0)
       (effects (font (size 1.27 1.27)) hide)
     )
@@
       (effects (font (size 1.27 1.27)) hide)
     )
-    (property "Distributor 1" "DigiKey" (at 195.58 127 0)
+    (property "Distributor 1" "JLCPCB" (at 195.58 127 0)
       (effects (font (size 1.27 1.27)) hide)
     )
-    (property "Distributor 1 PN" "609-5189-ND" (at 195.58 127 0)
+    (property "Distributor 1 PN" "C3013509" (at 195.58 127 0)
       (effects (font (size 1.27 1.27)) hide)
     )
@@
       (effects (font (size 1.27 1.27)) hide)
     )
+    (property "Distributor 2" "DigiKey" (at 195.58 127 0)
+      (effects (font (size 1.27 1.27)) hide)
+    )
+    (property "Distributor 2 PN" "609-5189-ND" (at 195.58 127 0)
+      (effects (font (size 1.27 1.27)) hide)
+    )

Commit message: Adding files to preserve while fixing merge conflicts.
Parts:
- J?: MPN https://www.amazon.com/Pc-Accessories-Connectors-Connector-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 -> LD09S13A4GX00LF; MPN 2 LD09S13A4GX00LF -> https://www.amazon.com/Pc-Accessories-Connectors-Connector-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; Manufacturer Connectors Pro -> Amphenol ICC (FCI); Manufacturer 2 Amphenol ICC (FCI) -> Connectors Pro
- U?: value MAX3232 -> MAX3232IDWR; MPN MAX3232ID -> MAX3232IDWR
Changed lines of the file:
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@@
       (effects (font (size 1.27 1.27)) hide)
     )
-    (property "MPN 2" "LD09S13A4GX00LF" (at 195.58 127 0)
+    (property "MPN 2" "https://www.amazon.com/Pc-Accessories-Connectors-Connector-20-Pack/dp/B014IVD7L0/ref=sr_1_1" (at 195.58 127 0)
       (effects (font (size 1.27 1.27)) hide)
     )
-    (property "Manufacturer 2" "Amphenol ICC (FCI)" (at 195.58 127 0)
+    (property "Manufacturer 2" "Connectors Pro" (at 195.58 127 0)
       (effects (font (size 1.27 1.27)) hide)
     )
@@
       (effects (font (size 1.27 1.27)) hide)
     )
-    (property "MPN" "https://www.amazon.com/Pc-Accessories-Connectors-Connector-20-Pack/dp/B014IVD7L0/ref=sr_1_1" (at 195.58 127 0)
+    (property "MPN" "LD09S13A4GX00LF" (at 195.58 127 0)
       (effects (font (size 1.27 1.27)) hide)
     )
-    (property "Manufacturer" "Connectors Pro" (at 195.58 127 0)
+    (property "Manufacturer" "Amphenol ICC (FCI)" (at 195.58 127 0)
+      (effects (font (size 1.27 1.27)) hide)
+    )
+    (property "Distributor 2" "DigiKey" (at 195.58 127 0)
+      (effects (font (size 1.27 1.27)) hide)
+    )
+    (property "Distributor 2 PN" "609-5189-ND" (at 195.58 127 0)
       (effects (font (size 1.27 1.27)) hide)
     )
@@
       (effects (font (size 1.27 1.27)))
     )
-    (property "Value" "MAX3232" (at 104.14 78.105 0)
+    (property "Value" "MAX3232IDWR" (at 104.14 78.105 0)
       (effects (font (size 1.27 1.27)))
     )
@@
       (effects (font (size 1.27 1.27)) hide)
     )
-    (property "MPN" "MAX3232ID" (at 104.14 106.68 0)
+    (property "MPN" "MAX3232IDWR" (at 104.14 106.68 0)
       (effects (font (size 1.27 1.27)) hide)
     )
