File: PWA_REV2/RS232.kicad_sch (KiCad schematic)
At the start: 21 parts

Commit message: fixed kicad project issue.
Parts:
- removed MF403 (x2): Male-Female-Cylinder-Jackscrews_4-40, symbol GPAD_SCH_LIB:Nut_4-40_0.1875
Changed lines of the file:
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@@
-    )
-  )
-  (symbol (lib_id "GPAD_SCH_LIB:Nut_4-40_0.1875") (at 208.28 142.24 0) (unit 1)
-    (in_bom yes) (on_board no) (dnp no) (fields_autoplaced)
-    (property "Reference" "MF403" (at 213.995 140.9699 0)
-      (effects (font (size 1.27 1.27)) (justify left))
-    )
-    (property "Value" "Male-Female-Cylinder-Jackscrews_4-40" (at 213.995 143.5099 0)
-      (effects (font (size 1.27 1.27)) (justify left))
-    )
-    (property "Footprint" "" (at 208.28 142.24 0)
-      (effects (font (size 1.27 1.27)) hide)
-    )
-    (property "Datasheet" "" (at 208.28 142.24 0)
-      (effects (font (size 1.27 1.27)) hide)
-    )
-    (property "Distributor 1" "Amazon" (at 208.28 142.24 0)
-      (effects (font (size 1.27 1.27)) hide)
-    )
-    (property "Distributor 1 PN" "https://www.amazon.com/Ochoos-Male-Female-Cylinder-Jackscrew-Motherboard/dp/B07R66WYND" (at 208.28 142.24 0)
-      (effects (font (size 1.27 1.27)) hide)
-    )
-    (property "Cost" "0.35" (at 208.28 142.24 0)
-      (effects (font (size 1.27 1.27)) hide)
-    )
-    (property "MPN 2" "" (at 208.28 142.24 0)
-      (effects (font (size 1.27 1.27)) hide)
-    )
-    (property "Manufacturer 2" "" (at 208.28 142.24 0)
-      (effects (font (size 1.27 1.27)) hide)
-    )
-    (property "AssemblyType" "HAND" (at 208.28 142.24 0)
-      (effects (font (size 1.27 1.27)) hide)
-    )
-    (property "MPN" "4694" (at 208.28 142.24 0)
-      (effects (font (size 1.27 1.27)) hide)
-    )
-    (property "Manufacturer" "" (at 208.28 142.24 0)
-      (effects (font (size 1.27 1.27)) hide)
-    )
-    (property "Description" "25X Brass Copper #4-40x5+7 M-F Male-Female Hex Cylinder Standoff Spacer Screw Jackscrew Nut" (at 208.28 142.24 0)
-      (effects (font (size 1.27 1.27)) hide)
-    )
-    (instances
-      (project "PWA_REV2"
-        (path "/412a327d-1ee3-473e-bc00-1545004b7edf/00000000-0000-0000-0000-000062b871ee"
-          (reference "MF403") (unit 1)
-        )
-        (path "/412a327d-1ee3-473e-bc00-1545004b7edf/b048976a-3284-45ec-9285-06d31a0a2b0c"
-          (reference "MF701") (unit 1)
-        )
-      )
     )
   )
@@
         )
       )
-    )
-  )
-  (symbol (lib_id "GPAD_SCH_LIB:Nut_4-40_0.1875") (at 208.28 152.4 0) (unit 1)
-    (in_bom yes) (on_board no) (dnp no) (fields_autoplaced)
-    (property "Reference" "MF403" (at 213.995 151.1299 0)
-      (effects (font (size 1.27 1.27)) (justify left))
-    )
-    (property "Value" "Male-Female-Cylinder-Jackscrews_4-40" (at 213.995 153.6699 0)
-      (effects (font (size 1.27 1.27)) (justify left))
-    )
-    (property "Footprint" "" (at 208.28 152.4 0)
-      (effects (font (size 1.27 1.27)) hide)
-    )
-    (property "Datasheet" "" (at 208.28 152.4 0)
-      (effects (font (size 1.27 1.27)) hide)
-    )
-    (property "Distributor 1" "Amazon" (at 208.28 152.4 0)
-      (effects (font (size 1.27 1.27)) hide)
-    )
-    (property "Distributor 1 PN" "https://www.amazon.com/Ochoos-Male-Female-Cylinder-Jackscrew-Motherboard/dp/B07R66WYND" (at 208.28 152.4 0)
-      (effects (font (size 1.27 1.27)) hide)
-    )
-    (property "Cost" "0.35" (at 208.28 152.4 0)
-      (effects (font (size 1.27 1.27)) hide)
-    )
-    (property "MPN 2" "" (at 208.28 152.4 0)
-      (effects (font (size 1.27 1.27)) hide)
-    )
-    (property "Manufacturer 2" "" (at 208.28 152.4 0)
-      (effects (font (size 1.27 1.27)) hide)
-    )
-    (property "AssemblyType" "HAND" (at 208.28 152.4 0)
-      (effects (font (size 1.27 1.27)) hide)
-    )
-    (property "MPN" "4694" (at 208.28 152.4 0)
-      (effects (font (size 1.27 1.27)) hide)
-    )
-    (property "Manufacturer" "" (at 208.28 152.4 0)
-      (effects (font (size 1.27 1.27)) hide)
-    )
-    (property "Description" "25X Brass Copper #4-40x5+7 M-F Male-Female Hex Cylinder Standoff Spacer Screw Jackscrew Nut" (at 208.28 152.4 0)
-      (effects (font (size 1.27 1.27)) hide)
-    )
-    (instances
-      (project "PWA_REV2"
-        (path "/412a327d-1ee3-473e-bc00-1545004b7edf/00000000-0000-0000-0000-000062b871ee"
-          (reference "MF403") (unit 1)
-        )
-        (path "/412a327d-1ee3-473e-bc00-1545004b7edf/b048976a-3284-45ec-9285-06d31a0a2b0c"
-          (reference "MF702") (unit 1)
-        )
-      )

Commit message: PWA_REV2/PWA_REV2.kicad_pcb, Update for the actualy Mute key cap. Fixed MAX3232 part number.
Parts:
- U?: value MAX3232IDWR -> MAX3232CDR; Distributor 1 PN C354119 -> C45843; MPN MAX3232IDWR -> MAX3232CDR; MPN 2 (none) -> MAX3232ID (JLCPCB Part # C354119)
Changed lines of the file:
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@@
       (effects (font (size 1.27 1.27)))
     )
-    (property "Value" "MAX3232IDWR" (at 104.14 78.105 0)
+    (property "Value" "MAX3232CDR" (at 104.14 78.105 0)
       (effects (font (size 1.27 1.27)))
     )
@@
       (effects (font (size 1.27 1.27)) (justify left) hide)
     )
-    (property "Datasheet" "https://datasheets.maximintegrated.com/en/ds/MAX3222-MAX3241.pdf" (at 105.41 119.38 0)
+    (property "Datasheet" "https://www.ti.com/lit/ds/symlink/max3232.pdf" (at 105.41 119.38 0)
       (effects (font (size 1.27 1.27)) hide)
     )
@@
       (effects (font (size 1.27 1.27)) hide)
     )
-    (property "MPN 2" "" (at 104.14 106.68 0)
+    (property "MPN 2" " MAX3232ID (JLCPCB Part # C354119)" (at 104.14 106.68 0)
       (effects (font (size 1.27 1.27)) hide)
     )
@@
       (effects (font (size 1.27 1.27)) hide)
     )
-    (property "Description" "250Kbps Transceiver 2/2 SOIC-16 RS232 ICs ROHS" (at 104.14 106.68 0)
+    (property "Description" "250Kbps Transceiver 2/2 SOIC-16 RS232 ICs ROHS MAX3232CDR" (at 104.14 106.68 0)
       (effects (font (size 1.27 1.27)) hide)
     )
-    (property "MPN" "MAX3232IDWR" (at 104.14 106.68 0)
+    (property "MPN" "MAX3232CDR" (at 104.14 106.68 0)
       (effects (font (size 1.27 1.27)) hide)
     )
@@
       (effects (font (size 1.27 1.27)) hide)
     )
-    (property "Distributor 1 PN" "C354119" (at 104.14 106.68 0)
+    (property "Distributor 1 PN" "C45843" (at 104.14 106.68 0)
       (effects (font (size 1.27 1.27)) hide)
     )

Commit message: Hardware, PWA, Add a Jumper to BOM for J102 so that USB Connector Can Power Krake, issue 312.
:q
q
Parts:
- gave numbers to parts that had none: 9
- renumbered R503 to R701, R503 to R702, R503 to R703, R503 to R704, R503 to R705, R503 to R706, R503 to R707, R503 to R708, R503 to R709, R503 to R710

Commit message: Revert "Hardware, PWA, Add a Jumper to BOM for J102 so that USB Connector Can Power Krake, issue 312."
This reverts commit c2819b8ee4999f733f52d823f88f6aefd6456fcc.
Parts:
- renumbered C705 to C?, C706 to C?, C701 to C?, C702 to C?, C704 to C?, C703 to C?, J701 to J?, R702 to R503, R707 to R503, R710 to R503, R703 to R503, R704 to R503, R706 to R503, R709 to R503, R708 to R503, R701 to R503, R705 to R503, R711 to R?, U701 to U?
