File: PWA_REV2/PWA_REV2.kicad_pcb (KiCad board)
At the start: 2 copper layers, 137.2 x 83.8 mm, 212 parts, among them J101 Barrel_Jack_Switch_SMT, J102 0.100_2Pin, J103 0.100_2Pin, J104 Conn_01x14 1mm, J106 Conn_01x14 1mm, J107 Conn_01x10 1mm, J401 RJ12_6P6C_HORZ, J501 USB_C_Receptacle_USB2.0, J601 1X2P 1.25 mm Header, J602 0.100_2Pin, J603 DFPlayermini, J604 2mm_2Pin, J701 DE9_Receptacle_MountingHoles, Q201 MMBT2222A-7-F, Q202 MMBT2222A-7-F, Q203 MMBT2222A-7-F, Q204 MMBT2222A-7-F, Q205 MMBT2222A-7-F, Q206 MMBT2222A-7-F, Q207 MMBT2222A-7-F, Q301 BSS138, Q302 BSS138, Q303 BSS138, Q304 BSS138, Q305 BSS138, Q401 BSS138, Q402 BSS138, SW101 RotaryEncoder_Switch, T101 ToolingHole_Pad_1.152mm, T102 ToolingHole_Pad_1.152mm, T103 ToolingHole_Pad_1.152mm, U101 LM7805_TO220, U102 ESP32-WROOM-32E-N4, U103 AMS1117-3.3, U301 PCF8574AT_3_518, U302 LCD_20x4_Character-GPAD_SCH_L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, U501 CH340B, U701 MAX3232

Commit message: PWA_REV2, MOved U501 to the same X coordinates of u501 in Rev1.
Parts:
- moved U501 66.4 mm to (107.4, 138.4)
Changed lines of the file:
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@@
   )
   (footprint "Package_SO:SOIC-16_3.9x9.9mm_P1.27mm" (layer "F.Cu")
-    (at 173.863 138.873 90)
+    (at 107.4305 138.43 90)
     (descr "SOIC, 16 Pin (JEDEC MS-012AC, https://www.analog.com/media/en/package-pcb-resources/package/pkg_pdf/soic_narrow-r/r_16.pdf), generated with kicad-footprint-generator ipc_gullwing_generator.py")
     (tags "SOIC SO")
@@
     (pts (xy 55.88 101.6) (xy 193.04 101.6))
     (height 55.88)
-    (gr_text "137.1600 mm" (at 124.46 156.33) (layer "Dwgs.User")
+    (gr_text "5400.0000 mils" (at 124.46 156.33) (layer "Dwgs.User")
       (effects (font (size 1 1) (thickness 0.15)))
     )
@@
     (pts (xy 193.04 101.6) (xy 193.04 17.78))
     (height 37.465)
-    (gr_text "83.8200 mm" (at 229.355 59.69 90) (layer "Dwgs.User")
+    (gr_text "3300.0000 mils" (at 229.355 59.69 90) (layer "Dwgs.User")
       (effects (font (size 1 1) (thickness 0.15)))
     )
@@
     (pts (xy 71.12 73.66) (xy 71.12 101.6))
     (height 24.13)
-    (gr_text "27.9400 mm" (at 45.84 87.63 90) (layer "Dwgs.User")
+    (gr_text "1100.0000 mils" (at 45.84 87.63 90) (layer "Dwgs.User")
       (effects (font (size 1 1) (thickness 0.15)))
     )
@@
     (pts (xy 71.12 73.66) (xy 55.88 73.66))
     (height -38.735)
-    (gr_text "15.2400 mm" (at 63.5 111.245) (layer "Dwgs.User")
+    (gr_text "600.0000 mils" (at 63.5 111.245) (layer "Dwgs.User")
       (effects (font (size 1 1) (thickness 0.15)))
     )
@@
     (pts (xy 71.12 73.66) (xy 71.12 60.96))
     (height -23.495)
-    (gr_text "12.7000 mm" (at 46.475 67.31 90) (layer "Dwgs.User")
+    (gr_text "500.0000 mils" (at 46.475 67.31 90) (layer "Dwgs.User")
       (effects (font (size 1 1) (thickness 0.15)))
     )
@@
     (pts (xy 110.49 99.06) (xy 55.88 99.06))
     (height -20.32)
-    (gr_text "54.6100 mm" (at 83.185 118.23) (layer "Dwgs.User")
+    (gr_text "2150.0000 mils" (at 83.185 118.23) (layer "Dwgs.User")
       (effects (font (size 1 1) (thickness 0.15)))
     )
@@
     (pts (xy 87.63 91.44) (xy 55.88 91.44))
     (height -24.13)
-    (gr_text "31.7500 mm" (at 71.755 114.42) (layer "Dwgs.User")
+    (gr_text "1250.0000 mils" (at 71.755 114.42) (layer "Dwgs.User")
       (effects (font (size 1 1) (thickness 0.15)))
     )
@@
     (pts (xy 71.12 35.56) (xy 71.12 22.86))
     (height -19.685)
-    (gr_text "12.7000 mm" (at 50.285 29.21 90) (layer "Dwgs.User")
+    (gr_text "500.0000 mils" (at 50.285 29.21 90) (layer "Dwgs.User")
       (effects (font (size 1 1) (thickness 0.15)))
     )
@@
     (pts (xy 127 50.8) (xy 127 101.6))
     (height -91.44)
-    (gr_text "50.8000 mm" (at 217.29 76.2 90) (layer "Dwgs.User")
+    (gr_text "2000.0000 mils" (at 217.29 76.2 90) (layer "Dwgs.User")
       (effects (font (size 1 1) (thickness 0.15)))
     )
@@
     (pts (xy 124.46 96.52) (xy 55.88 96.52))
     (height -26.035)
-    (gr_text "68.5800 mm" (at 90.17 121.405) (layer "Dwgs.User")
+    (gr_text "2700.0000 mils" (at 90.17 121.405) (layer "Dwgs.User")
       (effects (font (size 1 1) (thickness 0.15)))
     )
@@
     (pts (xy 175.26 96.52) (xy 55.88 96.52))
     (height -36.195)
-    (gr_text "119.3800 mm" (at 115.57 131.565) (layer "Dwgs.User")
+    (gr_text "4700.0000 mils" (at 115.57 131.565) (layer "Dwgs.User")
       (effects (font (size 1 1) (thickness 0.15)))
     )
@@
     (pts (xy 154.305 96.52) (xy 55.88 96.52))
     (height -33.02)
-    (gr_text "98.4250 mm" (at 105.0925 128.39) (layer "Dwgs.User")
+    (gr_text "3875.0000 mils" (at 105.0925 128.39) (layer "Dwgs.User")
       (effects (font (size 1 1) (thickness 0.15)))
     )
@@
     (pts (xy 134.62 73.406) (xy 55.88 73.025))
     (height -93.917448)
-    (gr_text "78.7409 mm" (at 94.80113 165.981862 -0.2772354792) (layer "Dwgs.User")
+    (gr_text "3100.0363 mils" (at 94.80113 165.981862 -0.2772354792) (layer "Dwgs.User")
       (effects (font (size 1 1) (thickness 0.15)))
     )
@@
     (pts (xy 60.96 96.52) (xy 60.96 101.6))
     (height 8.89)
-    (gr_text "5.0800 mm" (at 50.92 99.06 90) (layer "Dwgs.User")
+    (gr_text "200.0000 mils" (at 50.92 99.06 90) (layer "Dwgs.User")
       (effects (font (size 1 1) (thickness 0.15)))
     )
@@
     (pts (xy 187.96 54.61) (xy 55.88 54.61))
     (height -94.615)
-    (gr_text "132.0800 mm" (at 121.92 148.075) (layer "Dwgs.User")
+    (gr_text "5200.0000 mils" (at 121.92 148.075) (layer "Dwgs.User")
       (effects (font (size 1 1) (thickness 0.15)))
     )
@@
     (pts (xy 71.12 48.26) (xy 71.12 35.56))
     (height -20.32)
-    (gr_text "12.7000 mm" (at 49.65 41.91 90) (layer "Dwgs.User")
+    (gr_text "500.0000 mils" (at 49.65 41.91 90) (layer "Dwgs.User")
       (effects (font (size 1 1) (thickness 0.15)))
     )
@@
     (pts (xy 187.96 96.52) (xy 55.88 96.52))
     (height -40.64)
-    (gr_text "132.0800 mm" (at 121.92 136.01) (layer "Dwgs.User")
+    (gr_text "5200.0000 mils" (at 121.92 136.01) (layer "Dwgs.User")
       (effects (font (size 1 1) (thickness 0.15)))
     )
@@
     (pts (xy 187.96 54.61) (xy 187.96 101.6))
     (height -10.795)
-    (gr_text "46.9900 mm" (at 197.605 78.105 90) (layer "Dwgs.User")
+    (gr_text "1850.0000 mils" (at 197.605 78.105 90) (layer "Dwgs.User")
       (effects (font (size 1 1) (thickness 0.15)))
     )
@@
     (pts (xy 185.42 38.735) (xy 55.88 38.735))
     (height -104.14)
-    (gr_text "129.5400 mm" (at 120.65 141.725) (layer "Dwgs.User")
+    (gr_text "5100.0000 mils" (at 120.65 141.725) (layer "Dwgs.User")
       (effects (font (size 1 1) (thickness 0.15)))
     )
@@
     (pts (xy 185.42 38.735) (xy 185.42 101.6))
     (height -20.955)
-    (gr_text "62.8650 mm" (at 205.225 70.1675 90) (layer "Dwgs.User")
+    (gr_text "2475.0000 mils" (at 205.225 70.1675 90) (layer "Dwgs.User")
       (effects (font (size 1 1) (thickness 0.15)))
     )
@@
     (pts (xy 134.62 73.406) (xy 134.62 101.476))
     (height -61.595)
-    (gr_text "28.0700 mm" (at 195.065 87.441 90) (layer "Dwgs.User")
+    (gr_text "1105.1181 mils" (at 195.065 87.441 90) (layer "Dwgs.User")
       (effects (font (size 1 1) (thickness 0.15)))
     )
@@
     (pts (xy 127 50.8) (xy 55.88 50.8))
     (height 36.83)
-    (gr_text "71.1200 mm" (at 91.44 12.82) (layer "Dwgs.User")
+    (gr_text "2800.0000 mils" (at 91.44 12.82) (layer "Dwgs.User")
       (effects (font (size 1 1) (thickness 0.15)))
     )
@@
     (pts (xy 137.16 101.6) (xy 55.88 101.6))
     (height -24.765)
-    (gr_text "81.2800 mm" (at 96.52 125.215) (layer "Dwgs.User")
+    (gr_text "3200.0000 mils" (at 96.52 125.215) (layer "Dwgs.User")
       (effects (font (size 1 1) (thickness 0.15)))
     )
@@
     (pts (xy 71.12 86.36) (xy 71.12 101.6))
     (height 21.59)
-    (gr_text "15.2400 mm" (at 48.38 93.98 90) (layer "Dwgs.User")
+    (gr_text "600.0000 mils" (at 48.38 93.98 90) (layer "Dwgs.User")
       (effects (font (size 1 1) (thickness 0.15)))
     )
@@
     (pts (xy 60.96 96.52) (xy 55.88 96.52))
     (height -10.16)
-    (gr_text "5.0800 mm" (at 58.42 105.53) (layer "Dwgs.User")
+    (gr_text "200.0000 mils" (at 58.42 105.53) (layer "Dwgs.User")
       (effects (font (size 1 1) (thickness 0.15)))
     )
@@
     (pts (xy 71.12 60.96) (xy 71.12 48.26))
     (height -22.225)
-    (gr_text "12.7000 mm" (at 47.745 54.61 90) (layer "Dwgs.User")
+    (gr_text "500.0000 mils" (at 47.745 54.61 90) (layer "Dwgs.User")
       (effects (font (size 1 1) (thickness 0.15)))
     )
@@
     (pts (xy 130.302 101.6) (xy 130.35 87.421))
     (height 9.161362)
-    (gr_text "14.1791 mm" (at 138.337317 94.537621 89.80603802) (layer "Cmts.User")
+    (gr_text "558.2315 mils" (at 138.337317 94.537621 89.80603802) (layer "Cmts.User")
       (effects (font (size 1 1) (thickness 0.15)))
     )
@@
     (pts (xy 114.865 101.961) (xy 145.835 101.961))
     (height 7.513)
-    (gr_text "30.9700 mm" (at 130.35 108.324) (layer "Cmts.User")
+    (gr_text "1219.2913 mils" (at 130.35 108.324) (layer "Cmts.User")
       (effects (font (size 1 1) (thickness 0.15)))
     )
@@
     (pts (xy 130.302 101.6) (xy 55.88 101.6))
     (height -88.392)
-    (gr_text "74.4220 mm" (at 93.091 188.842) (layer "Cmts.User")
+    (gr_text "2930.0000 mils" (at 93.091 188.842) (layer "Cmts.User")
       (effects (font (size 1 1) (thickness 0.15)))
     )

Commit message: PWA_REV2, Routed U501.
Parts:
- moved R217 69.3 mm to (103.1, 78.7), turned to -90 degrees
- moved TP204 55.0 mm to (117.3, 84.8)
- moved U501 50.8 mm to (107.4, 87.6)
- moved R215 16.3 mm to (118.1, 79.5), turned to 0 degrees
- moved C503 11.3 mm to (103.9, 92.5), turned to 180 degrees
- moved C501 5.18 mm to (101.6, 81.9)
- moved R213 3.77 mm to (98.9, 92.2), turned to 180 degrees
- moved TP203 3.61 mm to (115.6, 72.4)
- moved Q207 3.06 mm to (117.3, 76.7)
- moved TP202 1.52 mm to (97.8, 95.5)
- moved R504 0.85 mm to (111.0, 80.0)
- moved R214 0.72 mm to (104.9, 78.7)
- moved R211 0.54 mm to (112.4, 92.5), turned to 0 degrees
Routing:
- net Net-(Q207-E): track 0.00 -> 27.1 mm, vias 0 -> 3
- net Net-(Q207-C): track 18.5 -> 0.00 mm
- net /USB_UART/V3: track 31.4 -> 13.0 mm, vias 2 -> 0
- net Net-(Q207-B): track 17.4 -> 2.15 mm, vias 2 -> 0
- net Net-(Q206-E): track 18.1 -> 31.7 mm, vias 2 -> 4
- net GND: track 148.6 -> 135.3 mm
- net Net-(U501-RST#): track 0.00 -> 9.10 mm
- net Net-(U501-RXD): track 87.4 -> 80.3 mm, vias 4 -> 2
- net /USB_UART/3V3USB: track 34.0 -> 28.0 mm
- net Net-(U501-TXD): track 19.6 -> 14.8 mm, vias 2 -> 0
- net Net-(U501-~{CTS}): track 13.9 -> 17.4 mm, vias 3 -> 2
- net Net-(J501-CC2): track 3.33 -> 4.88 mm
- net GPIO0: track 57.6 -> 56.1 mm
- net Net-(U501-TNOW): track 4.87 -> 6.19 mm, vias 3 -> 0
- net Net-(Q206-B): track 18.0 -> 19.2 mm
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- removed copper zone on F.Cu, net /USB_UART/3V3USB

Commit message: PWA_REV2, Placed J601 and J604.
Parts:
- moved J604 55.6 mm to (145.8, 65.5), turned to 90 degrees
- turned J601 to 90 degrees
Routing:
- net Net-(J603-SPK_2): track 37.6 -> 42.9 mm
- net Net-(J603-SPK_1): track 42.5 -> 47.5 mm, vias 1 -> 2
- net GND: vias 136 -> 135

Commit message: USB_UART, moving the RX test point closer to where the tx of USB is.
Parts:
- moved TP104 110.1 mm to (58.4, 28.2)
- moved TP109 107.4 mm to (76.7, 29.0)
- moved TP105 80.1 mm to (189.0, 87.6)
- moved TP100 75.3 mm to (100.3, 49.0)
- moved TP106 60.6 mm to (66.8, 97.8)
- moved T101 11.1 mm to (65.3, 19.1)
- moved T102 9.88 mm to (57.4, 93.2)
Routing:
- net /3v3Controller: track 129.0 -> 130.3 mm
- net +3.3V: track 242.9 -> 244.0 mm
- net Switch_Mute: track 167.1 -> 167.8 mm
- net GND: vias 135 -> 134
