File: PWA_REV2/PWA_REV2.kicad_pcb (KiCad board)
At the start: 2 copper layers, 137.2 x 83.8 mm, 212 parts, among them J101 Barrel_Jack_Switch_SMT, J102 0.100_2Pin, J103 0.100_2Pin, J104 Conn_01x14 1mm, J106 Conn_01x14 1mm, J107 Conn_01x10 1mm, J401 RJ12_6P6C_HORZ, J501 USB_C_Receptacle_USB2.0, J601 1X2P 1.25 mm Header, J602 0.100_2Pin, J603 DFPlayermini, J604 2mm_2Pin, J701 DE9_Receptacle_MountingHoles, Q201 MMBT2222A-7-F, Q202 MMBT2222A-7-F, Q203 MMBT2222A-7-F, Q204 MMBT2222A-7-F, Q205 MMBT2222A-7-F, Q206 MMBT2222A-7-F, Q207 MMBT2222A-7-F, Q301 BSS138, Q302 BSS138, Q303 BSS138, Q304 BSS138, Q305 BSS138, Q401 BSS138, Q402 BSS138, SW101 RotaryEncoder_Switch, T101 ToolingHole_Pad_1.152mm, T102 ToolingHole_Pad_1.152mm, T103 ToolingHole_Pad_1.152mm, U101 LM7805_TO220, U102 ESP32-WROOM-32E-N4, U103 AMS1117-3.3, U301 PCF8574AT_3_518, U302 LCD_20x4_Character-GPAD_SCH_L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, U501 CH340B, U701 MAX3232

Commit message: USB_UART, moving the RX test point closer to where the tx of USB is.
Parts:
- removed TP107: U0_TX, TestPoint:TestPoint_Loop_D1.80mm_Drill1.0mm_Beaded
- added TP206: U0_TX, TestPoint:TestPoint_Loop_D1.80mm_Drill1.0mm_Beaded, F.Cu at (127.3, 67.3)
- moved TP108 72.0 mm to (123.2, 67.3)
- moved G*** 0.76 mm to (116.3, 67.1)
Routing:
- net GPIO0: track 56.1 -> 59.4 mm
- net Net-(U501-RXD): track 80.3 -> 82.4 mm
- net ControllerRX: track 72.0 -> 73.6 mm

Commit message: PWA_REV2, Placed testpoint and routed it. Changed the settings of some Values of old testpoints to be on silkscreen.
Parts:
- +5esp32, TP100, TP109, TP306, TP501: footprint TestPoint:TestPoint_Loop_D2.54mm_Drill1.5mm_Beaded -> TestPoint:TestPoint_Loop_D1.80mm_Drill1.0mm_Beaded
- moved TP205 76.9 mm to (88.3, 83.4), turned to -90 degrees
- moved TP306 74.3 mm to (171.4, 56.1)
- moved TP501 71.9 mm to (88.9, 78.7)
- moved TP305 60.1 mm to (144.3, 80.8)
- moved TP302 51.6 mm to (165.1, 87.4)
- moved TP301 51.0 mm to (165.1, 83.6)
- moved TP304 49.6 mm to (164.7, 99.2), turned to 90 degrees
- moved TP303 46.4 mm to (141.6, 85.0)
- moved TP202 3.64 mm to (99.3, 98.8)
Connections:
- TP501 pad 1: /AlarmAudio/5VDFP -> (no net)
Routing:
- net /SPI Peripherial/MOSI: track 9.14 -> 25.4 mm
- net /USB_UART/3V3USB: track 28.0 -> 39.4 mm
- net /SPI Peripherial/SS: track 3.80 -> 13.9 mm
- net /SPI Peripherial/+12in: track 6.45 -> 16.2 mm
- net /AlarmAudio/5VDFP: track 16.1 -> 20.4 mm
- net /SPI Peripherial/MISO: track 9.51 -> 13.6 mm
- net SPI_SCK: track 111.7 -> 115.7 mm
- net /USB_UART/V3: track 13.0 -> 15.9 mm
- net /SPI Peripherial/5VRaw: track 84.1 -> 86.0 mm
- net ControllerVcc: track 18.3 -> 16.5 mm
- net VBus: track 26.2 -> 27.9 mm
- net Net-(D303-COM): track 34.2 -> 35.8 mm
- net Net-(D301-COM): track 21.0 -> 22.0 mm
- net Net-(D104-A): track 18.2 -> 19.0 mm
- net Net-(Q206-B): track 19.2 -> 19.8 mm
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Other:
- outline, holes or cut-outs redrawn
- board text added: "SPI PWR"
- board text removed: "Power from SPI"

Commit message: PWA_REV2, tweeked silkscreens for testPoints.
Routing:
- net /SPI Peripherial/MOSI: track 25.4 -> 29.0 mm
Other:
- board text removed: "CIPO"
- board text removed: "CLK"
- board text removed: "SCL"
- board text removed: "SDA"
- board text removed: "SPI PWR"
- board text removed: "nCS"
Changed lines of the file:
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@@
     (property "ki_keywords" "test point tp")
     (attr through_hole)
-    (fp_text reference "TP102" (at 3.81 -1.016) (layer "F.SilkS")
+    (fp_text reference "TP102" (at 3.302 -2.667) (layer "F.SilkS")
         (effects (font (size 1 1) (thickness 0.15)))
     )
-    (fp_text value "Vin" (at 2.286 -2.286) (layer "F.SilkS")
+    (fp_text value "Vin" (at 2.54 -1.397) (layer "F.SilkS")
         (effects (font (size 1 1) (thickness 0.15)))
     )
@@
         (effects (font (size 1 1) (thickness 0.15)))
     )
-    (fp_text value "CIPO" (at 3.302 -1.016) (layer "F.SilkS")
+    (fp_text value "CIPO" (at 3.175 1.524) (layer "F.SilkS")
         (effects (font (size 1 1) (thickness 0.15)))
     )
@@
     (property "ki_keywords" "test point tp")
     (attr through_hole)
-    (fp_text reference "TP202" (at 1.27 -3.556 90) (layer "F.SilkS")
+    (fp_text reference "TP202" (at -0.381 -3.683 90) (layer "F.SilkS")
         (effects (font (size 1 1) (thickness 0.15)))
     )
-    (fp_text value "V3" (at 0 -2.8 90) (layer "F.SilkS")
+    (fp_text value "V3" (at 0.889 -2.54 90) (layer "F.SilkS")
         (effects (font (size 1 1) (thickness 0.15)))
     )
@@
     (property "ki_keywords" "test point tp")
     (attr through_hole)
-    (fp_text reference "TP201" (at 1.778 -3.556 90) (layer "F.SilkS")
+    (fp_text reference "TP201" (at 0.508 -3.937 90) (layer "F.SilkS")
         (effects (font (size 1 1) (thickness 0.15)))
     )
-    (fp_text value "VBus" (at 0.508 -3.556 90) (layer "F.SilkS")
+    (fp_text value "VBus" (at 1.778 -3.556 90) (layer "F.SilkS")
         (effects (font (size 1 1) (thickness 0.15)))
     )
@@
         (effects (font (size 1 1) (thickness 0.15)))
     )
-    (fp_text value "SDA" (at 0 -2.8) (layer "F.Fab")
+    (fp_text value "SDA" (at 1.397 3.556) (layer "F.SilkS")
         (effects (font (size 1 1) (thickness 0.15)))
     )
@@
     (property "ki_keywords" "test point tp")
     (attr through_hole)
-    (fp_text reference "TP305" (at 2.159 0.127 90) (layer "F.SilkS")
+    (fp_text reference "TP305" (at 2.159 0.508 90) (layer "F.SilkS")
         (effects (font (size 1 1) (thickness 0.15)))
     )
-    (fp_text value "SS" (at 3.175 -0.762 90) (layer "F.SilkS")
+    (fp_text value "SS" (at 3.302 -0.635 90) (layer "F.SilkS")
         (effects (font (size 1 1) (thickness 0.15)))
     )
@@
     (effects (font (size 1 1) (thickness 0.15)) (justify mirror))
   )
-  (gr_text "CLK" (at 155.321 80.899) (layer "F.SilkS")
-    (effects (font (size 0.762 0.762) (thickness 0.1524)))
-  )
   (gr_text "Power In" (at 175.768 88.138) (layer "F.SilkS")
     (effects (font (size 1.016 1.016) (thickness 0.254)))
@@
     (effects (font (size 1.016 1.016) (thickness 0.254)))
   )
-  (gr_text "COPI" (at 149.733 80.772) (layer "F.SilkS")
-    (effects (font (size 0.762 0.762) (thickness 0.1524)))
-  )
   (gr_text "RESET" (at 89.916 54.356) (layer "F.SilkS")
     (effects (font (size 1.5 1.5) (thickness 0.2)) (justify left bottom))
   )
-  (gr_text "CIPO" (at 161.29 80.899) (layer "F.SilkS")
-    (effects (font (size 0.762 0.762) (thickness 0.1524)))
-  )
-  (gr_text "nCS" (at 152.273 80.772) (layer "F.SilkS")
-    (effects (font (size 0.762 0.762) (thickness 0.1524)))
-  )
   (gr_text "BOOT" (at 120.142 54.356) (layer "F.SilkS")
     (effects (font (size 1.5 1.5) (thickness 0.2)) (justify left bottom))
@@
     (effects (font (size 1 1) (thickness 0.15)))
   )
-  (gr_text "SDA" (at 130.2004 40.8432) (layer "F.SilkS")
-    (effects (font (size 0.762 0.762) (thickness 0.1524)))
-  )
-  (gr_text "SCL" (at 129.8956 35.9156) (layer "F.SilkS")
-    (effects (font (size 0.762 0.762) (thickness 0.1524)))
-  )
-  (gr_text "SPI PWR\n" (at 164.592 90.17) (layer "F.SilkS")
-    (effects (font (size 1 1) (thickness 0.1)))
-  )
   (gr_text "<-UNO Pin 1" (at 194.31 78.105 90) (layer "Dwgs.User")
     (effects (font (size 0.762 0.762) (thickness 0.1905)))
@@
   (via (at 151.13 85.725) (size 0.8) (drill 0.4) (layers "F.Cu" "B.Cu") (net 115))
   (segment (start 151.13 87.63) (end 151.13 85.725) (width 0.635) (layer "B.Cu") (net 115))
-  (segment (start 157.051288 91.205) (end 153.435 91.205) (width 0.25) (layer "F.Cu") (net 116))
-  (segment (start 164.719 98.872712) (end 157.051288 91.205) (width 0.25) (layer "F.Cu") (net 116))
-  (segment (start 153.435 91.205) (end 152.4 90.17) (width 0.25) (layer "F.Cu") (net 116))
+  (segment (start 155.194 93.091) (end 155.194 92.964) (width 0.25) (layer "F.Cu") (net 116))
   (segment (start 148.59 84.0975) (end 148.59 84.35519) (width 0.25) (layer "F.Cu") (net 116))
+  (segment (start 164.719 99.187) (end 164.719 98.806) (width 0.25) (layer "F.Cu") (net 116))
   (segment (start 148.59 84.35519) (end 149.274905 85.040095) (width 0.25) (layer "F.Cu") (net 116))
-  (segment (start 164.719 99.187) (end 164.719 98.872712) (width 0.25) (layer "F.Cu") (net 116))
+  (segment (start 155.194 92.964) (end 155.194 98.679) (width 0.25) (layer "F.Cu") (net 116))
+  (segment (start 155.702 99.187) (end 164.719 99.187) (width 0.25) (layer "F.Cu") (net 116))
+  (segment (start 155.194 98.679) (end 155.702 99.187) (width 0.25) (layer "F.Cu") (net 116))
+  (segment (start 155.194 92.964) (end 152.4 90.17) (width 0.25) (layer "F.Cu") (net 116))
   (via (at 149.274905 85.040095) (size 0.8) (drill 0.4) (layers "F.Cu" "B.Cu") (net 116))
   (segment (start 149.274905 89.584905) (end 149.274905 85.040095) (width 0.25) (layer "B.Cu") (net 116))

Commit message: PWA_REV2, Cleared clearance violatoin and thermal relief DRC errors.
Parts:
- moved C501 1.18 mm to (102.2, 82.9), turned to 180 degrees
- moved R216 1.02 mm to (98.2, 81.4), turned to 180 degrees
- moved TP305 0.51 mm to (144.8, 80.8)
- moved TP304 0.25 mm to (164.7, 98.9)
Routing:
- net GND: track 134.7 -> 145.9 mm, vias 134 -> 151
- net /USB_UART/3V3USB: track 39.4 -> 32.9 mm
- net /AlarmAudio/5VDFP: track 20.4 -> 16.6 mm
- net +3.3V: track 244.0 -> 242.4 mm
- net Net-(U301-P7): track 17.1 -> 15.9 mm
- net Net-(U501-UD+): track 11.0 -> 10.1 mm
- net /SPI Peripherial/MOSI: track 29.0 -> 28.3 mm
- net Net-(Q206-E): track 31.7 -> 31.0 mm
- net Net-(J603-SPK_1): vias 2 -> 1
Other:
- board text added: "COM"
- board text added: "USB"
