File: PWA_REV2/PWA_REV2.kicad_pcb (KiCad board)
At the start: 2 copper layers, 137.2 x 83.8 mm, 212 parts, among them J101 Barrel_Jack_Switch_SMT, J102 0.100_2Pin, J103 0.100_2Pin, J104 Conn_01x14 1mm, J106 Conn_01x14 1mm, J107 Conn_01x10 1mm, J401 RJ12_6P6C_HORZ, J501 USB_C_Receptacle_USB2.0, J601 1X2P 1.25 mm Header, J602 0.100_2Pin, J603 DFPlayermini, J604 2mm_2Pin, J701 DE9_Receptacle_MountingHoles, Q201 MMBT2222A-7-F, Q202 MMBT2222A-7-F, Q203 MMBT2222A-7-F, Q204 MMBT2222A-7-F, Q205 MMBT2222A-7-F, Q206 MMBT2222A-7-F, Q207 MMBT2222A-7-F, Q301 BSS138, Q302 BSS138, Q303 BSS138, Q304 BSS138, Q305 BSS138, Q401 BSS138, Q402 BSS138, SW101 RotaryEncoder_Switch, T101 ToolingHole_Pad_1.152mm, T102 ToolingHole_Pad_1.152mm, T103 ToolingHole_Pad_1.152mm, U101 LM7805_TO220, U102 ESP32-WROOM-32E-N4, U103 AMS1117-3.3, U301 PCF8574AT_3_518, U302 LCD_20x4_Character-GPAD_SCH_L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, U501 CH340B, U701 MAX3232

Commit message: PWA_REV2, Cleared DRC errors, fixed R211.
Parts:
- turned R211 to 180 degrees
Routing:
- net GND: track 145.9 -> 142.1 mm
- net Net-(J501-CC2): track 4.88 -> 3.20 mm
- net Net-(U501-UD+): track 10.1 -> 8.57 mm

Commit message: PWA_REV2, Cleared DRC errors, thermal relief on C103.
Parts:
- moved C503 0.25 mm to (103.9, 92.7)
Routing:
- net Net-(J501-CC1): track 10.5 -> 6.42 mm
- net GND: track 142.1 -> 139.5 mm, vias 151 -> 152
- net Net-(Q207-E): track 26.9 -> 28.7 mm
- net /USB_UART/V3: track 15.7 -> 16.8 mm

Commit message: PWA_REV2, Cleared DRC warning, connected 5vDFP testpoint.
Connections:
- TP501 pad 1: (no net) -> /AlarmAudio/5VDFP
Routing:
- net /AlarmAudio/5VDFP: track 16.6 -> 20.3 mm
Changed lines of the file:
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@@
     (fp_circle (center 0 0) (end 1.3 0)
       (stroke (width 0.12) (type solid)) (fill none) (layer "F.Fab"))
-    (pad "1" thru_hole circle (at 0 0) (size 2 2) (drill 1) (layers "*.Cu" "*.Mask"))
+    (pad "1" thru_hole circle (at 0 0) (size 2 2) (drill 1) (layers "*.Cu" "*.Mask")
+      (net 19 "/AlarmAudio/5VDFP") (pinfunction "1") (pintype "passive"))
     (model "${KICAD6_3DMODEL_DIR}/TestPoint.3dshapes/TestPoint_Loop_D1.80mm_Drill1.0mm_Beaded.wrl"
       (offset (xyz 0 0 0))
@@
   (segment (start 87.2725 71.882) (end 87.2725 69.596) (width 0.25) (layer "F.Cu") (net 19))
   (segment (start 88.138 68.7305) (end 87.2725 69.596) (width 0.25) (layer "F.Cu") (net 19))
+  (segment (start 88.9 78.74) (end 92.6095 78.74) (width 0.25) (layer "F.Cu") (net 19))
   (segment (start 92.979 74.20971) (end 89.60021 74.20971) (width 0.25) (layer "F.Cu") (net 19))
-  (segment (start 92.6095 78.74) (end 92.979 78.3705) (width 0.25) (layer "F.Cu") (net 19))
   (segment (start 88.138 66.97) (end 88.138 68.7305) (width 0.25) (layer "F.Cu") (net 19))
   (segment (start 88.0345 72.644) (end 87.2725 71.882) (width 0.25) (layer "F.Cu") (net 19))
@@
   (segment (start 89.60021 74.20971) (end 88.0345 72.644) (width 0.25) (layer "F.Cu") (net 19))
   (segment (start 92.979 78.3705) (end 92.979 74.20971) (width 0.889) (layer "F.Cu") (net 19))
+  (segment (start 92.6095 78.74) (end 92.964 78.3855) (width 0.25) (layer "F.Cu") (net 19))
   (segment (start 123.942 72.43) (end 123.5475 72.0355) (width 0.25) (layer "F.Cu") (net 20))
   (segment (start 126.15 72.43) (end 123.942 72.43) (width 0.25) (layer "F.Cu") (net 20))

Commit message: PWA_REV2, Clearing DRC warning, overlapping Silkscreen. enhanced LED standoffs footprint.
Parts:
- moved R102 0.78 mm to (86.1, 33.5)
- moved TP108 0.63 mm to (122.6, 67.3)
- moved C1100 0.38 mm to (87.8, 33.5)
- moved MF604 0.13 mm to (71.1, 34.3)
- moved R308 0.13 mm to (178.4, 38.6)
Routing:
- net /3v3Controller: track 130.3 -> 129.3 mm
