File: PWA_REV2/USB_UART.kicad_sch (KiCad schematic)
At the start: 21 parts, among them J501 USB_C_Receptacle_USB2.0, Q205 MMBT2222A-7-F, U501 CH340T

Commit message: Fixed the previous PWA_REV_2 file by added the changes of the USB UART. PCBa_krake is reverted to when no changes done to the schem.
Parts:
- removed U501: CH340T, GeneralPurposeAlarmDevicePCB:SSOP-20_5.3x7.2mm_P0.65mm_CH340T, symbol GPAD_SCH_LIB:CH340T
- added R217: 4K7, Resistor_SMD:R_0603_1608Metric_Pad0.98x0.95mm_HandSolder, symbol Device:R
- added TP204: nRST, TestPoint:TestPoint_Loop_D2.54mm_Drill1.5mm_Beaded, symbol Connector:TestPoint
- added U501: CH340B, Package_SO:SOIC-16_3.9x9.9mm_P1.27mm, symbol GPAD_SCH_LIB:CH340B
Connections:
- net GND: now also R217.1, U501.1 (GND)
- net GPIO0: now also Q205.3 (C); no longer Q205.2 (E)
- net at R502.2: now also U501.2 (TXD)
- net at R503.2: now also U501.3 (RXD)
- net at C503.1, R1.1, TP202.1: now also U501.4 (V3)
- net at C501.1, C502.1, R1.1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: now also U501.16 (VCC)
- net at R501.1: now also U501.15 (TNOW)
- net at R504.2, TP203.1: now also U501.9 (~{CTS})
- net at R505.1: now also Q205.2 (E), R217.2, U501.13 (~{DTR}); no longer Q205.3 (C)
- net at Q205.2 (E), R505.1: now also U501.14 (~{RTS})
- net at J501.A6 (D+), J501.B6 (D+): now also U501.5 (UD+)
- net at J501.A7 (D-), J501.B7 (D-): now also U501.6 (UD-)
- new net: TP204.1, U501.7 (RST#)
- no-connect marks 11 -> 5
Other:
- note added: "D501 indicates when data is transmitted. The serial port sends ongoing status indication, high level is active."
- note added: "The DTR# pin of CH340 is used as a configuration input pin before the USB configuration is complete. An external 4.7KΩ pull-down resistor (R217) can be connected with this pin to generate default low level during USB enumeration, apply larger supply current to the USB bus via the configuration descriptor."
- title: Krake Rev2 -> KRAKE_PCB
- moved on the sheet: R504, TP203

Commit message: PWA_REV2.kicad_sch, updated the footptint of the testpoint to 1mm hole and corrected description.
Parts:
- TP201, TP202, TP203, TP204: footprint TestPoint:TestPoint_Loop_D2.54mm_Drill1.5mm_Beaded -> TestPoint:TestPoint_Loop_D1.80mm_Drill1.0mm_Beaded
Changed lines of the file:
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@@
       (effects (font (size 1.27 1.27)) (justify left))
     )
-    (property "Footprint" "TestPoint:TestPoint_Loop_D2.54mm_Drill1.5mm_Beaded" (at 107.95 72.39 0)
+    (property "Footprint" "TestPoint:TestPoint_Loop_D1.80mm_Drill1.0mm_Beaded" (at 107.95 72.39 0)
       (effects (font (size 1.27 1.27)) hide)
     )
@@
       (effects (font (size 1.27 1.27)) hide)
     )
-    (property "Description" "Test Points/Test Rings ROHS red" (at 102.87 72.39 0)
+    (property "Description" "Test Points/Test Rings 1.25 mm Red" (at 102.87 72.39 0)
       (effects (font (size 1.27 1.27)) hide)
     )
@@
       (effects (font (size 1.27 1.27)) (justify left))
     )
-    (property "Footprint" "TestPoint:TestPoint_Loop_D2.54mm_Drill1.5mm_Beaded" (at 142.24 71.12 0)
+    (property "Footprint" "TestPoint:TestPoint_Loop_D1.80mm_Drill1.0mm_Beaded" (at 142.24 71.12 0)
       (effects (font (size 1.27 1.27)) hide)
     )
@@
       (effects (font (size 1.27 1.27)) hide)
     )
-    (property "Description" "Test Points/Test Rings ROHS red" (at 137.16 71.12 0)
+    (property "Description" "Test Points/Test Rings 1.25 mm Red" (at 137.16 71.12 0)
       (effects (font (size 1.27 1.27)) hide)
     )
@@
       (effects (font (size 1.27 1.27)) (justify left))
     )
-    (property "Footprint" "TestPoint:TestPoint_Loop_D2.54mm_Drill1.5mm_Beaded" (at 205.74 105.41 0)
+    (property "Footprint" "TestPoint:TestPoint_Loop_D1.80mm_Drill1.0mm_Beaded" (at 205.74 105.41 0)
       (effects (font (size 1.27 1.27)) hide)
     )
@@
       (effects (font (size 1.27 1.27)) hide)
     )
-    (property "Description" "Test Points/Test Rings ROHS yellow" (at 200.66 105.41 0)
+    (property "Description" "Test Points/Test Rings 1.25 mm Yellow" (at 200.66 105.41 0)
       (effects (font (size 1.27 1.27)) hide)
     )
@@
       (effects (font (size 1.27 1.27)) (justify left))
     )
-    (property "Footprint" "TestPoint:TestPoint_Loop_D2.54mm_Drill1.5mm_Beaded" (at 135.89 105.41 0)
+    (property "Footprint" "TestPoint:TestPoint_Loop_D1.80mm_Drill1.0mm_Beaded" (at 135.89 105.41 0)
       (effects (font (size 1.27 1.27)) hide)
     )
@@
       (effects (font (size 1.27 1.27)) hide)
     )
-    (property "Description" "Test Points/Test Rings ROHS yellow" (at 130.81 105.41 0)
-      (effects (font (size 1.27 1.27)) hide)
-    )
+    (property "Description" "Test Points/Test Rings 1.25 mm Yellow" (at 130.81 105.41 0)
+      (effects (font (size 1.27 1.27)) hide)
+    )

Commit message: PWA_REV2.kicad, Adding test points for the decoupling 3v3 resistors and for the VCC USB.
Parts:
- added TP205: 3V3USB, TestPoint:TestPoint_Loop_D1.80mm_Drill1.0mm_Beaded, symbol Connector:TestPoint
Connections:
- net V3: now reaches C503.1, R1.1, TP202.1, U501.4 (V3)
- net 3V3USB: now reaches C501.1, C502.1, R1.1, R1.2, U501.16 (VCC)
- net 3V3USB: now also TP205.1
Other:
- note removed: "Caution: the USB to UART does not work, U501 is missing a crystal and two capacitors Q207 emitter and collector are interchanged."
Changed lines of the file:
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@@
   (junction (at 172.72 125.73) (diameter 0) (color 0 0 0 0)
+  )
+  (junction (at 168.91 76.2) (diameter 0) (color 0 0 0 0)
   )
   (junction (at 102.87 72.39) (diameter 0) (color 0 0 0 0)
@@
     (stroke (width 0) (type default))
   )
-  (wire (pts (xy 161.29 76.2) (xy 198.12 76.2))
+  (wire (pts (xy 161.29 76.2) (xy 168.91 76.2))
     (stroke (width 0) (type default))
   )
@@
     (stroke (width 0) (type default))
   )
+  (wire (pts (xy 168.91 72.39) (xy 168.91 76.2))
+    (stroke (width 0) (type default))
+  )
   (wire (pts (xy 100.33 114.3) (xy 100.33 116.84))
     (stroke (width 0) (type default))
@@
   )
   (wire (pts (xy 137.16 72.39) (xy 137.16 78.74))
+    (stroke (width 0) (type default))
+  )
+  (wire (pts (xy 168.91 76.2) (xy 198.12 76.2))
     (stroke (width 0) (type default))
   )
@@
     (effects (font (size 1.27 1.27)) (justify right bottom))
   )
-  (text "Caution: the USB to UART does not work,\nU501 is missing a crystal and two capacitors \nQ207 emitter and collector are interchanged. "
-    (at 58.42 57.15 0)
-    (effects (font (face "Arial") (size 5.08 5.08) (thickness 1.016) bold (color 255 24 53 1)) (justify left bottom))
+  (label "3V3USB" (at 173.99 76.2 0) (fields_autoplaced)
+    (effects (font (size 1.27 1.27)) (justify left bottom))
+  )
+  (label "V3" (at 147.32 78.74 0) (fields_autoplaced)
+    (effects (font (size 1.27 1.27)) (justify left bottom))
   )
   (hierarchical_label "nRESET" (shape passive) (at 214.63 118.11 0) (fields_autoplaced)
@@
         )
       )
+    )
+  )
+  (symbol (lib_id "Connector:TestPoint") (at 168.91 72.39 0) (unit 1)
+    (in_bom yes) (on_board yes) (dnp no)
+    (property "Reference" "TP205" (at 170.18 68.58 0)
+      (effects (font (size 1.27 1.27)) (justify left))
+    )
+    (property "Value" "3V3USB" (at 170.18 71.12 0)
+      (effects (font (size 1.27 1.27)) (justify left))
+    )
+    (property "Footprint" "TestPoint:TestPoint_Loop_D1.80mm_Drill1.0mm_Beaded" (at 173.99 72.39 0)
+      (effects (font (size 1.27 1.27)) hide)
+    )
+    (property "Datasheet" "~" (at 173.99 72.39 0)
+      (effects (font (size 1.27 1.27)) hide)
+    )
+    (property "AssemblyType" "HAND" (at 168.91 72.39 0)
+      (effects (font (size 1.27 1.27)) hide)
+    )
+    (property "Description" "Test Points/Test Rings 1.25 mm Red" (at 168.91 72.39 0)
+      (effects (font (size 1.27 1.27)) hide)
+    )
+    (property "Distributor 1" "JLCPCB" (at 168.91 72.39 0)
+      (effects (font (size 1.27 1.27)) hide)
+    )
+    (property "Distributor 1 PN" "C5277086" (at 168.91 72.39 0)
+      (effects (font (size 1.27 1.27)) hide)
+    )
+    (property "MPN" "RH-5000" (at 168.91 72.39 0)
+      (effects (font (size 1.27 1.27)) hide)
+    )
+    (property "Manufacturer" "ronghe" (at 168.91 72.39 0)
+      (effects (font (size 1.27 1.27)) hide)
+    )
+    (property "Cost" "0.0717" (at 168.91 72.39 0)
+      (effects (font (size 1.27 1.27)) hide)
+    )
+    (property "MPN 2" "" (at 168.91 72.39 0)
+      (effects (font (size 1.27 1.27)) hide)
+    )
+    (property "Manufacturer 2" "" (at 168.91 72.39 0)
+      (effects (font (size 1.27 1.27)) hide)
+    )
+    (pin "1")
+    (instances
+      (project "PWA_REV2"
+        (path "/412a327d-1ee3-473e-bc00-1545004b7edf/00000000-0000-0000-0000-000062bc4e7e"
+          (reference "TP205") (unit 1)
+        )
+      )

Commit message: USB_UART, moving the RX test point closer to where the tx of USB is.
Parts:
- added TP404: U0_RX, TestPoint:TestPoint_Loop_D1.80mm_Drill1.0mm_Beaded, symbol Connector:TestPoint
Connections:
- net at R502.2, U501.2 (TXD): now also TP404.1
Changed lines of the file:
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@@
   (junction (at 189.23 125.73) (diameter 0) (color 0 0 0 0)
+  )
+  (junction (at 167.64 87.63) (diameter 0) (color 0 0 0 0)
   )
   (junction (at 137.16 78.74) (diameter 0) (color 0 0 0 0)
@@
     (stroke (width 0) (type default))
   )
-  (wire (pts (xy 165.1 87.63) (xy 168.91 87.63))
+  (wire (pts (xy 165.1 87.63) (xy 167.64 87.63))
     (stroke (width 0) (type default))
   )
@@
     (stroke (width 0) (type default))
   )
+  (wire (pts (xy 167.64 87.63) (xy 168.91 87.63))
+    (stroke (width 0) (type default))
+  )
   (wire (pts (xy 124.46 76.2) (xy 120.65 76.2))
     (stroke (width 0) (type default))
@@
     (stroke (width 0) (type default))
   )
+  (wire (pts (xy 167.64 83.82) (xy 167.64 87.63))
+    (stroke (width 0) (type default))
+  )
   (wire (pts (xy 125.73 72.39) (xy 124.46 72.39))
     (stroke (width 0) (type default))
@@
     (stroke (width 0) (type default))
   )
+  (wire (pts (xy 224.79 81.28) (xy 224.79 83.82))
+    (stroke (width 0) (type default))
+  )
   (wire (pts (xy 137.16 86.36) (xy 137.16 87.63))
     (stroke (width 0) (type default))
@@
   )
   (wire (pts (xy 86.36 97.79) (xy 86.36 100.33))
+    (stroke (width 0) (type default))
+  )
+  (wire (pts (xy 224.79 83.82) (xy 167.64 83.82))
     (stroke (width 0) (type default))
   )
@@
         )
       )
+    )
+  )
+  (symbol (lib_id "Connector:TestPoint") (at 224.79 81.28 0) (unit 1)
+    (in_bom yes) (on_board yes) (dnp no)
+    (property "Reference" "TP404" (at 224.79 74.93 0)
+      (effects (font (size 1.27 1.27)) (justify left))
+    )
+    (property "Value" "U0_RX" (at 226.06 77.47 0)
+      (effects (font (size 1.27 1.27)) (justify left))
+    )
+    (property "Footprint" "TestPoint:TestPoint_Loop_D1.80mm_Drill1.0mm_Beaded" (at 229.87 81.28 0)
+      (effects (font (size 1.27 1.27)) hide)
+    )
+    (property "Datasheet" "~" (at 229.87 81.28 0)
+      (effects (font (size 1.27 1.27)) hide)
+    )
+    (property "AssemblyType" "HAND" (at 224.79 81.28 0)
+      (effects (font (size 1.27 1.27)) hide)
+    )
+    (property "Distributor 1" "JLCPCB" (at 224.79 81.28 0)
+      (effects (font (size 1.27 1.27)) hide)
+    )
+    (property "Description" "Test Points/Test Rings 1.25 mm Yellow" (at 224.79 81.28 0)
+      (effects (font (size 1.27 1.27)) hide)
+    )
+    (property "Distributor 1 PN" "C5199804" (at 224.79 81.28 0)
+      (effects (font (size 1.27 1.27)) hide)
+    )
+    (property "MPN" "RH-5004" (at 224.79 81.28 0)
+      (effects (font (size 1.27 1.27)) hide)
+    )
+    (property "Manufacturer" "ronghe" (at 224.79 81.28 0)
+      (effects (font (size 1.27 1.27)) hide)
+    )
+    (property "Cost" "0.0800" (at 224.79 81.28 0)
+      (effects (font (size 1.27 1.27)) hide)
+    )
+    (property "MPN 2" "" (at 224.79 81.28 0)
+      (effects (font (size 1.27 1.27)) hide)
+    )
+    (property "Manufacturer 2" "" (at 224.79 81.28 0)
+      (effects (font (size 1.27 1.27)) hide)
+    )
+    (pin "1")
+    (instances
+      (project "PWA_REV2"
+        (path "/412a327d-1ee3-473e-bc00-1545004b7edf/00000000-0000-0000-0000-000062b871ee"
+          (reference "TP404") (unit 1)
+        )
+        (path "/412a327d-1ee3-473e-bc00-1545004b7edf"
+          (reference "TP108") (unit 1)
+        )
+        (path "/412a327d-1ee3-473e-bc00-1545004b7edf/00000000-0000-0000-0000-000062bc4e7e"
+          (reference "TP206") (unit 1)
+        )
+      )

Commit message: USB_UART, moving the RX test point closer to where the tx of USB is.
Parts:
- TP404: value U0_RX -> U0_TX
Connections:
- net at R502.2, U501.2 (TXD): no longer TP404.1
- net at R503.2, U501.3 (RXD): now also TP404.1
Changed lines of the file:
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@@
   (junction (at 86.36 100.33) (diameter 0) (color 0 0 0 0)
   )
+  (junction (at 168.91 90.17) (diameter 0) (color 0 0 0 0)
+  )
   (junction (at 193.04 142.24) (diameter 0) (color 0 0 0 0)
   )
@@
   )
   (junction (at 189.23 125.73) (diameter 0) (color 0 0 0 0)
-  )
-  (junction (at 167.64 87.63) (diameter 0) (color 0 0 0 0)
   )
   (junction (at 137.16 78.74) (diameter 0) (color 0 0 0 0)
@@
     (stroke (width 0) (type default))
   )
-  (wire (pts (xy 165.1 87.63) (xy 167.64 87.63))
+  (wire (pts (xy 165.1 87.63) (xy 168.91 87.63))
     (stroke (width 0) (type default))
   )
@@
     (stroke (width 0) (type default))
   )
-  (wire (pts (xy 167.64 87.63) (xy 168.91 87.63))
-    (stroke (width 0) (type default))
-  )
   (wire (pts (xy 124.46 76.2) (xy 120.65 76.2))
     (stroke (width 0) (type default))
@@
     (stroke (width 0) (type default))
   )
-  (wire (pts (xy 167.64 83.82) (xy 167.64 87.63))
-    (stroke (width 0) (type default))
-  )
   (wire (pts (xy 125.73 72.39) (xy 124.46 72.39))
     (stroke (width 0) (type default))
@@
     (stroke (width 0) (type default))
   )
+  (wire (pts (xy 229.87 86.36) (xy 229.87 90.17))
+    (stroke (width 0) (type default))
+  )
   (wire (pts (xy 166.37 101.6) (xy 166.37 95.25))
     (stroke (width 0) (type default))
@@
     (stroke (width 0) (type default))
   )
-  (wire (pts (xy 224.79 81.28) (xy 224.79 83.82))
-    (stroke (width 0) (type default))
-  )
   (wire (pts (xy 137.16 86.36) (xy 137.16 87.63))
     (stroke (width 0) (type default))
@@
     (stroke (width 0) (type default))
   )
+  (wire (pts (xy 229.87 90.17) (xy 168.91 90.17))
+    (stroke (width 0) (type default))
+  )
   (wire (pts (xy 168.91 76.2) (xy 198.12 76.2))
     (stroke (width 0) (type default))
@@
   )
   (wire (pts (xy 86.36 97.79) (xy 86.36 100.33))
-    (stroke (width 0) (type default))
-  )
-  (wire (pts (xy 224.79 83.82) (xy 167.64 83.82))
     (stroke (width 0) (type default))
   )
@@
     )
   )
+  (symbol (lib_id "Connector:TestPoint") (at 229.87 86.36 0) (unit 1)
+    (in_bom yes) (on_board yes) (dnp no)
+    (property "Reference" "TP404" (at 229.87 80.01 0)
+      (effects (font (size 1.27 1.27)) (justify left))
+    )
+    (property "Value" "U0_TX" (at 231.14 82.55 0)
+      (effects (font (size 1.27 1.27)) (justify left))
+    )
+    (property "Footprint" "TestPoint:TestPoint_Loop_D1.80mm_Drill1.0mm_Beaded" (at 234.95 86.36 0)
+      (effects (font (size 1.27 1.27)) hide)
+    )
+    (property "Datasheet" "~" (at 234.95 86.36 0)
+      (effects (font (size 1.27 1.27)) hide)
+    )
+    (property "AssemblyType" "HAND" (at 229.87 86.36 0)
+      (effects (font (size 1.27 1.27)) hide)
+    )
+    (property "Distributor 1" "JLCPCB" (at 229.87 86.36 0)
+      (effects (font (size 1.27 1.27)) hide)
+    )
+    (property "Description" "Test Points/Test Rings 1.25 mm Yellow" (at 229.87 86.36 0)
+      (effects (font (size 1.27 1.27)) hide)
+    )
+    (property "Distributor 1 PN" "C5199804" (at 229.87 86.36 0)
+      (effects (font (size 1.27 1.27)) hide)
+    )
+    (property "MPN" "RH-5004" (at 229.87 86.36 0)
+      (effects (font (size 1.27 1.27)) hide)
+    )
+    (property "Manufacturer" "ronghe" (at 229.87 86.36 0)
+      (effects (font (size 1.27 1.27)) hide)
+    )
+    (property "Cost" "0.0800" (at 229.87 86.36 0)
+      (effects (font (size 1.27 1.27)) hide)
+    )
+    (property "MPN 2" "" (at 229.87 86.36 0)
+      (effects (font (size 1.27 1.27)) hide)
+    )
+    (property "Manufacturer 2" "" (at 229.87 86.36 0)
+      (effects (font (size 1.27 1.27)) hide)
+    )
+    (pin "1")
+    (instances
+      (project "PWA_REV2"
+        (path "/412a327d-1ee3-473e-bc00-1545004b7edf/00000000-0000-0000-0000-000062b871ee"
+          (reference "TP404") (unit 1)
+        )
+        (path "/412a327d-1ee3-473e-bc00-1545004b7edf"
+          (reference "TP107") (unit 1)
+        )
+        (path "/412a327d-1ee3-473e-bc00-1545004b7edf/00000000-0000-0000-0000-000062bc4e7e"
+          (reference "TP206") (unit 1)
+        )
+      )
+    )
+  )
   (symbol (lib_id "power:GND") (at 100.33 116.84 0) (unit 1)
     (in_bom yes) (on_board yes) (dnp no)
@@
         )
       )
-    )
-  )
-  (symbol (lib_id "Connector:TestPoint") (at 224.79 81.28 0) (unit 1)
-    (in_bom yes) (on_board yes) (dnp no)
-    (property "Reference" "TP404" (at 224.79 74.93 0)
-      (effects (font (size 1.27 1.27)) (justify left))
-    )
-    (property "Value" "U0_RX" (at 226.06 77.47 0)
-      (effects (font (size 1.27 1.27)) (justify left))
-    )
-    (property "Footprint" "TestPoint:TestPoint_Loop_D1.80mm_Drill1.0mm_Beaded" (at 229.87 81.28 0)
-      (effects (font (size 1.27 1.27)) hide)
-    )
-    (property "Datasheet" "~" (at 229.87 81.28 0)
-      (effects (font (size 1.27 1.27)) hide)
-    )
-    (property "AssemblyType" "HAND" (at 224.79 81.28 0)
-      (effects (font (size 1.27 1.27)) hide)
-    )
-    (property "Distributor 1" "JLCPCB" (at 224.79 81.28 0)
-      (effects (font (size 1.27 1.27)) hide)
-    )
-    (property "Description" "Test Points/Test Rings 1.25 mm Yellow" (at 224.79 81.28 0)
-      (effects (font (size 1.27 1.27)) hide)
-    )
-    (property "Distributor 1 PN" "C5199804" (at 224.79 81.28 0)
-      (effects (font (size 1.27 1.27)) hide)
-    )
-    (property "MPN" "RH-5004" (at 224.79 81.28 0)
-      (effects (font (size 1.27 1.27)) hide)
-    )
-    (property "Manufacturer" "ronghe" (at 224.79 81.28 0)
-      (effects (font (size 1.27 1.27)) hide)
-    )
-    (property "Cost" "0.0800" (at 224.79 81.28 0)
-      (effects (font (size 1.27 1.27)) hide)
-    )
-    (property "MPN 2" "" (at 224.79 81.28 0)
-      (effects (font (size 1.27 1.27)) hide)
-    )
-    (property "Manufacturer 2" "" (at 224.79 81.28 0)
-      (effects (font (size 1.27 1.27)) hide)
-    )
-    (pin "1")
-    (instances
-      (project "PWA_REV2"
-        (path "/412a327d-1ee3-473e-bc00-1545004b7edf/00000000-0000-0000-0000-000062b871ee"
-          (reference "TP404") (unit 1)
-        )
-        (path "/412a327d-1ee3-473e-bc00-1545004b7edf"
-          (reference "TP108") (unit 1)
-        )
-        (path "/412a327d-1ee3-473e-bc00-1545004b7edf/00000000-0000-0000-0000-000062bc4e7e"
-          (reference "TP206") (unit 1)
-        )
-      )
