File: PWA_REV2/USB_UART.kicad_sch (KiCad schematic)
At the start: 25 parts, among them J501 USB_C_Receptacle_USB2.0, Q205 MMBT2222A-7-F, U501 CH340B

Commit message: PWA_REV2, We corrected Assembly Type for some components, and we added the JLCPCB PN for the DB9 and the CH340B.
Parts:
- U501: AssemblyType (none) -> SMT; Cost (none) -> 1.05; Distributor 1 (none) -> JLCPCB; Distributor 1 PN (none) -> C81010
Changed lines of the file:
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@@
+      (effects (font (size 1.27 1.27)) hide)
+    )
+    (property "Cost" "1.05" (at 154.94 97.79 0)
+      (effects (font (size 1.27 1.27)) hide)
+    )
+    (property "Distributor 1" "JLCPCB" (at 154.94 97.79 0)
+      (effects (font (size 1.27 1.27)) hide)
+    )
+    (property "Distributor 1 PN" "C81010" (at 154.94 97.79 0)
+      (effects (font (size 1.27 1.27)) hide)
+    )
+    (property "AssemblyType" "SMT" (at 154.94 97.79 0)
       (effects (font (size 1.27 1.27)) hide)
     )

Commit message: USB_UART.kicad_sch, Adding description and MPN for CH340B.
Parts:
- U501: MPN (none) -> CH340B
Changed lines of the file:
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@@
+      (effects (font (size 1.27 1.27)) hide)
+    )
+    (property "Description" "2Mbps 3.3V Transceiver USB 2.0 SOP-16 USB Converters ROHS" (at 154.94 97.79 0)
+      (effects (font (size 1.27 1.27)) hide)
+    )
+    (property "MPN" "CH340B" (at 154.94 97.79 0)
       (effects (font (size 1.27 1.27)) hide)
     )
