File: PWA_REV2/LCD And I2C Interface.kicad_sch (KiCad schematic)
At the start: 44 parts, among them Q301 BSS138, Q401 BSS138, Q402 BSS138, U301 PCF8574AT_3_518, U302 LCD_20x4_Character-GPAD_SCH_L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, U303 Conn_01x16

Commit message: Fixed the previous PWA_REV_2 file by added the changes of the USB UART. PCBa_krake is reverted to when no changes done to the schem.
Connections:
- no-connect marks 0 -> 16
Other:
- title: Krake Rev2 -> KRAKE_PCB

Commit message: PWA_REV2, kicad project, changed to CH340B, changed the polarity of Q207, added I2C address table.
Other:
- note added: "The six resistors connected to A0 A1 A2 define the I2C address ref to table 5 below:"
- moved on the sheet: MF401, MF402, MF403, MF404, MF405, MF406, MF407, MF408, MF409, MF410, MF411, MF412

Commit message: PWA_REV2.kicad_sch, updated the footptint of the testpoint to 1mm hole and corrected description.
Parts:
- TP102, TP401, TP402, TP403, TP404: footprint TestPoint:TestPoint_Loop_D2.54mm_Drill1.5mm_Beaded -> TestPoint:TestPoint_Loop_D1.80mm_Drill1.0mm_Beaded
Changed lines of the file:
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@@
       (effects (font (size 1.27 1.27)) (justify left))
     )
-    (property "Footprint" "TestPoint:TestPoint_Loop_D2.54mm_Drill1.5mm_Beaded" (at 134.62 106.68 0)
+    (property "Footprint" "TestPoint:TestPoint_Loop_D1.80mm_Drill1.0mm_Beaded" (at 134.62 106.68 0)
       (effects (font (size 1.27 1.27)) hide)
     )
@@
       (effects (font (size 1.27 1.27)) hide)
     )
-    (property "Description" "Test Points/Test Rings ROHS yellow" (at 139.7 106.68 0)
+    (property "Description" "Test Points/Test Rings 1.25 mm Yellow" (at 139.7 106.68 0)
       (effects (font (size 1.27 1.27)) hide)
     )
@@
       (effects (font (size 1.27 1.27)) (justify left))
     )
-    (property "Footprint" "TestPoint:TestPoint_Loop_D2.54mm_Drill1.5mm_Beaded" (at 219.71 60.96 0)
+    (property "Footprint" "TestPoint:TestPoint_Loop_D1.80mm_Drill1.0mm_Beaded" (at 219.71 60.96 0)
       (effects (font (size 1.27 1.27)) hide)
     )
@@
       (effects (font (size 1.27 1.27)) hide)
     )
-    (property "Description" "Test Points/Test Rings ROHS red" (at 214.63 60.96 0)
+    (property "Description" "Test Points/Test Rings 1.25 mm Red" (at 214.63 60.96 0)
       (effects (font (size 1.27 1.27)) hide)
     )
@@
       (effects (font (size 1.27 1.27)) (justify left))
     )
-    (property "Footprint" "TestPoint:TestPoint_Loop_D2.54mm_Drill1.5mm_Beaded" (at 139.7 67.31 0)
+    (property "Footprint" "TestPoint:TestPoint_Loop_D1.80mm_Drill1.0mm_Beaded" (at 139.7 67.31 0)
       (effects (font (size 1.27 1.27)) hide)
     )
@@
       (effects (font (size 1.27 1.27)) hide)
     )
-    (property "Description" "Test Points/Test Rings ROHS yellow" (at 134.62 67.31 0)
+    (property "Description" "Test Points/Test Rings 1.25 mm Yellow" (at 134.62 67.31 0)
       (effects (font (size 1.27 1.27)) hide)
     )
@@
       (effects (font (size 1.27 1.27)) (justify left))
     )
-    (property "Footprint" "TestPoint:TestPoint_Loop_D2.54mm_Drill1.5mm_Beaded" (at 228.6 35.56 0)
+    (property "Footprint" "TestPoint:TestPoint_Loop_D1.80mm_Drill1.0mm_Beaded" (at 228.6 35.56 0)
       (effects (font (size 1.27 1.27)) hide)
     )
@@
       (effects (font (size 1.27 1.27)) hide)
     )
-    (property "Description" "Test Points/Test Rings ROHS red" (at 223.52 35.56 0)
+    (property "Description" "Test Points/Test Rings 1.25 mm Red" (at 223.52 35.56 0)
       (effects (font (size 1.27 1.27)) hide)
     )
@@
       (effects (font (size 1.27 1.27)) (justify left))
     )
-    (property "Footprint" "TestPoint:TestPoint_Loop_D2.54mm_Drill1.5mm_Beaded" (at 134.62 71.12 0)
+    (property "Footprint" "TestPoint:TestPoint_Loop_D1.80mm_Drill1.0mm_Beaded" (at 134.62 71.12 0)
       (effects (font (size 1.27 1.27)) hide)
     )
@@
       (effects (font (size 1.27 1.27)) hide)
     )
-    (property "Description" "Test Points/Test Rings ROHS yellow" (at 129.54 71.12 0)
-      (effects (font (size 1.27 1.27)) hide)
-    )
+    (property "Description" "Test Points/Test Rings 1.25 mm Yellow" (at 129.54 71.12 0)
+      (effects (font (size 1.27 1.27)) hide)
+    )

Commit message: PWA_REV2, solved issue 239, added functionality discription to D106, and similarly we corrected Schematic and PCB text for MENU BOOT RESET MUTE CONTRAST POWER.
Other:
- note added: "CONTRAST"
Changed lines of the file:
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@@
     (effects (font (size 1.27 1.27)) (justify left bottom))
+  )
+  (text "CONTRAST" (at 203.2 81.28 0)
+    (effects (font (size 2.54 2.54)) (justify left bottom))
   )
   (text "The six resistors connected to A0 A1 A2 \ndefine the I2C address ref to table 5 below:"
@@
       (effects (font (size 1.27 1.27)) hide)
     )
-    (property "Value" "GND" (at 209.677 79.3242 0)
+    (property "Value" "GND" (at 207.01 74.93 0)
       (effects (font (size 1.27 1.27)))
     )
@@
   )
   (symbol (lib_id "GPAD_SCH_LIB:POT 0.375 10K") (at 209.55 68.58 180) (unit 1)
-    (in_bom yes) (on_board yes) (dnp no) (fields_autoplaced)
-    (property "Reference" "RV301" (at 207.01 72.5171 0)
+    (in_bom yes) (on_board yes) (dnp no)
+    (property "Reference" "RV301" (at 210.82 66.04 0)
       (effects (font (size 1.27 1.27)) (justify right))
     )
-    (property "Value" "POT 0.375 10K" (at 207.01 69.9771 0)
+    (property "Value" "POT 0.375 10K" (at 210.82 68.58 0)
       (effects (font (size 1.27 1.27)) (justify right))
     )
@@
       (effects (font (size 1.27 1.27)) hide)
     )
-    (property "Distributor 2 PN" "3386P-103LF-ND" (at 207.01 64.8971 0)
-      (effects (font (size 1.27 1.27)) (justify right))
-    )
-    (property "Cost" "0.6963" (at 209.55 68.58 0)
-      (effects (font (size 1.27 1.27)))
+    (property "Distributor 2 PN" "3386P-103LF-ND" (at 205.74 74.93 0)
+      (effects (font (size 1.27 1.27)) (justify right) hide)
+    )
+    (property "Cost" "0.6963" (at 201.93 69.85 0)
+      (effects (font (size 1.27 1.27)) hide)
     )
     (property "Manufacturer" "BOURNS" (at 209.55 68.58 0)
