File: PWA_REV2/Enclosure.kicad_sch (KiCad schematic)
At the start: 2 parts

Commit message: Fixed the previous PWA_REV_2 file by added the changes of the USB UART. PCBa_krake is reverted to when no changes done to the schem.
Other:
- title: Krake Rev2 -> KRAKE_PCB
Changed lines of the file:
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@@
   (paper "A4")
   (title_block
-    (title "Krake Rev2")
-    (date "2025-07-16")
-    (rev "2.0")
+    (title "KRAKE_PCB")
+    (date "2024-11-23")
+    (rev "1.0")
     (company "PublicInvention")
     (comment 1 "GNU Affero General Public License v3.0")
@@
     )
     (instances
-      (project "PWA_REV2"
+      (project "PCBa_KRAKE"
         (path "/412a327d-1ee3-473e-bc00-1545004b7edf"
           (reference "MF102") (unit 1)
@@
     )
     (instances
-      (project "PWA_REV2"
+      (project "PCBa_KRAKE"
         (path "/412a327d-1ee3-473e-bc00-1545004b7edf"
           (reference "MF101") (unit 1)

Commit message: PWA_REV2.kicad_sch, add screws for PWA to enclosure, Enclosure shell top to bottom. Add lable symbol to schematic.
Parts:
- added LB801: Krake_Model_Serial, symbol GPAD_SCH_LIB:Label_Product
- added MF401 (x4): Screw_#6x1/2"PanTorxHeadSelfTapping, symbol GPAD_SCH_LIB:Screw_4-40_0.375_Phillips
- added MF401 (x4): Screw_2-32x3/8_Phillips_Pan_Self_Tapping, symbol GPAD_SCH_LIB:Screw_4-40_0.375_Phillips
Other:
- note added: "Screws hold PWA into enclosure"
- note added: "Screws hold enclosure top shell to bottom shell"
- moved on the sheet: MF101, MF102

Commit message: PWA_REV2.kicad_sch, add 28mm speaker enclosure parts including key cap and encoder knob.
Parts:
- removed MF102: ENCLOSURE_KRAKE_VER1, symbol GPAD_SCH_LIB:ENCLOSURE_GPAD_VER1
- added MF102: ENCODER_KNOB_D_KRAKE, symbol GPAD_SCH_LIB:ENCLOSURE_GPAD_VER1
- added MF102: ENCLOSURE_KRAKE_FRONP_PANEL_28mmSPEAKER, symbol GPAD_SCH_LIB:ENCLOSURE_GPAD_VER1
- added MF102: ENCLOSURE_KRAKE_BOTTOM_SHELL_28mmSPEAKER, symbol GPAD_SCH_LIB:ENCLOSURE_GPAD_VER1
- added MF102: KEY_CAP_12MM_KRAKE_MUTE_BUTTON, symbol GPAD_SCH_LIB:ENCLOSURE_GPAD_VER1
- added MF102: ENCLOSURE_KRAKE_REAR_PANNEL_28mmSPEAKER, symbol GPAD_SCH_LIB:ENCLOSURE_GPAD_VER1
- added MF102: ENCLOSURE_KRAKE_TOP_SHELL_28mmSPEAKER, symbol GPAD_SCH_LIB:ENCLOSURE_GPAD_VER1
Other:
- moved on the sheet: MF401

Commit message: fixed kicad project issue.
Parts:
- removed LB801: Krake_Model_Serial, symbol GPAD_SCH_LIB:Label_Product
- removed MF102: ENCODER_KNOB_D_KRAKE, symbol GPAD_SCH_LIB:ENCLOSURE_GPAD_VER1
- removed MF102: ENCLOSURE_KRAKE_FRONP_PANEL_28mmSPEAKER, symbol GPAD_SCH_LIB:ENCLOSURE_GPAD_VER1
- removed MF102: ENCLOSURE_KRAKE_BOTTOM_SHELL_28mmSPEAKER, symbol GPAD_SCH_LIB:ENCLOSURE_GPAD_VER1
- removed MF102: KEY_CAP_12MM_KRAKE_MUTE_BUTTON, symbol GPAD_SCH_LIB:ENCLOSURE_GPAD_VER1
- removed MF102: ENCLOSURE_KRAKE_REAR_PANNEL_28mmSPEAKER, symbol GPAD_SCH_LIB:ENCLOSURE_GPAD_VER1
- removed MF102: ENCLOSURE_KRAKE_TOP_SHELL_28mmSPEAKER, symbol GPAD_SCH_LIB:ENCLOSURE_GPAD_VER1
- removed MF401 (x4): Screw_#6x1/2"PanTorxHeadSelfTapping, symbol GPAD_SCH_LIB:Screw_4-40_0.375_Phillips
- removed MF401 (x4): Screw_2-32x3/8_Phillips_Pan_Self_Tapping, symbol GPAD_SCH_LIB:Screw_4-40_0.375_Phillips
- added MF102: ENCLOSURE_KRAKE_VER1, symbol GPAD_SCH_LIB:ENCLOSURE_GPAD_VER1
Other:
- note removed: "Screws hold PWA into enclosure"
- note removed: "Screws hold enclosure top shell to bottom shell"
- moved on the sheet: MF101

Commit message: Hardware, PWA, Add a Jumper to BOM for J102 so that USB Connector Can Power Krake, issue 312.
:q
q
Parts:
- renumbered MF102 to MF801, MF101 to MF802
