File: PWA_REV2/Enclosure.kicad_sch (KiCad schematic)
At the start: 2 parts

Commit message: Revert "Hardware, PWA, Add a Jumper to BOM for J102 so that USB Connector Can Power Krake, issue 312."
This reverts commit c2819b8ee4999f733f52d823f88f6aefd6456fcc.
Parts:
- renumbered MF802 to MF101, MF801 to MF102
